Commit message: Rotate joints 3 and 5 to fix arm

File: tiago_sea_arm_description/urdf/arm.urdf.xacro (robot description, xacro)
@@ -139,5 +139,5 @@
     <!-- ARM 3 JOINT -->
     <joint name="${name}_3_joint" type="revolute">
-      <origin xyz="-0.02 0.16991 -0.04491" rpy="1.5708 1.5708 0" />
+      <origin xyz="-0.02 0.16991 -0.04491" rpy="-1.5707 0 0" />
       <parent link="${name}_2_link" />
       <child link="${name}_3_link" />
@@ -213,5 +213,5 @@
     <!-- ARM 5 JOINT -->
     <joint name="${name}_5_joint" type="revolute">
-      <origin xyz="-0.02 0.16991 -0.04491" rpy="1.5708 1.5708 0" />
+      <origin xyz="-0.02 0.16991 -0.04491" rpy="-1.5708 0 0" />
       <parent link="${name}_4_link" />
       <child link="${name}_5_link" />

Commit message: Separate joint limits in extra file, set convention for joints

File: tiago_sea_arm_description/urdf/arm.urdf.xacro (robot description, xacro)
@@ -15,4 +15,6 @@
 <!-- Transmissions file -->
 <xacro:include filename="$(find tiago_sea_arm_description)/urdf/arm.transmission.xacro"/>
+<!-- Joint Limits file -->
+<xacro:include filename="$(find tiago_sea_arm_description)/urdf/arm.limits.xacro"/>
 <!-- Constant parameters -->
 <xacro:property name="arm_friction"       value="1.0" />
@@ -69,5 +71,5 @@
       <child link="${name}_1_link" />
       <axis xyz="0 0 1" />
-      <limit lower="-2.6" upper="2.6" effort="${arm_1_max_effort}" velocity="${arm_1_max_velocity}" />
+      <limit lower="${arm_1_joint_lb}" upper="${arm_1_joint_ub}" effort="${arm_1_max_effort}" velocity="${arm_1_max_velocity}" />
     </joint>
     <!-- ARM 2 LINK -->
@@ -106,5 +108,5 @@
       <child link="${name}_2_link" />
       <axis xyz="0 0 -1" />
-      <limit lower="-1.05" upper="2.45" effort="${arm_2_max_effort}" velocity="${arm_2_max_velocity}" />
+      <limit lower="${arm_2_joint_lb}" upper="${arm_2_joint_ub}" effort="${arm_2_max_effort}" velocity="${arm_2_max_velocity}" />
     </joint>
     <!-- ARM 3 LINK -->
@@ -139,9 +141,10 @@
     <!-- ARM 3 JOINT -->
     <joint name="${name}_3_joint" type="revolute">
-      <origin xyz="-0.02 0.16991 -0.04491" rpy="-1.5707 0 0" />
+      <!-- Mechanics provided {r p y} = {-1.5707 0 0} -->
+      <origin xyz="-0.02 0.16991 -0.04491" rpy="${reflect * 1.5707} 0 ${(reflect + 1) * 0.5 * 3.1415}" />
       <parent link="${name}_2_link" />
       <child link="${name}_3_link" />
       <axis xyz="0 0 1" />
-      <limit lower="-2.6" upper="2.6" effort="${arm_3_max_effort}" velocity="${arm_3_max_velocity}" />
+      <limit lower="${arm_3_joint_lb}" upper="${arm_3_joint_ub}" effort="${arm_3_max_effort}" velocity="${arm_3_max_velocity}" />
     </joint>
     <!-- ARM 4 LINK -->
@@ -180,5 +183,5 @@
       <child link="${name}_4_link" />
       <axis xyz="0 0 -1" />
-      <limit lower="-1.05" upper="2.45" effort="${arm_4_max_effort}" velocity="${arm_4_max_velocity}" />
+      <limit lower="${arm_4_joint_lb}" upper="${arm_4_joint_ub}" effort="${arm_4_max_effort}" velocity="${arm_4_max_velocity}" />
     </joint>
     <!-- ARM 5 LINK -->
@@ -217,5 +220,5 @@
       <child link="${name}_5_link" />
       <axis xyz="0 0 1" />
-      <limit lower="-2.6" upper="2.6" effort="${arm_5_max_effort}" velocity="${arm_5_max_velocity}" />
+      <limit lower="${arm_5_joint_lb}" upper="${arm_5_joint_ub}" effort="${arm_5_max_effort}" velocity="${arm_5_max_velocity}" />
     </joint>
     <!-- ARM 6 LINK -->
@@ -254,5 +257,5 @@
       <child link="${name}_6_link" />
       <axis xyz="0 0 1" />
-      <limit lower="-2" upper="2" effort="${arm_6_max_effort}" velocity="${arm_6_max_velocity}" />
+      <limit lower="${arm_6_joint_lb}" upper="${arm_6_joint_ub}" effort="${arm_6_max_effort}" velocity="${arm_6_max_velocity}" />
     </joint>
     <!-- ARM 7 LINK -->
@@ -291,5 +294,5 @@
       <child link="${name}_7_link" />
       <axis xyz="0 0 1" />
-      <limit lower="-2.6" upper="2.6" effort="${arm_7_max_effort}" velocity="${arm_7_max_velocity}" />
+      <limit lower="${arm_7_joint_lb}" upper="${arm_7_joint_ub}" effort="${arm_7_max_effort}" velocity="${arm_7_max_velocity}" />
     </joint>
     <!-- TRANSMISSIONS -->

Commit message: elbow aligned with joint 2

File: tiago_sea_arm_description/urdf/arm.urdf.xacro (robot description, xacro)
@@ -142,5 +142,5 @@
     <joint name="${name}_3_joint" type="revolute">
       <!-- Mechanics provided {r p y} = {-1.5707 0 0} -->
-      <origin xyz="-0.02 0.16991 -0.04491" rpy="${reflect * 1.5707} 0 ${(reflect + 1) * 0.5 * 3.1415}" />
+      <origin xyz="-0.02 0.16991 -0.04491" rpy="${reflect * 1.5707} 1.5707 ${(reflect + 1) * 0.5 * 3.1415}" />
       <parent link="${name}_2_link" />
       <child link="${name}_3_link" />
@@ -216,5 +216,5 @@
     <!-- ARM 5 JOINT -->
     <joint name="${name}_5_joint" type="revolute">
-      <origin xyz="-0.02 0.16991 -0.04491" rpy="-1.5708 0 0" />
+      <origin xyz="-0.02 0.16991 -0.04491" rpy="-1.5708 1.5707 0" />
       <parent link="${name}_4_link" />
       <child link="${name}_5_link" />

Commit message: rotate arm_7_link axis to point outwards

File: tiago_sea_arm_description/urdf/arm.urdf.xacro (robot description, xacro)
@@ -290,5 +290,5 @@
     <!-- ARM 7 JOINT -->
     <joint name="${name}_7_joint" type="revolute">
-      <origin xyz="0 0.135 -0.0431" rpy="1.5708 1.5708 0" />
+      <origin xyz="0 0.135 -0.0431" rpy="-1.5708 1.5708 0" />
       <parent link="${name}_6_link" />
       <child link="${name}_7_link" />

Commit message: added more mass

File: tiago_sea_arm_description/urdf/arm.urdf.xacro (robot description, xacro)
@@ -40,5 +40,5 @@
       <inertial>
         <origin xyz="0.0049601 0.014951 0.13623" rpy="0 0 0" />
-        <mass value="0.47419" />
+        <mass value="1.0" />
         <inertia
           ixx="0.0011142"
@@ -77,5 +77,5 @@
       <inertial>
         <origin xyz="-0.018757 0.1146 -0.041335" rpy="0 0 0" />
-        <mass value="0.41866" />
+        <mass value="1.0" />
         <inertia
           ixx="0.00072176"
@@ -114,5 +114,5 @@
       <inertial>
         <origin xyz="-0.0049601 -0.014951 0.13627" rpy="0 0 0" />
-        <mass value="0.47419" />
+        <mass value="1.0" />
         <inertia
           ixx="0.0011142"
@@ -152,5 +152,5 @@
       <inertial>
         <origin xyz="-0.018757 0.1146 -0.041335" rpy="0 0 0" />
-        <mass value="0.41866" />
+        <mass value="1" />
         <inertia
           ixx="0.00072176"
@@ -189,5 +189,5 @@
       <inertial>
         <origin xyz="-0.0034877 0.0007088 0.10161" rpy="0 0 0" />
-        <mass value="1.3606" />
+        <mass value="0.65" /> <!--1.3606-->
         <inertia
           ixx="0.0042327"
@@ -226,5 +226,5 @@
       <inertial>
         <origin xyz="-3.3166E-06 0.051142 -0.045664" rpy="0 0 0" />
-        <mass value="0.87439" />
+        <mass value="0.65" />
         <inertia
           ixx="0.0012166"
@@ -295,4 +295,31 @@
       <axis xyz="0 0 1" />
       <limit lower="${arm_7_joint_lb}" upper="${arm_7_joint_ub}" effort="${arm_7_max_effort}" velocity="${arm_7_max_velocity}" />
+    </joint>
+ <!--***********************-->
+    <!--        TOOL           -->
+    <!--***********************-->
+    <link name="${name}_tool_link">
+      <inertial>
+        <mass value="0.1" />
+        <inertia ixx="8.33E-07" ixy="0.0" ixz="0.0" iyy="8.33E-07" iyz="0.0" izz="1.25E-06" />
+      </inertial>
+      <visual>
+        <origin xyz="0.001 0 0" rpy="0 1.5708 0" />
+        <geometry>
+          <cylinder radius="0.005" length="0.005"/>
+        </geometry>
+        <material name="LightGrey" />
+      </visual>
+      <collision>
+        <origin xyz="0.001 0 0" rpy="0 1.5708 0" />
+        <geometry>
+          <cylinder radius="0.005" length="0.005"/>
+        </geometry>
+      </collision>
+    </link>
+    <joint name="${name}_tool_joint" type="fixed">
+      <parent link="${name}_7_link" />
+      <child link="${name}_tool_link" />
+        <origin xyz="0 0 -0.07" rpy="3.1415 0 0" />
     </joint>
     <!-- TRANSMISSIONS -->

Commit message: fixed tool_link position

File: tiago_sea_arm_description/urdf/arm.urdf.xacro (robot description, xacro)
@@ -321,5 +321,5 @@
       <parent link="${name}_7_link" />
       <child link="${name}_tool_link" />
-        <origin xyz="0 0 -0.07" rpy="3.1415 0 0" />
+        <origin xyz="0 0 0" rpy="0 0 0" />
     </joint>
     <!-- TRANSMISSIONS -->
