Commit message: Update stl + frames + collision of the ft_sensor

File: tiago_sea_arm_description/urdf/end_effector/end_effector.urdf.xacro (robot description, xacro)
@@ -27,5 +27,4 @@
     <!-- Add nothing -->
   </xacro:if>
-  <!-- TODO: Get correct transform for new gripper -->
   <!-- PAL Pro Gripper -->
   <xacro:if value="${type == 'pal-pro-gripper'}">

File: tiago_sea_arm_description/urdf/sensors/ft_sensor.urdf.xacro (robot description, xacro)
@@ -20,8 +20,8 @@
         <inertial>
           <mass value="0.2657" />
-          <inertia ixx="268925.36" ixy="3102.05" ixz="5074.07" iyy="160140.92" iyz="4096.6" izz="268336.32" />
+          <inertia ixx="2.9766E-04" ixy="1.87E-06" ixz="8.95E-06" iyy="3.095E-04" iyz="2.07E-06" izz="1.6632E-04" />
         </inertial>
         <visual>
-          <origin xyz="0.0 0.0 -0.050" rpy="${90.0 * deg_to_rad} 0 ${45.0 * deg_to_rad if reflect == '1' else 135 * deg_to_rad}"/>
+          <origin xyz="0.0 0.0 0.0" rpy="0.0 0.0 0.0"/>
           <geometry>
             <mesh filename="package://tiago_sea_arm_description/meshes/sensors/ati_ft_sensor.STL"/>
@@ -32,5 +32,5 @@
         </visual>
         <collision>
-          <origin xyz="0 0 -0.025" rpy="0 0 0" />
+          <origin xyz="0 0 -0.030" rpy="0 0 0" />
           <geometry>
             <cylinder radius="0.035" length="0.05"/>
@@ -38,7 +38,7 @@
         </collision>
         <collision>
-          <origin xyz="0.047 0 -0.040" rpy="0 0 0" />
+          <origin xyz="0.035 0.011 -0.035" rpy="0 0 ${25.0 * deg_to_rad}" />
           <geometry>
-            <box size="0.025 0.012 0.04"/>
+            <box size="0.0395 0.0496 0.053"/>
           </geometry>
         </collision>
@@ -47,5 +47,5 @@
       <parent link="${parent}" />
       <child link="${name}_ft_link" />
-      <origin xyz="0.050 0 0" rpy="${-90.0 * deg_to_rad} ${45.0 * deg_to_rad} ${-90.0 * deg_to_rad}" />
+      <origin xyz="0.045 0 0" rpy="${-90.0 * deg_to_rad} ${45.0 * deg_to_rad} ${-90.0 * deg_to_rad}" />
     </joint>
     <!--***********************-->
@@ -56,5 +56,5 @@
       <parent link="${name}_ft_link" />
       <child link="${name}_ft_tool_link" />
-      <origin xyz="0 0 0.0" rpy="${45.0 * deg_to_rad} ${-90.0 * deg_to_rad} ${0.0 * deg_to_rad}" />
+      <origin xyz="0 0 0.005" rpy="${45.0 * deg_to_rad} ${-90.0 * deg_to_rad} ${0.0 * deg_to_rad}" />
     </joint>
 </xacro:macro>
