Commit message: Separate origin of first joint to robot xacro

File: tiago_sea_arm_description/robots/tiago_sea_arm.urdf.xacro (robot description, xacro)
@@ -44,4 +44,6 @@
   </link>
   <!-- ARM -->
-  <xacro:tiago_sea_arm name="arm" parent="base_link" reflect="1" arm_1_offset="0" arm_2_offset="0" arm_3_offset="0" arm_4_offset="0" arm_5_offset="0" arm_6_offset="0" arm_7_offset="0" />
+  <xacro:tiago_sea_arm name="arm" parent="base_link" reflect="1" arm_1_offset="0" arm_2_offset="0" arm_3_offset="0" arm_4_offset="0" arm_5_offset="0" arm_6_offset="0" arm_7_offset="0">
+    <origin xyz="0 0 0.01991" rpy="0 0 3.1416" />
+  </xacro:tiago_sea_arm>
 </robot>

File: tiago_sea_arm_description/urdf/arm.urdf.xacro (robot description, xacro)
@@ -32,5 +32,5 @@
 <xacro:property name="arm_6_max_effort"   value="26" />
 <xacro:property name="arm_7_max_effort"   value="26" />
-<xacro:macro name="tiago_sea_arm" params="name parent reflect arm_1_offset arm_2_offset arm_3_offset arm_4_offset arm_5_offset arm_6_offset arm_7_offset no_safety_eps:=False">
+<xacro:macro name="tiago_sea_arm" params="name parent reflect *origin arm_1_offset arm_2_offset arm_3_offset arm_4_offset arm_5_offset arm_6_offset arm_7_offset no_safety_eps:=False">
   <xacro:property name="arm_eps"       value="${0.00 if no_safety_eps else 0.07}"/>
     <!-- ARM 1 LINK -->
@@ -65,5 +65,5 @@
     </link>
     <joint name="${name}_1_joint" type="revolute">
-      <origin xyz="0 0 0.01991" rpy="0 0 3.1416" />
+      <xacro:insert_block name="origin"/>
       <parent link="${parent}" />
       <child link="${name}_1_link" />

Commit message: update models + urdf

File: tiago_sea_arm_description/robots/tiago_sea_arm.urdf.xacro (robot description, xacro)
@@ -13,18 +13,12 @@
 -->
 <robot xmlns:xacro="http://ros.org/wiki/xacro" name="tiago_sea_arm">
-  <xacro:include filename="$(find tiago_sea_arm_description)/urdf/arm.urdf.xacro"/>
+  <xacro:include filename="$(find tiago_sea_arm_description)/urdf/arm/arm.urdf.xacro"/>
+  <xacro:include filename="$(find tiago_sea_arm_description)/urdf/end_effector/end_effector.urdf.xacro"/>
+  <xacro:arg name="end_effector" default="false"/>
+  <xacro:arg name="ft_sensor" default="false"/>
+  <xacro:property name="end_effector" value="$(arg end_effector)" />
+  <xacro:property name="ft_sensor" value="$(arg ft_sensor)" />
   <!-- BASE LINK -->
   <link name="base_link">
-    <inertial>
-      <origin xyz="2.601E-19 4.0232E-18 -0.015448" rpy="0 0 0" />
-      <mass value="0.28971" />
-      <inertia
-        ixx="0.00022379"
-        ixy="1.5836E-20"
-        ixz="5.2063E-21"
-        iyy="0.00022379"
-        iyz="-5.1333E-21"
-        izz="0.00019673" />
-    </inertial>
     <visual>
       <origin xyz="0 0 0" rpy="0 0 0" />
@@ -44,6 +38,5 @@
   </link>
   <!-- ARM -->
-  <xacro:tiago_sea_arm name="arm" parent="base_link" reflect="1" arm_1_offset="0" arm_2_offset="0" arm_3_offset="0" arm_4_offset="0" arm_5_offset="0" arm_6_offset="0" arm_7_offset="0">
-    <origin xyz="0 0 0.01991" rpy="0 0 3.1416" />
-  </xacro:tiago_sea_arm>
+  <xacro:tiago_sea_arm name="arm_right" parent="base_link" reflect="1" ft_sensor="${ft_sensor}" arm_1_offset="0" arm_2_offset="0" arm_3_offset="0" arm_4_offset="0" arm_5_offset="0" arm_6_offset="0" arm_7_offset="0"/>
+  <xacro:tiago_sea_arm_end_effector name="gripper" parent="arm_right_7_link" type="${end_effector}"/>
 </robot>

File: tiago_sea_arm_description/urdf/arm/arm.transmission.xacro (robot description, xacro)
@@ -1,15 +1,3 @@
-<?xml version="1.0" encoding="UTF-8"?>
-<!--
-  Copyright (c) 2022 PAL Robotics S.L. All rights reserved.
-  Licensed under the Apache License, Version 2.0 (the "License");
-  you may not use this file except in compliance with the License.
-  You may obtain a copy of the License at
-      http://www.apache.org/licenses/LICENSE-2.0
-  Unless required by applicable law or agreed to in writing, software
-  distributed under the License is distributed on an "AS IS" BASIS,
-  WITHOUT WARRANTIES OR CONDITIONS OF ANY KIND, either express or implied.
-  See the License for the specific language governing permissions and
-  limitations under the License.
--->
+<?xml version="1.0"?>
 <robot xmlns:xacro="http://ros.org/wiki/xacro">
   <xacro:macro name="arm_simple_transmission" params="name number reduction offset_value" >
@@ -22,6 +10,20 @@
         <offset>${offset_value}</offset>
         <hardwareInterface>hardware_interface/PositionJointInterface</hardwareInterface>
+        <hardwareInterface>hardware_interface/EffortJointInterface</hardwareInterface>
         <hardwareInterface>hardware_interface/VelocityJointInterface</hardwareInterface>
+        <hardwareInterface>hardware_interface/JointStateInterface</hardwareInterface>
+      </joint>
+    </transmission>
+  </xacro:macro>
+  <xacro:macro name="arm_sea_simple_transmission" params="name number offset_value" >
+    <transmission name="${name}_${number}_trans">
+      <type>sea_transmissions/SeaSimpleTransmission</type><!--transmission_interface/SeaTransmission-->
+      <actuator name="${name}_${number}_motor" >
+      </actuator>
+      <joint name="${name}_${number}_joint">
+        <offset>${offset_value}</offset>
+        <hardwareInterface>hardware_interface/PositionJointInterface</hardwareInterface>
         <hardwareInterface>hardware_interface/EffortJointInterface</hardwareInterface>
+        <hardwareInterface>hardware_interface/VelocityJointInterface</hardwareInterface>
         <hardwareInterface>hardware_interface/JointStateInterface</hardwareInterface>
       </joint>

Commit message: remove old meshes, only uses the right arm, add calibration constants

File: tiago_sea_arm_description/robots/tiago_sea_arm.urdf.xacro (robot description, xacro)
@@ -19,22 +19,4 @@
   <xacro:property name="end_effector" value="$(arg end_effector)" />
   <xacro:property name="ft_sensor" value="$(arg ft_sensor)" />
-  <!-- BASE LINK -->
-  <link name="base_link">
-    <visual>
-      <origin xyz="0 0 0" rpy="0 0 0" />
-      <geometry>
-        <mesh filename="package://tiago_sea_arm_description/meshes/base_link.STL" />
-      </geometry>
-      <material name="">
-        <color rgba="0.75294 0.75294 0.75294 1" />
-      </material>
-    </visual>
-    <collision>
-      <origin xyz="0 0 0" rpy="0 0 0" />
-      <geometry>
-        <mesh filename="package://tiago_sea_arm_description/meshes/base_link.STL" />
-      </geometry>
-    </collision>
-  </link>
   <!-- ARM -->
   <xacro:tiago_sea_arm name="arm_right" parent="base_link" reflect="1" ft_sensor="${ft_sensor}" arm_1_offset="0" arm_2_offset="0" arm_3_offset="0" arm_4_offset="0" arm_5_offset="0" arm_6_offset="0" arm_7_offset="0"/>
