Commit message: remove old meshes, only uses the right arm, add calibration constants

File: tiago_sea_arm_description/urdf/calibration_constants.urdf.xacro (robot description, xacro)
@@ -7,4 +7,10 @@
  	<xacro:include filename="$(find tiago_sea_arm_description)/urdf/deg_to_rad.xacro" />
 	<!--Constant parameters-->
+	<xacro:property name="camera_position_x" value="0.0908" />
+	<xacro:property name="camera_position_y" value="0.08" />
+	<xacro:property name="camera_position_z" value="0.0" />
+	<xacro:property name="camera_orientation_r" value="${-90 * deg_to_rad}" />
+	<xacro:property name="camera_orientation_p" value="0.0" />
+	<xacro:property name="camera_orientation_y" value="0.0" />
 	<xacro:property name="head_2_joint_offset" value="0" />
 	<xacro:property name="head_1_joint_offset" value="0" />

Commit message: Update robot urdf

File: tiago_sea_arm_description/robots/tiago_sea_arm.urdf.xacro (robot description, xacro)
@@ -19,6 +19,35 @@
   <xacro:property name="end_effector" value="$(arg end_effector)" />
   <xacro:property name="ft_sensor" value="$(arg ft_sensor)" />
+   <link name="world"/>
+    <joint name="world_fixed" type="fixed">
+        <origin xyz="0 0 0" rpy="0 0 0"/>
+        <parent link="world"/>
+        <child link="arm_root_link"/>
+    </joint>
+    <link name="arm_root_link">
+        <visual>
+            <origin xyz="0 0 0.5" rpy="0 0 0"/>
+            <geometry>
+                <box size="0.1 0.1 1.0"/>
+            </geometry>
+        </visual>
+        <collision>
+            <origin xyz="0 0 0.5" rpy="0 0 0"/>
+            <geometry>
+                <box size="0.1 0.1 1.0"/>
+            </geometry>
+        </collision>
+        <inertial>
+            <mass value="1e2" />
+            <origin xyz="0.0 0.0 0.0" />
+            <inertia ixx = "0.000001" ixy = "0.000000" ixz = "0.000000"
+                     iyx = "0.000000" iyy = "0.000001" iyz = "0.000000"
+                     izx = "0.000000" izy = "0.000000" izz = "0.000001" />
+        </inertial>
+    </link>
   <!-- ARM -->
-  <xacro:tiago_sea_arm name="arm_right" parent="base_link" reflect="1" ft_sensor="${ft_sensor}" arm_1_offset="0" arm_2_offset="0" arm_3_offset="0" arm_4_offset="0" arm_5_offset="0" arm_6_offset="0" arm_7_offset="0"/>
-  <xacro:tiago_sea_arm_end_effector name="gripper" parent="arm_right_7_link" type="${end_effector}"/>
+  <xacro:tiago_sea_arm name="arm" parent="arm_root_link" reflect="1" ft_sensor="${ft_sensor}" tiago_dual="-1" arm_1_offset="0" arm_2_offset="0" arm_3_offset="0" arm_4_offset="0" arm_5_offset="0" arm_6_offset="0" arm_7_offset="0">
+          <origin xyz="0.05 0 0.85" rpy="0 1.5708 0"/>
+  </xacro:tiago_sea_arm>
+  <xacro:tiago_sea_arm_end_effector name="gripper" parent="arm_7_link" type="${end_effector}"/>
 </robot>

Commit message: Add ft_sensor to TIAGo sea

File: tiago_sea_arm_description/robots/tiago_sea_arm.urdf.xacro (robot description, xacro)
@@ -15,41 +15,56 @@
   <xacro:include filename="$(find tiago_sea_arm_description)/urdf/arm/arm.urdf.xacro"/>
   <xacro:include filename="$(find tiago_sea_arm_description)/urdf/end_effector/end_effector.urdf.xacro"/>
+  <xacro:include filename="$(find tiago_sea_arm_description)/urdf/sensors/ft_sensor.urdf.xacro" />
+  <!-- Materials for visualization -->
+  <xacro:include filename="$(find tiago_description)/urdf/materials.urdf.xacro" />
   <xacro:arg name="end_effector" default="false"/>
   <xacro:arg name="ft_sensor" default="false"/>
   <xacro:property name="end_effector" value="$(arg end_effector)" />
   <xacro:property name="ft_sensor" value="$(arg ft_sensor)" />
-   <link name="world"/>
-    <joint name="world_fixed" type="fixed">
-        <origin xyz="0 0 0" rpy="0 0 0"/>
-        <parent link="world"/>
-        <child link="arm_root_link"/>
-    </joint>
-    <link name="arm_root_link">
-        <visual>
-            <origin xyz="0 0 0.5" rpy="0 0 0"/>
-            <geometry>
-                <box size="0.1 0.1 1.0"/>
-            </geometry>
-        </visual>
-        <collision>
-            <origin xyz="0 0 0.5" rpy="0 0 0"/>
-            <geometry>
-                <box size="0.1 0.1 1.0"/>
-            </geometry>
-        </collision>
-        <inertial>
-            <mass value="1e2" />
-            <origin xyz="0.0 0.0 0.0" />
-            <inertia ixx = "0.000001" ixy = "0.000000" ixz = "0.000000"
-                     iyx = "0.000000" iyy = "0.000001" iyz = "0.000000"
-                     izx = "0.000000" izy = "0.000000" izz = "0.000001" />
-        </inertial>
-    </link>
+  <xacro:if value="${end_effector not in ['false', False, 'pal-pro-gripper']}">
+    <xacro:wrong_end_effector/>
+  </xacro:if>
+  <xacro:if value="${ft_sensor not in ['false', False, 'ati']}">
+    <xacro:wrong_ft_sensor/>
+  </xacro:if>
+  <xacro:property name="has_ft_sensor"           value="${ft_sensor in ['ati']}"/>
+  <xacro:property name="has_end_effector"        value="${end_effector not in ['false', False, 'no-ee']}"/>
+  <xacro:property name="end_effector_link"       value="${'arm_ft_tool_link' if has_ft_sensor else 'arm_tool_link'}"/>
+  <link name="world"/>
+  <joint name="world_fixed" type="fixed">
+      <origin xyz="0 0 0" rpy="0 0 0"/>
+      <parent link="world"/>
+      <child link="arm_root_link"/>
+  </joint>
+  <link name="arm_root_link">
+      <visual>
+          <origin xyz="0 0 0.5" rpy="0 0 0"/>
+          <geometry>
+              <box size="0.1 0.1 1.0"/>
+          </geometry>
+      </visual>
+      <collision>
+          <origin xyz="0 0 0.5" rpy="0 0 0"/>
+          <geometry>
+              <box size="0.1 0.1 1.0"/>
+          </geometry>
+      </collision>
+      <inertial>
+          <mass value="1e2" />
+          <origin xyz="0.0 0.0 0.0" />
+          <inertia ixx = "0.000001" ixy = "0.000000" ixz = "0.000000"
+                   iyx = "0.000000" iyy = "0.000001" iyz = "0.000000"
+                   izx = "0.000000" izy = "0.000000" izz = "0.000001" />
+      </inertial>
+  </link>
   <!-- Generic simulator_gazebo plugins -->
-  <xacro:include filename="$(find tiago_sea_description)/gazebo/gazebo.urdf.xacro" />
+  <xacro:include filename="$(find tiago_sea_arm_description)/gazebo/gazebo.urdf.xacro" />
   <!-- ARM -->
   <xacro:tiago_sea_arm name="arm" parent="arm_root_link" reflect="1" ft_sensor="${ft_sensor}" tiago_dual="-1" arm_1_offset="0" arm_2_offset="0" arm_3_offset="0" arm_4_offset="0" arm_5_offset="0" arm_6_offset="0" arm_7_offset="0">
-          <origin xyz="0.05 0 0.85" rpy="0 1.5708 0"/>
+          <origin xyz="0 0 1.0" rpy="0 0 0"/>
   </xacro:tiago_sea_arm>
-  <xacro:tiago_sea_arm_end_effector name="gripper" parent="arm_7_link" type="${end_effector}"/>
+  <xacro:tiago_sea_arm_end_effector name="gripper" parent="${end_effector_link}" type="${end_effector}" has_end_effector="${has_end_effector}" reflect="1"/>
+  <xacro:if value="${ft_sensor == 'ati'}">
+    <xacro:ft_sensor name="arm" parent="arm_tool_link" reflect="1"/>
+  </xacro:if>
 </robot>

File: tiago_sea_arm_description/urdf/arm/arm.urdf.xacro (robot description, xacro)
@@ -348,29 +348,9 @@
     <!--        TOOL           -->
     <!--***********************-->
-    <link name="${name}_tool_link">
-      <inertial>
-        <mass value="0.1" />
-        <inertia ixx="8.33E-07" ixy="0.0" ixz="0.0" iyy="8.33E-07" iyz="0.0" izz="1.25E-06" />
-      </inertial>
-      <visual>
-        <origin xyz="0.001 0 0" rpy="0 ${90.0 * deg_to_rad} 0" />
-        <geometry>
-          <cylinder radius="0.005" length="0.005"/>
-        </geometry>
-        <material name="LightGrey" />
-      </visual>
-      <collision>
-        <origin xyz="0.001 0 0" rpy="0 ${90.0 * deg_to_rad} 0" />
-        <geometry>
-          <cylinder radius="0.005" length="0.005"/>
-        </geometry>
-      </collision>
-    </link>
-    <!-- TODO: get correct offset with and without ft -->
-    <xacro:property name="tool_link_z_offset"           value="${ 0.046 if ft_sensor == 'ati' else 0.0573 }"/>
+    <link name="${name}_tool_link"/>
     <joint name="${name}_tool_joint" type="fixed">
       <parent link="${name}_7_link" />
       <child link="${name}_tool_link" />
-      <origin xyz="0 0 ${-reflect * tool_link_z_offset}" rpy="${0.0 * deg_to_rad} ${90.0 * reflect * deg_to_rad} ${0 * deg_to_rad}" />
+      <origin xyz="0 0 0" rpy="${0.0 * deg_to_rad} ${90.0 * reflect * deg_to_rad} ${0 * deg_to_rad}" />
     </joint>
    <gazebo reference="${name}_1_link">

File: tiago_sea_arm_description/urdf/end_effector/end_effector.urdf.xacro (robot description, xacro)
@@ -1,5 +1,5 @@
 <?xml version="1.0"?>
 <!--
-  Copyright (c) 2023 PAL Robotics S.L. All rights reserved.
+  Copyright (c) 2021 PAL Robotics S.L. All rights reserved.
   Licensed under the Apache License, Version 2.0 (the "License");
   you may not use this file except in compliance with the License.
@@ -13,13 +13,48 @@
 -->
 <robot xmlns:xacro="http://ros.org/wiki/xacro">
+  <!--File includes-->
   <xacro:include filename="$(find tiago_sea_arm_description)/urdf/deg_to_rad.xacro" />
-  <xacro:macro name="tiago_sea_arm_end_effector" params="name parent type">
-  <!-- Robotiq 2F-85 Gripper -->
-    <xacro:if value="${type == 'pal-pro-gripper'}">
-      <xacro:include filename="$(find pal_pro_gripper_description)/urdf/pro_gripper.urdf.xacro" />
-      <xacro:pal_pro_gripper name="${name}" parent="${parent}" >
-        <origin xyz="0 0 0" rpy="${0*deg_to_rad} ${180*deg_to_rad} ${0*deg_to_rad}"/>
-      </xacro:pal_pro_gripper>
+  <!--
+    Utiliy to create a tiago end effector (right or left).
+    Parameters:
+    - name: End effector name. The created links and joints are prepended with 'name_'
+    - parent: Parent link
+    - reflect: Set to 1 for a right end effector, or to -1 for a left end effector
+  -->
+  <xacro:macro name="tiago_sea_arm_end_effector" params="name parent type has_end_effector reflect is_dual:=false">
+  <!-- No end-effector -->
+  <xacro:if value="${not has_end_effector}">
+    <!-- Add nothing -->
+  </xacro:if>
+  <!-- TODO: Get correct transform for new gripper -->
+  <!-- PAL Pro Gripper -->
+  <xacro:if value="${type == 'pal-pro-gripper'}">
+    <xacro:include filename="$(find pal_pro_gripper_description)/urdf/pro_gripper.urdf.xacro" />
+    <xacro:pal_pro_gripper name="${name}" parent="${parent}" >
+      <origin xyz="0.052 0.0 0.0" rpy="0 ${90 * deg_to_rad} 0"/>
+    </xacro:pal_pro_gripper>
+  </xacro:if>
+  <!-- Custom -->
+  <xacro:if value="${type == 'custom' and not is_dual}">
+    <xacro:include filename="$(find custom_ee_description)/urdf/end-effector.urdf.xacro" />
+    <xacro:end_effector parent="${parent}">
+      <origin xyz="0.0 0 0" rpy="0 0 0"/>
+    </xacro:end_effector>
+  </xacro:if>
+  <!-- Custom dual-->
+  <xacro:if value="${type == 'custom' and is_dual}">
+    <xacro:if value="${reflect == 1}"> <!-- If right -->
+    <xacro:include filename="$(find custom_dual_ee_description)/urdf/end-effector-right.urdf.xacro" />
+    <xacro:end_effector_right parent="${parent}">
+      <origin xyz="0.0 0 0" rpy="0 0 0"/>
+    </xacro:end_effector_right>
     </xacro:if>
+    <xacro:if value="${reflect == -1}"> <!-- If left -->
+    <xacro:include filename="$(find custom_dual_ee_description)/urdf/end-effector-left.urdf.xacro" />
+    <xacro:end_effector_left parent="${parent}">
+      <origin xyz="0.0 0 0" rpy="0 0 0"/>
+    </xacro:end_effector_left>
+    </xacro:if>
+  </xacro:if>
   </xacro:macro>
 </robot>

File: tiago_sea_arm_description/urdf/sensors/ft_sensor.urdf.xacro (robot description, xacro)
@@ -13,60 +13,48 @@
 -->
 <robot xmlns:xacro="http://ros.org/wiki/xacro">
-  <xacro:macro name="ft_sensor" params="name parent">
+  <xacro:macro name="ft_sensor" params="name parent reflect">
     <!--************************-->
     <!--        ft sensor       -->
     <!--************************-->
     <link name="${name}_ft_link">
-      <inertial>
-        <mass value="0.1" />
-        <inertia ixx="1.6E-05" ixy="-2.0E-06" ixz="0.0" iyy="1.6E-05" iyz="0.0" izz="2.7E-05" />
-      </inertial>
-      <visual>
-        <origin xyz="0 0 0" rpy="0 0 0" />
-        <geometry>
-          <cylinder radius="${0.045*0.5}" length="0.0157"/>
-        </geometry>
-        <material name="LightGrey" />
-      </visual>
-      <collision>
-        <origin xyz="0 0 0" rpy="0 0 0" />
-        <geometry>
-          <cylinder radius="${0.045*0.5}" length="0.0157"/>
-        </geometry>
-      </collision>
+        <inertial>
+          <mass value="0.2657" />
+          <inertia ixx="268925.36" ixy="3102.05" ixz="5074.07" iyy="160140.92" iyz="4096.6" izz="268336.32" />
+        </inertial>
+        <visual>
+          <origin xyz="0.0 0.0 -0.050" rpy="${90.0 * deg_to_rad} 0 ${45.0 * deg_to_rad if reflect == '1' else 135 * deg_to_rad}"/>
+          <geometry>
+            <mesh filename="package://tiago_sea_arm_description/meshes/sensors/ati_ft_sensor.STL"/>
+          </geometry>
+          <material name="">
+            <color rgba="0.752941176470588 0.752941176470588 0.752941176470588 1" />
+          </material>
+        </visual>
+        <collision>
+          <origin xyz="0 0 -0.025" rpy="0 0 0" />
+          <geometry>
+            <cylinder radius="0.035" length="0.05"/>
+          </geometry>
+        </collision>
+        <collision>
+          <origin xyz="0.047 0 -0.040" rpy="0 0 0" />
+          <geometry>
+            <box size="0.025 0.012 0.04"/>
+          </geometry>
+        </collision>
     </link>
-<!-- TODO: Fix origin -->
     <joint name="${name}_ft_joint" type="fixed">
       <parent link="${parent}" />
       <child link="${name}_ft_link" />
-      <origin xyz="0 0 0" rpy="${90.0 * deg_to_rad} 0 ${90.0 * deg_to_rad}" />
+      <origin xyz="0.050 0 0" rpy="${-90.0 * deg_to_rad} ${45.0 * deg_to_rad} ${-90.0 * deg_to_rad}" />
     </joint>
     <!--***********************-->
     <!--       FT TOOL         -->
     <!--***********************-->
-    <link name="${name}_ft_tool_link">
-      <inertial>
-        <mass value="0.1" />
-        <inertia ixx="1.64E-05" ixy="0.0" ixz="0.0" iyy="1.64E-05" iyz="0.0" izz="3.125E-05" />
-      </inertial>
-      <visual>
-        <origin xyz="0.0 0 0" rpy="0 ${90.0 * deg_to_rad} 0" />
-        <geometry>
-          <cylinder radius="${0.05*0.5}" length="0.00975"/>
-        </geometry>
-        <material name="FlatBlack" />
-      </visual>
-      <collision>
-        <origin xyz="0.0 0 0" rpy="0 ${90.0 * deg_to_rad} 0" />
-        <geometry>
-          <cylinder radius="${0.05*0.5}" length="0.00975"/>
-        </geometry>
-      </collision>
-    </link>
-<!-- TODO: Fix origin -->
-    <joint name="${name}_tool_joint" type="fixed">
+    <link name="${name}_ft_tool_link"/>
+    <joint name="${name}_ft_tool_joint" type="fixed">
       <parent link="${name}_ft_link" />
       <child link="${name}_ft_tool_link" />
-      <origin xyz="0 0 0" rpy="${-90.0 * deg_to_rad} ${-90.0 * deg_to_rad} 0" />
+      <origin xyz="0 0 0.0" rpy="${45.0 * deg_to_rad} ${-90.0 * deg_to_rad} ${0.0 * deg_to_rad}" />
     </joint>
 </xacro:macro>

Commit message: Change ati to rokubi

File: tiago_sea_arm_description/robots/tiago_sea_arm.urdf.xacro (robot description, xacro)
@@ -25,8 +25,8 @@
     <xacro:wrong_end_effector/>
   </xacro:if>
-  <xacro:if value="${ft_sensor not in ['false', False, 'ati']}">
+  <xacro:if value="${ft_sensor not in ['false', False, 'rokubi']}">
     <xacro:wrong_ft_sensor/>
   </xacro:if>
-  <xacro:property name="has_ft_sensor"           value="${ft_sensor in ['ati']}"/>
+  <xacro:property name="has_ft_sensor"           value="${ft_sensor in ['rokubi']}"/>
   <xacro:property name="has_end_effector"        value="${end_effector not in ['false', False, 'no-ee']}"/>
   <xacro:property name="end_effector_link"       value="${'arm_ft_tool_link' if has_ft_sensor else 'arm_tool_link'}"/>
@@ -65,6 +65,6 @@
   </xacro:tiago_sea_arm>
   <xacro:tiago_sea_arm_end_effector name="gripper" parent="${end_effector_link}" type="${end_effector}" has_end_effector="${has_end_effector}" reflect="1"/>
-  <xacro:if value="${ft_sensor == 'ati'}">
-    <xacro:ft_sensor name="arm" parent="arm_tool_link" reflect="1"/>
+  <xacro:if value="${has_ft_sensor}">
+    <xacro:ft_sensor name="arm" parent="arm_tool_link"/>
   </xacro:if>
 </robot>

File: tiago_sea_arm_description/urdf/sensors/ft_sensor.urdf.xacro (robot description, xacro)
@@ -13,5 +13,5 @@
 -->
 <robot xmlns:xacro="http://ros.org/wiki/xacro">
-  <xacro:macro name="ft_sensor" params="name parent reflect">
+  <xacro:macro name="ft_sensor" params="name parent">
     <!--************************-->
     <!--        ft sensor       -->
@@ -25,5 +25,5 @@
           <origin xyz="0.0 0.0 0.0" rpy="0.0 0.0 0.0"/>
           <geometry>
-            <mesh filename="package://tiago_sea_arm_description/meshes/sensors/ati_ft_sensor.STL"/>
+            <mesh filename="package://tiago_sea_arm_description/meshes/sensors/rokubi_ft_sensor.STL"/>
           </geometry>
           <material name="">

Commit message: Add new meshes of the arm

File: tiago_sea_arm_description/robots/tiago_sea_arm.urdf.xacro (robot description, xacro)
@@ -61,5 +61,5 @@
   <xacro:include filename="$(find tiago_sea_arm_description)/gazebo/gazebo.urdf.xacro" />
   <!-- ARM -->
-  <xacro:tiago_sea_arm name="arm" parent="arm_root_link" reflect="1" ft_sensor="${ft_sensor}" tiago_dual="-1" arm_1_offset="0" arm_2_offset="0" arm_3_offset="0" arm_4_offset="0" arm_5_offset="0" arm_6_offset="0" arm_7_offset="0">
+  <xacro:tiago_sea_arm name="arm" parent="arm_root_link" reflect="-1" ft_sensor="${ft_sensor}" tiago_dual="-1" arm_1_offset="0" arm_2_offset="0" arm_3_offset="0" arm_4_offset="0" arm_5_offset="0" arm_6_offset="0" arm_7_offset="0">
           <origin xyz="0 0 1.0" rpy="0 0 0"/>
   </xacro:tiago_sea_arm>

File: tiago_sea_arm_description/urdf/arm/arm.urdf.xacro (robot description, xacro)
@@ -76,5 +76,5 @@
     <xacro:property name="arm_1_lower_limit"       value="${-90 if tiago_dual == 1 else 0.0}"/>
     <joint name="${name}_1_joint" type="revolute">
-      <origin xyz="0.0 0.0 0.02" rpy=" 0 ${(90 - 90 * reflect) * deg_to_rad } ${-90 * deg_to_rad}" />
+      <origin xyz="0.0 0.0 0.0" rpy=" 0 ${(90 - 90 * reflect) * deg_to_rad } 0" />
       <parent link="${name}_base_link" />
       <child link="${name}_1_link" />
@@ -117,6 +117,6 @@
     <xacro:property name="arm_2_lower_limit"       value="${-90 if tiago_dual == 1 else -62.5}"/>
     <joint name="${name}_2_joint" type="revolute">
-      <origin xyz="0.13 -0.0483 ${-0.04* reflect}"
-        rpy="${90 * reflect * deg_to_rad} 0 ${180 * deg_to_rad}" />
+      <origin xyz="0 0.13 ${-0.01989* reflect}"
+        rpy="${90 * reflect * deg_to_rad} 0 -1.5708" />
       <parent link="${name}_1_link" />
       <child link="${name}_2_link" />
@@ -160,6 +160,6 @@
     <xacro:property name="arm_3_upper_limit"       value="${225 if tiago_dual == 1 else 170}"/>
     <joint name="${name}_3_joint" type="revolute">
-     <origin xyz="-0.1549 0 ${0.05 * reflect}"
-        rpy="0 ${90 * reflect * deg_to_rad} 0" />
+     <origin xyz="-0.13455 0 ${-0.0019939 * reflect}"
+        rpy="3.1416 ${90 * reflect * deg_to_rad} 0" />
       <parent link="${name}_2_link" />
       <child
@@ -203,6 +203,6 @@
     </link>
     <joint name="${name}_4_joint" type="revolute">
-     <origin xyz="0.05 0.02 ${-0.1651 * reflect}"
-        rpy="${90 * reflect * deg_to_rad} ${-25 * reflect * deg_to_rad} ${-90 * deg_to_rad}" />
+     <origin xyz="0.0019939 0.02 ${0.18521 * reflect}"
+        rpy="0 ${90 * reflect * deg_to_rad} 0" />
       <parent
         link="${name}_3_link" />
@@ -246,6 +246,6 @@
     </link>
     <joint name="${name}_5_joint" type="revolute">
-     <origin xyz="-0.04738 -0.1489 ${0.05 * reflect}"
-        rpy="${90 * reflect * deg_to_rad} 0 ${155 * deg_to_rad}" />
+     <origin xyz="-0.1345 -0.02 ${-0.0022914 * reflect}"
+        rpy="3.1416 ${90 * reflect * deg_to_rad}  0" />
       <parent link="${name}_4_link" />
       <child
@@ -289,6 +289,6 @@
     </link>
     <joint name="${name}_6_joint" type="revolute">
-     <origin xyz="0 -0.0395 ${-0.1651 * reflect}"
-        rpy="${90 * reflect * deg_to_rad} 0 ${180 * deg_to_rad}" />
+     <origin xyz="0.0022914 0 ${0.18516 * reflect}"
+        rpy="0 ${90 * reflect * deg_to_rad} 0" />
       <parent link="${name}_5_link" />
       <child
@@ -332,6 +332,6 @@
     </link>
     <joint name="${name}_7_joint" type="revolute">
-     <origin xyz="0 -0.146 ${0.039 * reflect}"
-        rpy="0 ${90 * reflect * deg_to_rad} ${90 * deg_to_rad}" />
+     <origin xyz="-0.1278 0 ${-0.001497 * reflect}"
+        rpy="3.1416 ${90 * reflect * deg_to_rad} 0" />
       <parent link="${name}_6_link" />
       <child
@@ -370,5 +370,5 @@
       <parent link="${name}_7_link" />
       <child link="${name}_tool_link" />
-      <origin xyz="0 0 0" rpy="${0.0 * deg_to_rad} ${90.0 * reflect * deg_to_rad} ${0 * deg_to_rad}" />
+      <origin xyz="0 0 0" rpy="${0.0 * deg_to_rad} ${-90.0 * reflect * deg_to_rad} ${0 * deg_to_rad}" />
     </joint>
    <gazebo reference="${name}_1_link">
