Commit message: update arm joint limits based on visual limit

File: tiago_sea_arm_description/urdf/arm/arm.limits.xacro (robot description, xacro)
@@ -6,12 +6,12 @@
   <xacro:property name="arm_k_velocity" value="20"/>
   <!-- TODO: Check these values -->
-  <xacro:property name="arm_4_joint_ub" value="1.60868" />
-  <xacro:property name="arm_4_joint_lb" value="-2.41302" />
-  <xacro:property name="arm_5_joint_ub" value="2.54185" />
-  <xacro:property name="arm_5_joint_lb" value="-2.54185" />
-  <xacro:property name="arm_6_joint_ub" value="2.1562" />
-  <xacro:property name="arm_6_joint_lb" value="-2.1562" />
-  <xacro:property name="arm_7_joint_ub" value="1.3701" />
-  <xacro:property name="arm_7_joint_lb" value="-3.6" />
+  <xacro:property name="arm_4_joint_ub" value="60" />
+  <xacro:property name="arm_4_joint_lb" value="-130" />
+  <xacro:property name="arm_5_joint_ub" value="145" />
+  <xacro:property name="arm_5_joint_lb" value="-145" />
+  <xacro:property name="arm_6_joint_ub" value="114" />
+  <xacro:property name="arm_6_joint_lb" value="-114" />
+  <xacro:property name="arm_7_joint_ub" value="145" />
+  <xacro:property name="arm_7_joint_lb" value="-145" />
   <xacro:property name="arm_1_max_velocity"      value="1.95" />
   <xacro:property name="arm_2_max_velocity"      value="1.95" />

File: tiago_sea_arm_description/urdf/arm/arm.urdf.xacro (robot description, xacro)
@@ -2,4 +2,5 @@
 <robot xmlns:xacro="http://ros.org/wiki/xacro">
   <!-- File includes -->
+  <xacro:include filename="$(find tiago_sea_arm_description)/urdf/deg_to_rad.xacro" />
   <xacro:include filename="$(find tiago_sea_arm_description)/urdf/arm/arm.transmission.xacro" />
   <xacro:include filename="$(find tiago_sea_arm_description)/urdf/arm/arm.limits.xacro" />
@@ -72,4 +73,6 @@
       </collision>
     </link>
+    <xacro:property name="arm_1_upper_limit"       value="${90.0 if tiago_dual == 1 else 180}"/>
+    <xacro:property name="arm_1_lower_limit"       value="${-67.5 if tiago_dual == 1 else 0.0}"/>
     <joint name="${name}_1_joint" type="revolute">
       <origin xyz="0.0 0.0 0.02" rpy=" 0 ${(90 - 90 * reflect) * deg_to_rad } ${-90 * deg_to_rad}" />
@@ -77,8 +80,8 @@
       <child link="${name}_1_link" />
       <axis xyz="0 0 ${1}" />
-      <limit lower="-0.8480" upper="1.5639" effort="${arm_1_max_effort}" velocity="${arm_1_max_velocity}" />
+      <limit lower="${arm_1_lower_limit * deg_to_rad}" upper="${arm_1_upper_limit * deg_to_rad}" effort="${arm_1_max_effort}" velocity="${arm_1_max_velocity}" />
       <dynamics friction="${arm_friction}" damping="${arm_damping}"/>
-      <safety_controller k_position="${arm_k_position}" k_velocity="${arm_k_velocity}" soft_lower_limit="${-0.8480  + arm_eps}"
-        soft_upper_limit="${1.5639 - arm_eps}" />
+      <safety_controller k_position="${arm_k_position}" k_velocity="${arm_k_velocity}" soft_lower_limit="${arm_1_lower_limit * deg_to_rad  + arm_eps}"
+        soft_upper_limit="${arm_1_upper_limit * deg_to_rad - arm_eps}" />
     </joint>
     <link name="${name}_2_link">
@@ -111,4 +114,6 @@
       </collision>
     </link>
+    <xacro:property name="arm_2_upper_limit"       value="${90.0 if tiago_dual == 1 else 62.5}"/>
+    <xacro:property name="arm_2_lower_limit"       value="${-67.5 if tiago_dual == 1 else -90.0}"/>
     <joint name="${name}_2_joint" type="revolute">
       <origin xyz="0.13 -0.0483 ${-0.04* reflect}"
@@ -117,8 +122,8 @@
       <child link="${name}_2_link" />
       <axis xyz="0 0 ${1}" />
-      <limit lower="-1.5922" upper="1.5922" effort="${arm_2_max_effort}" velocity="${arm_2_max_velocity}" />
+      <limit lower="${arm_2_lower_limit * deg_to_rad}" upper="${arm_2_upper_limit * deg_to_rad}" effort="${arm_2_max_effort}" velocity="${arm_2_max_velocity}" />
       <dynamics friction="${arm_friction}" damping="${arm_damping}"/>
-      <safety_controller k_position="${arm_k_position}" k_velocity="${arm_k_velocity}" soft_lower_limit="${-1.5922  + arm_eps}"
-        soft_upper_limit="${1.5922 - arm_eps}" />
+      <safety_controller k_position="${arm_k_position}" k_velocity="${arm_k_velocity}" soft_lower_limit="${arm_2_lower_limit * deg_to_rad  + arm_eps}"
+        soft_upper_limit="${arm_2_upper_limit * deg_to_rad - arm_eps}" />
     </joint>
     <link name="${name}_3_link">
@@ -152,4 +157,6 @@
       </collision>
     </link>
+    <xacro:property name="arm_3_lower_limit"       value="${-45 if tiago_dual == 1 else -148}"/>
+    <xacro:property name="arm_3_upper_limit"       value="${225 if tiago_dual == 1 else 148}"/>
     <joint name="${name}_3_joint" type="revolute">
      <origin xyz="-0.1549 0 ${0.05 * reflect}"
@@ -159,10 +166,10 @@
         link="${name}_3_link" />
       <axis xyz="0 0 1" />
-      <limit lower="-2.53135" upper="2.53135"
+      <limit lower="${arm_3_lower_limit * deg_to_rad}" upper="${arm_3_upper_limit * deg_to_rad}"
         effort="${arm_3_max_effort}" velocity="${arm_3_max_velocity}" />
        <dynamics friction="${arm_friction}" damping="${arm_damping}"/>
       <safety_controller k_position="${arm_k_position}" k_velocity="${arm_k_velocity}"
-        soft_lower_limit="${-2.53135  + arm_eps}"
-        soft_upper_limit="${2.53135 - arm_eps}" />
+        soft_lower_limit="${arm_3_lower_limit * deg_to_rad  + arm_eps}"
+        soft_upper_limit="${arm_3_upper_limit * deg_to_rad - arm_eps}" />
     </joint>
     <link name="${name}_4_link">
@@ -203,9 +210,9 @@
       <axis xyz="0 0 1" />
       <limit
-        lower="${arm_4_joint_lb}" upper="${arm_4_joint_ub}" effort="${arm_4_max_effort}" velocity="${arm_4_max_velocity}" />
+        lower="${arm_4_joint_lb * deg_to_rad}" upper="${arm_4_joint_ub * deg_to_rad}" effort="${arm_4_max_effort}" velocity="${arm_4_max_velocity}" />
        <dynamics friction="${arm_friction}" damping="${arm_damping}"/>
       <safety_controller
-        k_position="${arm_k_position}" k_velocity="${arm_k_velocity}" soft_lower_limit="${arm_4_joint_lb  + arm_eps}"
-        soft_upper_limit="${arm_4_joint_ub - arm_eps}" />
+        k_position="${arm_k_position}" k_velocity="${arm_k_velocity}" soft_lower_limit="${arm_4_joint_lb * deg_to_rad  + arm_eps}"
+        soft_upper_limit="${arm_4_joint_ub * deg_to_rad - arm_eps}" />
     </joint>
     <link name="${name}_5_link">
@@ -246,9 +253,9 @@
       <axis xyz="0 0 1" />
       <limit
-        lower="${arm_5_joint_lb}" upper="${arm_5_joint_ub}" effort="${arm_5_max_effort}" velocity="${arm_5_max_velocity}" />
+        lower="${arm_5_joint_lb * deg_to_rad}" upper="${arm_5_joint_ub * deg_to_rad}" effort="${arm_5_max_effort}" velocity="${arm_5_max_velocity}" />
        <dynamics friction="${arm_friction}" damping="${arm_damping}"/>
       <safety_controller
-        k_position="${arm_k_position}" k_velocity="${arm_k_velocity}" soft_lower_limit="${arm_5_joint_lb  + arm_eps}"
-        soft_upper_limit="${arm_5_joint_ub - arm_eps}" />
+        k_position="${arm_k_position}" k_velocity="${arm_k_velocity}" soft_lower_limit="${arm_5_joint_lb * deg_to_rad  + arm_eps}"
+        soft_upper_limit="${arm_5_joint_ub * deg_to_rad - arm_eps}" />
     </joint>
     <link name="${name}_6_link">
@@ -289,9 +296,9 @@
       <axis xyz="0 0 1" />
       <limit
-        lower="${arm_6_joint_lb}" upper="${arm_6_joint_ub}" effort="${arm_6_max_effort}" velocity="${arm_6_max_velocity}" />
+        lower="${arm_6_joint_lb * deg_to_rad}" upper="${arm_6_joint_ub * deg_to_rad}" effort="${arm_6_max_effort}" velocity="${arm_6_max_velocity}" />
        <dynamics friction="${arm_friction}" damping="${arm_damping}"/>
       <safety_controller
-        k_position="${arm_k_position}" k_velocity="${arm_k_velocity}" soft_lower_limit="${arm_6_joint_lb  + arm_eps}"
-        soft_upper_limit="${arm_6_joint_ub - arm_eps}" />
+        k_position="${arm_k_position}" k_velocity="${arm_k_velocity}" soft_lower_limit="${arm_6_joint_lb * deg_to_rad  + arm_eps}"
+        soft_upper_limit="${arm_6_joint_ub * deg_to_rad - arm_eps}" />
     </joint>
     <link name="${name}_7_link">
@@ -332,9 +339,9 @@
       <axis xyz="0 0 1" />
       <limit
-        lower="${arm_7_joint_lb}" upper="${arm_7_joint_ub}" effort="${arm_7_max_effort}" velocity="${arm_7_max_velocity}" />
+        lower="${arm_7_joint_lb * deg_to_rad}" upper="${arm_7_joint_ub * deg_to_rad}" effort="${arm_7_max_effort}" velocity="${arm_7_max_velocity}" />
        <dynamics friction="${arm_friction}" damping="${arm_damping}"/>
       <safety_controller
-        k_position="${arm_k_position}" k_velocity="${arm_k_velocity}" soft_lower_limit="${arm_7_joint_lb  + arm_eps}"
-        soft_upper_limit="${arm_7_joint_ub - arm_eps}" />
+        k_position="${arm_k_position}" k_velocity="${arm_k_velocity}" soft_lower_limit="${arm_7_joint_lb * deg_to_rad  + arm_eps}"
+        soft_upper_limit="${arm_7_joint_ub * deg_to_rad - arm_eps}" />
     </joint>
     <!--***********************-->

Commit message: Update joint limits for tiago dual

File: tiago_sea_arm_description/urdf/arm/arm.limits.xacro (robot description, xacro)
@@ -6,6 +6,6 @@
   <xacro:property name="arm_k_velocity" value="20"/>
   <!-- TODO: Check these values -->
-  <xacro:property name="arm_4_joint_ub" value="60" />
-  <xacro:property name="arm_4_joint_lb" value="-130" />
+  <xacro:property name="arm_4_joint_ub" value="90" />
+  <xacro:property name="arm_4_joint_lb" value="-140" />
   <xacro:property name="arm_5_joint_ub" value="145" />
   <xacro:property name="arm_5_joint_lb" value="-145" />

File: tiago_sea_arm_description/urdf/arm/arm.urdf.xacro (robot description, xacro)
@@ -74,5 +74,5 @@
     </link>
     <xacro:property name="arm_1_upper_limit"       value="${90.0 if tiago_dual == 1 else 180}"/>
-    <xacro:property name="arm_1_lower_limit"       value="${-67.5 if tiago_dual == 1 else 0.0}"/>
+    <xacro:property name="arm_1_lower_limit"       value="${-48.5 if tiago_dual == 1 else 0.0}"/>
     <joint name="${name}_1_joint" type="revolute">
       <origin xyz="0.0 0.0 0.02" rpy=" 0 ${(90 - 90 * reflect) * deg_to_rad } ${-90 * deg_to_rad}" />
@@ -115,5 +115,5 @@
     </link>
     <xacro:property name="arm_2_upper_limit"       value="${90.0 if tiago_dual == 1 else 90}"/>
-    <xacro:property name="arm_2_lower_limit"       value="${-67.5 if tiago_dual == 1 else -90.0}"/>
+    <xacro:property name="arm_2_lower_limit"       value="${-90 if tiago_dual == 1 else -90.0}"/>
     <joint name="${name}_2_joint" type="revolute">
       <origin xyz="0.13 -0.0483 ${-0.04* reflect}"
@@ -157,6 +157,6 @@
       </collision>
     </link>
-    <xacro:property name="arm_3_lower_limit"       value="${-45 if tiago_dual == 1 else -170}"/>
-    <xacro:property name="arm_3_upper_limit"       value="${225 if tiago_dual == 1 else 170}"/>
+    <xacro:property name="arm_3_lower_limit"       value="${-145 if tiago_dual == 1 else -170}"/>
+    <xacro:property name="arm_3_upper_limit"       value="${145 if tiago_dual == 1 else 170}"/>
     <joint name="${name}_3_joint" type="revolute">
      <origin xyz="-0.1549 0 ${0.05 * reflect}"

Commit message: Update arm limits

File: tiago_sea_arm_description/urdf/arm/arm.limits.xacro (robot description, xacro)
@@ -8,6 +8,6 @@
   <xacro:property name="arm_1_joint_ub" value="90"/>
   <xacro:property name="arm_1_joint_lb" value="-90"/>
-  <xacro:property name="arm_2_joint_ub" value="62.5"/>
-  <xacro:property name="arm_2_joint_lb" value="-90"/>
+  <xacro:property name="arm_2_joint_ub" value="90"/>
+  <xacro:property name="arm_2_joint_lb" value="-62.5"/>
   <xacro:property name="arm_3_joint_ub" value="170"/>
   <xacro:property name="arm_3_joint_lb" value="-170"/>
