Commit message: Urdf only using meshes of right arm

File: tiago_sea_arm_description/urdf/arm/arm.urdf.xacro (robot description, xacro)
@@ -49,5 +49,5 @@
   <!-- ARM MACRO -->
   <!-- reflect: Set to 1 for a right arm, or to -1 for a left arm -->
-  <xacro:macro name="tiago_sea_arm" params="name parent reflect ft_sensor arm_1_offset arm_2_offset arm_3_offset arm_4_offset arm_5_offset arm_6_offset arm_7_offset no_safety_eps:=False">
+  <xacro:macro name="tiago_sea_arm" params="name parent *origin reflect ft_sensor tiago_dual arm_1_offset arm_2_offset arm_3_offset arm_4_offset arm_5_offset arm_6_offset arm_7_offset no_safety_eps:=False">
     <xacro:property name="arm_eps"       value="${0.00 if no_safety_eps else 0.07}"/>
     <!--  arm 1  -->

Commit message: Add joint transmissions and damping to urdf

File: tiago_sea_arm_description/urdf/arm/arm.urdf.xacro (robot description, xacro)
@@ -79,4 +79,5 @@
       <axis xyz="0 0 ${1}" />
       <limit lower="-0.8480" upper="1.5639" effort="${arm_1_max_effort}" velocity="${arm_1_max_velocity}" />
+      <dynamics friction="${arm_friction}" damping="${arm_damping}"/>
       <safety_controller k_position="${arm_k_position}" k_velocity="${arm_k_velocity}" soft_lower_limit="${-0.8480  + arm_eps}"
         soft_upper_limit="${1.5639 - arm_eps}" />
@@ -118,4 +119,5 @@
       <axis xyz="0 0 ${1}" />
       <limit lower="-1.5922" upper="1.5922" effort="${arm_2_max_effort}" velocity="${arm_2_max_velocity}" />
+      <dynamics friction="${arm_friction}" damping="${arm_damping}"/>
       <safety_controller k_position="${arm_k_position}" k_velocity="${arm_k_velocity}" soft_lower_limit="${-1.5922  + arm_eps}"
         soft_upper_limit="${1.5922 - arm_eps}" />
@@ -160,4 +162,5 @@
       <limit lower="-2.53135" upper="2.53135"
         effort="${arm_3_max_effort}" velocity="${arm_3_max_velocity}" />
+       <dynamics friction="${arm_friction}" damping="${arm_damping}"/>
       <safety_controller k_position="${arm_k_position}" k_velocity="${arm_k_velocity}"
         soft_lower_limit="${-2.53135  + arm_eps}"
@@ -202,4 +205,5 @@
       <limit
         lower="${arm_4_joint_lb}" upper="${arm_4_joint_ub}" effort="${arm_4_max_effort}" velocity="${arm_4_max_velocity}" />
+       <dynamics friction="${arm_friction}" damping="${arm_damping}"/>
       <safety_controller
         k_position="${arm_k_position}" k_velocity="${arm_k_velocity}" soft_lower_limit="${arm_4_joint_lb  + arm_eps}"
@@ -244,4 +248,5 @@
       <limit
         lower="${arm_5_joint_lb}" upper="${arm_5_joint_ub}" effort="${arm_5_max_effort}" velocity="${arm_5_max_velocity}" />
+       <dynamics friction="${arm_friction}" damping="${arm_damping}"/>
       <safety_controller
         k_position="${arm_k_position}" k_velocity="${arm_k_velocity}" soft_lower_limit="${arm_5_joint_lb  + arm_eps}"
@@ -286,4 +291,5 @@
       <limit
         lower="${arm_6_joint_lb}" upper="${arm_6_joint_ub}" effort="${arm_6_max_effort}" velocity="${arm_6_max_velocity}" />
+       <dynamics friction="${arm_friction}" damping="${arm_damping}"/>
       <safety_controller
         k_position="${arm_k_position}" k_velocity="${arm_k_velocity}" soft_lower_limit="${arm_6_joint_lb  + arm_eps}"
@@ -328,4 +334,5 @@
       <limit
         lower="${arm_7_joint_lb}" upper="${arm_7_joint_ub}" effort="${arm_7_max_effort}" velocity="${arm_7_max_velocity}" />
+       <dynamics friction="${arm_friction}" damping="${arm_damping}"/>
       <safety_controller
         k_position="${arm_k_position}" k_velocity="${arm_k_velocity}" soft_lower_limit="${arm_7_joint_lb  + arm_eps}"
@@ -361,4 +368,67 @@
       <origin xyz="0 0 ${-reflect * tool_link_z_offset}" rpy="${0.0 * deg_to_rad} ${90.0 * reflect * deg_to_rad} ${0 * deg_to_rad}" />
     </joint>
+   <gazebo reference="${name}_1_link">
+     <mu1>0.9</mu1>
+     <mu2>0.9</mu2>
+     <material>Gazebo/DarkGrey</material>
+   </gazebo>
+   <gazebo reference="${name}_2_link">
+     <mu1>0.9</mu1>
+     <mu2>0.9</mu2>
+     <material>Gazebo/DarkGrey</material>
+   </gazebo>
+   <gazebo reference="${name}_3_link">
+     <mu1>0.9</mu1>
+     <mu2>0.9</mu2>
+     <material>Gazebo/DarkGrey</material>
+   </gazebo>
+   <gazebo reference="${name}_4_link">
+     <mu1>0.9</mu1>
+     <mu2>0.9</mu2>
+     <material>Gazebo/DarkGrey</material>
+   </gazebo>
+    <gazebo reference="${name}_5_link">
+     <mu1>0.9</mu1>
+     <mu2>0.9</mu2>
+     <material>Gazebo/DarkGrey</material>
+   </gazebo>
+    <gazebo reference="${name}_6_link">
+     <mu1>0.9</mu1>
+     <mu2>0.9</mu2>
+     <material>Gazebo/DarkGrey</material>
+   </gazebo>
+    <gazebo reference="${name}_7_link">
+     <mu1>0.9</mu1>
+     <mu2>0.9</mu2>
+     <material>Gazebo/DarkGrey</material>
+   </gazebo>
+   <gazebo reference="${name}_1_joint">
+      <implicitSpringDamper>1</implicitSpringDamper>
+   </gazebo>
+   <gazebo reference="${name}_2_joint">
+      <implicitSpringDamper>1</implicitSpringDamper>
+   </gazebo>
+   <gazebo reference="${name}_3_joint">
+      <implicitSpringDamper>1</implicitSpringDamper>
+   </gazebo>
+   <gazebo reference="${name}_4_joint">
+      <implicitSpringDamper>1</implicitSpringDamper>
+   </gazebo>
+   <gazebo reference="${name}_5_joint">
+      <implicitSpringDamper>1</implicitSpringDamper>
+   </gazebo>
+   <gazebo reference="${name}_6_joint">
+      <implicitSpringDamper>1</implicitSpringDamper>
+   </gazebo>
+   <gazebo reference="${name}_7_joint">
+      <implicitSpringDamper>1</implicitSpringDamper>
+   </gazebo>
+    <xacro:arm_simple_transmission name="${name}" number="1" reduction="1.0" offset_value="${arm_1_offset}"/>
+    <xacro:arm_simple_transmission name="${name}" number="2" reduction="1.0" offset_value="${arm_2_offset}"/>
+    <xacro:arm_simple_transmission name="${name}" number="3" reduction="1.0" offset_value="${arm_3_offset}"/>
+    <xacro:arm_simple_transmission name="${name}" number="4" reduction="1.0" offset_value="${arm_4_offset}"/>
+    <xacro:arm_simple_transmission name="${name}" number="5" reduction="1.0" offset_value="${arm_4_offset}"/>
+    <xacro:arm_simple_transmission name="${name}" number="6" reduction="1.0" offset_value="${arm_4_offset}"/>
+    <xacro:arm_simple_transmission name="${name}" number="7" reduction="1.0" offset_value="${arm_4_offset}"/>
   </xacro:macro>
 </robot>

Commit message: Update joint limits based on visuals

File: tiago_sea_arm_description/urdf/arm/arm.urdf.xacro (robot description, xacro)
@@ -114,5 +114,5 @@
       </collision>
     </link>
-    <xacro:property name="arm_2_upper_limit"       value="${90.0 if tiago_dual == 1 else 62.5}"/>
+    <xacro:property name="arm_2_upper_limit"       value="${90.0 if tiago_dual == 1 else 90}"/>
     <xacro:property name="arm_2_lower_limit"       value="${-67.5 if tiago_dual == 1 else -90.0}"/>
     <joint name="${name}_2_joint" type="revolute">
@@ -157,6 +157,6 @@
       </collision>
     </link>
-    <xacro:property name="arm_3_lower_limit"       value="${-45 if tiago_dual == 1 else -148}"/>
-    <xacro:property name="arm_3_upper_limit"       value="${225 if tiago_dual == 1 else 148}"/>
+    <xacro:property name="arm_3_lower_limit"       value="${-45 if tiago_dual == 1 else -170}"/>
+    <xacro:property name="arm_3_upper_limit"       value="${225 if tiago_dual == 1 else 170}"/>
     <joint name="${name}_3_joint" type="revolute">
      <origin xyz="-0.1549 0 ${0.05 * reflect}"

Commit message: Update inertias

File: tiago_sea_arm_description/urdf/arm/arm.urdf.xacro (robot description, xacro)
@@ -48,7 +48,7 @@
         <origin xyz="0.1046 -0.0136 ${-0.0310 * reflect}" rpy="0 0 0" />
         <mass value="0.8770" />
-        <inertia ixx="1.8531E-03" ixy="8.3565E-05" ixz="${2.5620E-05 * reflect}"
-                 iyy="6.0021E-04" iyz="${-3.3154E-04 * reflect}"
-                 izz="1.6564E-03" />
+        <inertia ixx="6.0149E-04" ixy="8.3434E-05" ixz="${3.1716E-04 * reflect}"
+                 iyy="1.8511E-03" iyz="${-2.4871E-05 * reflect}"
+                 izz="1.6552E-03" />
       </inertial>
       <visual>
@@ -89,5 +89,5 @@
         <origin xyz="-0.1032 0 ${0.0403 * reflect}" rpy="0 0 0" />
         <mass value="0.7941" />
-        <inertia ixx="7.8558E-04" ixy="-2.0052E-07" ixz="${-2.8139E-04 * reflect}"
+        <inertia ixx="7.8558E-04" ixy="-2.0052E-07" ixz="${2.8139E-04 * reflect}"
           iyy="1.2374E-03" iyz="${-9.5016E-07 * reflect}"
           izz="1.2876E-03" />
@@ -177,5 +177,5 @@
         <origin xyz="-0.02709 -0.0989 ${reflect * 0.0405}" rpy="0 0 0" />
         <mass value="0.8229" />
-        <inertia ixx="1.3428E-03" ixy="1.0575E-04" ixz="${8.8477E-05 * reflect}"
+        <inertia ixx="1.3428E-03" ixy="-1.0575E-04" ixz="${8.8477E-05 * reflect}"
           iyy="8.2512E-04" iyz="${3.0671E-04 * reflect}"
           izz="1.3987E-03" />

Commit message: update arm_link_1 limit for tiago_dual

File: tiago_sea_arm_description/urdf/arm/arm.urdf.xacro (robot description, xacro)
@@ -74,5 +74,5 @@
     </link>
     <xacro:property name="arm_1_upper_limit"       value="${90.0 if tiago_dual == 1 else 180}"/>
-    <xacro:property name="arm_1_lower_limit"       value="${-48.5 if tiago_dual == 1 else 0.0}"/>
+    <xacro:property name="arm_1_lower_limit"       value="${-90 if tiago_dual == 1 else 0.0}"/>
     <joint name="${name}_1_joint" type="revolute">
       <origin xyz="0.0 0.0 0.02" rpy=" 0 ${(90 - 90 * reflect) * deg_to_rad } ${-90 * deg_to_rad}" />

Commit message: Update arm joint limits

File: tiago_sea_arm_description/urdf/arm/arm.urdf.xacro (robot description, xacro)
@@ -115,5 +115,5 @@
     </link>
     <xacro:property name="arm_2_upper_limit"       value="${90.0 if tiago_dual == 1 else 90}"/>
-    <xacro:property name="arm_2_lower_limit"       value="${-90 if tiago_dual == 1 else -90.0}"/>
+    <xacro:property name="arm_2_lower_limit"       value="${-90 if tiago_dual == 1 else -62.5}"/>
     <joint name="${name}_2_joint" type="revolute">
       <origin xyz="0.13 -0.0483 ${-0.04* reflect}"
@@ -157,6 +157,6 @@
       </collision>
     </link>
-    <xacro:property name="arm_3_lower_limit"       value="${-145 if tiago_dual == 1 else -170}"/>
-    <xacro:property name="arm_3_upper_limit"       value="${145 if tiago_dual == 1 else 170}"/>
+    <xacro:property name="arm_3_lower_limit"       value="${-45 if tiago_dual == 1 else -170}"/>
+    <xacro:property name="arm_3_upper_limit"       value="${225 if tiago_dual == 1 else 170}"/>
     <joint name="${name}_3_joint" type="revolute">
      <origin xyz="-0.1549 0 ${0.05 * reflect}"

Commit message: Update center of mass for the links

File: tiago_sea_arm_description/urdf/arm/arm.urdf.xacro (robot description, xacro)
@@ -15,9 +15,9 @@
     <link name="${name}_base_link">
       <inertial>
-        <origin xyz="3.2628E-04 -3.2799E-03 -0.0322" rpy="0 0 0" />
+        <origin xyz="-3.2799E-03 -3.2628E-04 -0.0322" rpy="0 0 0" />
         <mass value="0.8021" />
         <inertia
-          ixx="5.5663E-04" ixy="-5.9227E-06" ixz="5.7113E-06"
-          iyy="5.3024E-04" iyz="1.0828E-06"
+          ixx="5.3024E-04" ixy="5.9227E-06" ixz="1.0828E-06"
+          iyy="5.5663E-04" iyz="-5.7113E-06"
           izz="6.8971E-04" />
       </inertial>
@@ -46,9 +46,9 @@
     <link name="${name}_1_link">
       <inertial>
-        <origin xyz="0.0106 0.1082 ${-0.0328 * reflect}" rpy="0 0 0" />
+        <origin xyz="0.1082 -0.0106 ${-0.0328 * reflect}" rpy="0 0 0" />
         <mass value="1.0267" />
       <inertia
-        ixx="1.9301E-03" ixy="-8.52034E-05" ixz="${1.9426E-05 * reflect}"
-        iyy="8.0603E-04" iyz="${3.0124E-04 * reflect}"
+        ixx="8.0603E-04" ixy="8.52034E-05" ixz="${3.0124E-04 * reflect}"
+        iyy="1.9301E-03" iyz="${-1.9426E-05 * reflect}"
         izz="1.8484E-03" />
       </inertial>
@@ -88,9 +88,9 @@
     <link name="${name}_2_link">
       <inertial>
-        <origin xyz="-8.2340E-03 -0.0941 ${0.0414 * reflect}" rpy="0 0 0" />
+        <origin xyz="-0.0941 2.6612E-04  ${0.0414 * reflect}" rpy="0 0 0" />
         <mass value="0.9496" />
         <inertia
-          ixx="1.4185E-03" ixy="5.7830E-06" ixz="${-5.8148E-06 * reflect}"
-          iyy="8.4202E-04" iyz="${-2.6145E-04 * reflect}"
+          ixx="8.4202E-04" ixy="-5.7830E-06" ixz="${2.6145E-04 * reflect}"
+          iyy="1.4185E-03" iyz="${-5.8148E-06 * reflect}"
           izz="1.4729E-03" />
       </inertial>
@@ -131,5 +131,5 @@
     <link name="${name}_3_link">
       <inertial>
-        <origin xyz="0.0151 0.0121 ${0.1344 * reflect}"
+        <origin xyz="0.0121 0.0151 ${-0.1344 * reflect}"
           rpy="0 0 0" />
         <mass value="1.0676" />
@@ -178,5 +178,5 @@
     <link name="${name}_4_link">
       <inertial>
-        <origin xyz="-0.018 -0.1025 ${-0.0419 * reflect}" rpy="0 0 0" />
+        <origin xyz="0.018 -0.1025 ${0.0419 * reflect}" rpy="0 0 0" />
         <mass value="0.9494" />
       <inertia
@@ -222,5 +222,5 @@
     <link name="${name}_5_link">
       <inertial>
-        <origin xyz="0 2.5984E-03 ${0.1278 * reflect}" rpy="0 0 0" />
+        <origin xyz="2.5984E-03 0 ${-0.1278 * reflect}" rpy="0 0 0" />
         <mass value="0.7489" />
         <inertia
@@ -266,5 +266,5 @@
     <link name="${name}_6_link">
       <inertial>
-        <origin xyz="0 -0.0939 ${-0.0329 * reflect}" rpy="0 0 0" />
+        <origin xyz="0 -0.0939 ${0.0329 * reflect}" rpy="0 0 0" />
         <mass value="0.7078" />
         <inertia

Commit message: added collision and description values of the tool link

File: tiago_sea_arm_description/urdf/arm/arm.urdf.xacro (robot description, xacro)
@@ -348,5 +348,23 @@
     <!--        TOOL           -->
     <!--***********************-->
-    <link name="${name}_tool_link"/>
+    <link name="${name}_tool_link">
+      <inertial>
+        <mass value="0.1" />
+        <inertia ixx="8.33E-07" ixy="0.0" ixz="0.0" iyy="8.33E-07" iyz="0.0" izz="1.25E-06" />
+      </inertial>
+      <visual>
+        <origin xyz="0.001 0 0" rpy="0 ${90.0 * deg_to_rad} 0" />
+        <geometry>
+          <cylinder radius="0.005" length="0.005"/>
+        </geometry>
+        <material name="LightGrey" />
+      </visual>
+      <collision>
+        <origin xyz="0.001 0 0" rpy="0 ${90.0 * deg_to_rad} 0" />
+        <geometry>
+          <cylinder radius="0.005" length="0.005"/>
+        </geometry>
+      </collision>
+    </link>
     <joint name="${name}_tool_joint" type="fixed">
       <parent link="${name}_7_link" />

Commit message: Update stl origins of arm

File: tiago_sea_arm_description/urdf/arm/arm.urdf.xacro (robot description, xacro)
@@ -15,8 +15,8 @@
     <link name="${name}_base_link">
       <inertial>
-        <origin xyz="-3.2799E-03 -3.2628E-04 -0.0322" rpy="0 0 0" />
+        <origin xyz="3.2799E-03 -3.2628E-04 -0.0322" rpy="0 0 0" />
         <mass value="0.8021" />
         <inertia
-          ixx="5.3024E-04" ixy="5.9227E-06" ixz="1.0828E-06"
+          ixx="5.3024E-04" ixy="-5.9227E-06" ixz="-1.0828E-06"
           iyy="5.5663E-04" iyz="-5.7113E-06"
           izz="6.8971E-04" />
@@ -46,9 +46,9 @@
     <link name="${name}_1_link">
       <inertial>
-        <origin xyz="0.1082 -0.0106 ${-0.0328 * reflect}" rpy="0 0 0" />
+        <origin xyz="0.1082 -0.0106 ${0.0328 * reflect}" rpy="0 0 0" />
         <mass value="1.0267" />
       <inertia
-        ixx="8.0603E-04" ixy="8.52034E-05" ixz="${3.0124E-04 * reflect}"
-        iyy="1.9301E-03" iyz="${1.9426E-05 * reflect}"
+        ixx="8.0603E-04" ixy="8.52034E-05" ixz="${-3.0124E-04 * reflect}"
+        iyy="1.9301E-03" iyz="${-1.9426E-05 * reflect}"
         izz="1.8484E-03" />
       </inertial>
@@ -77,5 +77,5 @@
     <xacro:property name="arm_1_lower_limit"       value="-90"/>
     <joint name="${name}_1_joint" type="revolute">
-      <origin xyz="0.0 0.0 0.0" rpy=" 0 ${(90 - 90 * reflect) * deg_to_rad } ${(90 + 90 * reflect) * deg_to_rad}" />
+      <origin xyz="0.0 0.0 0.0" rpy=" 0 ${(90 + 90 * reflect) * deg_to_rad } ${(90 + 90 * reflect) * deg_to_rad}" />
       <parent link="${name}_base_link" />
       <child link="${name}_1_link" />
@@ -119,5 +119,5 @@
     <xacro:property name="arm_2_lower_limit"       value="${-90 if tiago_dual == 1 else -62.5}"/>
     <joint name="${name}_2_joint" type="revolute">
-      <origin xyz="0.13 -0.0483 ${-0.04* reflect}"
+      <origin xyz="0.13 -0.0483 ${0.04* reflect}"
         rpy="${90 * reflect * deg_to_rad} 0 ${180 * deg_to_rad}" />
       <parent link="${name}_1_link" />

Commit message: Change meshes orientation according to the robot

File: tiago_sea_arm_description/urdf/arm/arm.urdf.xacro (robot description, xacro)
@@ -49,9 +49,9 @@
     <link name="${name}_1_link">
       <inertial>
-        <origin xyz="0.1082 -0.0106 ${0.0328 * reflect}" rpy="0 0 0" />
+        <origin xyz="0.1082 -0.0106 ${-0.0328 * reflect}" rpy="0 0 0" />
         <mass value="1.0267" />
       <inertia
-        ixx="8.0603E-04" ixy="8.52034E-05" ixz="${-3.0124E-04 * reflect}"
-        iyy="1.9301E-03" iyz="${-1.9426E-05 * reflect}"
+        ixx="8.0603E-04" ixy="8.52034E-05" ixz="${3.0124E-04 * reflect}"
+        iyy="1.9301E-03" iyz="${1.9426E-05 * reflect}"
         izz="1.8484E-03" />
       </inertial>
@@ -78,5 +78,5 @@
     </link>
     <joint name="${name}_1_joint" type="revolute">
-      <origin xyz="0.0 0.0 0.0" rpy=" 0 ${(90 + 90 * reflect) * deg_to_rad } ${(90 + 90 * reflect) * deg_to_rad}" />
+      <origin xyz="0.0 0.0 0.0" rpy=" 0 ${(90 - 90 * reflect) * deg_to_rad } ${(90 - 90 * reflect) * deg_to_rad}" />
       <parent link="${name}_base_link" />
       <child link="${name}_1_link" />
@@ -118,5 +118,5 @@
     </link>
     <joint name="${name}_2_joint" type="revolute">
-      <origin xyz="0.13 -0.0483 ${0.04* reflect}"
+      <origin xyz="0.13 -0.0483 ${-0.04* reflect}"
         rpy="${90 * reflect * deg_to_rad} 0 ${180 * deg_to_rad}" />
       <parent link="${name}_1_link" />
@@ -337,5 +337,6 @@
     <joint name="${name}_7_joint" type="revolute">
      <origin xyz="0 -0.146 ${0.039 * reflect}"
-        rpy="0 ${90 * reflect * deg_to_rad} ${90 * deg_to_rad}" />
+        rpy="${-90 * reflect * deg_to_rad} 0 0" />
+        <!-- rpy="0 ${90 * reflect * deg_to_rad} ${90 * deg_to_rad}" /> -->
       <parent link="${name}_6_link" />
       <child

Commit message: Update mirror arm_1 link

File: tiago_sea_arm_description/urdf/arm/arm.urdf.xacro (robot description, xacro)
@@ -49,8 +49,8 @@
     <link name="${name}_1_link">
       <inertial>
-        <origin xyz="0.1082 -0.0106 ${-0.0328 * reflect}" rpy="0 0 0" />
+        <origin xyz="0.1082 0.0106 ${0.0328 * reflect}" rpy="0 0 0" />
         <mass value="1.0267" />
       <inertia
-        ixx="8.0603E-04" ixy="8.52034E-05" ixz="${3.0124E-04 * reflect}"
+        ixx="8.0603E-04" ixy="-8.52034E-05" ixz="${-3.0124E-04 * reflect}"
         iyy="1.9301E-03" iyz="${1.9426E-05 * reflect}"
         izz="1.8484E-03" />
@@ -78,5 +78,6 @@
     </link>
     <joint name="${name}_1_joint" type="revolute">
-      <origin xyz="0.0 0.0 0.0" rpy=" 0 ${(90 - 90 * reflect) * deg_to_rad } ${(90 - 90 * reflect) * deg_to_rad}" />
+      <!-- <origin xyz="0.0 0.0 0.0" rpy=" 0 ${(90 - 90 * reflect) * deg_to_rad } ${(90 - 90 * reflect) * deg_to_rad}" /> -->
+      <origin xyz="0.0 0.0 0.0" rpy=" ${(90 + 90 * reflect) * deg_to_rad } 0 0" />
       <parent link="${name}_base_link" />
       <child link="${name}_1_link" />
@@ -118,6 +119,6 @@
     </link>
     <joint name="${name}_2_joint" type="revolute">
-      <origin xyz="0.13 -0.0483 ${-0.04* reflect}"
-        rpy="${90 * reflect * deg_to_rad} 0 ${180 * deg_to_rad}" />
+      <origin xyz="0.13 0.0483 ${0.04* reflect}"
+        rpy="${-90 * reflect * deg_to_rad} 0 ${180 * deg_to_rad}" />
       <parent link="${name}_1_link" />
       <child link="${name}_2_link" />
