Commit message: updated joint limits to match real robot

File: pal_sea_arm_description/urdf/arm/limits/arm_tiago-sea-dual.limits.xacro (robot description, xacro)
@@ -12,12 +12,12 @@
   <xacro:property name="arm_3_joint_ub" value="210"/>
   <xacro:property name="arm_3_joint_lb" value="-90"/>
-  <xacro:property name="arm_4_joint_ub" value="90" />
+  <xacro:property name="arm_4_joint_ub" value="100" />
   <xacro:property name="arm_4_joint_lb" value="-125" />
-  <xacro:property name="arm_5_joint_ub" value="145" />
-  <xacro:property name="arm_5_joint_lb" value="-145" />
-  <xacro:property name="arm_6_joint_ub" value="115" />
-  <xacro:property name="arm_6_joint_lb" value="-115" />
-  <xacro:property name="arm_7_joint_ub" value="135" />
-  <xacro:property name="arm_7_joint_lb" value="-135" />
+  <xacro:property name="arm_5_joint_ub" value="150" />
+  <xacro:property name="arm_5_joint_lb" value="-150" />
+  <xacro:property name="arm_6_joint_ub" value="120" />
+  <xacro:property name="arm_6_joint_lb" value="-120" />
+  <xacro:property name="arm_7_joint_ub" value="140" />
+  <xacro:property name="arm_7_joint_lb" value="-140" />
   <xacro:property name="arm_1_max_velocity"      value="1.95" />
   <xacro:property name="arm_2_max_velocity"      value="1.95" />
