Commit message: add the SEA simple transmissions for all the arm joints

File: pal_sea_arm_description/urdf/arm/arm.transmission.xacro (robot description, xacro)
@@ -16,14 +16,16 @@
     </transmission>
   </xacro:macro>
-  <xacro:macro name="arm_pro_simple_transmission" params="name number offset_value" >
+  <xacro:macro name="arm_sea_simple_transmission" params="name number reduction offset_value" >
     <transmission name="${name}_${number}_trans">
-      <type>sea_transmissions/SeaSimpleTransmission</type><!--transmission_interface/SeaTransmission-->
+      <type>sea_transmissions/SeaSimpleTransmission</type>
       <actuator name="${name}_${number}_motor" >
+        <mechanicalReduction>${reduction}</mechanicalReduction>
       </actuator>
       <joint name="${name}_${number}_joint">
-        <offset>${offset_value}</offset>
+        <actuators_data_ns>/actuators_data/${name}_${number}_motor</actuators_data_ns>
+        <joint_offset_ns>/${name}_${number}_motor/output_offset</joint_offset_ns>
         <hardwareInterface>hardware_interface/PositionJointInterface</hardwareInterface>
+        <hardwareInterface>hardware_interface/VelocityJointInterface</hardwareInterface>
         <hardwareInterface>hardware_interface/EffortJointInterface</hardwareInterface>
-        <hardwareInterface>hardware_interface/VelocityJointInterface</hardwareInterface>
         <hardwareInterface>hardware_interface/JointStateInterface</hardwareInterface>
       </joint>

File: pal_sea_arm_description/urdf/arm/arm.urdf.xacro (robot description, xacro)
@@ -331,11 +331,11 @@
     </gazebo>
     <!-- TRANSMISSIONS -->
-    <xacro:arm_simple_transmission name="${name}" number="1" reduction="1.0" offset_value="${arm_1_offset}"/>
-    <xacro:arm_simple_transmission name="${name}" number="2" reduction="1.0" offset_value="${arm_2_offset}"/>
-    <xacro:arm_simple_transmission name="${name}" number="3" reduction="1.0" offset_value="${arm_3_offset}"/>
-    <xacro:arm_simple_transmission name="${name}" number="4" reduction="1.0" offset_value="${arm_4_offset}"/>
-    <xacro:arm_simple_transmission name="${name}" number="5" reduction="1.0" offset_value="${arm_5_offset}"/>
-    <xacro:arm_simple_transmission name="${name}" number="6" reduction="1.0" offset_value="${arm_6_offset}"/>
-    <xacro:arm_simple_transmission name="${name}" number="7" reduction="1.0" offset_value="${arm_7_offset}"/>
+    <xacro:arm_sea_simple_transmission name="${name}" number="1" reduction="121.0" offset_value="${arm_1_offset}"/>
+    <xacro:arm_sea_simple_transmission name="${name}" number="2" reduction="121.0" offset_value="${arm_2_offset}"/>
+    <xacro:arm_sea_simple_transmission name="${name}" number="3" reduction="101.0" offset_value="${arm_3_offset}"/>
+    <xacro:arm_sea_simple_transmission name="${name}" number="4" reduction="101.0" offset_value="${arm_4_offset}"/>
+    <xacro:arm_sea_simple_transmission name="${name}" number="5" reduction="101.0" offset_value="${arm_4_offset}"/>
+    <xacro:arm_sea_simple_transmission name="${name}" number="6" reduction="101.0" offset_value="${arm_4_offset}"/>
+    <xacro:arm_sea_simple_transmission name="${name}" number="7" reduction="101.0" offset_value="${arm_4_offset}"/>
   </xacro:macro>
 </robot>

Commit message: rename the macro to arm_pro_simple_transmission and fix a minor bug

File: pal_sea_arm_description/urdf/arm/arm.transmission.xacro (robot description, xacro)
@@ -16,5 +16,5 @@
     </transmission>
   </xacro:macro>
-  <xacro:macro name="arm_sea_simple_transmission" params="name number reduction offset_value" >
+  <xacro:macro name="arm_pro_simple_transmission" params="name number reduction offset_value" >
     <transmission name="${name}_${number}_trans">
       <type>sea_transmissions/SeaSimpleTransmission</type>

File: pal_sea_arm_description/urdf/arm/arm.urdf.xacro (robot description, xacro)
@@ -331,11 +331,11 @@
     </gazebo>
     <!-- TRANSMISSIONS -->
-    <xacro:arm_sea_simple_transmission name="${name}" number="1" reduction="121.0" offset_value="${arm_1_offset}"/>
-    <xacro:arm_sea_simple_transmission name="${name}" number="2" reduction="121.0" offset_value="${arm_2_offset}"/>
-    <xacro:arm_sea_simple_transmission name="${name}" number="3" reduction="101.0" offset_value="${arm_3_offset}"/>
-    <xacro:arm_sea_simple_transmission name="${name}" number="4" reduction="101.0" offset_value="${arm_4_offset}"/>
-    <xacro:arm_sea_simple_transmission name="${name}" number="5" reduction="101.0" offset_value="${arm_4_offset}"/>
-    <xacro:arm_sea_simple_transmission name="${name}" number="6" reduction="101.0" offset_value="${arm_4_offset}"/>
-    <xacro:arm_sea_simple_transmission name="${name}" number="7" reduction="101.0" offset_value="${arm_4_offset}"/>
+    <xacro:arm_pro_simple_transmission name="${name}" number="1" reduction="121.0" offset_value="${arm_1_offset}"/>
+    <xacro:arm_pro_simple_transmission name="${name}" number="2" reduction="121.0" offset_value="${arm_2_offset}"/>
+    <xacro:arm_pro_simple_transmission name="${name}" number="3" reduction="101.0" offset_value="${arm_3_offset}"/>
+    <xacro:arm_pro_simple_transmission name="${name}" number="4" reduction="101.0" offset_value="${arm_4_offset}"/>
+    <xacro:arm_pro_simple_transmission name="${name}" number="5" reduction="101.0" offset_value="${arm_5_offset}"/>
+    <xacro:arm_pro_simple_transmission name="${name}" number="6" reduction="101.0" offset_value="${arm_6_offset}"/>
+    <xacro:arm_pro_simple_transmission name="${name}" number="7" reduction="101.0" offset_value="${arm_7_offset}"/>
   </xacro:macro>
 </robot>
