Commit message: Adding absolute_position joint state interface

File: pal_sea_arm_description/urdf/arm/arm.ros2_control.xacro (robot description, xacro)
@@ -13,5 +13,5 @@
  -->
 <robot xmlns:xacro="http://ros.org/wiki/xacro">
-  <xacro:macro name="ros2_control_arm" params="name reduction offset_value" >
+  <xacro:macro name="ros2_control_arm" params="name reduction offset_value">
     <joint name="${name}_joint">
       <command_interface name="position" />
@@ -22,7 +22,8 @@
       <state_interface name="effort" />
       <state_interface name="torque"/>
+      <state_interface name="absolute_position"/>
     </joint>
-  <xacro:include filename="$(find pal_sea_arm_description)/ros2_control/transmissions.urdf.xacro" />
-  <xacro:pal_sea_arm_simple_transmission name="${name}" reduction="${reduction}" offset_value="${offset_value}" />
+    <xacro:include filename="$(find pal_sea_arm_description)/ros2_control/transmissions.urdf.xacro" />
+    <xacro:pal_sea_arm_simple_transmission name="${name}" reduction="${reduction}" offset_value="${offset_value}" />
   </xacro:macro>
 </robot>

Commit message: SEA transmission optional loading

File: pal_sea_arm_description/urdf/arm/arm.ros2_control.xacro (robot description, xacro)
@@ -13,5 +13,5 @@
  -->
 <robot xmlns:xacro="http://ros.org/wiki/xacro">
-  <xacro:macro name="ros2_control_arm" params="name reduction offset_value">
+  <xacro:macro name="ros2_control_arm" params="name reduction offset_value use_sea_transmission:=false">
     <joint name="${name}_joint">
       <command_interface name="position" />
@@ -21,9 +21,19 @@
       <state_interface name="velocity" />
       <state_interface name="effort" />
-      <state_interface name="torque"/>
-      <state_interface name="absolute_position"/>
+      <!-- SEA specific joint interfaces -->
+      <xacro:if value="${use_sea_transmission}">
+        <state_interface name="torque"/>
+        <state_interface name="absolute_position"/>
+      </xacro:if>
     </joint>
     <xacro:include filename="$(find pal_sea_arm_description)/ros2_control/transmissions.urdf.xacro" />
-    <xacro:pal_sea_arm_simple_transmission name="${name}" reduction="${reduction}" offset_value="${offset_value}" />
+    <xacro:if value="${use_sea_transmission}">
+      <!-- Reduction needed for the torque estimation -->
+      <xacro:pal_sea_arm_simple_transmission name="${name}" reduction="${reduction}" offset_value="${offset_value}" />
+    </xacro:if>
+    <xacro:unless value="${use_sea_transmission}">
+      <!-- Reduction already applied in the RT layer, harcoded here to 1.0 -->
+      <xacro:arm_pro_simple_transmission name="${name}" reduction="1.0" offset_value="${offset_value}" />
+    </xacro:unless>
   </xacro:macro>
 </robot>

Commit message: added mujoco command interface

File: pal_sea_arm_description/urdf/arm/arm.ros2_control.xacro (robot description, xacro)
@@ -14,35 +14,28 @@
 <robot xmlns:xacro="http://ros.org/wiki/xacro">
   <xacro:macro name="ros2_control_arm" params="name reduction offset_value use_sea_transmission:=false">
-    <xacro:if value="${mujoco}">
-       <joint name="${name}_joint">
-        <xacro:unless value="${mj_simulate}">
-            <param name="position_kp">700</param>
-            <param name="position_ki">1</param>
-            <param name="position_kd">10</param>
-            <param name="position_i_max">0</param>
-            <command_interface name="position_pid" />
-            <!-- <command_interface name="effort" />
-            <command_interface name="velocity" /> -->
-        </xacro:unless>
-        <state_interface name="position" />
-        <state_interface name="velocity" />
-        <state_interface name="effort" />
-      </joint>
-    </xacro:if>
-    <xacro:unless value="${mujoco}">
-      <joint name="${name}_joint">
+    <joint name="${name}_joint">
+      <xacro:if value="${sim_type == 'mujoco-ros2-control'}">
+        <param name="position_kp">700</param>
+        <param name="position_ki">1</param>
+        <param name="position_kd">10</param>
+        <param name="position_i_max">0</param>
+        <command_interface name="position_pid" />
+      </xacro:if>
+      <xacro:if value="${sim_type == 'gazebo'}">
         <command_interface name="position" />
-        <command_interface name="velocity" />
-        <command_interface name="effort" />
-        <state_interface name="position" />
-        <state_interface name="velocity" />
-        <state_interface name="effort" />
-        <!-- SEA specific joint interfaces -->
-        <xacro:if value="${use_sea_transmission}">
-          <state_interface name="torque"/>
-          <state_interface name="absolute_position"/>
-        </xacro:if>
-      </joint>
-      <xacro:include filename="$(find pal_sea_arm_description)/ros2_control/transmissions.urdf.xacro" />
+      </xacro:if>
+      <command_interface name="velocity" />
+      <command_interface name="effort" />
+      <state_interface name="position" />
+      <state_interface name="velocity" />
+      <state_interface name="effort" />
+      <!-- SEA specific joint interfaces -->
+      <xacro:if value="${use_sea_transmission and sim_type == 'gazebo'}">
+        <state_interface name="torque"/>
+        <state_interface name="absolute_position"/>
+      </xacro:if>
+    </joint>
+    <xacro:include filename="$(find pal_sea_arm_description)/ros2_control/transmissions.urdf.xacro" />
+    <xacro:if value="${sim_type == 'gazebo'}">
       <xacro:if value="${use_sea_transmission}">
         <!-- Reduction needed for the torque estimation -->
@@ -53,5 +46,5 @@
         <xacro:simple_transmission name="${name}" reduction="1.0" offset_value="${offset_value}" />
       </xacro:unless>
-    </xacro:unless>
+    </xacro:if>
   </xacro:macro>
 </robot>
