Commit message: Remove base_link from arm urdf

File: pal_sea_arm_description/urdf/arm/arm.urdf.xacro (robot description, xacro)
@@ -345,35 +345,4 @@
     </xacro:if>
     <xacro:if value="${arm_model in ['tiago-sea', 'tiago-sea-dual']}">
-      <!-- BASE LINK -->
-      <link name="${name}_base_link">
-        <inertial>
-          <origin xyz="3.2799E-03 -3.2628E-04 -0.0322" rpy="0 0 0" />
-          <mass value="0.8021" />
-          <inertia
-            ixx="5.3024E-04" ixy="-5.9227E-06" ixz="-1.0828E-06"
-            iyy="5.5663E-04" iyz="-5.7113E-06"
-            izz="6.8971E-04" />
-        </inertial>
-        <visual>
-          <origin xyz="0 0 0" rpy="0 0 0" />
-          <geometry>
-            <mesh filename="package://pal_sea_arm_description/meshes/arm_tiago_sea/base_link.stl" />
-          </geometry>
-          <material name="">
-            <color rgba="0.75294 0.75294 0.75294 1" />
-          </material>
-        </visual>
-        <collision>
-          <origin xyz="0 0 0" rpy="0 0 0" />
-          <geometry>
-            <mesh filename="package://pal_sea_arm_description/meshes/arm_tiago_sea/base_link.stl" />
-          </geometry>
-        </collision>
-      </link>
-      <joint name="${name}_base_joint" type="fixed">
-        <xacro:insert_block name="origin" />
-        <parent link="${parent}" />
-        <child link="${name}_base_link" />
-      </joint>
       <!-- ARM 1 LINK -->
       <link name="${name}_1_link">
@@ -409,7 +378,6 @@
       <!-- ARM 1 JOINT -->
       <joint name="${name}_1_joint" type="revolute">
-        <!-- <origin xyz="0.0 0.0 0.0" rpy=" 0 ${(90 - 90 * reflect) * deg_to_rad } ${(90 - 90 * reflect) * deg_to_rad}" /> -->
-        <origin xyz="0.0 0.0 0.0" rpy=" ${(90 + 90 * reflect) * deg_to_rad } 0 0" />
-        <parent link="${name}_base_link" />
+        <xacro:insert_block name="origin" />
+        <parent link="${parent}" />
         <child link="${name}_1_link" />
         <axis xyz="0 0 ${1}" />

Commit message: Improve wheight of the links + fix link collision that was to small to visualize the marker in moveit

File: pal_sea_arm_description/urdf/arm/arm.urdf.xacro (robot description, xacro)
@@ -257,5 +257,5 @@
         <origin xyz="0.001 0 0" rpy="0 ${90.0 * deg_to_rad} 0" />
         <geometry>
-          <cylinder radius="0.005" length="0.005"/>
+          <cylinder radius="0.032" length="0.01"/>
         </geometry>
         <material name="pal/DarkGrey"/>
@@ -264,5 +264,5 @@
         <origin xyz="0.001 0 0" rpy="0 ${90.0 * deg_to_rad} 0" />
         <geometry>
-          <cylinder radius="0.005" length="0.005"/>
+          <cylinder radius="0.032" length="0.01"/>
         </geometry>
       </collision>

File: pal_sea_arm_description/urdf/arm/arm_properties/arm_tiago-sea-dual.properties.xacro (robot description, xacro)
@@ -6,5 +6,5 @@
         rpy="0 0 0" />
         <mass
-        value="1.0267" />
+        value="1.121" />
         <inertia
         ixx="8.0603E-04"
@@ -22,5 +22,5 @@
         rpy="0 0 0" />
         <mass
-        value="0.9496" />
+        value="1.04393478668639" />
         <inertia
         ixx="8.4202E-04"
@@ -41,5 +41,5 @@
         rpy="0 0 0" />
         <mass
-        value="1.0816" />
+        value="1.16187501225607" />
         <inertia
         ixx="2.4587E-03"
@@ -60,5 +60,5 @@
         rpy="0 0 0" />
         <mass
-        value="0.99204" />
+        value="1.04356953296638" />
         <inertia
         ixx="1.3967E-03"
@@ -79,5 +79,5 @@
         rpy="0 0 0" />
         <mass
-        value="0.52538" />
+        value="0.87162300950021" />
         <inertia
         ixx="1.9033E-03"
@@ -98,5 +98,5 @@
         rpy="0 0 0" />
         <mass
-        value="0.66725" />
+        value="0.707831170710613" />
         <inertia
         ixx="8.7604E-04"

File: pal_sea_arm_description/urdf/sensors/ft_sensor.urdf.xacro (robot description, xacro)
@@ -57,5 +57,23 @@
     <!--       FT TOOL         -->
     <!--***********************-->
-    <link name="${name}_ft_tool_link"/>
+    <link name="${name}_ft_tool_link">
+      <inertial>
+        <mass value="0.1" />
+        <inertia ixx="1.64E-05" ixy="0.0" ixz="0.0" iyy="1.64E-05" iyz="0.0" izz="3.125E-05" />
+      </inertial>
+      <visual>
+        <origin xyz="0.001 0 0" rpy="0 ${90.0 * deg_to_rad} 0" />
+        <geometry>
+          <cylinder radius="0.032" length="0.01"/>
+        </geometry>
+        <material name="pal/DarkGrey"/>
+      </visual>
+      <collision>
+        <origin xyz="0.001 0 0" rpy="0 ${90.0 * deg_to_rad} 0" />
+        <geometry>
+          <cylinder radius="0.032" length="0.01"/>
+        </geometry>
+      </collision>
+    </link>
     <joint name="${name}_ft_tool_joint" type="fixed">
       <parent link="${name}_ft_link" />

Commit message: Suggested changes

File: pal_sea_arm_description/urdf/arm/arm.urdf.xacro (robot description, xacro)
@@ -19,5 +19,5 @@
     <xacro:property name="mesh_folder"/>
     <!-- Tiago Pro -->
-    <xacro:if value="${arm_type in ['tiago-pro']}">
+    <xacro:if value="${arm_type in ['tiago-pro', 'pal-sea-arm-standalone']}">
       <xacro:property name="mesh_folder" value="arm_tiago_pro"/>
     </xacro:if>

File: pal_sea_arm_description/urdf/arm/arm_properties/pal-sea-arm-standalone/arm.properties.xacro (robot description, xacro)
@@ -1,42 +1,64 @@
 <robot xmlns:xacro="http://ros.org/wiki/xacro">
+    <xacro:macro name="inertial_base_link" params="reflect">
+        <inertial>
+            <origin xyz="-0.00069237 0.00052761 -0.012575" rpy="0 0 0" />
+            <mass value="0.76084" />
+            <inertia ixx="0.00052192" ixy="8.9882E-06" ixz="-6.4075E-06" iyy="0.00052523" iyz="8.9275E-06" izz="0.00054849" />
+        </inertial>
+    </xacro:macro>
     <xacro:macro name="inertial_link_1" params="reflect">
         <inertial>
-            <origin xyz="0.0023908 0.015901 0.1545" rpy="0 0 0" />
-            <mass value="0.2" />
-            <inertia ixx="0.0024426" ixy="2.3307E-05" ixz="5.9333E-05" iyy="0.0023089" iyz="-0.00020369" izz="0.00092843" />
+            <origin xyz="0.0043916 0.016184 0.15576" rpy="0 0 0" />
+            <mass value="1.1325" />
+            <inertia ixx="0.0025497" ixy="2.6206E-05" ixz="6.2082E-05" iyy="0.0023517" iyz="-0.00020617" izz="0.00097131" />
         </inertial>
+    </xacro:macro>
+    <xacro:macro name="origin_joint_1" params="reflect">
+        <origin xyz="0 0 0" rpy="0 0 0" />
     </xacro:macro>
     <xacro:macro name="inertial_link_2" params="reflect">
         <inertial>
-            <origin xyz="-0.11649 -0.017864 0.0053772" rpy="0 0 0" />
-            <mass value="0.01" />
-            <inertia ixx="0.00077294" ixy="-0.00011001" ixz="-0.00016136" iyy="0.0014605" iyz="-1.3224E-05" izz="0.0015605" />
+            <origin xyz="0.01786 -0.11956 -0.032097" rpy="0 0 0" />
+            <mass value="1.0436" />
+            <inertia ixx="0.0015021" ixy="0.00011264" ixz="1.0692E-05" iyy="0.00088017" iyz="-0.00015843" izz="0.0016021" />
         </inertial>
     </xacro:macro>
     <xacro:macro name="origin_joint_2" params="reflect">
-        <origin xyz="0.0 0.02 0.18" rpy="0 1.5708 0" />
+        <origin xyz="0.0371099999999995 0.02 0.18" rpy="-1.57079632679489 0 -1.5707963267949" />
     </xacro:macro>
     <xacro:macro name="inertial_link_3" params="reflect">
         <inertial>
-            <origin xyz="0.0023908 0.015901 0.1545" rpy="0 0 0" />
-            <mass value="0.1" />
-            <inertia ixx="0.0024426" ixy="2.3307E-05" ixz="5.9333E-05" iyy="0.0023089" iyz="-0.00020369" izz="0.00092843" />
+            <origin xyz="0.016184 -0.0043916 0.13565" rpy="0 0 0" />
+            <mass value="1.1325" />
+            <inertia ixx="0.0023517" ixy="-2.6206E-05" ixz="-0.00020617" iyy="0.0025497" iyz="-6.2082E-05" izz="0.00097131" />
         </inertial>
     </xacro:macro>
     <xacro:macro name="origin_joint_3" params="reflect">
-        <origin xyz="-0.15 -0.02 0" rpy="3.1415 1.5707 0" />
+        <origin xyz="0.019999999999999 -0.17011 -0.037110000000001" rpy="1.5707963267949 0 0" />
     </xacro:macro>
     <xacro:macro name="inertial_link_4" params="reflect">
         <inertial>
-            <origin xyz="-0.11649 -0.017864 0.0053772" rpy="0 0 0" />
-            <mass value="0.1" />
-            <inertia ixx="0.00077294" ixy="-0.00011001" ixz="-0.00016136" iyy="0.0014605" iyz="-1.3224E-05" izz="0.0015605" />
+            <origin xyz="-0.01786 0.11956 -0.032097" rpy="0 0 0" />
+            <mass value="1.0436" />
+            <inertia ixx="0.0015021" ixy="0.00011264" ixz="-1.0692E-05" iyy="0.00088017" iyz="0.00015843" izz="0.0016021" />
         </inertial>
     </xacro:macro>
     <xacro:macro name="origin_joint_4" params="reflect">
-        <origin xyz="0 0.02 0.18" rpy="0 1.5708 0" />
+        <origin xyz="0.0199999999999993 -0.0371100000000008 0.15989" rpy="1.57079632679489 0 0" />
     </xacro:macro>
     <xacro:macro name="origin_joint_5" params="reflect">
-        <origin xyz="-0.15 -0.02 0" rpy="0 -1.5708 0" />
+        <origin xyz="-0.0199999999999971 0.17011 -0.037110000000002" rpy="-1.5707963267949 0 0" />
+    </xacro:macro>
+    <!-- Tool changer (can be present in both wrists)-->
+    <xacro:macro name="inertial_tool_changer_link" params="reflect">
+        <inertial>
+            <origin xyz="0.0019481 0.0017558 -0.0084934" rpy="0 0 0" />
+            <mass value="0.12272" />
+            <inertia ixx="5.1385E-05" ixy="8.5364E-07" ixz="-9.0329E-08" iyy="4.7962E-05" iyz="-1.8035E-07" izz="9.2935E-05" />
+        </inertial>
+    </xacro:macro>
+    <xacro:macro name="origin_joint_tool_changer" params="reflect">
+        <!-- @Lucien needs to fix -->
+        <origin xyz="0 0 0.017" rpy="0 0 0" />
     </xacro:macro>
 </robot>

File: pal_sea_arm_description/urdf/arm/arm_properties/pal-sea-arm-standalone/straight-wrist.properties.xacro (robot description, xacro)
@@ -2,38 +2,28 @@
     <xacro:macro name="inertial_link_5" params="reflect">
         <inertial>
-            <origin xyz="0.0004859 0.00014289 0.129" rpy="0 0 0" />
-            <mass value="0.12538" />
-            <inertia ixx="0.0019111" ixy="-1.4245E-08" ixz="3.8663E-05" iyy="0.0018565" iyz="1.1356E-06" izz="0.00046496" />
+            <origin xyz="8.9806E-06 -0.00053878 0.13058" rpy="0 0 0" />
+            <mass value="0.84847" />
+            <inertia ixx="0.0020531" ixy="-8.9232E-07" ixz="1.6668E-06" iyy="0.0020434" iyz="3.7824E-05" izz="0.00067121" />
         </inertial>
     </xacro:macro>
     <xacro:macro name="inertial_link_6" params="reflect">
         <inertial>
-            <origin xyz="-0.086822 -7.7905E-06 0.0045258" rpy="0 0 0" />
-            <mass value="0.1725" />
-            <inertia ixx="0.00035696" ixy="1.6019E-07" ixz="-9.5191E-05" iyy="0.00073846" iyz="2.118E-08" izz="0.00075321" />
+            <origin xyz="-0.016007 0.052767 3.7676E-05" rpy="0 0 0" />
+            <mass value="0.15792" />
+            <inertia ixx="0.00043323" ixy="9.3978E-05" ixz="-2.1216E-08" iyy="0.00013569" iyz="1.5995E-07" izz="0.00041746" />
         </inertial>
     </xacro:macro>
     <xacro:macro name="origin_joint_6" params="reflect">
-        <origin xyz="0 0 0.185" rpy="0 1.5708 0" />
+        <origin xyz="0 0.0354 0.16489" rpy="1.5708 0 1.5708" />
     </xacro:macro>
     <xacro:macro name="inertial_link_7" params="reflect">
         <inertial>
-            <origin xyz="-6.764E-18 -1.4549E-16 0.018549" rpy="0 0 0" />
-            <mass value="0.10189" />
-            <inertia ixx="5.1076E-05" ixy="-1.0899E-21" ixz="-5.93E-21" iyy="5.0882E-05" iyz="-8.5344E-21" izz="9.705E-05" />
+            <origin xyz="-7.5568E-05 1.3009E-17 -0.037565" rpy="0 0 0" />
+            <mass value="0.51032" />
+            <inertia ixx="0.00032034" ixy="-7.8169E-21" ixz="1.0206E-06" iyy="0.00032121" iyz="7.188E-20" izz="0.00022179" />
         </inertial>
     </xacro:macro>
     <xacro:macro name="origin_joint_7" params="reflect">
-        <origin xyz="-0.1166 0 0" rpy="0 -1.5708 0" />
-    </xacro:macro>
-    <xacro:macro name="inertial_tool_link" params="reflect">
-        <inertial>
-            <origin xyz="5.0493E-18 -4.4892E-17 -0.0068514" rpy="0 0 0" />
-            <mass value="0.10189" />
-            <inertia ixx="5.1076E-05" ixy="-1.0374E-21" ixz="-5.9164E-21" iyy="5.0882E-05" iyz="-8.5211E-21" izz="9.705E-05" />
-        </inertial>
-    </xacro:macro>
-    <xacro:macro name="origin_joint_tool" params="reflect">
-        <origin xyz="0 0 0.0184" rpy="0 ${-90.0 * deg_to_rad} ${90.0 * deg_to_rad}" />
+        <origin xyz="-0.0354 0.135 0" rpy="-1.5708 0 0" />
     </xacro:macro>
 </robot>

File: pal_sea_arm_description/urdf/arm/arm_properties/tiago-sea-dual/arm.properties.xacro (robot description, xacro)
@@ -40,3 +40,15 @@
         <origin xyz="0.02 -0.1546 ${0.05 * reflect}" rpy="${90 * reflect * deg_to_rad} 0 ${180 * deg_to_rad}" />
     </xacro:macro>
+    <!-- Tool changer (can be present in both wrists)-->
+    <xacro:macro name="inertial_tool_changer_link" params="reflect">
+        <inertial>
+            <origin xyz="0.0019481 0.0017558 -0.0084934" rpy="0 0 0" />
+            <mass value="0.12272" />
+            <inertia ixx="5.1385E-05" ixy="8.5364E-07" ixz="-9.0329E-08" iyy="4.7962E-05" iyz="-1.8035E-07" izz="9.2935E-05" />
+        </inertial>
+    </xacro:macro>
+    <xacro:macro name="origin_joint_tool_changer" params="reflect">
+        <!-- @Lucien needs to fix -->
+        <origin xyz="0 0 0.017" rpy="0 0 0" />
+    </xacro:macro>
 </robot>

File: pal_sea_arm_description/urdf/arm/arm_properties/tiago-sea-dual/straight-wrist.properties.xacro (robot description, xacro)
@@ -25,15 +25,5 @@
     </xacro:macro>
     <xacro:macro name="origin_joint_7" params="reflect">
-        <origin xyz="0 -0.146 ${0.039 * reflect}" rpy="${-90 * reflect * deg_to_rad} 0 0" />
-    </xacro:macro>
-    <xacro:macro name="inertial_tool_link" params="reflect">
-        <inertial>
-            <origin xyz="0 0 0" rpy="0 0 0" />
-            <mass value="0.1" />
-            <inertia ixx="8.33E-07" ixy="0.0" ixz="0.0" iyy="8.33E-07" iyz="0.0" izz="1.25E-06" />
-        </inertial>
-    </xacro:macro>
-    <xacro:macro name="origin_joint_tool" params="reflect">
-        <origin xyz="0 0 0" rpy="${0.0 * deg_to_rad} ${90.0 * reflect * deg_to_rad} ${0 * deg_to_rad}" />
+        <origin xyz="0 -0.146 ${0.039 * reflect}" rpy="${-90 * reflect * deg_to_rad} 0 3.14" />
     </xacro:macro>
 </robot>

File: pal_sea_arm_description/urdf/arm/arm_properties/tiago-sea/arm.properties.xacro (robot description, xacro)
@@ -1,42 +1,64 @@
 <robot xmlns:xacro="http://ros.org/wiki/xacro">
+    <xacro:macro name="inertial_base_link" params="reflect">
+        <inertial>
+            <origin xyz="-0.00069237 0.00052761 -0.012575" rpy="0 0 0" />
+            <mass value="0.76084" />
+            <inertia ixx="0.00052192" ixy="8.9882E-06" ixz="-6.4075E-06" iyy="0.00052523" iyz="8.9275E-06" izz="0.00054849" />
+        </inertial>
+    </xacro:macro>
     <xacro:macro name="inertial_link_1" params="reflect">
         <inertial>
-            <origin xyz="0.1082 0.0106 ${0.0328 * reflect}" rpy="0 0 0" />
-            <mass value="1.0267" />
-            <inertia ixx="8.0603E-04" ixy="-8.52034E-05" ixz="${-3.0124E-04 * reflect}" iyy="1.9301E-03" iyz="${1.9426E-05 * reflect}" izz="1.8484E-03" />
+            <origin xyz="0.0043916 0.016184 0.15576" rpy="0 0 0" />
+            <mass value="1.1325" />
+            <inertia ixx="0.0025497" ixy="2.6206E-05" ixz="6.2082E-05" iyy="0.0023517" iyz="-0.00020617" izz="0.00097131" />
         </inertial>
+    </xacro:macro>
+    <xacro:macro name="origin_joint_1" params="reflect">
+        <origin xyz="0 0 0" rpy="0 0 0" />
     </xacro:macro>
     <xacro:macro name="inertial_link_2" params="reflect">
         <inertial>
-            <origin xyz="-0.0941 2.6612E-04  ${0.0414 * reflect}" rpy="0 0 0" />
-            <mass value="0.9496" />
-            <inertia ixx="8.4202E-04" ixy="-5.7830E-06" ixz="${2.6145E-04 * reflect}" iyy="1.4185E-03" iyz="${-5.8148E-06 * reflect}" izz="1.4729E-03" />
+            <origin xyz="0.01786 -0.11956 -0.032097" rpy="0 0 0" />
+            <mass value="1.0436" />
+            <inertia ixx="0.0015021" ixy="0.00011264" ixz="1.0692E-05" iyy="0.00088017" iyz="-0.00015843" izz="0.0016021" />
         </inertial>
     </xacro:macro>
     <xacro:macro name="origin_joint_2" params="reflect">
-        <origin xyz="0.13 0.0483 ${0.04* reflect}" rpy="${-90 * reflect * deg_to_rad} 0 ${180 * deg_to_rad}" />
+        <origin xyz="0.0371099999999995 0.02 0.18" rpy="-1.57079632679489 0 -1.5707963267949" />
     </xacro:macro>
     <xacro:macro name="inertial_link_3" params="reflect">
         <inertial>
-            <origin xyz="0.0121 0.0151 ${-0.1344 * reflect}" rpy="0 0 0" />
-            <mass value="1.0816" />
-            <inertia ixx="2.4587E-03" ixy="-1.2107E-05" ixz="${2.1354E-04 * reflect}" iyy="2.7652E-03" iyz="${6.0550E-05 * reflect}" izz="9.3005E-04" />
+            <origin xyz="0.016184 -0.0043916 0.13565" rpy="0 0 0" />
+            <mass value="1.1325" />
+            <inertia ixx="0.0023517" ixy="-2.6206E-05" ixz="-0.00020617" iyy="0.0025497" iyz="-6.2082E-05" izz="0.00097131" />
         </inertial>
     </xacro:macro>
     <xacro:macro name="origin_joint_3" params="reflect">
-        <origin xyz="-0.1549 0 ${0.05 * reflect}" rpy="0 ${90 * reflect * deg_to_rad} 0" />
+        <origin xyz="0.019999999999999 -0.17011 -0.037110000000001" rpy="1.5707963267949 0 0" />
     </xacro:macro>
     <xacro:macro name="inertial_link_4" params="reflect">
         <inertial>
-            <origin xyz="0.018 -0.1025 ${0.0419 * reflect}" rpy="0 0 0" />
-            <mass value="0.99204" />
-            <inertia ixx="1.3967E-03" ixy="1.0609E-04" ixz="${-4.2876E-05 * reflect}" iyy="8.5657E-04" iyz="${2.5436E-04 * reflect}" izz="1.4862E-03" />
+            <origin xyz="-0.01786 0.11956 -0.032097" rpy="0 0 0" />
+            <mass value="1.0436" />
+            <inertia ixx="0.0015021" ixy="0.00011264" ixz="-1.0692E-05" iyy="0.00088017" iyz="0.00015843" izz="0.0016021" />
         </inertial>
     </xacro:macro>
     <xacro:macro name="origin_joint_4" params="reflect">
-        <origin xyz="0.05 0.02 ${-0.1651 * reflect}" rpy="${90 * reflect * deg_to_rad} ${-0 * reflect * deg_to_rad} ${-90 * deg_to_rad}" />
+        <origin xyz="0.0199999999999993 -0.0371100000000008 0.15989" rpy="1.57079632679489 0 0" />
     </xacro:macro>
     <xacro:macro name="origin_joint_5" params="reflect">
-        <origin xyz="0.02 -0.1546 ${0.05 * reflect}" rpy="${90 * reflect * deg_to_rad} 0 ${180 * deg_to_rad}" />
+        <origin xyz="-0.0199999999999971 0.17011 -0.037110000000002" rpy="-1.5707963267949 0 0" />
+    </xacro:macro>
+    <!-- Tool changer (can be present in both wrists)-->
+    <xacro:macro name="inertial_tool_changer_link" params="reflect">
+        <inertial>
+            <origin xyz="0.0019481 0.0017558 -0.0084934" rpy="0 0 0" />
+            <mass value="0.12272" />
+            <inertia ixx="5.1385E-05" ixy="8.5364E-07" ixz="-9.0329E-08" iyy="4.7962E-05" iyz="-1.8035E-07" izz="9.2935E-05" />
+        </inertial>
+    </xacro:macro>
+    <xacro:macro name="origin_joint_tool_changer" params="reflect">
+        <!-- @Lucien needs to fix -->
+        <origin xyz="0 0 0.017" rpy="0 0 0" />
     </xacro:macro>
 </robot>

File: pal_sea_arm_description/urdf/arm/arm_properties/tiago-sea/straight-wrist.properties.xacro (robot description, xacro)
@@ -25,15 +25,5 @@
     </xacro:macro>
     <xacro:macro name="origin_joint_7" params="reflect">
-        <origin xyz="0 -0.146 ${0.039 * reflect}" rpy="${-90 * reflect * deg_to_rad} 0 0" />
-    </xacro:macro>
-    <xacro:macro name="inertial_tool_link" params="reflect">
-        <inertial>
-            <origin xyz="0 0 0" rpy="0 0 0" />
-            <mass value="0.1" />
-            <inertia ixx="8.33E-07" ixy="0.0" ixz="0.0" iyy="8.33E-07" iyz="0.0" izz="1.25E-06" />
-        </inertial>
-    </xacro:macro>
-    <xacro:macro name="origin_joint_tool" params="reflect">
-        <origin xyz="0 0 0" rpy="${0.0 * deg_to_rad} ${90.0 * reflect * deg_to_rad} ${0 * deg_to_rad}" />
+        <origin xyz="0 -0.146 ${0.039 * reflect}" rpy="${-90 * reflect * deg_to_rad} 0 3.14" />
     </xacro:macro>
 </robot>

Commit message: Standalone meshes

File: pal_sea_arm_description/urdf/arm/arm.urdf.xacro (robot description, xacro)
@@ -21,4 +21,8 @@
     <xacro:if value="${arm_type in ['tiago-pro', 'pal-sea-arm-standalone']}">
       <xacro:property name="mesh_folder" value="arm_tiago_pro"/>
+    </xacro:if>
+    <!-- Standalone arm -->
+    <xacro:if value="${arm_type in ['pal-sea-arm-standalone']}">
+      <xacro:property name="mesh_folder" value="pal_sea_arm_standalone"/>
     </xacro:if>
     <!-- Tiago SEA -->

Commit message: Orientation std

File: pal_sea_arm_description/urdf/arm/arm.urdf.xacro (robot description, xacro)
@@ -268,4 +268,6 @@
         <parent link="${name}_7_link" />
         <child link="${name}_tool_link" />
+        <!-- This is added so both grippers are oriented the same -->
+        <origin xyz="0 0 0" rpy="0 0 1.570796" />
       </joint>
     </xacro:unless>
