Commit message: Gripper with rokubi position fixed

File: pal_sea_arm_description/urdf/arm/arm.urdf.xacro (robot description, xacro)
@@ -268,6 +268,4 @@
         <parent link="${name}_7_link" />
         <child link="${name}_tool_link" />
-        <!-- This is added so both grippers are oriented the same -->
-        <!-- <origin xyz="0 0 0.0" rpy="0 0 1.570796" /> -->
       </joint>
     </xacro:unless>

File: pal_sea_arm_description/urdf/arm/arm_properties/tiago-pro/arm.properties.xacro (robot description, xacro)
@@ -59,6 +59,7 @@
     </xacro:macro>
     <xacro:macro name="origin_joint_tool_changer" params="reflect">
-        <!-- @Lucien needs to fix -->
-        <origin xyz="0 0 0.017" rpy="0 0 0" />
+        <!-- @Lucien needs to fix, rotation remove to std gripper rotations -->
+        <!-- <origin xyz="0 0 0.017" rpy="0 0 1.570796" /> -->
+        <origin xyz="0 0 0.017" rpy="0 0 0.0" />
     </xacro:macro>
 </robot>

File: pal_sea_arm_description/urdf/arm/arm_properties/tiago-sea-dual/arm.properties.xacro (robot description, xacro)
@@ -49,6 +49,7 @@
     </xacro:macro>
     <xacro:macro name="origin_joint_tool_changer" params="reflect">
-        <!-- @Lucien needs to fix -->
-        <origin xyz="0 0 0.017" rpy="0 0 0" />
+        <!-- @Lucien needs to fix, rotation remove to std gripper rotations -->
+        <!-- <origin xyz="0 0 0.017" rpy="0 0 1.570796" /> -->
+        <origin xyz="0 0 0.017" rpy="0 0 0.0" />
     </xacro:macro>
 </robot>

File: pal_sea_arm_description/urdf/arm/arm_properties/tiago-sea/arm.properties.xacro (robot description, xacro)
@@ -59,6 +59,7 @@
     </xacro:macro>
     <xacro:macro name="origin_joint_tool_changer" params="reflect">
-        <!-- @Lucien needs to fix -->
-        <origin xyz="0 0 0.017" rpy="0 0 0" />
+        <!-- @Lucien needs to fix, rotation remove to std gripper rotations -->
+        <!-- <origin xyz="0 0 0.017" rpy="0 0 1.570796" /> -->
+        <origin xyz="0 0 0.017" rpy="0 0 0.0" />
     </xacro:macro>
 </robot>

File: pal_sea_arm_description/urdf/sensors/ft_sensor/rokubi.urdf.xacro (robot description, xacro)
@@ -76,4 +76,5 @@
       <parent link="${name}_ft_link" />
       <child link="${name}_ft_tool_link" />
+      <origin xyz="0 0 0.0052" rpy="0 0 0" />
     </joint>
   </xacro:macro>

Commit message: Limits new structure

File: pal_sea_arm_description/urdf/arm/arm.urdf.xacro (robot description, xacro)
@@ -38,6 +38,6 @@
     </xacro:if> -->
     <!-- INCLUDES -->
-    <xacro:include filename="$(find pal_sea_arm_description)/urdf/arm/limits/arm_${arm_type}.limits.xacro"/>
-    <xacro:include filename="$(find pal_sea_arm_description)/urdf/arm/arm_properties/${arm_type}/arm.properties.xacro"/>
+    <xacro:include filename="$(find pal_sea_arm_description)/urdf/arm/arm_limits/${arm_type}/arm.limits.xacro"/>
+    <xacro:include filename="$(find pal_sea_arm_description)/urdf/arm/arm_limits/${arm_type}/${wrist_model}.limits.xacro"/>
     <xacro:include filename="$(find pal_sea_arm_description)/urdf/arm/arm_properties/${arm_type}/arm.properties.xacro"/>
     <xacro:include filename="$(find pal_sea_arm_description)/urdf/arm/arm_properties/${arm_type}/${wrist_model}.properties.xacro"/>

File: pal_sea_arm_description/urdf/arm/arm_limits/pal-sea-arm-standalone/arm.limits.xacro (robot description, xacro)
@@ -1,8 +1,9 @@
 <robot xmlns:xacro="http://ros.org/wiki/xacro">
   <!-- Constant parameters -->
-  <xacro:property name="arm_friction"       value="1.0" />
-  <xacro:property name="arm_damping"        value="1.0" />
+  <xacro:property name="arm_friction" value="1.0" />
+  <xacro:property name="arm_damping" value="1.0" />
   <xacro:property name="arm_k_position" value="20"/>
   <xacro:property name="arm_k_velocity" value="20"/>
+  <!-- Joint limits -->
   <xacro:property name="arm_1_joint_ub" value="148.97" />
   <xacro:property name="arm_1_joint_lb" value="-148.97" />
@@ -13,23 +14,13 @@
   <xacro:property name="arm_4_joint_ub" value="63.03" />
   <xacro:property name="arm_4_joint_lb" value="-139.8" />
-  <xacro:property name="arm_5_joint_ub" value="148.97" />
-  <xacro:property name="arm_5_joint_lb" value="-148.97" />
-  <xacro:property name="arm_6_joint_ub" value="114.59" />
-  <xacro:property name="arm_6_joint_lb" value="-114.59" />
-  <xacro:property name="arm_7_joint_ub" value="148.97" />
-  <xacro:property name="arm_7_joint_lb" value="-148.97" />
-  <xacro:property name="arm_1_max_velocity"      value="1.95" />
-  <xacro:property name="arm_2_max_velocity"      value="1.95" />
-  <xacro:property name="arm_3_max_velocity"      value="2.35" />
-  <xacro:property name="arm_4_max_velocity"      value="2.35" />
-  <xacro:property name="arm_5_max_velocity"      value="2.35" />
-  <xacro:property name="arm_6_max_velocity"      value="2.35" />
-  <xacro:property name="arm_7_max_velocity"      value="2.35" />
-  <xacro:property name="arm_1_max_effort"   value="43.0" />
-  <xacro:property name="arm_2_max_effort"   value="43.0" />
-  <xacro:property name="arm_3_max_effort"   value="26" />
-  <xacro:property name="arm_4_max_effort"   value="26" />
-  <xacro:property name="arm_5_max_effort"   value="26" />
-  <xacro:property name="arm_6_max_effort"   value="26" />
-  <xacro:property name="arm_7_max_effort"   value="26" />
+  <!-- Velocity limits -->
+  <xacro:property name="arm_1_max_velocity" value="1.95" />
+  <xacro:property name="arm_2_max_velocity" value="1.95" />
+  <xacro:property name="arm_3_max_velocity" value="2.35" />
+  <xacro:property name="arm_4_max_velocity" value="2.35" />
+  <!-- Effort limits -->
+  <xacro:property name="arm_1_max_effort" value="43.0" />
+  <xacro:property name="arm_2_max_effort" value="43.0" />
+  <xacro:property name="arm_3_max_effort" value="26" />
+  <xacro:property name="arm_4_max_effort" value="26" />
 </robot>

File: pal_sea_arm_description/urdf/arm/arm_limits/tiago-pro/arm.limits.xacro (robot description, xacro)
@@ -5,4 +5,5 @@
   <xacro:property name="arm_k_position" value="20"/>
   <xacro:property name="arm_k_velocity" value="20"/>
+  <!-- Joint limits -->
   <xacro:property name="arm_1_joint_ub" value="148.97" />
   <xacro:property name="arm_1_joint_lb" value="-148.97" />
@@ -13,23 +14,13 @@
   <xacro:property name="arm_4_joint_ub" value="63.03" />
   <xacro:property name="arm_4_joint_lb" value="-139.8" />
-  <xacro:property name="arm_5_joint_ub" value="148.97" />
-  <xacro:property name="arm_5_joint_lb" value="-148.97" />
-  <xacro:property name="arm_6_joint_ub" value="114.59" />
-  <xacro:property name="arm_6_joint_lb" value="-114.59" />
-  <xacro:property name="arm_7_joint_ub" value="148.97" />
-  <xacro:property name="arm_7_joint_lb" value="-148.97" />
+  <!-- Velocity limits -->
   <xacro:property name="arm_1_max_velocity" value="1.95" />
   <xacro:property name="arm_2_max_velocity" value="1.95" />
   <xacro:property name="arm_3_max_velocity" value="2.35" />
   <xacro:property name="arm_4_max_velocity" value="2.35" />
-  <xacro:property name="arm_5_max_velocity" value="2.35" />
-  <xacro:property name="arm_6_max_velocity" value="2.35" />
-  <xacro:property name="arm_7_max_velocity" value="2.35" />
+  <!-- Effort limits -->
   <xacro:property name="arm_1_max_effort" value="43.0" />
   <xacro:property name="arm_2_max_effort" value="43.0" />
   <xacro:property name="arm_3_max_effort" value="26" />
   <xacro:property name="arm_4_max_effort" value="26" />
-  <xacro:property name="arm_5_max_effort" value="26" />
-  <xacro:property name="arm_6_max_effort" value="26" />
-  <xacro:property name="arm_7_max_effort" value="26" />
 </robot>

File: pal_sea_arm_description/urdf/arm/arm_properties/tiago-pro/arm.properties.xacro (robot description, xacro)
@@ -56,5 +56,5 @@
     </xacro:macro>
     <xacro:macro name="origin_joint_tool_changer" params="reflect">
-        <!-- @Lucien needs to fix, rotation remove to std gripper rotations -->
+        <!-- Align with @Lucien -->
         <origin xyz="0 0 0.017" rpy="0 0 1.570796" />
         <!-- <origin xyz="0 0 0.017" rpy="0 0 0.0" /> -->

Commit message: Update on link 7 + fix joint limits

File: pal_sea_arm_description/urdf/arm/arm.urdf.xacro (robot description, xacro)
@@ -14,5 +14,5 @@
 <robot xmlns:xacro="http://ros.org/wiki/xacro">
   <!-- Transmissions file -->
-  <xacro:macro name="pal_sea_arm" params="name parent *origin arm_type tool_changer wrist_model reflect:=1 arm_1_offset arm_2_offset arm_3_offset arm_4_offset arm_5_offset arm_6_offset arm_7_offset no_safety_eps:=False">
+  <xacro:macro name="pal_sea_arm" params="name parent *origin arm_type tool_changer wrist_model reflect:=1 first_joint_reflect:=1 arm_1_offset arm_2_offset arm_3_offset arm_4_offset arm_5_offset arm_6_offset arm_7_offset no_safety_eps:=False">
     <!-- PROPERTIES -->
     <xacro:property name="arm_eps" value="${0.00 if no_safety_eps else 0.07}"/>
@@ -268,4 +268,5 @@
         <parent link="${name}_7_link" />
         <child link="${name}_tool_link" />
+        <origin xyz="0 0 0" rpy="0 ${0 if reflect is 1 else 180 * deg_to_rad} 0.0" />
       </joint>
     </xacro:unless>

File: pal_sea_arm_description/urdf/arm/arm_limits/pal-sea-arm-standalone/spherical-wrist.limits.xacro (robot description, xacro)
@@ -1,5 +1,5 @@
 <robot xmlns:xacro="http://ros.org/wiki/xacro">
   <!-- Joint limits -->
-  <xacro:property name="arm_5_joint_ub" value="230" />
+  <xacro:property name="arm_5_joint_ub" value="210" />
   <xacro:property name="arm_5_joint_lb" value="-90" />
   <xacro:property name="arm_6_joint_ub" value="114.59" />

File: pal_sea_arm_description/urdf/arm/arm_limits/tiago-pro/arm.limits.xacro (robot description, xacro)
@@ -6,6 +6,6 @@
   <xacro:property name="arm_k_velocity" value="20"/>
   <!-- Joint limits -->
-  <xacro:property name="arm_1_joint_ub" value="148.97" />
-  <xacro:property name="arm_1_joint_lb" value="-148.97" />
+  <xacro:property name="arm_1_joint_ub" value="${30 if first_joint_reflect is 1 else 270}" />
+  <xacro:property name="arm_1_joint_lb" value="${-270 if first_joint_reflect is 1 else -30}" />
   <xacro:property name="arm_2_joint_ub" value="63.03" />
   <xacro:property name="arm_2_joint_lb" value="-139.8" />

File: pal_sea_arm_description/urdf/arm/arm_properties/pal-sea-arm-standalone/spherical-wrist.properties.xacro (robot description, xacro)
@@ -25,5 +25,5 @@
     </xacro:macro>
     <xacro:macro name="origin_joint_7" params="reflect">
-        <origin xyz="0.07 -0.0534 -0.0422" rpy="1.5708 0 0" />
+        <origin xyz="-0.07 -0.0534 0.0422" rpy="1.5708 -1.5708 0" />
     </xacro:macro>
 </robot>

File: pal_sea_arm_description/urdf/arm/arm_properties/tiago-pro/spherical-wrist.properties.xacro (robot description, xacro)
@@ -29,5 +29,5 @@
     </xacro:macro>
     <xacro:macro name="origin_joint_7" params="reflect">
-        <origin xyz="-0.07 -0.0534 0.0422" rpy="1.5708 0 0" />
+        <origin xyz="-0.07 -0.0534 0.0422" rpy="1.5708 -1.5708 0" />
     </xacro:macro>
 </robot>

File: pal_sea_arm_description/urdf/arm/arm_properties/tiago-sea-dual/arm.properties.xacro (robot description, xacro)
@@ -51,5 +51,5 @@
         <!-- @Lucien needs to fix, rotation remove to std gripper rotations -->
         <!-- <origin xyz="0 0 0.017" rpy="0 0 1.570796" /> -->
-        <origin xyz="0 0 0.017" rpy="0 0 0.0" />
+        <origin xyz="0 0 0.017" rpy="0 ${0 if reflect is 1 else 180 * deg_to_rad} 0.0" />
     </xacro:macro>
 </robot>

Commit message: Fixing the 6 axis joint

File: pal_sea_arm_description/urdf/arm/arm.urdf.xacro (robot description, xacro)
@@ -200,5 +200,5 @@
       <parent link="${name}_5_link" />
       <child link="${name}_6_link" />
-      <axis xyz="0 0 1" />
+      <axis xyz="0 0 -1" />
       <limit lower="${arm_6_joint_lb * deg_to_rad}" upper="${arm_6_joint_ub * deg_to_rad}" effort="${arm_6_max_effort}" velocity="${arm_6_max_velocity}" />
       <dynamics friction="${arm_friction}" damping="${arm_damping}"/>

Commit message: add material + fix 7th joint

File: pal_sea_arm_description/urdf/arm/arm.urdf.xacro (robot description, xacro)
@@ -244,7 +244,5 @@
             <mesh filename="package://pal_sea_arm_description/meshes/${mesh_folder}/tool_changer_link.stl" scale="1 1 ${reflect}" />
           </geometry>
-          <material name="">
-            <color rgba="0.29804 0.29804 0.29804 1" />
-          </material>
+          <material name="pal/DarkGrey"/>
         </visual>
         <collision>

File: pal_sea_arm_description/urdf/arm/arm_properties/tiago-pro/arm.properties.xacro (robot description, xacro)
@@ -57,5 +57,5 @@
     <xacro:macro name="origin_joint_tool_changer" params="reflect">
         <!-- Align with @Lucien -->
-        <origin xyz="0 0 0.017" rpy="0 0 1.570796" />
+        <origin xyz="0 0 0.017" rpy="0 0 0" />
         <!-- <origin xyz="0 0 0.017" rpy="0 0 0.0" /> -->
     </xacro:macro>

File: pal_sea_arm_description/urdf/sensors/ft_sensor/ati.urdf.xacro (robot description, xacro)
@@ -42,4 +42,9 @@
       </collision>
     </link>
+    <gazebo reference="${name}_ft_sensor_base_link">
+      <material>Gazebo/DarkGrey</material>
+      <mu1>0.9</mu1>
+      <mu2>0.9</mu2>
+    </gazebo>
     <joint name="${name}_ft_sensor_base_joint" type="fixed">
       <parent link="${parent}" />
@@ -68,4 +73,9 @@
       </collision>
     </link>
+    <gazebo reference="${name}_ft_sensor_link">
+      <material>Gazebo/DarkGrey</material>
+      <mu1>0.9</mu1>
+      <mu2>0.9</mu2>
+    </gazebo>
     <joint name="${name}_ft_sensor_joint" type="fixed">
       <!-- <origin xyz="0 0 0.033998" rpy="0 0 0" /> -->
@@ -95,4 +105,9 @@
       </collision>
     </link>
+    <gazebo reference="${name}_ft_tool_link">
+      <material>Gazebo/DarkGrey</material>
+      <mu1>0.9</mu1>
+      <mu2>0.9</mu2>
+    </gazebo>
     <joint name="${name}_ft_tool_joint" type="fixed">
       <origin xyz="0 0 0.039998" rpy="0 0 0" />

File: pal_sea_arm_description/urdf/sensors/ft_sensor/rokubi.urdf.xacro (robot description, xacro)
@@ -26,7 +26,5 @@
           <mesh filename="package://pal_sea_arm_description/meshes/sensors/rokubi/rokubi_ft_sensor.stl"/>
         </geometry>
-        <material name="">
-          <color rgba="0.29804 0.29804 0.29804 1" />
-        </material>
+        <material name="pal/DarkGrey"/>
       </visual>
       <collision>

Commit message: Fix to use same urdf for tiago sea and tiago pro

File: pal_sea_arm_description/urdf/arm/arm.urdf.xacro (robot description, xacro)
@@ -200,5 +200,5 @@
       <parent link="${name}_5_link" />
       <child link="${name}_6_link" />
-      <axis xyz="0 0 -1" />
+      <axis xyz="0 0 ${-1 if wrist_model=='spherical-wrist' else 1}" />
       <limit lower="${arm_6_joint_lb * deg_to_rad}" upper="${arm_6_joint_ub * deg_to_rad}" effort="${arm_6_max_effort}" velocity="${arm_6_max_velocity}" />
       <dynamics friction="${arm_friction}" damping="${arm_damping}"/>

Commit message: Add reflect on the 5th joint

File: pal_sea_arm_description/urdf/arm/arm.urdf.xacro (robot description, xacro)
@@ -14,5 +14,5 @@
 <robot xmlns:xacro="http://ros.org/wiki/xacro">
   <!-- Transmissions file -->
-  <xacro:macro name="pal_sea_arm" params="name parent *origin arm_type tool_changer wrist_model reflect:=1 first_joint_reflect:=1 arm_1_offset arm_2_offset arm_3_offset arm_4_offset arm_5_offset arm_6_offset arm_7_offset no_safety_eps:=False">
+  <xacro:macro name="pal_sea_arm" params="name parent *origin arm_type tool_changer wrist_model reflect:=1 joint_reflect:=1 arm_1_offset arm_2_offset arm_3_offset arm_4_offset arm_5_offset arm_6_offset arm_7_offset no_safety_eps:=False">
     <!-- PROPERTIES -->
     <xacro:property name="arm_eps" value="${0.00 if no_safety_eps else 0.07}"/>

File: pal_sea_arm_description/urdf/arm/arm_limits/tiago-pro/arm.limits.xacro (robot description, xacro)
@@ -6,6 +6,6 @@
   <xacro:property name="arm_k_velocity" value="20"/>
   <!-- Joint limits -->
-  <xacro:property name="arm_1_joint_ub" value="${30 if first_joint_reflect is 1 else 270}" />
-  <xacro:property name="arm_1_joint_lb" value="${-270 if first_joint_reflect is 1 else -30}" />
+  <xacro:property name="arm_1_joint_ub" value="${30 if joint_reflect is 1 else 270}" />
+  <xacro:property name="arm_1_joint_lb" value="${-270 if joint_reflect is 1 else -30}" />
   <xacro:property name="arm_2_joint_ub" value="63.03" />
   <xacro:property name="arm_2_joint_lb" value="-139.8" />

File: pal_sea_arm_description/urdf/arm/arm_limits/tiago-pro/spherical-wrist.limits.xacro (robot description, xacro)
@@ -1,6 +1,6 @@
 <robot xmlns:xacro="http://ros.org/wiki/xacro">
   <!-- Joint limits -->
-  <xacro:property name="arm_5_joint_ub" value="210" />
-  <xacro:property name="arm_5_joint_lb" value="-90" />
+  <xacro:property name="arm_5_joint_ub" value="${210 if joint_reflect is 1 else 90}" />
+  <xacro:property name="arm_5_joint_lb" value="${-90 if joint_reflect is 1 else -210}" />
   <xacro:property name="arm_6_joint_ub" value="172" />
   <xacro:property name="arm_6_joint_lb" value="-108" />

Commit message: Adding real 5th mesh

File: pal_sea_arm_description/urdf/arm/arm.urdf.xacro (robot description, xacro)
@@ -164,5 +164,5 @@
         <origin xyz="0 0 0" rpy="0 0 0" />
         <geometry>
-          <mesh filename="package://pal_sea_arm_description/meshes/${mesh_folder}/${wrist_model}/arm_5_link_collision.stl" scale="1 1 ${reflect}" />
+          <mesh filename="package://pal_sea_arm_description/meshes/${mesh_folder}/${wrist_model}/arm_5_link.stl" scale="1 1 ${reflect}" />
         </geometry>
       </collision>

Commit message: Simplify arm_7_link + update ATI meshes and inertia

File: pal_sea_arm_description/urdf/arm/arm.urdf.xacro (robot description, xacro)
@@ -218,5 +218,5 @@
         <origin xyz="0 0 0" rpy="0 0 0" />
         <geometry>
-          <mesh filename="package://pal_sea_arm_description/meshes/${mesh_folder}/${wrist_model}/arm_7_link_collision.stl" scale="1 1 ${reflect}" />
+          <cylinder radius="0.0375" length="0.0366"/>
         </geometry>
       </collision>
@@ -237,20 +237,5 @@
     <!-- With tool changer (the tool link is the tool changer)-->
     <xacro:if value="${tool_changer}">
-      <link name="${name}_tool_link">
-        <xacro:inertial_tool_changer_link reflect="${reflect}"/>
-        <visual>
-          <origin xyz="0 0 0" rpy="0 0 0" />
-          <geometry>
-            <mesh filename="package://pal_sea_arm_description/meshes/${mesh_folder}/tool_changer_link.stl" scale="1 1 ${reflect}" />
-          </geometry>
-          <material name="pal/DarkGrey"/>
-        </visual>
-        <collision>
-          <origin xyz="0 0 0" rpy="0 0 0" />
-          <geometry>
-            <mesh filename="package://pal_sea_arm_description/meshes/${mesh_folder}/tool_changer_link_collision.stl" scale="1 1 ${reflect}" />
-          </geometry>
-        </collision>
-      </link>
+      <link name="${name}_tool_link"/>
       <joint name="${name}_tool_joint" type="fixed">
         <parent link="${name}_7_link" />

File: pal_sea_arm_description/urdf/arm/arm_properties/tiago-pro/arm.properties.xacro (robot description, xacro)
@@ -47,12 +47,4 @@
         <origin xyz="0.0199999999999993 -0.0371100000000008 0.15989" rpy="1.57079632679489 0 0" />
     </xacro:macro>
-    <!-- Tool changer (can be present in both wrists)-->
-    <xacro:macro name="inertial_tool_changer_link" params="reflect">
-        <inertial>
-            <origin xyz="0.003414871500006 0.002458561521477 -0.001077004696741" rpy="0 0 0" />
-            <mass value="0.0655061851536" />
-            <inertia ixx="1.79461992752602E-05" ixy="1.70670100210845E-06" ixz="-2.54814948767968E-09" iyy="1.47274432150498E-05" iyz="1.09471559381518E-07" izz="3.12924968277541E-05" />
-        </inertial>
-    </xacro:macro>
     <xacro:macro name="origin_joint_tool_changer" params="reflect">
         <!-- Align with @Lucien -->

File: pal_sea_arm_description/urdf/sensors/ft_sensor/ati.urdf.xacro (robot description, xacro)
@@ -36,7 +36,7 @@
       </visual>
       <collision>
-        <origin xyz="0 0 0" rpy="0 0 0" />
+        <origin xyz="0 0 0.0229" rpy="0 0 0" />
         <geometry>
-          <mesh filename="package://pal_sea_arm_description/meshes/sensors/ati/base_link.stl"/>
+          <cylinder radius="0.0375" length="0.045898"/>
         </geometry>
       </collision>
@@ -52,5 +52,5 @@
       <axis xyz="0 0 0" />
     </joint>
-    <!-- FT sensor link  -->
+    <!-- FT sensor link; the inertia and visual needs to exist for the ft sensor gazebo plugin to work -->
     <link name="${name}_ft_sensor_link">
       <inertial>
@@ -60,14 +60,14 @@
       </inertial>
       <visual>
-        <origin xyz="0 0 0" rpy="0 0 0" />
+        <origin xyz="0 0 0.01" rpy="0 0 0" />
         <geometry>
-          <mesh filename="package://pal_sea_arm_description/meshes/sensors/ati/ft_sensor_link.stl"/>
+          <cylinder radius="0.03" length="0.02"/>
         </geometry>
         <material name="pal/DarkGrey"/>
       </visual>
       <collision>
-        <origin xyz="0 0 0" rpy="0 0 0" />
+        <origin xyz="0 0 0.01" rpy="0 0 0" />
         <geometry>
-          <mesh filename="package://pal_sea_arm_description/meshes/sensors/ati/ft_sensor_link.stl"/>
+          <cylinder radius="0.03" length="0.02"/>
         </geometry>
       </collision>
@@ -84,5 +84,5 @@
       <axis xyz="0 0 0" />
     </joint>
-    <!-- FT out link -->
+    <!-- FT out link; the inertia and visual needs to exist for the ft sensor gazebo plugin to work -->
     <link name="${name}_ft_tool_link">
       <inertial>
@@ -92,14 +92,14 @@
       </inertial>
       <visual>
-        <origin xyz="0 0 0" rpy="0 0 0" />
+        <origin xyz="0 0 -0.01" rpy="0 0 0" />
         <geometry>
-          <mesh filename="package://pal_sea_arm_description/meshes/sensors/ati/ft_out_link.stl"/>
+          <cylinder radius="0.03" length="0.02"/>
         </geometry>
         <material name="pal/DarkGrey"/>
       </visual>
       <collision>
-        <origin xyz="0 0 0" rpy="0 0 0" />
+        <origin xyz="0 0 -0.01" rpy="0 0 0" />
         <geometry>
-          <mesh filename="package://pal_sea_arm_description/meshes/sensors/ati/ft_out_link.stl"/>
+          <cylinder radius="0.03" length="0.02"/>
         </geometry>
       </collision>

Commit message: Update collision model to match the link5 specific shape

File: pal_sea_arm_description/urdf/arm/arm.urdf.xacro (robot description, xacro)
@@ -164,5 +164,5 @@
         <origin xyz="0 0 0" rpy="0 0 0" />
         <geometry>
-          <mesh filename="package://pal_sea_arm_description/meshes/${mesh_folder}/${wrist_model}/arm_5_link.stl" scale="1 1 ${reflect}" />
+          <mesh filename="package://pal_sea_arm_description/meshes/${mesh_folder}/${wrist_model}/arm_5_link_collision.stl" scale="1 1 ${reflect}" />
         </geometry>
       </collision>
