Commit message: Fix inertia parameter

File: pal_sea_arm_description/urdf/arm/arm.urdf.xacro (robot description, xacro)
@@ -18,8 +18,14 @@
     <xacro:property name="arm_eps" value="${0.00 if no_safety_eps else 0.07}"/>
     <xacro:property name="mesh_folder"/>
+    <xacro:property name="inertia_version"/>
     <!-- Tiago Pro -->
     <xacro:if value="${arm_type in ['tiago-pro', 'tiago-pro-s']}">
       <xacro:property name="mesh_folder" value="arm_tiago_pro"/>
-      <xacro:property name="inertia_version" value="${arm_type}"/>
+      <xacro:if value="${arm_type == 'tiago-pro'}">
+        <xacro:property name="inertia_version" value="tiago-pro"/>
+      </xacro:if>
+      <xacro:if value="${arm_type == 'tiago-pro-s'}">
+        <xacro:property name="inertia_version" value="tiago-pro-s"/>
+      </xacro:if>
       <xacro:property name="arm_type" value="tiago-pro"/>
     </xacro:if>

File: pal_sea_arm_description/urdf/arm/arm_properties/tiago-pro/arm.properties.xacro (robot description, xacro)
@@ -8,5 +8,5 @@
     </xacro:macro>
     <xacro:macro name="inertial_link_1" params="reflect">
-        <xacro:if value="${inertia_version in ['tiago-pro-s']}">
+        <xacro:if value="${inertia_version == 'tiago-pro-s'}">
             <inertial>
                 <origin xyz="0.00476 0.01532 0.15274" rpy="0 0 0" />
@@ -15,5 +15,5 @@
             </inertial>
         </xacro:if>
-        <xacro:if value="${inertia_version in ['tiago-pro']}">
+        <xacro:if value="${inertia_version == 'tiago-pro'}">
             <inertial>
                 <origin xyz="0.0043916 0.016184 0.15576" rpy="0 0 0" />
@@ -27,5 +27,5 @@
     </xacro:macro>
     <xacro:macro name="inertial_link_2" params="reflect">
-        <xacro:if value="${inertia_version in ['tiago-pro-s']}">
+        <xacro:if value="${inertia_version == 'tiago-pro-s'}">
             <inertial>
                 <origin xyz="0.01715 -0.11231 -0.03000" rpy="0 0 0" />
@@ -34,5 +34,5 @@
             </inertial>
         </xacro:if>
-        <xacro:if value="${inertia_version in ['tiago-pro']}">
+        <xacro:if value="${inertia_version == 'tiago-pro'}">
             <inertial>
                 <origin xyz="0.01786 -0.11956 -0.032097" rpy="0 0 0" />
@@ -46,5 +46,5 @@
     </xacro:macro>
     <xacro:macro name="inertial_link_3" params="reflect">
-        <xacro:if value="${inertia_version in ['tiago-pro-s']}">
+        <xacro:if value="${inertia_version == 'tiago-pro-s'}">
             <inertial>
                 <origin xyz="0.01530 -0.00471 0.13242" rpy="0 0 0" />
@@ -53,5 +53,5 @@
             </inertial>
         </xacro:if>
-        <xacro:if value="${inertia_version in ['tiago-pro']}">
+        <xacro:if value="${inertia_version == 'tiago-pro'}">
             <inertial>
                 <origin xyz="0.016184 -0.0043916 0.13565" rpy="0 0 0" />
@@ -65,5 +65,5 @@
     </xacro:macro>
     <xacro:macro name="inertial_link_4" params="reflect">
-        <xacro:if value="${inertia_version in ['tiago-pro-s']}">
+        <xacro:if value="${inertia_version == 'tiago-pro-s'}">
             <inertial>
                 <origin xyz="-0.01715 0.11231 -0.03000" rpy="0 0 0" />
@@ -72,5 +72,5 @@
             </inertial>
         </xacro:if>
-        <xacro:if value="${inertia_version in ['tiago-pro']}">
+        <xacro:if value="${inertia_version == 'tiago-pro'}">
             <inertial>
                 <origin xyz="-0.01786 0.11956 -0.032097" rpy="0 0 0" />

Commit message: adding limit j1

File: pal_sea_arm_description/urdf/arm/arm.urdf.xacro (robot description, xacro)
@@ -75,4 +75,5 @@
       <child link="${name}_1_link" />
       <axis xyz="0 0 1" />
+      <limit effort="${arm_1_max_effort}" velocity="${arm_1_max_velocity}"/>
       <xacro:if value="${joint_type == 'revolute'}">
         <xacro:if value="${limits_v2}">

Commit message: Fix rotate axe for joint 6

File: pal_sea_arm_description/urdf/arm/arm.urdf.xacro (robot description, xacro)
@@ -226,14 +226,14 @@
         </collision>
       </link>
-      <!-- ARM 6 JOINT -->
-      <joint name="${name}_6_joint" type="revolute">
-        <xacro:origin_joint_6 reflect="${reflect}"/>
-        <parent link="${name}_5_link" />
-        <child link="${name}_6_link" />
-        <axis xyz="0 0 ${-1 if wrist_model=='spherical-wrist' else 1}" />
-        <limit lower="${arm_6_joint_lb * deg_to_rad}" upper="${arm_6_joint_ub * deg_to_rad}" effort="${arm_6_max_effort}" velocity="${arm_6_max_velocity}" />
-        <dynamics friction="${arm_friction}" damping="${arm_damping}"/>
-        <safety_controller k_position="${arm_k_position}" k_velocity="${arm_k_velocity}" soft_lower_limit="${arm_6_joint_lb * deg_to_rad  + arm_eps}" soft_upper_limit="${arm_6_joint_ub * deg_to_rad - arm_eps}" />
-      </joint>
+    <!-- ARM 6 JOINT -->
+    <joint name="${name}_6_joint" type="revolute">
+      <xacro:origin_joint_6 reflect="${reflect}"/>
+      <parent link="${name}_5_link" />
+      <child link="${name}_6_link" />
+      <axis xyz="0 0 ${-1 if wrist_model=='spherical-wrist' else 1}" />
+      <limit lower="${arm_6_joint_lb * deg_to_rad}" upper="${arm_6_joint_ub * deg_to_rad}" effort="${arm_6_max_effort}" velocity="${arm_6_max_velocity}" />
+      <dynamics friction="${arm_friction}" damping="${arm_damping}"/>
+      <safety_controller k_position="${arm_k_position}" k_velocity="${arm_k_velocity}" soft_lower_limit="${arm_6_joint_lb * deg_to_rad  + arm_eps}" soft_upper_limit="${arm_6_joint_ub * deg_to_rad - arm_eps}" />
+    </joint>
     <!-- ARM 7 LINK -->
       <link name="${name}_7_link">

Commit message: fix 1st joint

File: pal_sea_arm_description/urdf/arm/arm.urdf.xacro (robot description, xacro)
@@ -75,5 +75,7 @@
       <child link="${name}_1_link" />
       <axis xyz="0 0 1" />
-      <limit effort="${arm_1_max_effort}" velocity="${arm_1_max_velocity}"/>
+      <xacro:if value="${joint_type == 'continuous'}">
+        <limit effort="${arm_1_max_effort}" velocity="${arm_1_max_velocity}" />
+      </xacro:if>
       <xacro:if value="${joint_type == 'revolute'}">
         <xacro:if value="${limits_v2}">

Commit message: remove use_sim_time

File: pal_sea_arm_description/urdf/arm/arm.urdf.xacro (robot description, xacro)
@@ -14,5 +14,5 @@
 <robot xmlns:xacro="http://ros.org/wiki/xacro">
   <!-- Transmissions file -->
-  <xacro:macro name="pal_sea_arm" params="name parent use_sim_time:=^|false *origin arm_type tool_changer wrist_model reflect:=1 joint_reflect:=1 arm_1_offset arm_2_offset arm_3_offset arm_4_offset arm_5_offset arm_6_offset arm_7_offset no_safety_eps:=False limits_v2:=False">
+  <xacro:macro name="pal_sea_arm" params="name parent *origin arm_type tool_changer wrist_model reflect:=1 joint_reflect:=1 arm_1_offset arm_2_offset arm_3_offset arm_4_offset arm_5_offset arm_6_offset arm_7_offset no_safety_eps:=False limits_v2:=False">
     <!-- PROPERTIES -->
     <xacro:property name="arm_eps" value="${0.00 if no_safety_eps else 0.07}"/>

Commit message: add 7th link collision

File: pal_sea_arm_description/urdf/arm/arm.urdf.xacro (robot description, xacro)
@@ -250,5 +250,5 @@
           <origin xyz="0 0 0" rpy="0 0 0" />
           <geometry>
-            <cylinder radius="0.0375" length="0.0366"/>
+            <mesh filename="package://pal_sea_arm_description/meshes/${mesh_folder}/${wrist_model}/arm_7_link_collision.stl" scale="1 1 ${reflect}" />
           </geometry>
         </collision>

Commit message: set 3th and 5th as infinite joints

File: pal_sea_arm_description/urdf/arm/arm.urdf.xacro (robot description, xacro)
@@ -134,18 +134,24 @@
     </link>
     <!-- ARM 3 JOINT -->
-    <joint name="${name}_3_joint" type="revolute">
+    <xacro:property name="joint_type" value="${'continuous' if arm_type == 'pal-sea-arm-standalone' else 'revolute'}" />
+    <joint name="${name}_3_joint" type="${joint_type}">
       <xacro:origin_joint_3 reflect="${reflect}"/>
       <parent link="${name}_2_link" />
       <child link="${name}_3_link" />
       <axis xyz="0 0 1" />
-      <xacro:if value="${limits_v2}">
-        <limit lower="${arm_3_joint_lb_v2 * deg_to_rad}" upper="${arm_3_joint_ub_v2 * deg_to_rad}" effort="${arm_3_max_effort}" velocity="${arm_3_max_velocity}" />
-      <safety_controller k_position="${arm_k_position}" k_velocity="${arm_k_velocity}" soft_lower_limit="${arm_3_joint_lb_v2 * deg_to_rad  + arm_eps}" soft_upper_limit="${arm_3_joint_ub_v2 * deg_to_rad - arm_eps}" />
-      </xacro:if>
-      <xacro:unless value="${limits_v2}">
-        <limit lower="${arm_3_joint_lb * deg_to_rad}" upper="${arm_3_joint_ub * deg_to_rad}" effort="${arm_3_max_effort}" velocity="${arm_3_max_velocity}" />
-        <safety_controller k_position="${arm_k_position}" k_velocity="${arm_k_velocity}" soft_lower_limit="${arm_3_joint_lb * deg_to_rad  + arm_eps}" soft_upper_limit="${arm_3_joint_ub * deg_to_rad - arm_eps}" />
-      </xacro:unless>
-      <dynamics friction="${arm_friction}" damping="${arm_damping}"/>
+      <xacro:if value="${joint_type == 'continuous'}">
+        <limit effort="${arm_3_max_effort}" velocity="${arm_3_max_velocity}" />
+      </xacro:if>
+      <xacro:if value="${joint_type == 'revolute'}">
+        <xacro:if value="${limits_v2}">
+          <limit lower="${arm_3_joint_lb_v2 * deg_to_rad}" upper="${arm_3_joint_ub_v2 * deg_to_rad}" effort="${arm_3_max_effort}" velocity="${arm_3_max_velocity}" />
+        <safety_controller k_position="${arm_k_position}" k_velocity="${arm_k_velocity}" soft_lower_limit="${arm_3_joint_lb_v2 * deg_to_rad  + arm_eps}" soft_upper_limit="${arm_3_joint_ub_v2 * deg_to_rad - arm_eps}" />
+        </xacro:if>
+        <xacro:unless value="${limits_v2}">
+          <limit lower="${arm_3_joint_lb * deg_to_rad}" upper="${arm_3_joint_ub * deg_to_rad}" effort="${arm_3_max_effort}" velocity="${arm_3_max_velocity}" />
+          <safety_controller k_position="${arm_k_position}" k_velocity="${arm_k_velocity}" soft_lower_limit="${arm_3_joint_lb * deg_to_rad  + arm_eps}" soft_upper_limit="${arm_3_joint_ub * deg_to_rad - arm_eps}" />
+        </xacro:unless>
+      </xacro:if>
+        <dynamics friction="${arm_friction}" damping="${arm_damping}"/>
     </joint>
     <!-- ARM 4 LINK -->
@@ -194,17 +200,23 @@
     </link>
     <!-- ARM 5 JOINT -->
-    <joint name="${name}_5_joint" type="revolute">
+    <xacro:property name="joint_type" value="${'continuous' if arm_type == 'pal-sea-arm-standalone' else 'revolute'}" />
+    <joint name="${name}_5_joint" type="${joint_type}">
       <xacro:origin_joint_5 reflect="${reflect}"/>
       <parent link="${name}_4_link" />
       <child link="${name}_5_link" />
       <axis xyz="0 0 1" />
-      <xacro:if value="${limits_v2}">
-        <limit lower="${arm_5_joint_lb_v2 * deg_to_rad}" upper="${arm_5_joint_ub_v2 * deg_to_rad}" effort="${arm_5_max_effort}" velocity="${arm_5_max_velocity}" />
-        <safety_controller k_position="${arm_k_position}" k_velocity="${arm_k_velocity}" soft_lower_limit="${arm_5_joint_lb_v2 * deg_to_rad  + arm_eps}" soft_upper_limit="${arm_5_joint_ub_v2 * deg_to_rad - arm_eps}" />
-      </xacro:if>
-      <xacro:unless value="${limits_v2}">
-        <limit lower="${arm_5_joint_lb * deg_to_rad}" upper="${arm_5_joint_ub * deg_to_rad}" effort="${arm_5_max_effort}" velocity="${arm_5_max_velocity}" />
-        <safety_controller k_position="${arm_k_position}" k_velocity="${arm_k_velocity}" soft_lower_limit="${arm_5_joint_lb * deg_to_rad  + arm_eps}" soft_upper_limit="${arm_5_joint_ub * deg_to_rad - arm_eps}" />
-      </xacro:unless>
+      <xacro:if value="${joint_type == 'continuous'}">
+        <limit effort="${arm_5_max_effort}" velocity="${arm_5_max_velocity}" />
+      </xacro:if>
+      <xacro:if value="${joint_type == 'revolute'}">
+        <xacro:if value="${limits_v2}">
+          <limit lower="${arm_5_joint_lb_v2 * deg_to_rad}" upper="${arm_5_joint_ub_v2 * deg_to_rad}" effort="${arm_5_max_effort}" velocity="${arm_5_max_velocity}" />
+          <safety_controller k_position="${arm_k_position}" k_velocity="${arm_k_velocity}" soft_lower_limit="${arm_5_joint_lb_v2 * deg_to_rad  + arm_eps}" soft_upper_limit="${arm_5_joint_ub_v2 * deg_to_rad - arm_eps}" />
+        </xacro:if>
+        <xacro:unless value="${limits_v2}">
+          <limit lower="${arm_5_joint_lb * deg_to_rad}" upper="${arm_5_joint_ub * deg_to_rad}" effort="${arm_5_max_effort}" velocity="${arm_5_max_velocity}" />
+          <safety_controller k_position="${arm_k_position}" k_velocity="${arm_k_velocity}" soft_lower_limit="${arm_5_joint_lb * deg_to_rad  + arm_eps}" soft_upper_limit="${arm_5_joint_ub * deg_to_rad - arm_eps}" />
+        </xacro:unless>
+      </xacro:if>
       <dynamics friction="${arm_friction}" damping="${arm_damping}"/>
     </joint>

File: pal_sea_arm_description/urdf/arm/arm_limits/pal-sea-arm-standalone/arm.limits.xacro (robot description, xacro)
@@ -8,6 +8,4 @@
   <xacro:property name="arm_2_joint_ub" value="63.03" />
   <xacro:property name="arm_2_joint_lb" value="-139.8" />
-  <xacro:property name="arm_3_joint_ub" value="150" />
-  <xacro:property name="arm_3_joint_lb" value="-150" />
   <xacro:property name="arm_4_joint_ub" value="63.03" />
   <xacro:property name="arm_4_joint_lb" value="-139.8" />

File: pal_sea_arm_description/urdf/arm/arm_limits/pal-sea-arm-standalone/spherical-wrist.limits.xacro (robot description, xacro)
@@ -1,6 +1,4 @@
 <robot xmlns:xacro="http://ros.org/wiki/xacro">
   <!-- Joint limits -->
-  <xacro:property name="arm_5_joint_ub" value="210" />
-  <xacro:property name="arm_5_joint_lb" value="-90" />
   <xacro:property name="arm_6_joint_ub" value="114.59" />
   <xacro:property name="arm_6_joint_lb" value="-114.59" />

File: pal_sea_arm_description/urdf/arm/arm_limits/pal-sea-arm-standalone/straight-wrist.limits.xacro (robot description, xacro)
@@ -1,6 +1,4 @@
 <robot xmlns:xacro="http://ros.org/wiki/xacro">
   <!-- Joint limits -->
-  <xacro:property name="arm_5_joint_ub" value="148.97" />
-  <xacro:property name="arm_5_joint_lb" value="-148.97" />
   <xacro:property name="arm_6_joint_ub" value="114.59" />
   <xacro:property name="arm_6_joint_lb" value="-114.59" />

Commit message: fix property joint_type

File: pal_sea_arm_description/urdf/arm/arm.urdf.xacro (robot description, xacro)
@@ -50,4 +50,5 @@
     <xacro:include filename="$(find pal_sea_arm_description)/urdf/arm/arm_properties/${arm_type}/${wrist_model}.properties.xacro"/>
     <!-- ARM DEFINITION -->
+    <xacro:property name="joint_type" value="${'continuous' if arm_type == 'pal-sea-arm-standalone' else 'revolute'}" />
     <!-- ARM 1 LINK -->
     <link name="${name}_1_link">
@@ -68,5 +69,4 @@
     </link>
     <!-- ARM 1 JOINT -->
-    <xacro:property name="joint_type" value="${'continuous' if arm_type == 'pal-sea-arm-standalone' else 'revolute'}" />
     <joint name="${name}_1_joint" type="${joint_type}">
       <xacro:insert_block name="origin"/>
@@ -134,5 +134,4 @@
     </link>
     <!-- ARM 3 JOINT -->
-    <xacro:property name="joint_type" value="${'continuous' if arm_type == 'pal-sea-arm-standalone' else 'revolute'}" />
     <joint name="${name}_3_joint" type="${joint_type}">
       <xacro:origin_joint_3 reflect="${reflect}"/>
@@ -200,5 +199,4 @@
     </link>
     <!-- ARM 5 JOINT -->
-    <xacro:property name="joint_type" value="${'continuous' if arm_type == 'pal-sea-arm-standalone' else 'revolute'}" />
     <joint name="${name}_5_joint" type="${joint_type}">
       <xacro:origin_joint_5 reflect="${reflect}"/>
@@ -239,15 +237,15 @@
         </collision>
       </link>
-    <!-- ARM 6 JOINT -->
-    <joint name="${name}_6_joint" type="revolute">
-      <xacro:origin_joint_6 reflect="${reflect}"/>
-      <parent link="${name}_5_link" />
-      <child link="${name}_6_link" />
-      <axis xyz="0 0 ${-1 if wrist_model=='spherical-wrist' else 1}" />
-      <limit lower="${arm_6_joint_lb * deg_to_rad}" upper="${arm_6_joint_ub * deg_to_rad}" effort="${arm_6_max_effort}" velocity="${arm_6_max_velocity}" />
-      <dynamics friction="${arm_friction}" damping="${arm_damping}"/>
-      <safety_controller k_position="${arm_k_position}" k_velocity="${arm_k_velocity}" soft_lower_limit="${arm_6_joint_lb * deg_to_rad  + arm_eps}" soft_upper_limit="${arm_6_joint_ub * deg_to_rad - arm_eps}" />
-    </joint>
-    <!-- ARM 7 LINK -->
+      <!-- ARM 6 JOINT -->
+      <joint name="${name}_6_joint" type="revolute">
+        <xacro:origin_joint_6 reflect="${reflect}"/>
+        <parent link="${name}_5_link" />
+        <child link="${name}_6_link" />
+        <axis xyz="0 0 ${-1 if wrist_model=='spherical-wrist' else 1}" />
+        <limit lower="${arm_6_joint_lb * deg_to_rad}" upper="${arm_6_joint_ub * deg_to_rad}" effort="${arm_6_max_effort}" velocity="${arm_6_max_velocity}" />
+        <dynamics friction="${arm_friction}" damping="${arm_damping}"/>
+        <safety_controller k_position="${arm_k_position}" k_velocity="${arm_k_velocity}" soft_lower_limit="${arm_6_joint_lb * deg_to_rad  + arm_eps}" soft_upper_limit="${arm_6_joint_ub * deg_to_rad - arm_eps}" />
+      </joint>
+      <!-- ARM 7 LINK -->
       <link name="${name}_7_link">
         <xacro:inertial_link_7 reflect="${reflect}"/>
@@ -266,5 +264,5 @@
         </collision>
       </link>
-    <!-- ARM 7 JOINT -->
+      <!-- ARM 7 JOINT -->
       <joint name="${name}_7_joint" type="revolute">
         <xacro:origin_joint_7 reflect="${reflect}"/>
