Commit message: update limits for joint 4 + weights

File: pal_sea_arm_description/urdf/arm/arm_properties/arm_pal-sea-arm-standalone.properties.xacro (robot description, xacro)
@@ -6,5 +6,5 @@
         rpy="0 0 0" />
         <mass
-        value="1.0816" />
+        value="0.2" />
         <inertia
         ixx="0.0024426"
@@ -22,5 +22,5 @@
         rpy="0 0 0" />
         <mass
-        value="0.99204" />
+        value="0.01" />
         <inertia
         ixx="0.00077294"
@@ -41,5 +41,5 @@
         rpy="0 0 0" />
         <mass
-        value="1.0816" />
+        value="0.1" />
         <inertia
         ixx="0.0024426"
@@ -60,5 +60,5 @@
         rpy="0 0 0" />
         <mass
-        value="0.99204" />
+        value="0.1" />
         <inertia
         ixx="0.00077294"
@@ -79,5 +79,5 @@
         rpy="0 0 0" />
         <mass
-        value="0.52538" />
+        value="0.12538" />
         <inertia
         ixx="0.0019111"
@@ -98,5 +98,5 @@
         rpy="0 0 0" />
         <mass
-        value="0.66725" />
+        value="0.1725" />
         <inertia
         ixx="0.00035696"

File: pal_sea_arm_description/urdf/arm/limits/arm_pal-sea-arm-standalone.limits.xacro (robot description, xacro)
@@ -11,6 +11,6 @@
   <xacro:property name="arm_3_joint_ub" value="148.97" />
   <xacro:property name="arm_3_joint_lb" value="-148.97" />
-  <xacro:property name="arm_4_joint_ub" value="139.8" />
-  <xacro:property name="arm_4_joint_lb" value="-63.03" />
+  <xacro:property name="arm_4_joint_ub" value="63.03" />
+  <xacro:property name="arm_4_joint_lb" value="-139.8" />
   <xacro:property name="arm_5_joint_ub" value="148.97" />
   <xacro:property name="arm_5_joint_lb" value="-148.97" />
