Commit message: Address comments

File: pal_sea_arm_description/urdf/arm/arm_properties/tiago-pro/spherical-wrist.properties.xacro (robot description, xacro)
@@ -1,18 +1,9 @@
 <robot xmlns:xacro="http://ros.org/wiki/xacro">
     <xacro:macro name="inertial_link_5" params="reflect">
-        <xacro:if value="${inertia_version in ['tiago-pro-s']}">
-            <inertial>
-                <origin xyz="0.00017 -0.02738 0.06749" rpy="0 0 0" />
-                <mass value="0.31298" />
-                <inertia ixx="0.00157" ixy="0.00000" ixz="0.00000" iyy="0.00154" iyz="-0.00038" izz="0.00043" />
-            </inertial>
-        </xacro:if>
-        <xacro:if value="${inertia_version in ['tiago-pro']}">
-            <inertial>
-                <origin xyz="1.1053306160504E-05 -0.027586177392457 0.067845360860401" rpy="0 0 0" />
-                <mass value="0.310763344920608" />
-                <inertia ixx="0.001401450896582" ixy="9.16506225733395E-08" ixz="-9.26253840796548E-08" iyy="0.001399994200261" iyz="0.000327712970358816" izz="0.000402007894416599" />
-            </inertial>
-        </xacro:if>
+        <inertial>
+            <origin xyz="-0.00017 -0.02738 0.06749" rpy="0 0 0" />
+            <mass value="0.31298" />
+            <inertia ixx="0.00157" ixy="0.00000" ixz="0.00000" iyy="0.00154" iyz="-0.00038" izz="0.00043" />
+        </inertial>
     </xacro:macro>
     <xacro:macro name="origin_joint_5" params="reflect">
@@ -21,18 +12,9 @@
     </xacro:macro>
     <xacro:macro name="inertial_link_6" params="reflect">
-        <xacro:if value="${inertia_version in ['tiago-pro-s']}">
-            <inertial>
-                <origin xyz="0.03179 -0.00642 -0.04078" rpy="0 0 0" />
-                <mass value="1.34957" />
-                <inertia ixx="0.00127" ixy="0.00036" ixz="0.00006" iyy="0.00261" iyz="-0.00001" izz="0.00273" />
-            </inertial>
-        </xacro:if>
-        <xacro:if value="${inertia_version in ['tiago-pro']}">
-            <inertial>
-                <origin xyz="0.031765231605914 -0.006515108863227 -0.040804517366422" rpy="0 0 0" />
-                <mass value="1.34587360139295" />
-                <inertia ixx="0.001098855044306" ixy="0.000130003468892" ixz="-5.88209416784623E-06" iyy="0.001164948561169" iyz="4.20092116284985E-07" izz="0.001189837857495" />
-            </inertial>
-        </xacro:if>
+        <inertial>
+            <origin xyz="0.031765231605914 -0.006515108863227 -0.040804517366422" rpy="0 0 0" />
+            <mass value="1.34587360139295" />
+            <inertia ixx="0.001098855044306" ixy="0.000130003468892" ixz="-5.88209416784623E-06" iyy="0.001164948561169" iyz="4.20092116284985E-07" izz="0.001189837857495" />
+        </inertial>
     </xacro:macro>
     <xacro:macro name="origin_joint_6" params="reflect">
