Commit message: Fixed link 6 and tool_changer rotation

File: pal_sea_arm_description/urdf/arm/arm_properties/tiago-pro/arm.properties.xacro (robot description, xacro)
@@ -60,5 +60,5 @@
     <xacro:macro name="origin_joint_tool_changer" params="reflect">
         <!-- @Lucien needs to fix -->
-        <origin xyz="0 0 0.017" rpy="0 0 0" />
+        <origin xyz="0 0 0.017" rpy="0 0 1.570796" />
     </xacro:macro>
 </robot>

File: pal_sea_arm_description/urdf/arm/arm_properties/tiago-pro/straight-wrist.properties.xacro (robot description, xacro)
@@ -15,5 +15,5 @@
     </xacro:macro>
     <xacro:macro name="origin_joint_6" params="reflect">
-        <origin xyz="0 0.0354 0.16489" rpy="1.5708 0 1.5708" />
+        <origin xyz="0 0.0354 0.16489" rpy="1.5708 0 0" />
     </xacro:macro>
     <xacro:macro name="inertial_link_7" params="reflect">
@@ -25,5 +25,5 @@
     </xacro:macro>
     <xacro:macro name="origin_joint_7" params="reflect">
-        <origin xyz="-0.0354 0.135 0" rpy="-1.5708 0 0" />
+        <origin xyz="0 0.135 0.0354" rpy="-1.5708 0 0" />
     </xacro:macro>
 </robot>

Commit message: Proper orientation of 5th joint in spherical wrist

File: pal_sea_arm_description/urdf/arm/arm_properties/tiago-pro/arm.properties.xacro (robot description, xacro)
@@ -47,7 +47,4 @@
         <origin xyz="0.0199999999999993 -0.0371100000000008 0.15989" rpy="1.57079632679489 0 0" />
     </xacro:macro>
-    <xacro:macro name="origin_joint_5" params="reflect">
-        <origin xyz="-0.0199999999999971 0.17011 -0.037110000000002" rpy="-1.5707963267949 0 0" />
-    </xacro:macro>
     <!-- Tool changer (can be present in both wrists)-->
     <xacro:macro name="inertial_tool_changer_link" params="reflect">
@@ -60,6 +57,6 @@
     <xacro:macro name="origin_joint_tool_changer" params="reflect">
         <!-- @Lucien needs to fix, rotation remove to std gripper rotations -->
-        <!-- <origin xyz="0 0 0.017" rpy="0 0 1.570796" /> -->
-        <origin xyz="0 0 0.017" rpy="0 0 0.0" />
+        <origin xyz="0 0 0.017" rpy="0 0 1.570796" />
+        <!-- <origin xyz="0 0 0.017" rpy="0 0 0.0" /> -->
     </xacro:macro>
 </robot>

File: pal_sea_arm_description/urdf/arm/arm_properties/tiago-pro/spherical-wrist.properties.xacro (robot description, xacro)
@@ -6,4 +6,8 @@
             <inertia ixx="0.0014015" ixy="9.1728E-08" ixz="-9.3079E-08" iyy="0.0014" iyz="0.00032771" izz="0.00040201" />
         </inertial>
+    </xacro:macro>
+    <xacro:macro name="origin_joint_5" params="reflect">
+        <!-- Check new limits -->
+        <origin xyz="-0.0199999999999971 0.17011 -0.037110000000002" rpy="-1.5707963267949 3.14 0" />
     </xacro:macro>
     <xacro:macro name="inertial_link_6" params="reflect">
@@ -15,5 +19,5 @@
     </xacro:macro>
     <xacro:macro name="origin_joint_6" params="reflect">
-        <origin xyz="0 -0.0422 0.1654" rpy="-1.5708 0 3.14" />
+        <origin xyz="0 -0.0422 0.1654" rpy="-1.5708 0 0" />
     </xacro:macro>
     <xacro:macro name="inertial_link_7" params="reflect">
@@ -25,5 +29,5 @@
     </xacro:macro>
     <xacro:macro name="origin_joint_7" params="reflect">
-        <origin xyz="0.07 -0.0534 -0.0422" rpy="1.5708 0 0" />
+        <origin xyz="-0.07 -0.0534 0.0422" rpy="1.5708 0 0" />
     </xacro:macro>
 </robot>

File: pal_sea_arm_description/urdf/arm/arm_properties/tiago-pro/straight-wrist.properties.xacro (robot description, xacro)
@@ -6,4 +6,8 @@
             <inertia ixx="0.0020531" ixy="-8.9232E-07" ixz="1.6668E-06" iyy="0.0020434" iyz="3.7824E-05" izz="0.00067121" />
         </inertial>
+    </xacro:macro>
+    <xacro:macro name="origin_joint_5" params="reflect">
+        <!-- Check new limits -->
+        <origin xyz="-0.0199999999999971 0.17011 -0.037110000000002" rpy="-1.5707963267949 0 0" />
     </xacro:macro>
     <xacro:macro name="inertial_link_6" params="reflect">

Commit message: Fix wrist inertia

File: pal_sea_arm_description/urdf/arm/arm_properties/tiago-pro/arm.properties.xacro (robot description, xacro)
@@ -50,7 +50,7 @@
     <xacro:macro name="inertial_tool_changer_link" params="reflect">
         <inertial>
-            <origin xyz="0.0019481 0.0017558 -0.0084934" rpy="0 0 0" />
-            <mass value="0.12272" />
-            <inertia ixx="5.1385E-05" ixy="8.5364E-07" ixz="-9.0329E-08" iyy="4.7962E-05" iyz="-1.8035E-07" izz="9.2935E-05" />
+            <origin xyz="0.003414871500006 0.002458561521477 -0.001077004696741" rpy="0 0 0" />
+            <mass value="0.0655061851536" />
+            <inertia ixx="1.79461992752602E-05" ixy="1.70670100210845E-06" ixz="-2.54814948767968E-09" iyy="1.47274432150498E-05" iyz="1.09471559381518E-07" izz="3.12924968277541E-05" />
         </inertial>
     </xacro:macro>

Commit message: Remove comments

File: pal_sea_arm_description/urdf/arm/arm_properties/tiago-pro/arm.properties.xacro (robot description, xacro)
@@ -48,7 +48,5 @@
     </xacro:macro>
     <xacro:macro name="origin_joint_tool_changer" params="reflect">
-        <!-- Align with @Lucien -->
         <origin xyz="0 0 0.017" rpy="0 0 0" />
-        <!-- <origin xyz="0 0 0.017" rpy="0 0 0.0" /> -->
     </xacro:macro>
 </robot>

Commit message: Update arm.properties.xacro

File: pal_sea_arm_description/urdf/arm/arm_properties/tiago-pro/arm.properties.xacro (robot description, xacro)
@@ -1,18 +1,9 @@
 <robot xmlns:xacro="http://ros.org/wiki/xacro">
     <xacro:macro name="inertial_base_link" params="reflect">
-        <xacro:if value="${inertia_version in ['tiago-pro-s']}">
-            <inertial>
-                <origin xyz="-0.00069 0.00053 -0.01258" rpy="0 0 0" />
-                <mass value="0.76084" />
-                <inertia ixx="0.00054" ixy="0.00001" ixz="-0.00001" iyy="0.00055" iyz="0.00001" izz="0.00055" />
-            </inertial>
-        </xacro:if>
-        <xacro:if value="${inertia_version in ['tiago-pro']}">
-            <inertial>
-                <origin xyz="-0.00069237 0.00052761 -0.012575" rpy="0 0 0" />
-                <mass value="0.76084" />
-                <inertia ixx="0.00052192" ixy="8.9882E-06" ixz="-6.4075E-06" iyy="0.00052523" iyz="8.9275E-06" izz="0.00054849" />
-            </inertial>
-        </xacro:if>
+        <inertial>
+            <origin xyz="-0.00069237 0.00052761 -0.012575" rpy="0 0 0" />
+            <mass value="0.76084" />
+            <inertia ixx="0.00052192" ixy="8.9882E-06" ixz="-6.4075E-06" iyy="0.00052523" iyz="8.9275E-06" izz="0.00054849" />
+        </inertial>
     </xacro:macro>
     <xacro:macro name="inertial_link_1" params="reflect">

Commit message: Remove difference between S+ and S- motors

File: pal_sea_arm_description/urdf/arm/arm_properties/tiago-pro/arm.properties.xacro (robot description, xacro)
@@ -30,5 +30,5 @@
             <inertial>
                 <origin xyz="0.01715 -0.11231 -0.03000" rpy="0 0 0" />
-                <mass value="1.13101" />
+                <mass value="1.08501" />
                 <inertia ixx="0.00357" ixy="0.00029" ixz="0.00007" iyy="0.00117" iyz="-0.00068" izz="0.00352" />
             </inertial>
@@ -37,5 +37,5 @@
             <inertial>
                 <origin xyz="0.01786 -0.11956 -0.032097" rpy="0 0 0" />
-                <mass value="1.0436" />
+                <mass value="0.9976" />
                 <inertia ixx="0.0015021" ixy="0.00011264" ixz="1.0692E-05" iyy="0.00088017" iyz="-0.00015843" izz="0.0016021" />
             </inertial>
@@ -49,5 +49,5 @@
             <inertial>
                 <origin xyz="0.01530 -0.00471 0.13242" rpy="0 0 0" />
-                <mass value="1.21628" />
+                <mass value="1.17028" />
                 <inertia ixx="0.00425" ixy="-0.00004" ixz="-0.00051" iyy="0.00437" iyz="-0.00015" izz="0.00121" />
             </inertial>
@@ -56,5 +56,5 @@
             <inertial>
                 <origin xyz="0.016184 -0.0043916 0.13565" rpy="0 0 0" />
-                <mass value="1.1325" />
+                <mass value="1.0865" />
                 <inertia ixx="0.0023517" ixy="-2.6206E-05" ixz="-0.00020617" iyy="0.0025497" iyz="-6.2082E-05" izz="0.00097131" />
             </inertial>
@@ -68,5 +68,5 @@
             <inertial>
                 <origin xyz="-0.01715 0.11231 -0.03000" rpy="0 0 0" />
-                <mass value="1.13101" />
+                <mass value="1.08501" />
                 <inertia ixx="0.00357" ixy="0.00029" ixz="-0.00007" iyy="0.00117" iyz="0.00068" izz="0.00352" />
             </inertial>
@@ -75,5 +75,5 @@
             <inertial>
                 <origin xyz="-0.01786 0.11956 -0.032097" rpy="0 0 0" />
-                <mass value="1.0436" />
+                <mass value="0.9976" />
                 <inertia ixx="0.0015021" ixy="0.00011264" ixz="-1.0692E-05" iyy="0.00088017" iyz="0.00015843" izz="0.0016021" />
             </inertial>

Commit message: Add the new weight taking into account the cables and screws

File: pal_sea_arm_description/urdf/arm/arm_properties/tiago-pro/arm.properties.xacro (robot description, xacro)
@@ -1,16 +1,18 @@
 <robot xmlns:xacro="http://ros.org/wiki/xacro">
-    <xacro:macro name="inertial_arm_base_link" params="reflect">
-        <inertial>
-            <origin xyz="-0.00069237 0.00052761 -0.012575" rpy="0 0 0" />
-            <mass value="0.76084" />
-            <inertia ixx="0.00052192" ixy="8.9882E-06" ixz="-6.4075E-06" iyy="0.00052523" iyz="8.9275E-06" izz="0.00054849" />
-        </inertial>
-    </xacro:macro>
     <xacro:macro name="inertial_link_1" params="reflect">
         <xacro:if value="${inertia_version == 'tiago-pro-s'}">
             <inertial>
-                <origin xyz="0.00476 0.01532 0.15274" rpy="0 0 0" />
-                <mass value="1.21459" />
-                <inertia ixx="0.00434" ixy="0.00004" ixz="0.00016" iyy="0.00421" iyz="-0.00051" izz="0.00121" />
+                <origin
+                    xyz="0.0047632 0.015281 0.15179"
+                    rpy="0 0 0" />
+                <mass
+                    value="1.2728" />
+                <inertia
+                    ixx="0.0026718"
+                    ixy="2.956E-05"
+                    ixz="9.1714E-05"
+                    iyy="0.0024708"
+                    iyz="-0.00021103"
+                    izz="0.0010181" />
             </inertial>
         </xacro:if>
@@ -29,7 +31,16 @@
         <xacro:if value="${inertia_version == 'tiago-pro-s'}">
             <inertial>
-                <origin xyz="0.01715 -0.11231 -0.03000" rpy="0 0 0" />
-                <mass value="1.08501" />
-                <inertia ixx="0.00357" ixy="0.00029" ixz="0.00007" iyy="0.00117" iyz="-0.00068" izz="0.00352" />
+                <origin
+                    xyz="0.016761 -0.11092 -0.029509"
+                    rpy="0 0 0" />
+                <mass
+                    value="1.0974" />
+                <inertia
+                    ixx="0.0017447"
+                    ixy="0.00015165"
+                    ixz="1.4253E-05"
+                    iyy="0.00092895"
+                    iyz="-0.00017788"
+                    izz="0.0018861" />
             </inertial>
         </xacro:if>
@@ -48,7 +59,16 @@
         <xacro:if value="${inertia_version == 'tiago-pro-s'}">
             <inertial>
-                <origin xyz="0.01530 -0.00471 0.13242" rpy="0 0 0" />
-                <mass value="1.17028" />
-                <inertia ixx="0.00425" ixy="-0.00004" ixz="-0.00051" iyy="0.00437" iyz="-0.00015" izz="0.00121" />
+                <origin
+                    xyz="0.014943 -0.0047866 0.12972"
+                    rpy="0 0 0" />
+                <mass
+                    value="1.1907" />
+                <inertia
+                    ixx="0.0024631"
+                    ixy="-2.9584E-05"
+                    ixz="-0.00021101"
+                    iyy="0.0026656"
+                    iyz="-9.1746E-05"
+                    izz="0.0010104" />
             </inertial>
         </xacro:if>
@@ -67,7 +87,16 @@
         <xacro:if value="${inertia_version == 'tiago-pro-s'}">
             <inertial>
-                <origin xyz="-0.01715 0.11231 -0.03000" rpy="0 0 0" />
-                <mass value="1.08501" />
-                <inertia ixx="0.00357" ixy="0.00029" ixz="-0.00007" iyy="0.00117" iyz="0.00068" izz="0.00352" />
+                <origin
+                    xyz="-0.016761 0.11092 -0.029509"
+                    rpy="0 0 0" />
+                <mass
+                    value="1.0974" />
+                <inertia
+                    ixx="0.0017447"
+                    ixy="0.00015165"
+                    ixz="-1.4253E-05"
+                    iyy="0.00092895"
+                    iyz="0.00017788"
+                    izz="0.0018861" />
             </inertial>
         </xacro:if>

File: pal_sea_arm_description/urdf/arm/arm_properties/tiago-pro/spherical-wrist.properties.xacro (robot description, xacro)
@@ -2,7 +2,16 @@
     <xacro:macro name="inertial_link_5" params="reflect">
         <inertial>
-            <origin xyz="-0.00017 -0.02738 0.06749" rpy="0 0 0" />
-            <mass value="0.31298" />
-            <inertia ixx="0.00157" ixy="0.00000" ixz="0.00000" iyy="0.00154" iyz="-0.00038" izz="0.00043" />
+            <origin
+                xyz="-6.6854E-07 -0.02662 0.067326"
+                rpy="0 0 0" />
+            <mass
+                value="0.34802" />
+            <inertia
+                ixx="0.0014602"
+                ixy="-1.4931E-08"
+                ixz="8.1828E-08"
+                iyy="0.0014558"
+                iyz="0.00033448"
+                izz="0.00040968" />
         </inertial>
     </xacro:macro>
@@ -13,7 +22,16 @@
     <xacro:macro name="inertial_link_6" params="reflect">
         <inertial>
-            <origin xyz="0.031765231605914 -0.006515108863227 -0.040804517366422" rpy="0 0 0" />
-            <mass value="1.34587360139295" />
-            <inertia ixx="0.001098855044306" ixy="0.000130003468892" ixz="-5.88209416784623E-06" iyy="0.001164948561169" iyz="4.20092116284985E-07" izz="0.001189837857495" />
+            <origin
+                xyz="0.031968 -0.0065097 -0.040676"
+                rpy="0 0 0" />
+            <mass
+                value="1.378" />
+            <inertia
+                ixx="0.0011002"
+                ixy="0.00012805"
+                ixz="-5.6797E-06"
+                iyy="0.0011658"
+                iyz="5.4596E-07"
+                izz="0.0011909" />
         </inertial>
     </xacro:macro>
@@ -23,7 +41,16 @@
     <xacro:macro name="inertial_link_7" params="reflect">
         <inertial>
-            <origin xyz="0.00174 -0.00223 0.0083" rpy="0 0 0" />
-            <mass value="0.12399" />
-            <inertia ixx="0.00008" ixy="0.0" ixz="0.0" iyy="0.00006" iyz="0.0" izz="0.00012" />
+            <origin
+                xyz="-0.0016034 0.001194 0.0075583"
+                rpy="0 0 0" />
+            <mass
+                value="0.1354" />
+            <inertia
+                ixx="5.0537E-05"
+                ixy="-8.1184E-07"
+                ixz="1.9023E-07"
+                iyy="5.1762E-05"
+                iyz="-3.2751E-07"
+                izz="9.5274E-05" />
         </inertial>
     </xacro:macro>
