Commit message: Fix SyntaxWarning messages when comparing values

File: pal_sea_arm_description/urdf/arm/arm_limits/tiago-pro/arm.limits.xacro (robot description, xacro)
@@ -6,6 +6,6 @@
   <xacro:property name="arm_k_velocity" value="20"/>
   <!-- Joint limits -->
-  <xacro:property name="arm_1_joint_ub" value="${30 if joint_reflect is 1 else 270}" />
-  <xacro:property name="arm_1_joint_lb" value="${-270 if joint_reflect is 1 else -30}" />
+  <xacro:property name="arm_1_joint_ub" value="${30 if joint_reflect == 1 else 270}" />
+  <xacro:property name="arm_1_joint_lb" value="${-270 if joint_reflect == 1 else -30}" />
   <xacro:property name="arm_2_joint_ub" value="63.03" />
   <xacro:property name="arm_2_joint_lb" value="-139.8" />

File: pal_sea_arm_description/urdf/arm/arm_limits/tiago-pro/spherical-wrist.limits.xacro (robot description, xacro)
@@ -1,6 +1,6 @@
 <robot xmlns:xacro="http://ros.org/wiki/xacro">
   <!-- Joint limits -->
-  <xacro:property name="arm_5_joint_ub" value="${210 if joint_reflect is 1 else 90}" />
-  <xacro:property name="arm_5_joint_lb" value="${-90 if joint_reflect is 1 else -210}" />
+  <xacro:property name="arm_5_joint_ub" value="${210 if joint_reflect == 1 else 90}" />
+  <xacro:property name="arm_5_joint_lb" value="${-90 if joint_reflect == 1 else -210}" />
   <xacro:property name="arm_6_joint_ub" value="172" />
   <xacro:property name="arm_6_joint_lb" value="-108" />

File: pal_sea_arm_description/urdf/arm/arm_properties/tiago-sea-dual/arm.properties.xacro (robot description, xacro)
@@ -51,5 +51,5 @@
         <!-- @Lucien needs to fix, rotation remove to std gripper rotations -->
         <!-- <origin xyz="0 0 0.017" rpy="0 0 1.570796" /> -->
-        <origin xyz="0 0 0.017" rpy="0 ${0 if reflect is 1 else 180 * deg_to_rad} 0.0" />
+        <origin xyz="0 0 0.017" rpy="0 ${0 if reflect == 1 else 180 * deg_to_rad} 0.0" />
     </xacro:macro>
 </robot>

Commit message: Fix joint limit

File: pal_sea_arm_description/urdf/arm/arm_limits/tiago-pro/arm.limits.xacro (robot description, xacro)
@@ -8,10 +8,10 @@
   <xacro:property name="arm_1_joint_ub" value="${30 if joint_reflect == 1 else 270}" />
   <xacro:property name="arm_1_joint_lb" value="${-270 if joint_reflect == 1 else -30}" />
-  <xacro:property name="arm_2_joint_ub" value="63.03" />
-  <xacro:property name="arm_2_joint_lb" value="-139.8" />
-  <xacro:property name="arm_3_joint_ub" value="148.97" />
-  <xacro:property name="arm_3_joint_lb" value="-148.97" />
-  <xacro:property name="arm_4_joint_ub" value="63.03" />
-  <xacro:property name="arm_4_joint_lb" value="-139.8" />
+  <xacro:property name="arm_2_joint_ub" value="65" />
+  <xacro:property name="arm_2_joint_lb" value="-140" />
+  <xacro:property name="arm_3_joint_ub" value="150" />
+  <xacro:property name="arm_3_joint_lb" value="-150" />
+  <xacro:property name="arm_4_joint_ub" value="65" />
+  <xacro:property name="arm_4_joint_lb" value="-140" />
   <!-- Velocity limits -->
   <xacro:property name="arm_1_max_velocity" value="2.50" />

File: pal_sea_arm_description/urdf/arm/arm_limits/tiago-pro/spherical-wrist.limits.xacro (robot description, xacro)
@@ -5,6 +5,6 @@
   <xacro:property name="arm_6_joint_ub" value="172" />
   <xacro:property name="arm_6_joint_lb" value="-108" />
-  <xacro:property name="arm_7_joint_ub" value="148.5" />
-  <xacro:property name="arm_7_joint_lb" value="-148.5" />
+  <xacro:property name="arm_7_joint_ub" value="150" />
+  <xacro:property name="arm_7_joint_lb" value="-150" />
   <!-- Velocity limits -->
   <xacro:property name="arm_5_max_velocity" value="2.50" />
