Commit message: Add missing limits_v2 for the arm_5_joint when using short-wrist

File: pal_sea_arm_description/urdf/arm/arm_limits/tiago-pro/short-wrist.limits.xacro (robot description, xacro)
@@ -3,4 +3,7 @@
   <xacro:property name="arm_5_joint_ub" value="${210 if joint_reflect == 1 else 90}" />
   <xacro:property name="arm_5_joint_lb" value="${-90 if joint_reflect == 1 else -210}" />
+  <!-- Joint limits v2 -->
+  <xacro:property name="arm_5_joint_ub_v2" value="${220 if joint_reflect == 1 else 100}" />
+  <xacro:property name="arm_5_joint_lb_v2" value="${-100 if joint_reflect == 1 else -220}" />
   <!-- Velocity limits -->
   <xacro:property name="arm_5_max_velocity" value="2.50" />
