Commit message: reduce limit 7 TP spherical

File: pal_sea_arm_description/urdf/arm/arm_limits/tiago-pro/spherical-wrist.limits.xacro (robot description, xacro)
@@ -5,6 +5,6 @@
   <xacro:property name="arm_6_joint_ub" value="172" />
   <xacro:property name="arm_6_joint_lb" value="-108" />
-  <xacro:property name="arm_7_joint_ub" value="150" />
-  <xacro:property name="arm_7_joint_lb" value="-150" />
+  <xacro:property name="arm_7_joint_ub" value="140" />
+  <xacro:property name="arm_7_joint_lb" value="-140" />
   <!-- Joint limtis v2 -->
   <xacro:property name="arm_5_joint_ub_v2" value="${220 if joint_reflect == 1 else 100}" />
