Commit message: Proper colors for ATI FT

File: pal_sea_arm_description/urdf/sensors/ft_sensor/ati.urdf.xacro (robot description, xacro)
@@ -15,4 +15,10 @@
   <xacro:macro name="ft_sensor" params="name parent">
     <!-- FT DEFINITION -->
+    <!-- Gazebo reference -->
+    <gazebo reference="${name}_ft_link">
+      <material>Gazebo/DarkGrey</material>
+      <mu1>0.9</mu1>
+      <mu2>0.9</mu2>
+    </gazebo>
     <!-- Base link -->
     <link name="${name}_ft_sensor_base_link">
@@ -27,7 +33,5 @@
           <mesh filename="package://pal_sea_arm_description/meshes/sensors/ati/base_link.stl"/>
         </geometry>
-        <material name="">
-          <color rgba="0.75294 0.75294 0.75294 1" />
-        </material>
+        <material name="pal/DarkGrey"/>
       </visual>
       <collision>
@@ -55,7 +59,5 @@
           <mesh filename="package://pal_sea_arm_description/meshes/sensors/ati/ft_sensor_link.stl"/>
         </geometry>
-        <material name="">
-          <color rgba="0.89412 0.91373 0.92941 1" />
-        </material>
+        <material name="pal/DarkGrey"/>
       </visual>
       <collision>
@@ -84,7 +86,5 @@
           <mesh filename="package://pal_sea_arm_description/meshes/sensors/ati/ft_out_link.stl"/>
         </geometry>
-        <material name="">
-          <color rgba="0.75294 0.75294 0.75294 1" />
-        </material>
+        <material name="pal/DarkGrey"/>
       </visual>
       <collision>
@@ -101,10 +101,4 @@
       <axis xyz="0 0 0" />
     </joint>
-    <!-- Gazebo reference -->
-    <gazebo reference="${name}_ft_link">
-      <material>Gazebo/DarkGrey</material>
-      <mu1>0.9</mu1>
-      <mu2>0.9</mu2>
-    </gazebo>
   </xacro:macro>
 </robot>

Commit message: Rename ati mesh because of a mujoco bug if 2 meshes are called the same

File: pal_sea_arm_description/urdf/sensors/ft_sensor/ati.urdf.xacro (robot description, xacro)
@@ -31,5 +31,5 @@
         <origin xyz="0 0 0" rpy="0 0 0" />
         <geometry>
-          <mesh filename="package://pal_sea_arm_description/meshes/sensors/ati/base_link.stl"/>
+          <mesh filename="package://pal_sea_arm_description/meshes/sensors/ati/ati_ft_sensor.stl"/>
         </geometry>
         <material name="pal/DarkGrey"/>

Commit message: Fix ATI sensor in gazebo simulation

File: pal_sea_arm_description/urdf/sensors/ft_sensor/ati.urdf.xacro (robot description, xacro)
@@ -62,5 +62,5 @@
         <origin xyz="0 0 0.01" rpy="0 0 0" />
         <geometry>
-          <cylinder radius="0.03" length="0.02"/>
+          <cylinder radius="0.03" length="0.01"/>
         </geometry>
         <material name="pal/DarkGrey"/>
@@ -69,5 +69,5 @@
         <origin xyz="0 0 0.01" rpy="0 0 0" />
         <geometry>
-          <cylinder radius="0.03" length="0.02"/>
+          <cylinder radius="0.03" length="0.01"/>
         </geometry>
       </collision>
@@ -79,5 +79,5 @@
     </gazebo>
     <joint name="${name}_ft_sensor_joint" type="fixed">
-      <!-- <origin xyz="0 0 0.033998" rpy="0 0 0" /> -->
+      <origin xyz="0 0 0.033998" rpy="0 0 0" />
       <parent link="${name}_ft_sensor_base_link" />
       <child link="${name}_ft_sensor_link" />
@@ -94,5 +94,5 @@
         <origin xyz="0 0 -0.01" rpy="0 0 0" />
         <geometry>
-          <cylinder radius="0.03" length="0.02"/>
+          <cylinder radius="0.03" length="0.01"/>
         </geometry>
         <material name="pal/DarkGrey"/>
@@ -101,5 +101,5 @@
         <origin xyz="0 0 -0.01" rpy="0 0 0" />
         <geometry>
-          <cylinder radius="0.03" length="0.02"/>
+          <cylinder radius="0.03" length="0.01"/>
         </geometry>
       </collision>

File: pal_sea_arm_description/urdf/sensors/ft_sensor/ft_sensor.gazebo.xacro (robot description, xacro)
@@ -9,16 +9,14 @@
 <robot name="pal_sea_arm" xmlns:xacro="http://ros.org/wiki/xacro">
 <xacro:macro name="pal_sea_arm_force_torque_sensor" params="name update_rate">
-  <gazebo reference="${name}">
-    <sensor name="${name}_contact_sensor" type="contact">
-      <pose>0.105 0.071 0 0 0 0</pose>
-      <always_on>1</always_on>
+  <gazebo reference="${name}_ft_sensor_joint">
+    <preserveFixedJoint>true</preserveFixedJoint>      <!-- in case this is in a fixed joint -->
+    <sensor name="${name}_ft_sensor" type="force_torque">
       <update_rate>${update_rate}</update_rate>
-      <contact>
-        <collision>${name}_collision</collision>
-      </contact>
+      <visualize>true</visualize>
+      <force_torque>
+        <frame>child</frame>
+        <measure_direction>child_to_parent</measure_direction>
+      </force_torque>
     </sensor>
-  </gazebo>
-  <gazebo reference="${name}">
-    <provideFeedback>1</provideFeedback>
   </gazebo>
 </xacro:macro>

File: pal_sea_arm_description/urdf/sensors/ft_sensor/ft_sensor.urdf.xacro (robot description, xacro)
@@ -2,5 +2,7 @@
     <xacro:macro name="ft_sensor" params="name parent type">
         <xacro:include filename="$(find pal_sea_arm_description)/urdf/sensors/ft_sensor/${type}.urdf.xacro" />
+        <xacro:include filename="$(find pal_sea_arm_description)/urdf/sensors/ft_sensor/ft_sensor.gazebo.xacro" />
         <xacro:ft_sensor name="${name}" parent="${parent}"/>
+        <xacro:pal_sea_arm_force_torque_sensor name="${name}" update_rate="30"/>
     </xacro:macro>
 </robot>
