Commit message: number arg deleted

File: pal_sea_arm_description/ros2_control/transmissions.urdf.xacro (robot description, xacro)
@@ -1,32 +1,22 @@
 <?xml version="1.0"?>
 <robot xmlns:xacro="http://ros.org/wiki/xacro">
-  <xacro:macro name="pal_sea_arm_simple_transmission" params="name number reduction offset_value" >
-    <transmission name="${name}_${number}_trans">
-      <type>transmission_interface/SimpleTransmission</type>
-      <actuator name="${name}_${number}_motor" >
-        <mechanicalReduction>${reduction}</mechanicalReduction>
-      </actuator>
-      <joint name="${name}_${number}_joint">
+  <xacro:macro name="pal_sea_arm_simple_transmission" params="name reduction offset_value" >
+    <transmission name="${name}_trans">
+      <plugin>transmission_interface/SimpleTransmission</plugin>
+      <actuator name="${name}_motor" role="actuator1"/>
+      <joint name="${name}_joint" role="joint1">
         <offset>${offset_value}</offset>
-        <hardwareInterface>hardware_interface/PositionJointInterface</hardwareInterface>
-        <hardwareInterface>hardware_interface/EffortJointInterface</hardwareInterface>
-        <hardwareInterface>hardware_interface/VelocityJointInterface</hardwareInterface>
-        <hardwareInterface>hardware_interface/JointStateInterface</hardwareInterface>
+        <mechanical_reduction>${reduction}</mechanical_reduction>
       </joint>
     </transmission>
   </xacro:macro>
-  <xacro:macro name="arm_pro_simple_transmission" params="name number reduction offset_value" >
-    <transmission name="${name}_${number}_trans">
-      <type>sea_transmissions/SeaSimpleTransmission</type>
-      <actuator name="${name}_${number}_motor" >
-        <mechanicalReduction>${reduction}</mechanicalReduction>
-      </actuator>
-      <joint name="${name}_${number}_joint">
-        <actuators_data_ns>/actuators_data/${name}_${number}_motor</actuators_data_ns>
-        <joint_offset_ns>/${name}_${number}_motor/output_offset</joint_offset_ns>
-        <hardwareInterface>hardware_interface/PositionJointInterface</hardwareInterface>
-        <hardwareInterface>hardware_interface/VelocityJointInterface</hardwareInterface>
-        <hardwareInterface>hardware_interface/EffortJointInterface</hardwareInterface>
-        <hardwareInterface>hardware_interface/JointStateInterface</hardwareInterface>
+  <xacro:macro name="arm_pro_simple_transmission" params="name reduction offset_value" >
+    <transmission name="${name}_trans">
+      <plugin>sea_transmissions/SeaSimpleTransmission</plugin>
+      <actuator name="${name}_motor" role="actuator1"/>
+      <joint name="${name}_joint" role="joint1">
+        <actuators_data_ns>/actuators_data/${name}_motor</actuators_data_ns>
+        <joint_offset_ns>/${name}_motor/output_offset</joint_offset_ns>
+        <mechanical_reduction>${reduction}</mechanical_reduction>
       </joint>
     </transmission>

File: pal_sea_arm_description/urdf/arm/arm.ros2_control.xacro (robot description, xacro)
@@ -13,5 +13,5 @@
  -->
 <robot xmlns:xacro="http://ros.org/wiki/xacro">
-  <xacro:macro name="ros2_control_arm" params="name number reduction offset_value" >
+  <xacro:macro name="ros2_control_arm" params="name reduction offset_value" >
     <joint name="${name}_joint">
       <command_interface name="position" />
@@ -23,5 +23,5 @@
     </joint>
   <xacro:include filename="$(find pal_sea_arm_description)/ros2_control/transmissions.urdf.xacro" />
-  <xacro:arm_pro_simple_transmission name="${name}" number="${number}" reduction="${reduction}" offset_value="${offset_value}" />
+  <xacro:arm_pro_simple_transmission name="${name}" reduction="${reduction}" offset_value="${offset_value}" />
   </xacro:macro>
 </robot>

Commit message: added paths to sea data

File: pal_sea_arm_description/ros2_control/transmissions.urdf.xacro (robot description, xacro)
@@ -2,4 +2,17 @@
 <robot xmlns:xacro="http://ros.org/wiki/xacro">
   <xacro:macro name="pal_sea_arm_simple_transmission" params="name reduction offset_value" >
+    <transmission name="${name}_trans">
+      <plugin>sea_transmissions/SeaSimpleTransmission</plugin>
+      <actuator name="${name}_actuator" role="actuator1"/>
+      <joint name="${name}_joint" role="joint1">
+        <offset>${offset_value}</offset>
+        <mechanical_reduction>${reduction}</mechanical_reduction>
+      </joint>
+      <param name="actuator_fingerprint_path">file:///etc/sea_data/${name}_actuator/fingerprint.csv</param>
+      <param name="actuator_metadata_path">file:///etc/sea_data/${name}_actuator/actuator_metadata.yaml</param>
+      <param name="actuator_data_path">file:///home/pal/.pal/rt_device_manager_cfg/actuators.yaml</param>
+    </transmission>
+  </xacro:macro>
+  <xacro:macro name="arm_pro_simple_transmission" params="name reduction offset_value" >
     <transmission name="${name}_trans">
       <plugin>transmission_interface/SimpleTransmission</plugin>
@@ -11,13 +24,3 @@
     </transmission>
   </xacro:macro>
-  <xacro:macro name="arm_pro_simple_transmission" params="name reduction offset_value" >
-    <transmission name="${name}_trans">
-      <plugin>sea_transmissions/SeaSimpleTransmission</plugin>
-      <actuator name="${name}_actuator" role="actuator1"/>
-      <joint name="${name}_joint" role="joint1">
-        <offset>${offset_value}</offset>
-        <mechanical_reduction>${reduction}</mechanical_reduction>
-      </joint>
-    </transmission>
-  </xacro:macro>
 </robot>

Commit message: Adapted to new data loading mechanism

File: pal_sea_arm_description/ros2_control/transmissions.urdf.xacro (robot description, xacro)
@@ -1,5 +1,5 @@
 <?xml version="1.0"?>
 <robot xmlns:xacro="http://ros.org/wiki/xacro">
-  <xacro:macro name="pal_sea_arm_simple_transmission" params="name reduction offset_value" >
+  <xacro:macro name="pal_sea_arm_simple_transmission" params="name reduction offset_value">
     <transmission name="${name}_trans">
       <plugin>sea_transmissions/SeaSimpleTransmission</plugin>
@@ -9,10 +9,8 @@
         <mechanical_reduction>${reduction}</mechanical_reduction>
       </joint>
-      <param name="actuator_fingerprint_path">file:///etc/sea_data/${name}_actuator/fingerprint.csv</param>
-      <param name="actuator_metadata_path">file:///etc/sea_data/${name}_actuator/actuator_metadata.yaml</param>
-      <param name="actuator_data_path">file:///home/pal/.pal/rt_device_manager_cfg/actuators.yaml</param>
+      <param name="sea_data_type">sea_data</param>
     </transmission>
   </xacro:macro>
-  <xacro:macro name="arm_pro_simple_transmission" params="name reduction offset_value" >
+  <xacro:macro name="arm_pro_simple_transmission" params="name reduction offset_value">
     <transmission name="${name}_trans">
       <plugin>transmission_interface/SimpleTransmission</plugin>

Commit message: Better transmissions names

File: pal_sea_arm_description/ros2_control/transmissions.urdf.xacro (robot description, xacro)
@@ -1,5 +1,5 @@
 <?xml version="1.0"?>
 <robot xmlns:xacro="http://ros.org/wiki/xacro">
-  <xacro:macro name="pal_sea_arm_simple_transmission" params="name reduction offset_value">
+  <xacro:macro name="sea_transmission" params="name reduction offset_value">
     <transmission name="${name}_trans">
       <plugin>sea_transmissions/SeaSimpleTransmission</plugin>
@@ -12,5 +12,5 @@
     </transmission>
   </xacro:macro>
-  <xacro:macro name="arm_pro_simple_transmission" params="name reduction offset_value">
+  <xacro:macro name="simple_transmission" params="name reduction offset_value">
     <transmission name="${name}_trans">
       <plugin>transmission_interface/SimpleTransmission</plugin>

File: pal_sea_arm_description/urdf/arm/arm.ros2_control.xacro (robot description, xacro)
@@ -30,9 +30,9 @@
     <xacro:if value="${use_sea_transmission}">
       <!-- Reduction needed for the torque estimation -->
-      <xacro:pal_sea_arm_simple_transmission name="${name}" reduction="${reduction}" offset_value="${offset_value}" />
+      <xacro:sea_transmission name="${name}" reduction="${reduction}" offset_value="${offset_value}" />
     </xacro:if>
     <xacro:unless value="${use_sea_transmission}">
       <!-- Reduction already applied in the RT layer, harcoded here to 1.0 -->
-      <xacro:arm_pro_simple_transmission name="${name}" reduction="1.0" offset_value="${offset_value}" />
+      <xacro:simple_transmission name="${name}" reduction="1.0" offset_value="${offset_value}" />
     </xacro:unless>
   </xacro:macro>
