Commit message: delete number element in the arm transmission

File: pal_sea_arm_description/ros2_control/ros2_control.urdf.xacro (robot description, xacro)
@@ -19,5 +19,5 @@
     <xacro:property name="end_effector" value="$(arg end_effector)" />
     <xacro:property name="has_ft_sensor" value="${ft_sensor != 'no-ft-sensor'}" />
-  <xacro:property name="ft_sensor" value="$(arg ft_sensor)" />
+    <xacro:property name="ft_sensor" value="$(arg ft_sensor)" />
     <xacro:include filename="$(find pal_sea_arm_description)/urdf/arm/arm.ros2_control.xacro" />
     <xacro:if value="${end_effector == 'pal-pro-gripper'}">
@@ -35,16 +35,16 @@
         </xacro:unless>
       </hardware>
-       <!-- arm -->
-       <xacro:ros2_control_arm name="arm_1" number= "1" reduction="121.0" offset_value="${arm_1_joint_offset}"/>
-       <xacro:ros2_control_arm name="arm_2" number= "2" reduction="121.0" offset_value="${arm_2_joint_offset}"/>
-       <xacro:ros2_control_arm name="arm_3" number= "3" reduction="101.0" offset_value="${arm_3_joint_offset}"/>
-       <xacro:ros2_control_arm name="arm_4" number= "4" reduction="101.0" offset_value="${arm_4_joint_offset}"/>
-       <xacro:ros2_control_arm name="arm_5" number= "5" reduction="101.0" offset_value="${arm_5_joint_offset}"/>
-       <xacro:ros2_control_arm name="arm_6" number= "6" reduction="101.0" offset_value="${arm_6_joint_offset}"/>
-       <xacro:ros2_control_arm name="arm_7" number= "7" reduction="101.0" offset_value="${arm_7_joint_offset}"/>
-        <xacro:if value="${end_effector == 'pal-pro-gripper'}">
-          <!-- pal-gripper -->
-          <xacro:ros2_control_pal_pro_gripper name="gripper_left_finger" reduction="1.0" />
-        </xacro:if>
+      <!-- arm -->
+      <xacro:ros2_control_arm name="arm_1" reduction="121.0" offset_value="${arm_1_joint_offset}"/>
+      <xacro:ros2_control_arm name="arm_2" reduction="121.0" offset_value="${arm_2_joint_offset}"/>
+      <xacro:ros2_control_arm name="arm_3" reduction="101.0" offset_value="${arm_3_joint_offset}"/>
+      <xacro:ros2_control_arm name="arm_4" reduction="101.0" offset_value="${arm_4_joint_offset}"/>
+      <xacro:ros2_control_arm name="arm_5" reduction="101.0" offset_value="${arm_5_joint_offset}"/>
+      <xacro:ros2_control_arm name="arm_6" reduction="101.0" offset_value="${arm_6_joint_offset}"/>
+      <xacro:ros2_control_arm name="arm_7" reduction="101.0" offset_value="${arm_7_joint_offset}"/>
+      <xacro:if value="${end_effector == 'pal-pro-gripper'}">
+        <!-- pal-gripper -->
+        <xacro:ros2_control_pal_pro_gripper name="gripper_finger" reduction="1.0" />
+      </xacro:if>
       <!-- Force Torque sensor -->
       <xacro:if value="${has_ft_sensor}">

Commit message: Add missing sim_type xacro args

File: pal_sea_arm_description/ros2_control/ros2_control.urdf.xacro (robot description, xacro)
@@ -13,5 +13,5 @@
  -->
 <robot xmlns:xacro="http://ros.org/wiki/xacro" name="pal_sea_arm">
-  <xacro:macro name="pal_sea_arm_ros2_control" params="use_sim_time:=^|false torque_estimation:=false">
+  <xacro:macro name="pal_sea_arm_ros2_control" params="use_sim_time:=^|false torque_estimation:=false sim_type:=no-simulation">
     <xacro:arg name="end_effector" default="no-end-effector"/>
     <xacro:arg name="ft_sensor" default="no-ft-sensor"/>

File: pal_sea_arm_description/urdf/arm/arm.ros2_control.xacro (robot description, xacro)
@@ -13,5 +13,5 @@
  -->
 <robot xmlns:xacro="http://ros.org/wiki/xacro">
-  <xacro:macro name="ros2_control_arm" params="name reduction offset_value use_sea_transmission:=false">
+  <xacro:macro name="ros2_control_arm" params="name reduction offset_value use_sea_transmission:=false sim_type:=no-simulation">
     <joint name="${name}_joint">
       <xacro:if value="${sim_type == 'mujoco-ros2-control'}">

Commit message: fix simulation and 7-link-mesh

File: pal_sea_arm_description/ros2_control/ros2_control.urdf.xacro (robot description, xacro)
@@ -13,5 +13,5 @@
  -->
 <robot xmlns:xacro="http://ros.org/wiki/xacro" name="pal_sea_arm">
-  <xacro:macro name="pal_sea_arm_ros2_control" params="use_sim_time:=^|false torque_estimation:=false sim_type:=no-simulation">
+  <xacro:macro name="pal_sea_arm_ros2_control" params="use_sim_time:=^|false torque_estimation:=false">
     <xacro:arg name="end_effector" default="no-end-effector"/>
     <xacro:arg name="ft_sensor" default="no-ft-sensor"/>

File: pal_sea_arm_description/urdf/arm/arm.ros2_control.xacro (robot description, xacro)
@@ -13,5 +13,5 @@
  -->
 <robot xmlns:xacro="http://ros.org/wiki/xacro">
-  <xacro:macro name="ros2_control_arm" params="name reduction offset_value use_sea_transmission:=false sim_type:=no-simulation">
+  <xacro:macro name="ros2_control_arm" params="name reduction offset_value use_sea_transmission:=false">
     <joint name="${name}_joint">
       <xacro:if value="${sim_type == 'mujoco-ros2-control'}">
