Commit message: changed macro name

File: pal_sea_arm_description/mujoco/mj_tags.xacro (robot description, xacro)
@@ -19,5 +19,5 @@
         </worldbody>
     </xacro:macro>
-    <xacro:macro name="arm_mj_motor_actuators">
+    <xacro:macro name="single_arm_mj_motor_actuators">
       <motor group="0" name="arm_1_joint_torque" joint="arm_left_1_joint" ctrlrange="-46 46" />
       <motor group="0" name="arm_2_joint_torque" joint="arm_left_2_joint" ctrlrange="-46 46" />
@@ -28,5 +28,5 @@
       <motor group="0" name="arm_7_joint_torque" joint="arm_left_7_joint" ctrlrange="-46 46" />
     </xacro:macro>
-    <xacro:macro name="arm_mj_position_actuators">
+    <xacro:macro name="single_arm_mj_position_actuators">
       <position group="2" name="arm_1_joint_position" joint="arm_1_joint" ctrlrange="-0.523599 4.71239" kp="1000" kv="50"/>
       <position group="2" name="arm_2_joint_position" joint="arm_2_joint" ctrlrange="-2.44346 1.13446" kp="1000" kv="60"/>
@@ -37,3 +37,35 @@
       <position group="2" name="arm_7_joint_position" joint="arm_7_joint" ctrlrange="-2.61799 2.61799" kp="500" kv="20"/>
     </xacro:macro>
+    <xacro:macro name="both_arms_mj_motor_actuators">
+      <motor group="0" name="arm_left_1_joint_torque" joint="arm_left_1_joint" ctrlrange="-46 46" />
+      <motor group="0" name="arm_left_2_joint_torque" joint="arm_left_2_joint" ctrlrange="-46 46" />
+      <motor group="0" name="arm_left_3_joint_torque" joint="arm_left_3_joint" ctrlrange="-46 46" />
+      <motor group="0" name="arm_left_4_joint_torque" joint="arm_left_4_joint" ctrlrange="-46 46" />
+      <motor group="0" name="arm_left_5_joint_torque" joint="arm_left_5_joint" ctrlrange="-46 46" />
+      <motor group="0" name="arm_left_6_joint_torque" joint="arm_left_6_joint" ctrlrange="-46 46" />
+      <motor group="0" name="arm_left_7_joint_torque" joint="arm_left_7_joint" ctrlrange="-46 46" />
+      <motor group="0" name="arm_right_1_joint_torque" joint="arm_right_1_joint" ctrlrange="-46 46" />
+      <motor group="0" name="arm_right_2_joint_torque" joint="arm_right_2_joint" ctrlrange="-46 46" />
+      <motor group="0" name="arm_right_3_joint_torque" joint="arm_right_3_joint" ctrlrange="-46 46" />
+      <motor group="0" name="arm_right_4_joint_torque" joint="arm_right_4_joint" ctrlrange="-46 46" />
+      <motor group="0" name="arm_right_5_joint_torque" joint="arm_right_5_joint" ctrlrange="-46 46" />
+      <motor group="0" name="arm_right_6_joint_torque" joint="arm_right_6_joint" ctrlrange="-46 46" />
+      <motor group="0" name="arm_right_7_joint_torque" joint="arm_right_7_joint" ctrlrange="-46 46" />
+    </xacro:macro>
+     <xacro:macro name="both_arms_mj_position_actuators">
+      <position group="2" name="arm_left_1_joint_position" joint="arm_left_1_joint" ctrlrange="-0.523599 4.71239" kp="1000" kv="50"/>
+      <position group="2" name="arm_left_2_joint_position" joint="arm_left_2_joint" ctrlrange="-2.44346 1.13446" kp="1000" kv="60"/>
+      <position group="2" name="arm_left_3_joint_position" joint="arm_left_3_joint" ctrlrange="-2.61799 2.61799" kp="1000" kv="50"/>
+      <position group="2" name="arm_left_4_joint_position" joint="arm_left_4_joint" ctrlrange="-2.44346 1.13446" kp="500" kv="20"/>
+      <position group="2" name="arm_left_5_joint_position" joint="arm_left_5_joint" ctrlrange="-2.61799 2.61799" kp="1000" kv="20"/>
+      <position group="2" name="arm_left_6_joint_position" joint="arm_left_6_joint" ctrlrange="-2.00713 2.00713" kp="1000" kv="20"/>
+      <position group="2" name="arm_left_7_joint_position" joint="arm_left_7_joint" ctrlrange="-2.61799 2.61799" kp="500" kv="20"/>
+      <position group="2" name="arm_right_1_joint_position" joint="arm_right_1_joint" ctrlrange="-4.71239 0.523599"  kp="1000" kv="50"/>
+      <position group="2" name="arm_right_2_joint_position" joint="arm_right_2_joint" ctrlrange="-2.44346 1.13446"   kp="1000" kv="60"/>
+      <position group="2" name="arm_right_3_joint_position" joint="arm_right_3_joint" ctrlrange="-2.61799 2.61799"   kp="1000" kv="50"/>
+      <position group="2" name="arm_right_4_joint_position" joint="arm_right_4_joint" ctrlrange="-2.44346 1.13446"  kp="500" kv="20"/>
+      <position group="2" name="arm_right_5_joint_position" joint="arm_right_5_joint" ctrlrange="-2.61799 2.61799"   kp="1000" kv="20"/>
+      <position group="2" name="arm_right_6_joint_position" joint="arm_right_6_joint" ctrlrange="-2.00713 2.00713"   kp="1000" kv="20"/>
+      <position group="2" name="arm_right_7_joint_position" joint="arm_right_7_joint" ctrlrange="-2.61799 2.61799"   kp="500" kv="20"/>
+    </xacro:macro>
 </robot>

Commit message: Improved logic for the mujoco robot description

File: pal_sea_arm_description/mujoco/mj_tags.xacro (robot description, xacro)
@@ -1,6 +1,6 @@
 <?xml version="1.0"?>
 <robot xmlns:xacro="http://ros.org/wiki/xacro" name="pal_sea_arm">
-    <!--  -->
-    <xacro:macro name="mj_common">
+    <!-- Mujoco environment for arm mujoco simulation-->
+    <xacro:macro name="mj_arm_common">
       <compiler strippath="false" discardvisual="false" balanceinertia="true" angle="radian" />
         <option integrator="implicitfast" />
@@ -19,53 +19,28 @@
         </worldbody>
     </xacro:macro>
-    <xacro:macro name="single_arm_mj_motor_actuators">
-      <motor group="0" name="arm_1_joint_torque" joint="arm_1_joint" ctrlrange="-46 46" />
-      <motor group="0" name="arm_2_joint_torque" joint="arm_2_joint" ctrlrange="-46 46" />
-      <motor group="0" name="arm_3_joint_torque" joint="arm_3_joint" ctrlrange="-46 46" />
-      <motor group="0" name="arm_4_joint_torque" joint="arm_4_joint" ctrlrange="-46 46" />
-      <motor group="0" name="arm_5_joint_torque" joint="arm_5_joint" ctrlrange="-46 46" />
-      <motor group="0" name="arm_6_joint_torque" joint="arm_6_joint" ctrlrange="-46 46" />
-      <motor group="0" name="arm_7_joint_torque" joint="arm_7_joint" ctrlrange="-46 46" />
-    </xacro:macro>
-    <xacro:macro name="single_arm_mj_position_actuators">
-      <position group="2" name="arm_1_joint_position" joint="arm_1_joint" ctrlrange="-4.71239 0.523599"  kp="1000"/>
-      <position group="2" name="arm_2_joint_position" joint="arm_2_joint" ctrlrange="-2.44346 1.13446"   kp="1000" />
-      <position group="2" name="arm_3_joint_position" joint="arm_3_joint" ctrlrange="-2.61799 2.61799"   kp="1000" />
-      <position group="2" name="arm_4_joint_position" joint="arm_4_joint" ctrlrange="-2.44346 1.13446"   kp="500" />
-      <position group="2" name="arm_5_joint_position" joint="arm_5_joint" ctrlrange="-2.61799 2.61799"   kp="1000" />
-      <position group="2" name="arm_6_joint_position" joint="arm_6_joint" ctrlrange="-2.00713 2.00713"   kp="1000"/>
-      <position group="2" name="arm_7_joint_position" joint="arm_7_joint" ctrlrange="-2.61799 2.61799"   kp="500"/>
-    </xacro:macro>
-    <xacro:macro name="both_arms_mj_motor_actuators">
-      <motor group="0" name="arm_left_1_joint_torque" joint="arm_left_1_joint" ctrlrange="-46 46" />
-      <motor group="0" name="arm_left_2_joint_torque" joint="arm_left_2_joint" ctrlrange="-46 46" />
-      <motor group="0" name="arm_left_3_joint_torque" joint="arm_left_3_joint" ctrlrange="-46 46" />
-      <motor group="0" name="arm_left_4_joint_torque" joint="arm_left_4_joint" ctrlrange="-46 46" />
-      <motor group="0" name="arm_left_5_joint_torque" joint="arm_left_5_joint" ctrlrange="-46 46" />
-      <motor group="0" name="arm_left_6_joint_torque" joint="arm_left_6_joint" ctrlrange="-46 46" />
-      <motor group="0" name="arm_left_7_joint_torque" joint="arm_left_7_joint" ctrlrange="-46 46" />
-      <motor group="0" name="arm_right_1_joint_torque" joint="arm_right_1_joint" ctrlrange="-46 46" />
-      <motor group="0" name="arm_right_2_joint_torque" joint="arm_right_2_joint" ctrlrange="-46 46" />
-      <motor group="0" name="arm_right_3_joint_torque" joint="arm_right_3_joint" ctrlrange="-46 46" />
-      <motor group="0" name="arm_right_4_joint_torque" joint="arm_right_4_joint" ctrlrange="-46 46" />
-      <motor group="0" name="arm_right_5_joint_torque" joint="arm_right_5_joint" ctrlrange="-46 46" />
-      <motor group="0" name="arm_right_6_joint_torque" joint="arm_right_6_joint" ctrlrange="-46 46" />
-      <motor group="0" name="arm_right_7_joint_torque" joint="arm_right_7_joint" ctrlrange="-46 46" />
-    </xacro:macro>
-     <xacro:macro name="both_arms_mj_position_actuators">
-      <position group="2" name="arm_left_1_joint_position" joint="arm_left_1_joint" ctrlrange="-0.523599 4.71239" kp="1000" kv="50"/>
-      <position group="2" name="arm_left_2_joint_position" joint="arm_left_2_joint" ctrlrange="-2.44346 1.13446" kp="1000" kv="60"/>
-      <position group="2" name="arm_left_3_joint_position" joint="arm_left_3_joint" ctrlrange="-2.61799 2.61799" kp="1000" kv="50"/>
-      <position group="2" name="arm_left_4_joint_position" joint="arm_left_4_joint" ctrlrange="-2.44346 1.13446" kp="500" kv="20"/>
-      <position group="2" name="arm_left_5_joint_position" joint="arm_left_5_joint" ctrlrange="-2.61799 2.61799" kp="1000" kv="20"/>
-      <position group="2" name="arm_left_6_joint_position" joint="arm_left_6_joint" ctrlrange="-2.00713 2.00713" kp="1000" kv="20"/>
-      <position group="2" name="arm_left_7_joint_position" joint="arm_left_7_joint" ctrlrange="-2.61799 2.61799" kp="500" kv="20"/>
-      <position group="2" name="arm_right_1_joint_position" joint="arm_right_1_joint" ctrlrange="-4.71239 0.523599"  kp="1000" kv="50"/>
-      <position group="2" name="arm_right_2_joint_position" joint="arm_right_2_joint" ctrlrange="-2.44346 1.13446"   kp="1000" kv="60"/>
-      <position group="2" name="arm_right_3_joint_position" joint="arm_right_3_joint" ctrlrange="-2.61799 2.61799"   kp="1000" kv="50"/>
-      <position group="2" name="arm_right_4_joint_position" joint="arm_right_4_joint" ctrlrange="-2.44346 1.13446"  kp="500" kv="20"/>
-      <position group="2" name="arm_right_5_joint_position" joint="arm_right_5_joint" ctrlrange="-2.61799 2.61799"   kp="1000" kv="20"/>
-      <position group="2" name="arm_right_6_joint_position" joint="arm_right_6_joint" ctrlrange="-2.00713 2.00713"   kp="1000" kv="20"/>
-      <position group="2" name="arm_right_7_joint_position" joint="arm_right_7_joint" ctrlrange="-2.61799 2.61799"   kp="500" kv="20"/>
+    <!-- Actuators -->
+    <xacro:macro name="mj_arm_actuators" params="side joint_reflect:=1">
+      <xacro:include filename="$(find pal_sea_arm_description)/urdf/arm/arm_limits/${arm_type}/arm.limits.xacro"/>
+      <xacro:include filename="$(find pal_sea_arm_description)/urdf/arm/arm_limits/${arm_type}/${wrist_model}.limits.xacro"/>
+      <xacro:include filename="$(find pal_sea_arm_description)/urdf/arm/arm_properties/${arm_type}/arm.properties.xacro"/>
+      <xacro:include filename="$(find pal_sea_arm_description)/urdf/arm/arm_properties/${arm_type}/${wrist_model}.properties.xacro"/>
+      <xacro:if value="${mj_controller == 'motor'}">
+        <motor name="${side}_1_joint_torque" joint="${side}_1_joint" ctrlrange="-46 46" />
+        <motor name="${side}_2_joint_torque" joint="${side}_2_joint" ctrlrange="-46 46" />
+        <motor name="${side}_3_joint_torque" joint="${side}_3_joint" ctrlrange="-46 46" />
+        <motor name="${side}_4_joint_torque" joint="${side}_4_joint" ctrlrange="-46 46" />
+        <motor name="${side}_5_joint_torque" joint="${side}_5_joint" ctrlrange="-46 46" />
+        <motor name="${side}_6_joint_torque" joint="${side}_6_joint" ctrlrange="-46 46" />
+        <motor name="${side}_7_joint_torque" joint="${side}_7_joint" ctrlrange="-46 46" />
+      </xacro:if>
+      <xacro:if value="${mj_controller == 'position'}">
+        <position name="${side}_1_joint_position" joint="${side}_1_joint" ctrlrange="${arm_1_joint_lb * deg_to_rad} ${arm_1_joint_ub * deg_to_rad}" kp="1000" kv="50"/>
+        <position name="${side}_2_joint_position" joint="${side}_2_joint" ctrlrange="${arm_2_joint_lb * deg_to_rad} ${arm_2_joint_ub * deg_to_rad}" kp="1000" kv="60"/>
+        <position name="${side}_3_joint_position" joint="${side}_3_joint" ctrlrange="${arm_3_joint_lb * deg_to_rad} ${arm_3_joint_ub * deg_to_rad}" kp="1000" kv="50"/>
+        <position name="${side}_4_joint_position" joint="${side}_4_joint" ctrlrange="${arm_4_joint_lb * deg_to_rad} ${arm_4_joint_ub * deg_to_rad}" kp="500" kv="20"/>
+        <position name="${side}_5_joint_position" joint="${side}_5_joint" ctrlrange="${arm_5_joint_lb * deg_to_rad} ${arm_5_joint_ub * deg_to_rad}" kp="1000" kv="20"/>
+        <position name="${side}_6_joint_position" joint="${side}_6_joint" ctrlrange="${arm_6_joint_lb * deg_to_rad} ${arm_6_joint_ub * deg_to_rad}" kp="1000" kv="20"/>
+        <position name="${side}_7_joint_position" joint="${side}_7_joint" ctrlrange="${arm_7_joint_lb * deg_to_rad} ${arm_7_joint_ub * deg_to_rad}" kp="500" kv="20"/>
+      </xacro:if>
     </xacro:macro>
 </robot>

File: pal_sea_arm_description/robots/pal_sea_arm.urdf.xacro (robot description, xacro)
@@ -31,6 +31,4 @@
   <!-- Mujoco args -->
   <xacro:arg name="mujoco" default="false" />
-  <xacro:arg name="mj_motor" default="false" />
-  <xacro:arg name="mj_position" default="false" />
   <xacro:arg name="mj_simulate" default="false" />
   <xacro:arg name="mj_control" default="false" />
@@ -45,5 +43,7 @@
   <!-- Mujoco properties -->
   <xacro:property name="mujoco" value="$(arg mujoco)" />
+  <xacro:property name="mj_simulate" value="$(arg mj_simulate)" />
   <xacro:property name="mj_control" value="$(arg mj_control)" />
+  <xacro:property name="mj_controller" value="${mj_control if mj_control != 'false' else 'no_controller'}"/>
   <xacro:if value="${end_effector not in ['no-end-effector', 'pal-pro-gripper', 'allegro-hand', 'custom']}">
     <xacro:wrong_end_effector/>
@@ -102,16 +102,29 @@
    <!-- Mujoco Tags -->
   <xacro:include filename="$(find pal_sea_arm_description)/mujoco/mj_tags.xacro" />
-  <xacro:if value="$(arg mujoco)">
+  <xacro:include filename="$(find pal_pro_gripper_description)/mujoco/mj_tags.xacro" />
+  <xacro:if value="${mujoco}">
     <mujoco>
-      <xacro:mj_common/>
-      <xacro:if value="$(arg mj_simulate)">
+       <!-- Mujoco environment -->
+      <xacro:mj_arm_common/>
+      <!-- Actuator-->
+      <xacro:if value="${mj_simulate}">
         <actuator>
-          <xacro:if value="$(arg mj_motor)">
-            <xacro:single_arm_mj_motor_actuators/>
-          </xacro:if>
-          <xacro:if value="$(arg mj_position)">
-            <xacro:single_arm_mj_position_actuators/>
+          <!-- Arm -->
+          <xacro:mj_arm_actuators side="arm" joint_reflect="1"/>
+          <xacro:if value="${has_end_effector}">
+            <!-- End-effector -->
+            <xacro:mj_gripper_actuators side="gripper" reflect="1"/>
           </xacro:if>
         </actuator>
+      </xacro:if>
+      <xacro:if value="${has_end_effector}">
+          <!-- Equality-->
+        <equality>
+          <xacro:mj_gripper_equality side="gripper" anchor_r="0.014 -0.0015 0" anchor_l="0.014 -0.001 0"/>
+        </equality>
+        <!-- Contact-->
+        <contact>
+          <xacro:mj_gripper_contact side="gripper"/>
+        </contact>
       </xacro:if>
     </mujoco>

File: pal_sea_arm_description/ros2_control/ros2_control.urdf.xacro (robot description, xacro)
@@ -29,8 +29,8 @@
       <hardware>
         <xacro:if value="$(arg use_sim_time)">
-          <xacro:if value="${mj_control}">
+          <xacro:if value="${mujoco and not mj_simulate}">
             <plugin>mujoco_ros2_control/MujocoSystem</plugin>
           </xacro:if>
-          <xacro:unless value="${mj_control}">
+          <xacro:unless value="${mujoco}">
             <plugin>gazebo_ros2_control/GazeboSystem</plugin>
           </xacro:unless>

File: pal_sea_arm_description/urdf/arm/arm.ros2_control.xacro (robot description, xacro)
@@ -14,26 +14,19 @@
 <robot xmlns:xacro="http://ros.org/wiki/xacro">
   <xacro:macro name="ros2_control_arm" params="name reduction offset_value use_sea_transmission:=false">
-    <xacro:if value="$(arg mujoco)">
+    <xacro:if value="${mujoco}">
        <joint name="${name}_joint">
-        <xacro:if value="$(arg mj_position)">
-          <xacro:if value="$(arg mj_simulate)">
-            <command_interface name="position" />
-          </xacro:if>
-          <xacro:unless value="$(arg mj_simulate)">
+        <xacro:unless value="${mj_simulate}">
             <param name="position_kp">700</param>
-            <param name="position_ki">0</param>
-            <param name="position_kd">1</param>
+            <param name="position_ki">1</param>
+            <param name="position_kd">10</param>
             <param name="position_i_max">0</param>
             <command_interface name="position_pid" />
-          </xacro:unless>
-        </xacro:if>
-        <xacro:unless value="$(arg mj_position)">
-          <command_interface name="effort" />
-          <command_interface name="velocity" />
+            <!-- <command_interface name="effort" />
+            <command_interface name="velocity" /> -->
         </xacro:unless>
         <state_interface name="position" />
         <state_interface name="velocity" />
         <state_interface name="effort" />
-       </joint>
+      </joint>
     </xacro:if>
     <xacro:unless value="$(arg mujoco)">

Commit message: Added arm_type and wrist_model argument

File: pal_sea_arm_description/mujoco/mj_tags.xacro (robot description, xacro)
@@ -20,5 +20,5 @@
     </xacro:macro>
     <!-- Actuators -->
-    <xacro:macro name="mj_arm_actuators" params="side joint_reflect:=1">
+    <xacro:macro name="mj_arm_actuators" params="side arm_type wrist_model joint_reflect">
       <xacro:include filename="$(find pal_sea_arm_description)/urdf/arm/arm_limits/${arm_type}/arm.limits.xacro"/>
       <xacro:include filename="$(find pal_sea_arm_description)/urdf/arm/arm_limits/${arm_type}/${wrist_model}.limits.xacro"/>

File: pal_sea_arm_description/robots/pal_sea_arm.urdf.xacro (robot description, xacro)
@@ -111,5 +111,5 @@
         <actuator>
           <!-- Arm -->
-          <xacro:mj_arm_actuators side="arm" joint_reflect="1"/>
+          <xacro:mj_arm_actuators side="arm" arm_type="${arm_type}" wrist_model="${wrist_model}" joint_reflect="1"/>
           <xacro:if value="${has_end_effector}">
             <!-- End-effector -->
