Commit message: Improved mujoco model structure

File: pal_sea_arm_description/mujoco/mj_tags.xacro (robot description, xacro)
@@ -1,22 +1,4 @@
 <?xml version="1.0"?>
 <robot xmlns:xacro="http://ros.org/wiki/xacro" name="pal_sea_arm">
-    <!-- Mujoco environment for arm mujoco simulation-->
-    <xacro:macro name="mj_arm_common">
-      <compiler strippath="false" discardvisual="false" balanceinertia="true" angle="radian" />
-        <option integrator="implicitfast" />
-        <asset>
-            <texture type="skybox" builtin="gradient" rgb1="0.3 0.5 0.7" rgb2="0 0 0" width="512"
-                height="3072" />
-            <texture type="2d" name="groundplane" builtin="checker" mark="edge" rgb1="0.2 0.3 0.4"
-                rgb2="0.1 0.2 0.3"
-                markrgb="0.8 0.8 0.8" width="300" height="300" />
-            <material name="groundplane" texture="groundplane" texuniform="true" texrepeat="5 5"
-                reflectance="0.2" />
-        </asset>
-        <worldbody>
-            <light name="spotlight" mode="targetbody" target="arm_1_link" pos="1 0 10" />
-            <geom name="floor" size="0 0 0.05" type="plane" material="groundplane" group="1" contype="1" conaffinity="1" friction="0.001 0.0 0.0"/>
-        </worldbody>
-    </xacro:macro>
     <!-- Actuators -->
     <xacro:macro name="mj_arm_actuators" params="side arm_type wrist_model joint_reflect">
@@ -25,5 +7,5 @@
       <xacro:include filename="$(find pal_sea_arm_description)/urdf/arm/arm_properties/${arm_type}/arm.properties.xacro"/>
       <xacro:include filename="$(find pal_sea_arm_description)/urdf/arm/arm_properties/${arm_type}/${wrist_model}.properties.xacro"/>
-      <xacro:if value="${mj_controller == 'motor'}">
+      <xacro:if value="${mj_control == 'motor'}">
         <motor name="${side}_1_joint_torque" joint="${side}_1_joint" ctrlrange="-46 46" />
         <motor name="${side}_2_joint_torque" joint="${side}_2_joint" ctrlrange="-46 46" />
@@ -34,5 +16,5 @@
         <motor name="${side}_7_joint_torque" joint="${side}_7_joint" ctrlrange="-46 46" />
       </xacro:if>
-      <xacro:if value="${mj_controller == 'position'}">
+      <xacro:if value="${mj_control == 'position'}">
         <position name="${side}_1_joint_position" joint="${side}_1_joint" ctrlrange="${arm_1_joint_lb * deg_to_rad} ${arm_1_joint_ub * deg_to_rad}" kp="1000" kv="50"/>
         <position name="${side}_2_joint_position" joint="${side}_2_joint" ctrlrange="${arm_2_joint_lb * deg_to_rad} ${arm_2_joint_ub * deg_to_rad}" kp="1000" kv="60"/>

File: pal_sea_arm_description/robots/pal_sea_arm.urdf.xacro (robot description, xacro)
@@ -30,7 +30,7 @@
   <xacro:arg name="namespace" default=""/>
   <!-- Mujoco args -->
-  <xacro:arg name="mujoco" default="false" />
-  <xacro:arg name="mj_simulate" default="false" />
+  <xacro:arg name="sim_type" default="gazebo" />
   <xacro:arg name="mj_control" default="false" />
+  <xacro:arg name="mj_world_name" default="floor" />
   <!-- PROPERTIES -->
   <xacro:property name="end_effector" value="$(arg end_effector)" />
@@ -41,9 +41,7 @@
   <xacro:property name="tool_changer" value="$(arg tool_changer)" />
   <xacro:property name="nsp" value="$(arg namespace)" />
-  <!-- Mujoco properties -->
-  <xacro:property name="mujoco" value="$(arg mujoco)" />
-  <xacro:property name="mj_simulate" value="$(arg mj_simulate)" />
-  <xacro:property name="mj_control" value="$(arg mj_control)" />
-  <xacro:property name="mj_controller" value="${mj_control if mj_control != 'false' else 'no_controller'}"/>
+  <xacro:property name="sim_type" value="$(arg sim_type)" />
+  <xacro:property name="mj_control" value="$(arg mj_control)"/>
+  <xacro:property name="mj_world_name" value="$(arg mj_world_name)"/>
   <xacro:if value="${end_effector not in ['no-end-effector', 'pal-pro-gripper', 'allegro-hand', 'custom']}">
     <xacro:wrong_end_effector/>
@@ -100,13 +98,14 @@
   <!-- End effector -->
   <xacro:pal_sea_arm_end_effector name="gripper" parent="${end_effector_link}" type="${end_effector}" tool_changer="${tool_changer}" reflect="1"/>
-   <!-- Mujoco Tags -->
-  <xacro:include filename="$(find pal_sea_arm_description)/mujoco/mj_tags.xacro" />
-  <xacro:include filename="$(find pal_pro_gripper_description)/mujoco/mj_tags.xacro" />
-  <xacro:if value="${mujoco}">
+  <xacro:if value="${sim_type == 'mujoco' or sim_type == 'mujoco-ros2-control'}">
     <mujoco>
+      <!-- Mujoco Includes -->
+      <xacro:include filename="$(find pal_sea_arm_description)/mujoco/mj_tags.xacro" />
+      <xacro:include filename="$(find pal_pro_gripper_description)/mujoco/mj_tags.xacro" />
+      <xacro:include filename="$(find pal_mujoco_scenes)/scenes/${mj_world_name}.xacro" />
        <!-- Mujoco environment -->
-      <xacro:mj_arm_common/>
+      <xacro:mj_common light_target="arm_1_link"/>
       <!-- Actuator-->
-      <xacro:if value="${mj_simulate}">
+      <xacro:if value="${sim_type == 'mujoco'}">
         <actuator>
           <!-- Arm -->
@@ -114,5 +113,5 @@
           <xacro:if value="${has_end_effector}">
             <!-- End-effector -->
-            <xacro:mj_gripper_actuators side="gripper" reflect="1"/>
+            <xacro:mj_gripper_actuators name="gripper"/>
           </xacro:if>
         </actuator>

Commit message: changed mujoco xacro parameter name

File: pal_sea_arm_description/mujoco/mj_tags.xacro (robot description, xacro)
@@ -2,5 +2,5 @@
 <robot xmlns:xacro="http://ros.org/wiki/xacro" name="pal_sea_arm">
     <!-- Actuators -->
-    <xacro:macro name="mj_arm_actuators" params="side arm_type wrist_model joint_reflect">
+    <xacro:macro name="mj_arm_actuators" params="name arm_type wrist_model joint_reflect">
       <xacro:include filename="$(find pal_sea_arm_description)/urdf/arm/arm_limits/${arm_type}/arm.limits.xacro"/>
       <xacro:include filename="$(find pal_sea_arm_description)/urdf/arm/arm_limits/${arm_type}/${wrist_model}.limits.xacro"/>
@@ -8,20 +8,20 @@
       <xacro:include filename="$(find pal_sea_arm_description)/urdf/arm/arm_properties/${arm_type}/${wrist_model}.properties.xacro"/>
       <xacro:if value="${mj_control == 'motor'}">
-        <motor name="${side}_1_joint_torque" joint="${side}_1_joint" ctrlrange="-46 46" />
-        <motor name="${side}_2_joint_torque" joint="${side}_2_joint" ctrlrange="-46 46" />
-        <motor name="${side}_3_joint_torque" joint="${side}_3_joint" ctrlrange="-46 46" />
-        <motor name="${side}_4_joint_torque" joint="${side}_4_joint" ctrlrange="-46 46" />
-        <motor name="${side}_5_joint_torque" joint="${side}_5_joint" ctrlrange="-46 46" />
-        <motor name="${side}_6_joint_torque" joint="${side}_6_joint" ctrlrange="-46 46" />
-        <motor name="${side}_7_joint_torque" joint="${side}_7_joint" ctrlrange="-46 46" />
+        <motor name="${name}_1_joint_torque" joint="${name}_1_joint" ctrlrange="-46 46" />
+        <motor name="${name}_2_joint_torque" joint="${name}_2_joint" ctrlrange="-46 46" />
+        <motor name="${name}_3_joint_torque" joint="${name}_3_joint" ctrlrange="-46 46" />
+        <motor name="${name}_4_joint_torque" joint="${name}_4_joint" ctrlrange="-46 46" />
+        <motor name="${name}_5_joint_torque" joint="${name}_5_joint" ctrlrange="-46 46" />
+        <motor name="${name}_6_joint_torque" joint="${name}_6_joint" ctrlrange="-46 46" />
+        <motor name="${name}_7_joint_torque" joint="${name}_7_joint" ctrlrange="-46 46" />
       </xacro:if>
       <xacro:if value="${mj_control == 'position'}">
-        <position name="${side}_1_joint_position" joint="${side}_1_joint" ctrlrange="${arm_1_joint_lb * deg_to_rad} ${arm_1_joint_ub * deg_to_rad}" kp="1000" kv="50"/>
-        <position name="${side}_2_joint_position" joint="${side}_2_joint" ctrlrange="${arm_2_joint_lb * deg_to_rad} ${arm_2_joint_ub * deg_to_rad}" kp="1000" kv="60"/>
-        <position name="${side}_3_joint_position" joint="${side}_3_joint" ctrlrange="${arm_3_joint_lb * deg_to_rad} ${arm_3_joint_ub * deg_to_rad}" kp="1000" kv="50"/>
-        <position name="${side}_4_joint_position" joint="${side}_4_joint" ctrlrange="${arm_4_joint_lb * deg_to_rad} ${arm_4_joint_ub * deg_to_rad}" kp="500" kv="20"/>
-        <position name="${side}_5_joint_position" joint="${side}_5_joint" ctrlrange="${arm_5_joint_lb * deg_to_rad} ${arm_5_joint_ub * deg_to_rad}" kp="1000" kv="20"/>
-        <position name="${side}_6_joint_position" joint="${side}_6_joint" ctrlrange="${arm_6_joint_lb * deg_to_rad} ${arm_6_joint_ub * deg_to_rad}" kp="1000" kv="20"/>
-        <position name="${side}_7_joint_position" joint="${side}_7_joint" ctrlrange="${arm_7_joint_lb * deg_to_rad} ${arm_7_joint_ub * deg_to_rad}" kp="500" kv="20"/>
+        <position name="${name}_1_joint_position" joint="${name}_1_joint" ctrlrange="${arm_1_joint_lb * deg_to_rad} ${arm_1_joint_ub * deg_to_rad}" kp="1000" kv="50"/>
+        <position name="${name}_2_joint_position" joint="${name}_2_joint" ctrlrange="${arm_2_joint_lb * deg_to_rad} ${arm_2_joint_ub * deg_to_rad}" kp="1000" kv="60"/>
+        <position name="${name}_3_joint_position" joint="${name}_3_joint" ctrlrange="${arm_3_joint_lb * deg_to_rad} ${arm_3_joint_ub * deg_to_rad}" kp="1000" kv="50"/>
+        <position name="${name}_4_joint_position" joint="${name}_4_joint" ctrlrange="${arm_4_joint_lb * deg_to_rad} ${arm_4_joint_ub * deg_to_rad}" kp="500" kv="20"/>
+        <position name="${name}_5_joint_position" joint="${name}_5_joint" ctrlrange="${arm_5_joint_lb * deg_to_rad} ${arm_5_joint_ub * deg_to_rad}" kp="1000" kv="20"/>
+        <position name="${name}_6_joint_position" joint="${name}_6_joint" ctrlrange="${arm_6_joint_lb * deg_to_rad} ${arm_6_joint_ub * deg_to_rad}" kp="1000" kv="20"/>
+        <position name="${name}_7_joint_position" joint="${name}_7_joint" ctrlrange="${arm_7_joint_lb * deg_to_rad} ${arm_7_joint_ub * deg_to_rad}" kp="500" kv="20"/>
       </xacro:if>
     </xacro:macro>
