Commit message: update velocity limits for S+, S- and XS

File: pal_sea_arm_description/urdf/arm/arm_limits/pal-sea-arm-standalone/arm.limits.xacro (robot description, xacro)
@@ -17,6 +17,6 @@
   <xacro:property name="arm_1_max_velocity" value="1.95" />
   <xacro:property name="arm_2_max_velocity" value="1.95" />
-  <xacro:property name="arm_3_max_velocity" value="2.35" />
-  <xacro:property name="arm_4_max_velocity" value="2.35" />
+  <xacro:property name="arm_3_max_velocity" value="3.95" />
+  <xacro:property name="arm_4_max_velocity" value="3.95" />
   <!-- Effort limits -->
   <xacro:property name="arm_1_max_effort" value="43.0" />

File: pal_sea_arm_description/urdf/arm/arm_limits/pal-sea-arm-standalone/spherical-wrist.limits.xacro (robot description, xacro)
@@ -8,7 +8,7 @@
   <xacro:property name="arm_7_joint_lb" value="-148.97" />
   <!-- Velocity limits -->
-  <xacro:property name="arm_5_max_velocity" value="2.35" />
-  <xacro:property name="arm_6_max_velocity" value="2.35" />
-  <xacro:property name="arm_7_max_velocity" value="2.35" />
+  <xacro:property name="arm_5_max_velocity" value="3.95" />
+  <xacro:property name="arm_6_max_velocity" value="3.95" />
+  <xacro:property name="arm_7_max_velocity" value="3.95" />
   <!-- Effort limits -->
   <xacro:property name="arm_5_max_effort" value="26" />

File: pal_sea_arm_description/urdf/arm/arm_limits/pal-sea-arm-standalone/straight-wrist.limits.xacro (robot description, xacro)
@@ -8,7 +8,7 @@
   <xacro:property name="arm_7_joint_lb" value="-148.97" />
   <!-- Velocity limits -->
-  <xacro:property name="arm_5_max_velocity" value="2.35" />
-  <xacro:property name="arm_6_max_velocity" value="2.35" />
-  <xacro:property name="arm_7_max_velocity" value="2.35" />
+  <xacro:property name="arm_5_max_velocity" value="3.95" />
+  <xacro:property name="arm_6_max_velocity" value="3.95" />
+  <xacro:property name="arm_7_max_velocity" value="3.95" />
   <!-- Effort limits -->
   <xacro:property name="arm_5_max_effort" value="26" />

File: pal_sea_arm_description/urdf/arm/arm_limits/tiago-pro/arm.limits.xacro (robot description, xacro)
@@ -15,8 +15,8 @@
   <xacro:property name="arm_4_joint_lb" value="-140" />
   <!-- Velocity limits -->
-  <xacro:property name="arm_1_max_velocity" value="2.50" />
-  <xacro:property name="arm_2_max_velocity" value="2.50" />
-  <xacro:property name="arm_3_max_velocity" value="2.50" />
-  <xacro:property name="arm_4_max_velocity" value="2.50" />
+  <xacro:property name="arm_1_max_velocity" value="1.95" />
+  <xacro:property name="arm_2_max_velocity" value="1.95" />
+  <xacro:property name="arm_3_max_velocity" value="3.95" />
+  <xacro:property name="arm_4_max_velocity" value="3.95" />
   <!-- Effort limits -->
   <xacro:property name="arm_1_max_effort" value="43.0" />

File: pal_sea_arm_description/urdf/arm/arm_limits/tiago-pro/spherical-wrist.limits.xacro (robot description, xacro)
@@ -8,7 +8,7 @@
   <xacro:property name="arm_7_joint_lb" value="-150" />
   <!-- Velocity limits -->
-  <xacro:property name="arm_5_max_velocity" value="2.50" />
-  <xacro:property name="arm_6_max_velocity" value="2.50" />
-  <xacro:property name="arm_7_max_velocity" value="2.50" />
+  <xacro:property name="arm_5_max_velocity" value="3.95" />
+  <xacro:property name="arm_6_max_velocity" value="3.95" />
+  <xacro:property name="arm_7_max_velocity" value="3.95" />
   <!-- Effort limits -->
   <xacro:property name="arm_5_max_effort" value="26" />

File: pal_sea_arm_description/urdf/arm/arm_limits/tiago-pro/straight-wrist.limits.xacro (robot description, xacro)
@@ -8,7 +8,7 @@
   <xacro:property name="arm_7_joint_lb" value="-150" />
   <!-- Velocity limits -->
-  <xacro:property name="arm_5_max_velocity" value="2.35" />
-  <xacro:property name="arm_6_max_velocity" value="2.35" />
-  <xacro:property name="arm_7_max_velocity" value="2.35" />
+  <xacro:property name="arm_5_max_velocity" value="3.95" />
+  <xacro:property name="arm_6_max_velocity" value="3.95" />
+  <xacro:property name="arm_7_max_velocity" value="3.95" />
   <!-- Effort limits -->
   <xacro:property name="arm_5_max_effort" value="26" />

Commit message: fix limits j1 and j3

File: pal_sea_arm_description/urdf/arm/arm_limits/pal-sea-arm-standalone/arm.limits.xacro (robot description, xacro)
@@ -6,10 +6,8 @@
   <xacro:property name="arm_k_velocity" value="20"/>
   <!-- Joint limits -->
-  <xacro:property name="arm_1_joint_ub" value="120" />
-  <xacro:property name="arm_1_joint_lb" value="-180" />
   <xacro:property name="arm_2_joint_ub" value="63.03" />
   <xacro:property name="arm_2_joint_lb" value="-139.8" />
-  <xacro:property name="arm_3_joint_ub" value="148.97" />
-  <xacro:property name="arm_3_joint_lb" value="-148.97" />
+  <xacro:property name="arm_3_joint_ub" value="-148.97" />
+  <xacro:property name="arm_3_joint_lb" value="148.97" />
   <xacro:property name="arm_4_joint_ub" value="63.03" />
   <xacro:property name="arm_4_joint_lb" value="-139.8" />

Commit message: change limits j3

File: pal_sea_arm_description/urdf/arm/arm_limits/pal-sea-arm-standalone/arm.limits.xacro (robot description, xacro)
@@ -8,6 +8,6 @@
   <xacro:property name="arm_2_joint_ub" value="63.03" />
   <xacro:property name="arm_2_joint_lb" value="-139.8" />
-  <xacro:property name="arm_3_joint_ub" value="-148.97" />
-  <xacro:property name="arm_3_joint_lb" value="148.97" />
+  <xacro:property name="arm_3_joint_ub" value="150" />
+  <xacro:property name="arm_3_joint_lb" value="-150" />
   <xacro:property name="arm_4_joint_ub" value="63.03" />
   <xacro:property name="arm_4_joint_lb" value="-139.8" />
