Commit message: change values limits joint6

File: pal_sea_arm_description/urdf/arm/arm_limits/pal-sea-arm-standalone/spherical-wrist.limits.xacro (robot description, xacro)
@@ -1,6 +1,6 @@
 <robot xmlns:xacro="http://ros.org/wiki/xacro">
   <!-- Joint limits -->
-  <xacro:property name="arm_6_joint_ub" value="114.59" />
-  <xacro:property name="arm_6_joint_lb" value="-114.59" />
+  <xacro:property name="arm_6_joint_ub" value="172" />
+  <xacro:property name="arm_6_joint_lb" value="-98" />
   <xacro:property name="arm_7_joint_ub" value="148.97" />
   <xacro:property name="arm_7_joint_lb" value="-148.97" />

Commit message: Reducing arm_7 upper/lower bound

File: pal_sea_arm_description/urdf/arm/arm_limits/pal-sea-arm-standalone/spherical-wrist.limits.xacro (robot description, xacro)
@@ -3,6 +3,6 @@
   <xacro:property name="arm_6_joint_ub" value="172" />
   <xacro:property name="arm_6_joint_lb" value="-98" />
-  <xacro:property name="arm_7_joint_ub" value="148.97" />
-  <xacro:property name="arm_7_joint_lb" value="-148.97" />
+  <xacro:property name="arm_7_joint_ub" value="140" />
+  <xacro:property name="arm_7_joint_lb" value="-140" />
   <!-- Velocity limits -->
   <xacro:property name="arm_5_max_velocity" value="3.95" />
