Commit message: reduce 7 limit for spherical and straight wrist

File: pal_sea_arm_description/urdf/arm/arm_limits/pal-sea-arm-standalone/straight-wrist.limits.xacro (robot description, xacro)
@@ -3,6 +3,6 @@
   <xacro:property name="arm_6_joint_ub" value="114.59" />
   <xacro:property name="arm_6_joint_lb" value="-114.59" />
-  <xacro:property name="arm_7_joint_ub" value="148.97" />
-  <xacro:property name="arm_7_joint_lb" value="-148.97" />
+  <xacro:property name="arm_7_joint_ub" value="140" />
+  <xacro:property name="arm_7_joint_lb" value="-140" />
   <!-- Velocity limits -->
   <xacro:property name="arm_5_max_velocity" value="3.95" />

File: pal_sea_arm_description/urdf/arm/arm_limits/tiago-pro/straight-wrist.limits.xacro (robot description, xacro)
@@ -5,6 +5,6 @@
   <xacro:property name="arm_6_joint_ub" value="120" />
   <xacro:property name="arm_6_joint_lb" value="-120" />
-  <xacro:property name="arm_7_joint_ub" value="150" />
-  <xacro:property name="arm_7_joint_lb" value="-150" />
+  <xacro:property name="arm_7_joint_ub" value="140" />
+  <xacro:property name="arm_7_joint_lb" value="-140" />
   <!-- Velocity limits -->
   <xacro:property name="arm_5_max_velocity" value="3.95" />

File: pal_sea_arm_description/urdf/arm/arm_limits/tiago-sea/straight-wrist.limits.xacro (robot description, xacro)
@@ -5,6 +5,6 @@
   <xacro:property name="arm_6_joint_ub" value="114" />
   <xacro:property name="arm_6_joint_lb" value="-114" />
-  <xacro:property name="arm_7_joint_ub" value="145" />
-  <xacro:property name="arm_7_joint_lb" value="-145" />
+  <xacro:property name="arm_7_joint_ub" value="140" />
+  <xacro:property name="arm_7_joint_lb" value="-140" />
   <!-- Velocity limits -->
   <xacro:property name="arm_5_max_velocity" value="1.95" />
