Commit message: fix 7th joint

File: pal_sea_arm_description/urdf/arm/arm_properties/pal-sea-arm-standalone/spherical-wrist.properties.xacro (robot description, xacro)
@@ -25,5 +25,5 @@
     </xacro:macro>
     <xacro:macro name="origin_joint_7" params="reflect">
-        <origin xyz="-0.07 -0.0534 0.0422" rpy="1.5708 -1.5708 0" />
+        <origin xyz="0.07 -0.0534 -0.0422" rpy="1.5708 -1.5708 0" />
     </xacro:macro>
 </robot>
