Commit message: changed mesh name

File: pal_sea_arm_description/urdf/arm/arm_properties/pal-sea-arm-standalone/arm.properties.xacro (robot description, xacro)
@@ -1,4 +1,4 @@
 <robot xmlns:xacro="http://ros.org/wiki/xacro">
-    <xacro:macro name="inertial_base_link" params="reflect">
+    <xacro:macro name="inertial_arm_base_link" params="reflect">
         <inertial>
             <origin xyz="-0.00069237 0.00052761 -0.012575" rpy="0 0 0" />

File: pal_sea_arm_description/urdf/arm/arm_properties/tiago-pro/arm.properties.xacro (robot description, xacro)
@@ -1,4 +1,4 @@
 <robot xmlns:xacro="http://ros.org/wiki/xacro">
-    <xacro:macro name="inertial_base_link" params="reflect">
+    <xacro:macro name="inertial_arm_base_link" params="reflect">
         <inertial>
             <origin xyz="-0.00069237 0.00052761 -0.012575" rpy="0 0 0" />

File: pal_sea_arm_description/urdf/arm/arm_properties/tiago-sea/arm.properties.xacro (robot description, xacro)
@@ -1,4 +1,4 @@
 <robot xmlns:xacro="http://ros.org/wiki/xacro">
-    <xacro:macro name="inertial_base_link" params="reflect">
+    <xacro:macro name="inertial_arm_base_link" params="reflect">
         <inertial>
             <origin xyz="-0.00069237 0.00052761 -0.012575" rpy="0 0 0" />

File: pal_sea_arm_description/urdf/end_effector/grasping_frames.xacro (robot description, xacro)
@@ -23,5 +23,5 @@
     <!-- Grasping frame X -->
     <joint name="${prefix}grasping_frame_joint" type="fixed">
-      <parent link="${prefix}base_link" />
+      <parent link="${prefix}arm_base_link" />
       <child link="${prefix}grasping_frame" />
       <origin xyz="${xyz}" rpy="0 -1.5708 0" />
@@ -30,5 +30,5 @@
     <!-- Grasping frame Y -->
     <joint name="${prefix}grasping_frame_Y_joint" type="fixed">
-      <parent link="${prefix}base_link" />
+      <parent link="${prefix}arm_base_link" />
       <child link="${prefix}grasping_frame_Y" />
       <origin xyz="${xyz}" rpy="1.5708 0 0" />
@@ -37,5 +37,5 @@
     <!-- Grasping frame Z -->
     <joint name="${prefix}grasping_frame_Z_joint" type="fixed">
-      <parent link="${prefix}base_link" />
+      <parent link="${prefix}arm_base_link" />
       <child link="${prefix}grasping_frame_Z" />
       <origin xyz="${xyz}" rpy="0 0 0" />

Commit message: Fix spherical wrist properties and origins

File: pal_sea_arm_description/urdf/arm/arm_properties/pal-sea-arm-standalone/arm.properties.xacro (robot description, xacro)
@@ -47,7 +47,4 @@
         <origin xyz="0.0199999999999993 -0.0371100000000008 0.15989" rpy="1.57079632679489 0 0" />
     </xacro:macro>
-    <xacro:macro name="origin_joint_5" params="reflect">
-        <origin xyz="-0.0199999999999971 0.17011 -0.037110000000002" rpy="-1.5707963267949 0 0" />
-    </xacro:macro>
     <!-- Tool changer (can be present in both wrists)-->
     <xacro:macro name="inertial_tool_changer_link" params="reflect">

File: pal_sea_arm_description/urdf/arm/arm_properties/pal-sea-arm-standalone/spherical-wrist.properties.xacro (robot description, xacro)
@@ -2,14 +2,36 @@
     <xacro:macro name="inertial_link_5" params="reflect">
         <inertial>
-            <origin xyz="-1.1035E-05 -0.027586 0.067845" rpy="0 0 0" />
-            <mass value="0.31076" />
-            <inertia ixx="0.0014015" ixy="9.1728E-08" ixz="-9.3079E-08" iyy="0.0014" iyz="0.00032771" izz="0.00040201" />
+            <origin
+                xyz="-6.6854E-07 -0.02662 0.067326"
+                rpy="0 0 0" />
+            <mass
+                value="0.34802" />
+            <inertia
+                ixx="0.0014602"
+                ixy="-1.4931E-08"
+                ixz="8.1828E-08"
+                iyy="0.0014558"
+                iyz="0.00033448"
+                izz="0.00040968" />
         </inertial>
+    </xacro:macro>
+    <xacro:macro name="origin_joint_5" params="reflect">
+        <!-- Check new limits -->
+        <origin xyz="-0.0199999999999971 0.17011 -0.037110000000002" rpy="-1.5707963267949 3.14 0" />
     </xacro:macro>
     <xacro:macro name="inertial_link_6" params="reflect">
         <inertial>
-            <origin xyz="-0.0083923 -0.00081501 0.039899" rpy="0 0 0" />
-            <mass value="0.83518" />
-            <inertia ixx="0.00077706" ixy="-0.00012999" ixz="-5.9554E-06" iyy="0.00094237" iyz="-1.5002E-06" izz="0.00086922" />
+            <origin
+                xyz="0.031968 -0.0065097 -0.040676"
+                rpy="0 0 0" />
+            <mass
+                value="1.378" />
+            <inertia
+                ixx="0.0011002"
+                ixy="0.00012805"
+                ixz="-5.6797E-06"
+                iyy="0.0011658"
+                iyz="5.4596E-07"
+                izz="0.0011909" />
         </inertial>
     </xacro:macro>
@@ -19,11 +41,20 @@
     <xacro:macro name="inertial_link_7" params="reflect">
         <inertial>
-            <origin xyz="2.1788E-15 7.5568E-05 -0.037565" rpy="0 0 0" />
-            <mass value="0.51032" />
-            <inertia ixx="0.00032121" ixy="-1.7628E-21" ixz="-7.178E-21" iyy="0.00032034" iyz="-1.0206E-06" izz="0.00022179" />
+            <origin
+                xyz="-0.0016034 0.001194 0.0075583"
+                rpy="0 0 0" />
+            <mass
+                value="0.1354" />
+            <inertia
+                ixx="5.0537E-05"
+                ixy="-8.1184E-07"
+                ixz="1.9023E-07"
+                iyy="5.1762E-05"
+                iyz="-3.2751E-07"
+                izz="9.5274E-05" />
         </inertial>
     </xacro:macro>
     <xacro:macro name="origin_joint_7" params="reflect">
-        <origin xyz="0.07 -0.0534 -0.0422" rpy="1.5708 -1.5708 0" />
+        <origin xyz="0.07 -0.0534 -0.0422" rpy="1.5708 0 0" />
     </xacro:macro>
 </robot>
