Commit message: add 5th joint in short and straight wrist properties

File: pal_sea_arm_description/urdf/arm/arm_properties/pal-sea-arm-standalone/short-wrist.properties.xacro (robot description, xacro)
@@ -7,3 +7,7 @@
         </inertial>
     </xacro:macro>
+    <xacro:macro name="origin_joint_5" params="reflect">
+        <!-- Check new limits -->
+        <origin xyz="-0.0199999999999971 0.17011 -0.037110000000002" rpy="-1.5707963267949 3.14 0" />
+    </xacro:macro>
 </robot>

File: pal_sea_arm_description/urdf/arm/arm_properties/pal-sea-arm-standalone/straight-wrist.properties.xacro (robot description, xacro)
@@ -6,4 +6,8 @@
             <inertia ixx="0.0020531" ixy="-8.9232E-07" ixz="1.6668E-06" iyy="0.0020434" iyz="3.7824E-05" izz="0.00067121" />
         </inertial>
+    </xacro:macro>
+    <xacro:macro name="origin_joint_5" params="reflect">
+        <!-- Check new limits -->
+        <origin xyz="-0.0199999999999971 0.17011 -0.037110000000002" rpy="-1.5707963267949 0 0" />
     </xacro:macro>
     <xacro:macro name="inertial_link_6" params="reflect">
@@ -25,5 +29,5 @@
     </xacro:macro>
     <xacro:macro name="origin_joint_7" params="reflect">
-        <origin xyz="-0.0354 0.135 0" rpy="-1.5708 0 0" />
+        <origin xyz="0 0.135 0.0354" rpy="-1.5708 0 0" />
     </xacro:macro>
 </robot>
