Commit message: fix 6th link standalone

File: pal_sea_arm_description/urdf/arm/arm_properties/pal-sea-arm-standalone/straight-wrist.properties.xacro (robot description, xacro)
@@ -9,5 +9,5 @@
     <xacro:macro name="origin_joint_5" params="reflect">
         <!-- Check new limits -->
-        <origin xyz="-0.0199999999999971 0.17011 -0.037110000000002" rpy="-1.5707963267949 0 0" />
+        <origin xyz="-0.0199999999999971 0.17011 -0.037110000000002" rpy="-1.5707963267949 3.14 0" />
     </xacro:macro>
     <xacro:macro name="inertial_link_6" params="reflect">
@@ -19,5 +19,5 @@
     </xacro:macro>
     <xacro:macro name="origin_joint_6" params="reflect">
-        <origin xyz="0 0.0354 0.16489" rpy="1.5708 0 1.5708" />
+        <origin xyz="0 -0.0354 0.16489" rpy="1.57 0 3.14" />
     </xacro:macro>
     <xacro:macro name="inertial_link_7" params="reflect">
@@ -31,3 +31,6 @@
         <origin xyz="0 0.135 0.0354" rpy="-1.5708 0 0" />
     </xacro:macro>
+    <xacro:macro name="origin_joint_tool_changer" params="reflect">
+        <origin xyz="0 0 0.017" rpy="0 0 0" />
+    </xacro:macro>
 </robot>
