Commit message: Add arguments to support the new gazebo

File: pal_sea_arm_description/gazebo/gazebo.urdf.xacro (robot description, xacro)
@@ -13,9 +13,20 @@
 -->
 <robot name="pal_sea_arm" xmlns:xacro="http://ros.org/wiki/xacro">
-  <gazebo>
-    <plugin filename="libgazebo_ros2_control.so" name="gazebo_ros2_control">
-      <parameters>$(find pal_sea_arm_controller_configuration)/config/gazebo_controller_manager_cfg.yaml</parameters>
-    </plugin>
-  </gazebo>
+  <xacro:if value="${gazebo_version == 'classic'}">
+    <gazebo>
+      <plugin filename="libgazebo_ros2_control.so" name="gazebo_ros2_control">
+        <parameters>$(find pal_sea_arm_controller_configuration)/config/gazebo_controller_manager_cfg.yaml</parameters>
+      </plugin>
+    </gazebo>
+  </xacro:if>
+  <xacro:if value="${gazebo_version == 'gazebo'}">
+    <gazebo>
+      <plugin filename="gz_ros2_control-system" name="gz_ros2_control::GazeboSimROS2ControlPlugin">
+        <robot_param>robot_description</robot_param>
+        <robot_param_node>robot_state_publisher</robot_param_node>
+        <parameters>$(find pal_sea_arm_controller_configuration)/config/gazebo_controller_manager_cfg.yaml</parameters>
+      </plugin>
+    </gazebo>
+  </xacro:if>
   <!-- define global properties -->
   <xacro:property name="M_PI" value="3.1415926535897931" />

File: pal_sea_arm_description/robots/pal_sea_arm.urdf.xacro (robot description, xacro)
@@ -180,4 +180,4 @@
   </xacro:if>
   <!-- ROS2 control -->
-  <xacro:pal_sea_arm_ros2_control use_sim_time="$(arg use_sim_time)" torque_estimation="${torque_estimation}"/>
+  <xacro:pal_sea_arm_ros2_control use_sim_time="$(arg use_sim_time)" torque_estimation="${torque_estimation}" gazebo_version="${gazebo_version}"/>
 </robot>

File: pal_sea_arm_description/ros2_control/ros2_control.urdf.xacro (robot description, xacro)
@@ -13,5 +13,5 @@
  -->
 <robot xmlns:xacro="http://ros.org/wiki/xacro" name="pal_sea_arm">
-  <xacro:macro name="pal_sea_arm_ros2_control" params="use_sim_time:=^|false torque_estimation:=false sim_type:=gazebo">
+  <xacro:macro name="pal_sea_arm_ros2_control" params="use_sim_time:=^|false torque_estimation:=false sim_type:=gazebo gazebo_version:=classic">
     <xacro:arg name="end_effector" default="no-end-effector"/>
     <xacro:arg name="ft_sensor" default="no-ft-sensor"/>
@@ -33,5 +33,10 @@
           </xacro:if>
           <xacro:if value="${sim_type == 'gazebo'}">
-            <plugin>gazebo_ros2_control/GazeboSystem</plugin>
+            <xacro:if value="${gazebo_version == 'classic'}">
+              <plugin>gazebo_ros2_control/GazeboSystem</plugin>
+            </xacro:if>
+            <xacro:if value="${gazebo_version == 'gazebo'}">
+              <plugin>gz_ros2_control/GazeboSimSystem</plugin>
+            </xacro:if>
           </xacro:if>
         </xacro:if>

File: pal_sea_arm_description/urdf/arm/arm.ros2_control.xacro (robot description, xacro)
@@ -25,6 +25,11 @@
         <command_interface name="position" />
       </xacro:if>
-      <command_interface name="velocity" />
-      <command_interface name="effort" />
+      <!-- TODO: Remove when moving to Gazebo Harmonic or ROS 2 Jazzy -->
+      <!-- Multiple command interfaces not working on Gazebo Fortress -->
+      <!-- https://github.com/ros-controls/gz_ros2_control/issues/182 -->
+      <xacro:if value="${gazebo_version == 'classic'}">
+        <command_interface name="velocity" />
+        <command_interface name="effort" />
+      </xacro:if>
       <state_interface name="position" />
       <state_interface name="velocity" />
