Commit message: TC working for all combinations

File: pal_sea_arm_description/urdf/end_effector/end_effector.urdf.xacro (robot description, xacro)
@@ -25,5 +25,5 @@
       <xacro:include filename="$(find pal_pro_gripper_description)/urdf/gripper.urdf.xacro" />
       <xacro:pal_pro_gripper name="${name}" parent="${parent}" tool_changer="${tool_changer}">
-        <origin xyz="0.0 0.0 -0.01" rpy="0 0 0"/>
+        <origin xyz="0.0 0.0 0.0" rpy="0 0 0"/>
       </xacro:pal_pro_gripper>
     </xacro:if>

Commit message: add pal_atc package

File: pal_sea_arm_description/urdf/end_effector/end_effector.urdf.xacro (robot description, xacro)
@@ -28,4 +28,5 @@
       </xacro:pal_pro_gripper>
     </xacro:if>
+<<<<<<< HEAD
     <!--Pen Gripper-->
     <xacro:if value="${type == 'pen-gripper'}">
@@ -70,4 +71,13 @@
       </link>
     </xacro:if>
+=======
+    <!-- PAL ATC -->
+    <xacro:if value="${type == 'pal-atc'}">
+      <xacro:include filename="$(find pal_atc_description)/urdf/gripper.urdf.xacro" />
+      <xacro:pal_atc name="${name}" parent="${parent}" tool_changer="${tool_changer}">
+        <origin xyz="0.0 0.0 0.0" rpy="0 0 0"/>
+      </xacro:pal_atc>
+    </xacro:if>
+>>>>>>> fe903b9 (add pal_atc package)
   <!--Allegro Hand-->
   <xacro:if value="${type == 'allegro-hand'}">
