Commit message: Link 5 short wrist with the tiago pro one

File: pal_sea_arm_description/urdf/arm/arm_properties/humanoid/5dof_arm.urdf.xacro (robot description, xacro)
@@ -6,4 +6,5 @@
   <xacro:property name="arm_5_max_effort"   value="43.0" />
   <xacro:macro name="kangaroo_5dof_arm" params="name side reflect parent *origin arm_1_offset:=0.0 arm_2_offset:=0.0 arm_3_offset:=0.0 arm_4_offset:=0.0">
+    <xacro:include filename="$(find pal_sea_arm_description)/urdf/arm/arm_properties/tiago-pro/short-wrist.properties.xacro"/>
     <!-- ARM 4 LINK -->
     <link name="${name}_${side}_4_link">
@@ -63,5 +64,5 @@
           <origin xyz="0 0 0" rpy="0 0 0" />
           <geometry>
-            <mesh filename="package://pal_sea_arm_description/meshes/humanoid/arm/arm5_tip_link.STL" />
+            <mesh filename="package://pal_sea_arm_description/meshes/arm_tiago_pro/short-wrist/arm_5_link.stl" scale="1 1 1" />
           </geometry>
           <material name="pal/DarkGrey" />
@@ -70,5 +71,5 @@
           mujoco="${sim_type in ['mujoco-ros2-control', 'mujoco']}"
           collision_type="${collision_type}"
-          mesh_file="package://pal_sea_arm_description/meshes/humanoid/arm/arm5_tip_link.STL"
+          mesh_file="package://pal_sea_arm_description/meshes/arm_tiago_pro/short-wrist/arm_5_link_collision.stl"
           scale="1 1 1"
           capsule_radius="0"
@@ -81,5 +82,5 @@
       </link>
       <joint name="${name}_${side}_5_joint" type="revolute">
-        <origin xyz="-0.17011 0.02 -0.03711" rpy="0 -1.5708 0" />
+        <origin xyz="-0.1999 0.02 -0.03711" rpy="0 -1.5708 0" />
         <parent link="${name}_${side}_4_link" />
         <child link="${name}_${side}_5_link" />

Commit message: Fix rotation direction

File: pal_sea_arm_description/urdf/arm/arm_properties/humanoid/5dof_arm.urdf.xacro (robot description, xacro)
@@ -85,5 +85,5 @@
         <parent link="${name}_${side}_4_link" />
         <child link="${name}_${side}_5_link" />
-        <axis xyz="0 0 -1" />
+        <axis xyz="0 0 1" />
         <limit
           lower="-1.57"

File: pal_sea_arm_description/urdf/arm/arm_properties/humanoid/7dof_arm.urdf.xacro (robot description, xacro)
@@ -36,5 +36,5 @@
       <parent link="${parent}" />
       <child link="${name}_${side}_5_link" />
-      <axis xyz="0 0 -1" />
+      <axis xyz="0 0 1" />
       <xacro:if value="${side == 'left'}">
         <limit lower="${deg_to_rad * -210}" upper="${deg_to_rad * 90}" effort="${arm_5_max_effort}" velocity="${arm_5_max_velocity}" />
@@ -121,5 +121,5 @@
       <parent link="${name}_${side}_6_link" />
       <child link="${name}_${side}_7_link" />
-      <axis xyz="0 0 -1" />
+      <axis xyz="0 0 1" />
       <limit lower="${deg_to_rad * -150}" upper="${deg_to_rad * 150}" effort="${arm_7_max_effort}" velocity="${arm_7_max_velocity}" />
     </joint>
