Commit message: Removing incorrect tool offset in 5dof

File: pal_sea_arm_description/urdf/arm/arm_properties/humanoid/arm.urdf.xacro (robot description, xacro)
@@ -19,5 +19,5 @@
       </xacro:kangaroo_5dof_arm>
       <xacro:property name="tip_link" value="5" />
-      <xacro:property name="tool_link_xyz" value="0 0 0.0303" />
+      <xacro:property name="tool_link_xyz" value="0 0 0" />
       <xacro:property name="tool_link_rpy" value="0 0 3.14159" />
     </xacro:if>
