Commit message: Split end effectors into sides

File: pal_sea_arm_description/urdf/arm/arm_properties/humanoid/4dof_arm.urdf.xacro (robot description, xacro)
@@ -23,5 +23,5 @@
         <origin xyz="0 0 0" rpy="0 0 0" />
         <geometry>
-          <mesh filename="package://kangaroo_description/meshes/arm/arm_base_link.STL" />
+          <mesh filename="package://pal_sea_arm_description/meshes/humanoid/arm/arm_base_link.STL" />
         </geometry>
         <material name="pal/DarkGrey" />
@@ -30,5 +30,5 @@
         mujoco="${sim_type in ['mujoco-ros2-control', 'mujoco']}"
         collision_type="${collision_type}"
-        mesh_file="package://kangaroo_description/meshes/arm/arm_base_link.STL"
+        mesh_file="package://pal_sea_arm_description/meshes/humanoid/arm/arm_base_link.STL"
         scale="1 1 1"
         capsule_radius="0"
@@ -61,5 +61,5 @@
         <origin xyz="0 0 0" rpy="0 0 0" />
         <geometry>
-          <mesh filename="package://kangaroo_description/meshes/arm/arm1_link.STL" />
+          <mesh filename="package://pal_sea_arm_description/meshes/humanoid/arm/arm1_link.STL" />
         </geometry>
         <material name="pal/DarkGrey" />
@@ -68,5 +68,5 @@
         mujoco="${sim_type in ['mujoco-ros2-control', 'mujoco']}"
         collision_type="${collision_type}"
-        mesh_file="package://kangaroo_description/meshes/arm/arm1_link.STL"
+        mesh_file="package://pal_sea_arm_description/meshes/humanoid/arm/arm1_link.STL"
         scale="1 1 1"
         capsule_radius="0"
@@ -101,5 +101,5 @@
         <origin xyz="0 0 0" rpy="0 0 0" />
         <geometry>
-          <mesh filename="package://kangaroo_description/meshes/arm/arm2_link.STL" />
+          <mesh filename="package://pal_sea_arm_description/meshes/humanoid/arm/arm2_link.STL" />
         </geometry>
         <material name="pal/DarkGrey" />
@@ -108,5 +108,5 @@
         mujoco="${sim_type in ['mujoco-ros2-control', 'mujoco']}"
         collision_type="${collision_type}"
-        mesh_file="package://kangaroo_description/meshes/arm/arm2_link.STL"
+        mesh_file="package://pal_sea_arm_description/meshes/humanoid/arm/arm2_link.STL"
         scale="1 1 1"
         capsule_radius="0"
@@ -141,5 +141,5 @@
         <origin xyz="0 0 0" rpy="0 0 0" />
         <geometry>
-          <mesh filename="package://kangaroo_description/meshes/arm/arm3_link.STL" />
+          <mesh filename="package://pal_sea_arm_description/meshes/humanoid/arm/arm3_link.STL" />
         </geometry>
         <material name="pal/DarkGrey" />
@@ -148,5 +148,5 @@
         mujoco="${sim_type in ['mujoco-ros2-control', 'mujoco']}"
         collision_type="${collision_type}"
-        mesh_file="package://kangaroo_description/meshes/arm/arm3_link.STL"
+        mesh_file="package://pal_sea_arm_description/meshes/humanoid/arm/arm3_link.STL"
         scale="1 1 1"
         capsule_radius="0"

File: pal_sea_arm_description/urdf/arm/arm_properties/humanoid/5dof_arm.urdf.xacro (robot description, xacro)
@@ -22,5 +22,5 @@
         <origin xyz="0 0 0" rpy="0 0 0" />
         <geometry>
-          <mesh filename="package://kangaroo_description/meshes/arm/arm4_link.STL" />
+          <mesh filename="package://pal_sea_arm_description/meshes/humanoid/arm/arm4_link.STL" />
         </geometry>
         <material name="pal/DarkGrey" />
@@ -29,5 +29,5 @@
         mujoco="${sim_type in ['mujoco-ros2-control', 'mujoco']}"
         collision_type="${collision_type}"
-        mesh_file="package://kangaroo_description/meshes/arm/arm4_link.STL"
+        mesh_file="package://pal_sea_arm_description/meshes/humanoid/arm/arm4_link.STL"
         scale="1 1 1"
         capsule_radius="0"
@@ -63,5 +63,5 @@
           <origin xyz="0 0 0" rpy="0 0 0" />
           <geometry>
-            <mesh filename="package://kangaroo_description/meshes/arm/arm5_tip_link.STL" />
+            <mesh filename="package://pal_sea_arm_description/meshes/humanoid/arm/arm5_tip_link.STL" />
           </geometry>
           <material name="pal/DarkGrey" />
@@ -70,5 +70,5 @@
           mujoco="${sim_type in ['mujoco-ros2-control', 'mujoco']}"
           collision_type="${collision_type}"
-          mesh_file="package://kangaroo_description/meshes/arm/arm5_tip_link.STL"
+          mesh_file="package://pal_sea_arm_description/meshes/humanoid/arm/arm5_tip_link.STL"
           scale="1 1 1"
           capsule_radius="0"

File: pal_sea_arm_description/urdf/arm/arm_properties/humanoid/7dof_arm.urdf.xacro (robot description, xacro)
@@ -24,5 +24,5 @@
         <origin xyz="0 0 0" rpy="0 0 0" />
         <geometry>
-          <mesh filename="package://kangaroo_description/meshes/arm/arm5_link.STL" />
+          <mesh filename="package://pal_sea_arm_description/meshes/humanoid/arm/arm5_link.STL" />
         </geometry>
         <material name="pal/DarkGrey" />
@@ -31,5 +31,5 @@
         mujoco="${sim_type in ['mujoco-ros2-control', 'mujoco']}"
         collision_type="${collision_type}"
-        mesh_file="package://kangaroo_description/meshes/arm/arm5_link.STL"
+        mesh_file="package://pal_sea_arm_description/meshes/humanoid/arm/arm5_link.STL"
         scale="1 1 1"
         capsule_radius="0"
@@ -69,5 +69,5 @@
         <origin xyz="0 0 0" rpy="0 0 0" />
         <geometry>
-          <mesh filename="package://kangaroo_description/meshes/arm/arm6_link.STL" />
+          <mesh filename="package://pal_sea_arm_description/meshes/humanoid/arm/arm6_link.STL" />
         </geometry>
         <material name="pal/DarkGrey" />
@@ -76,5 +76,5 @@
         mujoco="${sim_type in ['mujoco-ros2-control', 'mujoco']}"
         collision_type="${collision_type}"
-        mesh_file="package://kangaroo_description/meshes/arm/arm6_link.STL"
+        mesh_file="package://pal_sea_arm_description/meshes/humanoid/arm/arm6_link.STL"
         scale="1 1 1"
         capsule_radius="0"
@@ -109,5 +109,5 @@
         <origin xyz="0 0 0" rpy="0 0 0" />
         <geometry>
-          <mesh filename="package://kangaroo_description/meshes/arm/arm7_link.STL" />
+          <mesh filename="package://pal_sea_arm_description/meshes/humanoid/arm/arm7_link.STL" />
         </geometry>
         <material name="pal/DarkGrey" />
@@ -116,5 +116,5 @@
         mujoco="${sim_type in ['mujoco-ros2-control', 'mujoco']}"
         collision_type="${collision_type}"
-        mesh_file="package://kangaroo_description/meshes/arm/arm7_link.STL"
+        mesh_file="package://pal_sea_arm_description/meshes/humanoid/arm/arm7_link.STL"
         scale="1 1 1"
         capsule_radius="0"

File: pal_sea_arm_description/urdf/arm/arm_properties/humanoid/arm.urdf.xacro (robot description, xacro)
@@ -4,5 +4,5 @@
     <!-- 4DOF Arm -->
     <xacro:if value="${type in ['4dof', '5dof', '7dof']}">
-      <xacro:include filename="$(find kangaroo_description)/urdf/arm/4dof/4dof_arm.urdf.xacro" />
+      <xacro:include filename="$(find pal_sea_arm_description)/urdf/arm/arm_properties/humanoid/4dof_arm.urdf.xacro" />
       <xacro:kangaroo_4dof_arm name="${name}" side="${side}" reflect="${reflect}" parent="${parent}">
         <xacro:insert_block name="origin"/>
@@ -14,5 +14,5 @@
     <!-- 5DOF Arm -->
     <xacro:if value="${type in ['5dof', '7dof']}">
-      <xacro:include filename="$(find kangaroo_description)/urdf/arm/5dof/5dof_arm.urdf.xacro" />
+      <xacro:include filename="$(find pal_sea_arm_description)/urdf/arm/arm_properties/humanoid/5dof_arm.urdf.xacro" />
       <xacro:kangaroo_5dof_arm name="${name}" side="${side}" reflect="${reflect}" parent="${name}_${side}_3_link">
         <origin xyz="-0.03711 -0.02 -0.17011" rpy="0 -1.5708 0" />
@@ -24,5 +24,5 @@
     <!-- 7DOF Arm -->
     <xacro:if value="${type in ['7dof']}">
-      <xacro:include filename="$(find kangaroo_description)/urdf/arm/7dof/7dof_arm.urdf.xacro" />
+      <xacro:include filename="$(find pal_sea_arm_description)/urdf/arm/arm_properties/humanoid/7dof_arm.urdf.xacro" />
       <xacro:kangaroo_7dof_arm name="${name}" side="${side}" reflect="${reflect}" parent="${name}_${side}_4_link">
         <origin xyz="-0.17011 0.02 -0.03711" rpy="0 -1.5708 0" />

File: pal_sea_arm_description/urdf/arm/arm_properties/humanoid/arm_cover.urdf.xacro (robot description, xacro)
@@ -24,5 +24,5 @@
       <geometry>
         <mesh
-          filename="package://kangaroo_description/meshes/arm_cover/arm_cover_link.stl" />
+          filename="package://pal_sea_arm_description/meshes/humanoid/arm_cover/arm_cover_link.stl" />
       </geometry>
       <material name="pal/DarkGrey"/>
@@ -31,5 +31,5 @@
       mujoco="${sim_type in ['mujoco-ros2-control', 'mujoco']}"
       collision_type="${collision_type}"
-      mesh_file="package://kangaroo_description/meshes/arm_cover/arm_cover_link_collision.stl"
+      mesh_file="package://pal_sea_arm_description/meshes/humanoid/arm_cover/arm_cover_link_collision.stl"
       scale="1 1 1">
       <properties>

File: pal_sea_arm_description/urdf/arm/arm_properties/humanoid/ros2_control.urdf.xacro (robot description, xacro)
@@ -15,5 +15,5 @@
   <!-- INCLUDES -->
   <xacro:include filename="$(find kangaroo_description)/ros2_control/joint.ros2_control.xacro" />
-  <xacro:include filename="$(find kangaroo_description)/ros2_control/transmissions.urdf.xacro" />
+  <xacro:include filename="$(find pal_sea_arm_description)/ros2_control/transmissions.urdf.xacro" />
   <!-- MACRO DEFINITION-->
   <xacro:macro name="arm_ros2_control" params="side arm_type">

File: pal_sea_arm_description/urdf/end_effector/humanoid/fake_forearm.urdf.xacro (robot description, xacro)
@@ -19,5 +19,5 @@
         <origin xyz="0 0 0" rpy="0 0 0" />
         <geometry>
-          <mesh filename="package://pal_sea_arm_description/meshes/humanoid/fake_forearm_${side}_link.stl" scale="1 1 1"/>
+          <mesh filename="package://pal_sea_arm_description/meshes/humanoid/arm/fake_forearm_${side}_link.stl" scale="1 1 1"/>
         </geometry>
         <material name="pal/DarkGrey" />
@@ -26,5 +26,5 @@
         mujoco="${sim_type in ['mujoco-ros2-control', 'mujoco']}"
         collision_type="${collision_type}"
-        mesh_file="package://pal_sea_arm_description/meshes/humanoid/fake_forearm_${side}_link.stl"
+        mesh_file="package://pal_sea_arm_description/meshes/humanoid/arm/fake_forearm_${side}_link.stl"
         scale="1 1 1"
         capsule_radius="0.054849043041257713"

File: pal_sea_arm_description/urdf/end_effector/humanoid/ros2_control.urdf.xacro (robot description, xacro)
@@ -15,9 +15,9 @@
   <!-- MACRO DEFINITION-->
   <xacro:macro name="end_effector_ros2_control" params="side end_effector_type">
-    <xacro:if value="${end_effector_type == 'gripper'}">
+    <xacro:if value="${end_effector_${side} == 'gripper'}">
       <xacro:include filename="$(find pal_pro_gripper_description)/urdf/gripper.ros2_control.xacro" />
       <xacro:ros2_control_pal_pro_gripper name="gripper_${side}" reduction="1.0"  sim_type="${sim_type}"/>
     </xacro:if>
-    <xacro:if value="${end_effector_type == 'RH8D'}">
+    <xacro:if value="${end_effector_${side} == 'RH8D'}">
       <xacro:include filename="$(find rh8d_description)/urdf/hand/ros2_control.urdf.xacro" />
       <xacro:hand_ros2_control side="${side}" mimic="${use_mimic}"/>

Commit message: Fix axis

File: pal_sea_arm_description/urdf/arm/arm_properties/humanoid/4dof_arm.urdf.xacro (robot description, xacro)
@@ -82,5 +82,5 @@
       <parent link="${name}_${side}_base_link" />
       <child link="${name}_${side}_1_link" />
-      <axis xyz="0 0 -1" />
+      <axis xyz="0 0 1" />
       <limit lower="${deg_to_rad * -150}" upper="${deg_to_rad * 150}" effort="${arm_1_max_effort}" velocity="${arm_1_max_velocity}" />
     </joint>
@@ -162,5 +162,5 @@
       <parent link="${name}_${side}_2_link" />
       <child link="${name}_${side}_3_link" />
-      <axis xyz="0 0 -1" />
+      <axis xyz="0 0 1" />
       <limit lower="${deg_to_rad * -150}" upper="${deg_to_rad * 150}" effort="${arm_3_max_effort}" velocity="${arm_3_max_velocity}" />
     </joint>

File: pal_sea_arm_description/urdf/arm/arm_properties/humanoid/7dof_arm.urdf.xacro (robot description, xacro)
@@ -81,5 +81,5 @@
       <parent link="${name}_${side}_5_link" />
       <child link="${name}_${side}_6_link" />
-      <axis xyz="0 0 -1" />
+      <axis xyz="0 0 1" />
       <limit lower="${deg_to_rad * -108}" upper="${deg_to_rad * 172}" effort="${arm_6_max_effort}" velocity="${arm_6_max_velocity}" />
     </joint>

Commit message: Match axis with ROS 1 version

File: pal_sea_arm_description/urdf/arm/arm_properties/humanoid/4dof_arm.urdf.xacro (robot description, xacro)
@@ -82,5 +82,5 @@
       <parent link="${name}_${side}_base_link" />
       <child link="${name}_${side}_1_link" />
-      <axis xyz="0 0 1" />
+      <axis xyz="0 0 -1" />
       <limit lower="${deg_to_rad * -150}" upper="${deg_to_rad * 150}" effort="${arm_1_max_effort}" velocity="${arm_1_max_velocity}" />
     </joint>
@@ -162,5 +162,5 @@
       <parent link="${name}_${side}_2_link" />
       <child link="${name}_${side}_3_link" />
-      <axis xyz="0 0 1" />
+      <axis xyz="0 0 -1" />
       <limit lower="${deg_to_rad * -150}" upper="${deg_to_rad * 150}" effort="${arm_3_max_effort}" velocity="${arm_3_max_velocity}" />
     </joint>

File: pal_sea_arm_description/urdf/arm/arm_properties/humanoid/7dof_arm.urdf.xacro (robot description, xacro)
@@ -81,5 +81,5 @@
       <parent link="${name}_${side}_5_link" />
       <child link="${name}_${side}_6_link" />
-      <axis xyz="0 0 1" />
+      <axis xyz="0 0 -1" />
       <limit lower="${deg_to_rad * -108}" upper="${deg_to_rad * 172}" effort="${arm_6_max_effort}" velocity="${arm_6_max_velocity}" />
     </joint>

Commit message: Change fakeforearm to 4dof without end effector

File: pal_sea_arm_description/urdf/arm/arm_properties/humanoid/4dof_arm.urdf.xacro (robot description, xacro)
@@ -4,7 +4,9 @@
   <xacro:property name="arm_2_max_velocity"      value="1.95" />
   <xacro:property name="arm_3_max_velocity"      value="2.35" />
+  <xacro:property name="arm_4_max_velocity"      value="2.35" />
   <xacro:property name="arm_1_max_effort"   value="43.0" />
   <xacro:property name="arm_2_max_effort"   value="43.0" />
   <xacro:property name="arm_3_max_effort"   value="43.0" />
+  <xacro:property name="arm_4_max_effort"   value="43.0" />
   <xacro:macro name="kangaroo_4dof_arm" params="name side reflect parent *origin arm_1_offset:=0.0 arm_2_offset:=0.0 arm_3_offset:=0.0 arm_4_offset:=0.0">
     <link name="${name}_${side}_base_link">
@@ -165,4 +167,53 @@
       <limit lower="${deg_to_rad * -150}" upper="${deg_to_rad * 150}" effort="${arm_3_max_effort}" velocity="${arm_3_max_velocity}" />
     </joint>
+    <link name="${name}_${side}_4_link">
+        <inertial>
+          <origin xyz="-0.03711 -0.02 -0.17011" rpy="3.14159 1.5708 0" />
+          <mass value="1.4353488" />
+          <inertia
+            ixx="0.0012553"
+            ixy="-0.0012835"
+            ixz="9.49E-05"
+            iyy="0.0209442"
+            iyz="-1.1E-06"
+            izz="0.0210127" />
+        </inertial>
+        <visual>
+          <origin xyz="0 0 0" rpy="0 0 0" />
+          <geometry>
+            <mesh filename="package://pal_sea_arm_description/meshes/humanoid/arm/fake_forearm_${side}_link.stl" scale="1 1 1"/>
+          </geometry>
+          <material name="pal/DarkGrey" />
+        </visual>
+        <xacro:link_collision
+          mujoco="${sim_type in ['mujoco-ros2-control', 'mujoco']}"
+          collision_type="${collision_type}"
+          mesh_file="package://pal_sea_arm_description/meshes/humanoid/arm/fake_forearm_${side}_link.stl"
+          scale="1 1 1"
+          capsule_radius="0.054849043041257713"
+          capsule_length="0.43843343404800533">
+            <properties>
+              <xacro:origin xyz="0 0 0" rpy="0 0 0" condition="${collision_type == 'mesh'}"/>
+              <!-- Fake forearm capsule origin/rotation definition -->
+              <xacro:if value="${side == 'left'}">
+                <xacro:origin xyz="0.210246 -0.0167497 -0.0171982" rpy="0.805655 1.46244 0.73029" condition="${collision_type == 'capsule'}"/>
+              </xacro:if>
+              <xacro:if value="${side == 'right'}">
+                <xacro:origin xyz="0.210649 -0.0172373 -0.0265895" rpy="1.18814 1.49122 1.11539" condition="${collision_type == 'capsule'}"/>
+              </xacro:if>
+            </properties>
+        </xacro:link_collision>
+      </link>
+      <joint name="${name}_${side}_4_joint" type="revolute">
+        <origin xyz="-0.03711 -0.02 -0.17011" rpy="3.14159 1.5708 0" />
+        <parent link="${name}_${side}_3_link" />
+        <child link="${name}_${side}_4_link" />
+        <axis xyz="0 0 1" />
+        <limit
+          lower="-1.1345"
+          upper="2.4435"
+          effort="${arm_4_max_effort}"
+          velocity="${arm_4_max_velocity}" />
+      </joint>
   </xacro:macro>
 </robot>

Commit message: Add condition for 4dof arm without ee

File: pal_sea_arm_description/urdf/arm/arm_properties/humanoid/4dof_arm.urdf.xacro (robot description, xacro)
@@ -9,5 +9,5 @@
   <xacro:property name="arm_3_max_effort"   value="43.0" />
   <xacro:property name="arm_4_max_effort"   value="43.0" />
-  <xacro:macro name="kangaroo_4dof_arm" params="name side reflect parent *origin arm_1_offset:=0.0 arm_2_offset:=0.0 arm_3_offset:=0.0 arm_4_offset:=0.0">
+  <xacro:macro name="kangaroo_4dof_arm" params="name side reflect parent *origin arm_type:='4dof' arm_1_offset:=0.0 arm_2_offset:=0.0 arm_3_offset:=0.0 arm_4_offset:=0.0">
     <link name="${name}_${side}_base_link">
       <inertial>
@@ -167,5 +167,6 @@
       <limit lower="${deg_to_rad * -150}" upper="${deg_to_rad * 150}" effort="${arm_3_max_effort}" velocity="${arm_3_max_velocity}" />
     </joint>
-    <link name="${name}_${side}_4_link">
+    <xacro:if value="${arm_type == '4dof'}">
+      <link name="${name}_${side}_4_link">
         <inertial>
           <origin xyz="-0.03711 -0.02 -0.17011" rpy="3.14159 1.5708 0" />
@@ -216,4 +217,5 @@
           velocity="${arm_4_max_velocity}" />
       </joint>
+    </xacro:if>
   </xacro:macro>
 </robot>

File: pal_sea_arm_description/urdf/arm/arm_properties/humanoid/arm.urdf.xacro (robot description, xacro)
@@ -5,5 +5,5 @@
     <xacro:if value="${type in ['4dof', '5dof', '7dof']}">
       <xacro:include filename="$(find pal_sea_arm_description)/urdf/arm/arm_properties/humanoid/4dof_arm.urdf.xacro" />
-      <xacro:kangaroo_4dof_arm name="${name}" side="${side}" reflect="${reflect}" parent="${parent}">
+      <xacro:kangaroo_4dof_arm name="${name}" side="${side}" reflect="${reflect}" parent="${parent}" arm_type="${type}">
         <xacro:insert_block name="origin"/>
       </xacro:kangaroo_4dof_arm>

Commit message: Remove rotation from arm link 4 inertia

File: pal_sea_arm_description/urdf/arm/arm_properties/humanoid/4dof_arm.urdf.xacro (robot description, xacro)
@@ -170,5 +170,5 @@
       <link name="${name}_${side}_4_link">
         <inertial>
-          <origin xyz="-0.03711 -0.02 -0.17011" rpy="3.14159 1.5708 0" />
+          <origin xyz="0.17011 0.02 -0.03711" rpy="0 0 0" />
           <mass value="1.4353488" />
           <inertia

Commit message: Arm link 4 : use same inertia origin as old fake-forearm link

File: pal_sea_arm_description/urdf/arm/arm_properties/humanoid/4dof_arm.urdf.xacro (robot description, xacro)
@@ -170,5 +170,5 @@
       <link name="${name}_${side}_4_link">
         <inertial>
-          <origin xyz="0.17011 0.02 -0.03711" rpy="0 0 0" />
+          <origin xyz="0.0752641 -0.0079317 -0.023427" rpy="0 0 0" />
           <mass value="1.4353488" />
           <inertia
