Commit message: Change parameter and naming

File: pal_sea_arm_description/robots/pal_sea_arm.urdf.xacro (robot description, xacro)
@@ -54,5 +54,5 @@
       <origin xyz="0 0 0" rpy="0 0 0" />
       <geometry>
-        <mesh filename="package://pal_sea_arm_description/meshes/base_link.STL" />
+        <mesh filename="package://pal_sea_arm_description/meshes/arm_tiago_pro/base_link.stl" />
       </geometry>
       <material name="">
@@ -63,5 +63,5 @@
       <origin xyz="0 0 0" rpy="0 0 0" />
       <geometry>
-        <mesh filename="package://pal_sea_arm_description/meshes/base_link.STL" />
+        <mesh filename="package://pal_sea_arm_description/meshes/arm_tiago_pro/base_link.stl" />
       </geometry>
     </collision>

File: pal_sea_arm_description/urdf/arm/arm.urdf.xacro (robot description, xacro)
@@ -15,8 +15,9 @@
   <!-- Transmissions file -->
   <xacro:include filename="$(find pal_sea_arm_description)/urdf/arm/arm.transmission.xacro"/>
-  <xacro:macro name="pal_sea_arm" params="name parent *origin arm_model reflect arm_1_offset arm_2_offset arm_3_offset arm_4_offset arm_5_offset arm_6_offset arm_7_offset no_safety_eps:=False">
+  <xacro:macro name="pal_sea_arm" params="name parent *origin arm_model reflect arm_1_offset arm_2_offset arm_3_offset arm_4_offset arm_5_offset arm_6_offset arm_7_offset
+                                          no_safety_eps:=False joint_limits_file:='$(find pal_sea_arm_description)/urdf/arm/limits/arm_${arm_model}.limits.xacro'">
     <xacro:property name="arm_eps"       value="${0.00 if no_safety_eps else 0.07}"/>
     <!-- Joint Limits file -->
-    <xacro:include filename="$(find pal_sea_arm_description)/urdf/arm/arm_${arm_model}.limits.xacro"/>
+    <xacro:include filename="${joint_limits_file}"/>
     <xacro:if value="${arm_model in ['tiago-pro', 'pal-sea-arm-standalone']}">
       <!-- ARM 1 LINK -->
@@ -357,5 +358,5 @@
           <origin xyz="0 0 0" rpy="0 0 0" />
           <geometry>
-            <mesh filename="package://pal_sea_arm_description/meshes/base_link.STL" />
+            <mesh filename="package://pal_sea_arm_description/meshes/arm_tiago_sea/base_link.stl" />
           </geometry>
           <material name="">
@@ -366,5 +367,5 @@
           <origin xyz="0 0 0" rpy="0 0 0" />
           <geometry>
-            <mesh filename="package://pal_sea_arm_description/meshes/base_link.STL" />
+            <mesh filename="package://pal_sea_arm_description/meshes/arm_tiago_sea/base_link.stl" />
           </geometry>
         </collision>
@@ -388,5 +389,5 @@
           <origin xyz="0 0 0" rpy="0 0 0" />
           <geometry>
-            <mesh filename="package://pal_sea_arm_description/meshes/arm/arm_1_link.STL"
+            <mesh filename="package://pal_sea_arm_description/meshes/arm_tiago_sea/arm_1_link.stl"
               scale="1 1 ${reflect}" />
           </geometry>
@@ -401,5 +402,5 @@
           <geometry>
             <mesh
-              filename="package://pal_sea_arm_description/meshes/arm/arm_1_link_convex.STL"
+              filename="package://pal_sea_arm_description/meshes/arm_tiago_sea/arm_1_link_convex.stl"
               scale="1 1 ${reflect}" />
           </geometry>
@@ -431,5 +432,5 @@
           <origin xyz="0 0 0" rpy="0 0 0" />
           <geometry>
-            <mesh filename="package://pal_sea_arm_description/meshes/arm/arm_2_link.STL"
+            <mesh filename="package://pal_sea_arm_description/meshes/arm_tiago_sea/arm_2_link.stl"
               scale="1 1 ${reflect}" />
           </geometry>
@@ -444,5 +445,5 @@
           <geometry>
             <mesh
-              filename="package://pal_sea_arm_description/meshes/arm/arm_2_link_convex.STL"
+              filename="package://pal_sea_arm_description/meshes/arm_tiago_sea/arm_2_link_convex.stl"
               scale="1 1 ${reflect}" />
           </geometry>
@@ -475,5 +476,5 @@
           <origin xyz="0 0 0" rpy="0 0 0" />
           <geometry>
-            <mesh filename="package://pal_sea_arm_description/meshes/arm/arm_3_link.STL"
+            <mesh filename="package://pal_sea_arm_description/meshes/arm_tiago_sea/arm_3_link.stl"
               scale="1 1 ${reflect}" />
           </geometry>
@@ -488,5 +489,5 @@
           <geometry>
             <mesh
-              filename="package://pal_sea_arm_description/meshes/arm/arm_3_link_convex.STL"
+              filename="package://pal_sea_arm_description/meshes/arm_tiago_sea/arm_3_link_convex.stl"
               scale="1 1 ${reflect}" />
           </geometry>
@@ -521,5 +522,5 @@
           <origin xyz="0 0 0" rpy="0 0 0" />
           <geometry>
-            <mesh filename="package://pal_sea_arm_description/meshes/arm/arm_4_link.STL"
+            <mesh filename="package://pal_sea_arm_description/meshes/arm_tiago_sea/arm_4_link.stl"
               scale="1 1 ${reflect}" />
           </geometry>
@@ -534,5 +535,5 @@
           <geometry>
             <mesh
-              filename="package://pal_sea_arm_description/meshes/arm/arm_4_link_convex.STL"
+              filename="package://pal_sea_arm_description/meshes/arm_tiago_sea/arm_4_link_convex.stl"
               scale="1 1 ${reflect}" />
           </geometry>
@@ -567,5 +568,5 @@
           <origin xyz="0 0 0" rpy="0 0 0" />
           <geometry>
-            <mesh filename="package://pal_sea_arm_description/meshes/arm/arm_5_link.STL"
+            <mesh filename="package://pal_sea_arm_description/meshes/arm_tiago_sea/arm_5_link.stl"
               scale="1 1 ${reflect}" />
           </geometry>
@@ -580,5 +581,5 @@
           <geometry>
             <mesh
-              filename="package://pal_sea_arm_description/meshes/arm/arm_5_link_convex.STL"
+              filename="package://pal_sea_arm_description/meshes/arm_tiago_sea/arm_5_link_convex.stl"
               scale="1 1 ${reflect}" />
           </geometry>
@@ -613,5 +614,5 @@
           <origin xyz="0 0 0" rpy="0 0 0" />
           <geometry>
-            <mesh filename="package://pal_sea_arm_description/meshes/arm/arm_6_link.STL"
+            <mesh filename="package://pal_sea_arm_description/meshes/arm_tiago_sea/arm_6_link.stl"
               scale="1 1 ${reflect}" />
           </geometry>
@@ -626,5 +627,5 @@
           <geometry>
             <mesh
-              filename="package://pal_sea_arm_description/meshes/arm/arm_6_link_convex.STL"
+              filename="package://pal_sea_arm_description/meshes/arm_tiago_sea/arm_6_link_convex.stl"
               scale="1 1 ${reflect}" />
           </geometry>
@@ -659,5 +660,5 @@
           <origin xyz="0 0 0" rpy="0 0 0" />
           <geometry>
-            <mesh filename="package://pal_sea_arm_description/meshes/arm/arm_7_link.STL"
+            <mesh filename="package://pal_sea_arm_description/meshes/arm_tiago_sea/arm_7_link.stl"
               scale="1 1 ${reflect}" />
           </geometry>
@@ -672,5 +673,5 @@
           <geometry>
             <mesh
-              filename="package://pal_sea_arm_description/meshes/arm/arm_7_link_convex.STL"
+              filename="package://pal_sea_arm_description/meshes/arm_tiago_sea/arm_7_link_convex.stl"
               scale="1 1 ${reflect}" />
           </geometry>
