Commit message: Extract inertial and joints parameters to fusion both urdf

File: pal_sea_arm_description/robots/pal_sea_arm.urdf.xacro (robot description, xacro)
@@ -19,5 +19,5 @@
   <xacro:arg name="end_effector" default="false"/>
   <xacro:arg name="ft_sensor" default="false"/>
-  <xacro:arg name="arm_model" default="tiago-pro"/>
+  <xacro:arg name="arm_model" default="pal-sea-arm-standalone"/>
   <xacro:property name="end_effector" value="$(arg end_effector)" />
   <xacro:property name="ft_sensor" value="$(arg ft_sensor)" />

File: pal_sea_arm_description/urdf/arm/arm.urdf.xacro (robot description, xacro)
@@ -15,704 +15,310 @@
   <!-- Transmissions file -->
   <xacro:include filename="$(find pal_sea_arm_description)/urdf/arm/arm.transmission.xacro"/>
-  <xacro:macro name="pal_sea_arm" params="name parent *origin arm_model reflect arm_1_offset arm_2_offset arm_3_offset arm_4_offset arm_5_offset arm_6_offset arm_7_offset
-                                          no_safety_eps:=False joint_limits_file:='$(find pal_sea_arm_description)/urdf/arm/limits/arm_${arm_model}.limits.xacro'">
+  <xacro:macro name="pal_sea_arm" params="name parent *origin arm_model reflect:=1 arm_1_offset arm_2_offset arm_3_offset arm_4_offset arm_5_offset arm_6_offset arm_7_offset
+                                          no_safety_eps:=False joint_limits_file:='$(find pal_sea_arm_description)/urdf/arm/limits/arm_${arm_model}.limits.xacro'
+                                          arm_properties_file:='$(find pal_sea_arm_description)/urdf/arm/arm_properties/arm_${arm_model}.properties.xacro'">
     <xacro:property name="arm_eps"       value="${0.00 if no_safety_eps else 0.07}"/>
     <!-- Joint Limits file -->
     <xacro:include filename="${joint_limits_file}"/>
+    <xacro:include filename="${arm_properties_file}"/>
+    <xacro:property name="mesh_folder"/>
     <xacro:if value="${arm_model in ['tiago-pro', 'pal-sea-arm-standalone']}">
-      <!-- ARM 1 LINK -->
-      <link name="${name}_1_link">
-        <inertial>
-          <origin
-            xyz="0.0023908 0.015901 0.1545"
-            rpy="0 0 0" />
-          <mass
-            value="1.0816" />
-          <inertia
-            ixx="0.0024426"
-            ixy="2.3307E-05"
-            ixz="5.9333E-05"
-            iyy="0.0023089"
-            iyz="-0.00020369"
-            izz="0.00092843" />
-        </inertial>
-        <visual>
-          <origin xyz="0 0 0" rpy="0 0 0" />
-          <geometry>
-            <mesh
-              filename="package://pal_sea_arm_description/meshes/arm_tiago_pro/arm_1_link.stl" />
-          </geometry>
-          <material name="">
-            <color rgba="0.29804 0.29804 0.29804 1" />
-          </material>
-        </visual>
-        <collision>
-          <origin xyz="0 0 0" rpy="0 0 0" />
-          <geometry>
-            <mesh filename="package://pal_sea_arm_description/meshes/arm_tiago_pro/arm_1_link_collision.stl" />
-          </geometry>
-        </collision>
-      </link>
-      <joint name="${name}_1_joint" type="revolute">
-        <xacro:insert_block name="origin"/>
-        <parent link="${parent}" />
-        <child link="${name}_1_link" />
-        <axis xyz="0 0 1" />
-        <limit lower="${arm_1_joint_lb}" upper="${arm_1_joint_ub}" effort="${arm_1_max_effort}" velocity="${arm_1_max_velocity}" />
-      </joint>
-      <!-- ARM 2 LINK -->
-      <link name="${name}_2_link">
-        <inertial>
-          <origin
-            xyz="-0.11649 -0.017864 0.0053772"
-            rpy="0 0 0" />
-          <mass
-            value="0.99204" />
-          <inertia
-            ixx="0.00077294"
-            ixy="-0.00011001"
-            ixz="-0.00016136"
-            iyy="0.0014605"
-            iyz="-1.3224E-05"
-            izz="0.0015605" />
-        </inertial>
-        <visual>
-          <origin xyz="0 0 0" rpy="0 0 0" />
-          <geometry>
-            <mesh filename="package://pal_sea_arm_description/meshes/arm_tiago_pro/arm_2_link.stl" />
-          </geometry>
-          <material name="">
-            <color rgba="0.29804 0.29804 0.29804 1" />
-          </material>
-        </visual>
-        <collision>
-          <origin xyz="0 0 0" rpy="0 0 0" />
-          <geometry>
-            <mesh filename="package://pal_sea_arm_description/meshes/arm_tiago_pro/arm_2_link_collision.stl" />
-          </geometry>
-        </collision>
-      </link>
-      <!-- ARM 2 JOINT -->
-      <joint name="${name}_2_joint" type="revolute">
-        <origin xyz="0.0 0.02 0.18" rpy="0 1.5708 0" />
-        <parent link="${name}_1_link" />
-        <child link="${name}_2_link" />
-        <axis xyz="0 0 1" />
-        <limit lower="${arm_2_joint_lb}" upper="${arm_2_joint_ub}" effort="${arm_2_max_effort}" velocity="${arm_2_max_velocity}" />
-      </joint>
-      <!-- ARM 3 LINK -->
-      <link name="${name}_3_link">
-        <inertial>
-          <origin
-            xyz="0.0023908 0.015901 0.1545"
-            rpy="0 0 0" />
-          <mass
-            value="1.0816" />
-          <inertia
-            ixx="0.0024426"
-            ixy="2.3307E-05"
-            ixz="5.9333E-05"
-            iyy="0.0023089"
-            iyz="-0.00020369"
-            izz="0.00092843" />
-        </inertial>
-        <visual>
-          <origin xyz="0 0 0" rpy="0 0 0" />
-          <geometry>
-            <mesh filename="package://pal_sea_arm_description/meshes/arm_tiago_pro/arm_3_link.stl" />
-          </geometry>
-          <material name="">
-            <color rgba="0.29804 0.29804 0.29804 1" />
-          </material>
-        </visual>
-        <collision>
-          <origin xyz="0 0 0" rpy="0 0 0" />
-          <geometry>
-            <mesh filename="package://pal_sea_arm_description/meshes/arm_tiago_pro/arm_3_link_collision.stl" />
-          </geometry>
-        </collision>
-      </link>
-      <!-- ARM 3 JOINT -->
-      <joint name="${name}_3_joint" type="revolute">
-        <origin
-        xyz="-0.15 -0.02 0"
-        rpy="3.1415 1.5707 0" />
-        <parent link="${name}_2_link" />
-        <child link="${name}_3_link" />
-        <axis xyz="0 0 1" />
-        <limit lower="${arm_3_joint_lb}" upper="${arm_3_joint_ub}" effort="${arm_3_max_effort}" velocity="${arm_3_max_velocity}" />
-      </joint>
-      <!-- ARM 4 LINK -->
-      <link name="${name}_4_link">
-        <inertial>
-          <origin
-            xyz="-0.11649 -0.017864 0.0053772"
-            rpy="0 0 0" />
-          <mass
-            value="0.99204" />
-          <inertia
-            ixx="0.00077294"
-            ixy="-0.00011001"
-            ixz="-0.00016136"
-            iyy="0.0014605"
-            iyz="-1.3224E-05"
-            izz="0.0015605" />
-        </inertial>
-        <visual>
-          <origin xyz="0 0 0" rpy="0 0 0" />
-          <geometry>
-            <mesh filename="package://pal_sea_arm_description/meshes/arm_tiago_pro/arm_4_link.stl" />
-          </geometry>
-          <material name="">
-            <color rgba="0.29804 0.29804 0.29804 1" />
-          </material>
-        </visual>
-        <collision>
-          <origin xyz="0 0 0" rpy="0 0 0" />
-          <geometry>
-            <mesh filename="package://pal_sea_arm_description/meshes/arm_tiago_pro/arm_4_link_collision.stl" />
-          </geometry>
-        </collision>
-      </link>
-      <!-- ARM 4 JOINT -->
-      <joint name="${name}_4_joint" type="revolute">
-        <origin xyz="0 0.02 0.18" rpy="0 1.5708 0" />
-        <parent link="${name}_3_link" />
-        <child link="${name}_4_link" />
-        <axis xyz="0 0 -1" />
-        <limit lower="${arm_4_joint_lb}" upper="${arm_4_joint_ub}" effort="${arm_4_max_effort}" velocity="${arm_4_max_velocity}" />
-      </joint>
-      <!-- ARM 5 LINK -->
-      <link name="${name}_5_link">
-        <inertial>
-          <origin
-            xyz="0.0004859 0.00014289 0.129"
-            rpy="0 0 0" />
-          <mass
-            value="0.52538" />
-          <inertia
-            ixx="0.0019111"
-            ixy="-1.4245E-08"
-            ixz="3.8663E-05"
-            iyy="0.0018565"
-            iyz="1.1356E-06"
-            izz="0.00046496" />
-        </inertial>
-        <visual>
-          <origin xyz="0 0 0" rpy="0 0 0" />
-          <geometry>
-            <mesh filename="package://pal_sea_arm_description/meshes/arm_tiago_pro/arm_5_link.stl" />
-          </geometry>
-          <material name="">
-            <color rgba="0.29804 0.29804 0.29804 1" />
-          </material>
-        </visual>
-        <collision>
-          <origin xyz="0 0 0" rpy="0 0 0" />
-          <geometry>
-            <mesh filename="package://pal_sea_arm_description/meshes/arm_tiago_pro/arm_5_link_collision.stl" />
-          </geometry>
-        </collision>
-      </link>
-      <!-- ARM 5 JOINT -->
-      <joint name="${name}_5_joint" type="revolute">
-        <origin xyz="-0.15 -0.02 0" rpy="0 -1.5708 0" />
-        <parent link="${name}_4_link" />
-        <child link="${name}_5_link" />
-        <axis xyz="0 0 1" />
-        <limit lower="${arm_5_joint_lb}" upper="${arm_5_joint_ub}" effort="${arm_5_max_effort}" velocity="${arm_5_max_velocity}" />
-      </joint>
-      <!-- ARM 6 LINK -->
-      <link name="${name}_6_link">
-        <inertial>
-          <origin
-            xyz="-0.086822 -7.7905E-06 0.0045258"
-            rpy="0 0 0" />
-          <mass
-            value="0.66725" />
-          <inertia
-            ixx="0.00035696"
-            ixy="1.6019E-07"
-            ixz="-9.5191E-05"
-            iyy="0.00073846"
-            iyz="2.118E-08"
-            izz="0.00075321" />
-        </inertial>
-        <visual>
-          <origin xyz="0 0 0" rpy="0 0 0" />
-          <geometry>
-            <mesh filename="package://pal_sea_arm_description/meshes/arm_tiago_pro/arm_6_link.stl" />
-          </geometry>
-          <material name="">
-            <color rgba="0.29804 0.29804 0.29804 1" />
-          </material>
-        </visual>
-        <collision>
-          <origin xyz="0 0 0" rpy="0 0 0" />
-          <geometry>
-            <mesh filename="package://pal_sea_arm_description/meshes/arm_tiago_pro/arm_6_link_collision.stl" />
-          </geometry>
-        </collision>
-      </link>
-      <!-- ARM 6 JOINT -->
-      <joint name="${name}_6_joint" type="revolute">
-        <origin xyz="0 0 0.185" rpy="0 1.5708 0" />
-        <parent link="${name}_5_link" />
-        <child link="${name}_6_link" />
-        <axis xyz="0 0 1" />
-        <limit lower="${arm_6_joint_lb}" upper="${arm_6_joint_ub}" effort="${arm_6_max_effort}" velocity="${arm_6_max_velocity}" />
-      </joint>
-      <!-- ARM 7 LINK -->
-      <link name="${name}_7_link">
-        <inertial>
-          <origin
-            xyz="-6.764E-18 -1.4549E-16 0.018549"
-            rpy="0 0 0" />
-          <mass
-            value="0.10189" />
-          <inertia
-            ixx="5.1076E-05"
-            ixy="-1.0899E-21"
-            ixz="-5.93E-21"
-            iyy="5.0882E-05"
-            iyz="-8.5344E-21"
-            izz="9.705E-05" />
-        </inertial>
-        <visual>
-          <origin xyz="0 0 0" rpy="0 0 0" />
-          <geometry>
-            <mesh filename="package://pal_sea_arm_description/meshes/arm_tiago_pro/arm_7_link.stl" />
-          </geometry>
-          <material name="">
-            <color rgba="0.29804 0.29804 0.29804 1" />
-          </material>
-        </visual>
-        <collision>
-          <origin xyz="0 0 0" rpy="0 0 0" />
-          <geometry>
-            <mesh filename="package://pal_sea_arm_description/meshes/arm_tiago_pro/arm_7_link_collision.stl" />
-          </geometry>
-        </collision>
-      </link>
-      <!-- ARM 7 JOINT -->
-      <joint name="${name}_7_joint" type="revolute">
-        <origin
-        xyz="-0.1166 0 0"
-        rpy="0 -1.5708 0" />
-        <parent link="${name}_6_link" />
-        <child link="${name}_7_link" />
-        <axis xyz="0 0 1" />
-        <limit lower="${arm_7_joint_lb}" upper="${arm_7_joint_ub}" effort="${arm_7_max_effort}" velocity="${arm_7_max_velocity}" />
-      </joint>
-      <!--***********************-->
-      <!--        TOOL           -->
-      <!--***********************-->
-      <link name="${name}_tool_link">
-        <inertial>
-          <origin
-            xyz="5.0493E-18 -4.4892E-17 -0.0068514"
-            rpy="0 0 0" />
-          <mass value="0.10189" />
-          <inertia
-            ixx="5.1076E-05"
-            ixy="-1.0374E-21"
-            ixz="-5.9164E-21"
-            iyy="5.0882E-05"
-            iyz="-8.5211E-21"
-            izz="9.705E-05" />
-        </inertial>
-        <visual>
-          <origin xyz="0.001 0 0" rpy="0 1.5708 0" />
-          <geometry>
-            <cylinder radius="0.005" length="0.005"/>
-          </geometry>
-          <material name="">
-            <color rgba="0.29804 0.29804 0.29804 1" />
-          </material>
-        </visual>
-        <collision>
-          <origin xyz="0.001 0 0" rpy="0 1.5708 0" />
-          <geometry>
-            <cylinder radius="0.005" length="0.005"/>
-          </geometry>
-        </collision>
-      </link>
-      <joint name="${name}_tool_joint" type="fixed">
-        <parent link="${name}_7_link" />
-        <child link="${name}_tool_link" />
-          <origin xyz="0 0 0.0184" rpy="0 ${-90.0 * deg_to_rad} ${90.0 * deg_to_rad}" />
-      </joint>
+      <xacro:property name="mesh_folder"       value="arm_tiago_pro"/>
     </xacro:if>
     <xacro:if value="${arm_model in ['tiago-sea', 'tiago-sea-dual']}">
-      <!-- ARM 1 LINK -->
-      <link name="${name}_1_link">
-        <inertial>
-          <origin xyz="0.1082 0.0106 ${0.0328 * reflect}" rpy="0 0 0" />
-          <mass value="1.0267" />
-        <inertia
-          ixx="8.0603E-04" ixy="-8.52034E-05" ixz="${-3.0124E-04 * reflect}"
-          iyy="1.9301E-03" iyz="${1.9426E-05 * reflect}"
-          izz="1.8484E-03" />
-        </inertial>
-        <visual>
-          <origin xyz="0 0 0" rpy="0 0 0" />
-          <geometry>
-            <mesh filename="package://pal_sea_arm_description/meshes/arm_tiago_sea/arm_1_link.stl"
-              scale="1 1 ${reflect}" />
-          </geometry>
-          <material
-            name="">
-            <color
-              rgba="0.752941176470588 0.752941176470588 0.752941176470588 1" />
-          </material>
-        </visual>
-        <collision>
-          <origin xyz="0 0 0" rpy="0 0 0" />
-          <geometry>
-            <mesh
-              filename="package://pal_sea_arm_description/meshes/arm_tiago_sea/arm_1_link_convex.stl"
-              scale="1 1 ${reflect}" />
-          </geometry>
-        </collision>
-      </link>
-      <!-- ARM 1 JOINT -->
-      <joint name="${name}_1_joint" type="revolute">
-        <xacro:insert_block name="origin" />
-        <parent link="${parent}" />
-        <child link="${name}_1_link" />
-        <axis xyz="0 0 ${1}" />
-        <limit lower="${arm_1_joint_lb * deg_to_rad}" upper="${arm_1_joint_ub * deg_to_rad}" effort="${arm_1_max_effort}" velocity="${arm_1_max_velocity}" />
-        <dynamics friction="${arm_friction}" damping="${arm_damping}"/>
-        <safety_controller k_position="${arm_k_position}" k_velocity="${arm_k_velocity}" soft_lower_limit="${arm_1_joint_lb * deg_to_rad  + arm_eps}"
-          soft_upper_limit="${arm_1_joint_ub * deg_to_rad - arm_eps}" />
-      </joint>
-      <!-- ARM 2 LINK -->
-      <link name="${name}_2_link">
-        <inertial>
-          <origin xyz="-0.0941 2.6612E-04  ${0.0414 * reflect}" rpy="0 0 0" />
-          <mass value="0.9496" />
-          <inertia
-            ixx="8.4202E-04" ixy="-5.7830E-06" ixz="${2.6145E-04 * reflect}"
-            iyy="1.4185E-03" iyz="${-5.8148E-06 * reflect}"
-            izz="1.4729E-03" />
-        </inertial>
-        <visual>
-          <origin xyz="0 0 0" rpy="0 0 0" />
-          <geometry>
-            <mesh filename="package://pal_sea_arm_description/meshes/arm_tiago_sea/arm_2_link.stl"
-              scale="1 1 ${reflect}" />
-          </geometry>
-          <material
-            name="">
-            <color
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
File: pal_sea_arm_description/urdf/arm/limits/arm_pal-sea-arm-standalone.limits.xacro (robot description, xacro)
@@ -5,18 +5,18 @@
   <xacro:property name="arm_k_position" value="20"/>
   <xacro:property name="arm_k_velocity" value="20"/>
-  <xacro:property name="arm_1_joint_ub" value="2.6" />
-  <xacro:property name="arm_1_joint_lb" value="-2.6" />
-  <xacro:property name="arm_2_joint_ub" value="1.10" />
-  <xacro:property name="arm_2_joint_lb" value="-2.44" />
-  <xacro:property name="arm_3_joint_ub" value="2.6" />
-  <xacro:property name="arm_3_joint_lb" value="-2.6" />
-  <xacro:property name="arm_4_joint_ub" value="2.44" />
-  <xacro:property name="arm_4_joint_lb" value="-1.1" />
-  <xacro:property name="arm_5_joint_ub" value="2.6" />
-  <xacro:property name="arm_5_joint_lb" value="-2.6" />
-  <xacro:property name="arm_6_joint_ub" value="2.0" />
-  <xacro:property name="arm_6_joint_lb" value="-2.0" />
-  <xacro:property name="arm_7_joint_ub" value="2.6" />
-  <xacro:property name="arm_7_joint_lb" value="-2.6" />
+  <xacro:property name="arm_1_joint_ub" value="148.97" />
+  <xacro:property name="arm_1_joint_lb" value="-148.97" />
+  <xacro:property name="arm_2_joint_ub" value="63.03" />
+  <xacro:property name="arm_2_joint_lb" value="-139.8" />
+  <xacro:property name="arm_3_joint_ub" value="148.97" />
+  <xacro:property name="arm_3_joint_lb" value="-148.97" />
+  <xacro:property name="arm_4_joint_ub" value="139.8" />
+  <xacro:property name="arm_4_joint_lb" value="-63.03" />
+  <xacro:property name="arm_5_joint_ub" value="148.97" />
+  <xacro:property name="arm_5_joint_lb" value="-148.97" />
+  <xacro:property name="arm_6_joint_ub" value="114.59" />
+  <xacro:property name="arm_6_joint_lb" value="-114.59" />
+  <xacro:property name="arm_7_joint_ub" value="148.97" />
+  <xacro:property name="arm_7_joint_lb" value="-148.97" />
   <xacro:property name="arm_1_max_velocity"      value="1.95" />
   <xacro:property name="arm_2_max_velocity"      value="1.95" />

Commit message: Address comments + fix colors

File: pal_sea_arm_description/robots/pal_sea_arm.urdf.xacro (robot description, xacro)
@@ -13,4 +13,7 @@
 -->
 <robot xmlns:xacro="http://ros.org/wiki/xacro" name="pal_sea_arm">
+  <!--File includes-->
+  <xacro:include filename="$(find pal_urdf_utils)/urdf/deg_to_rad.xacro" />
+  <xacro:include filename="$(find pal_urdf_utils)/urdf/materials.urdf.xacro" />
   <xacro:include filename="$(find pal_sea_arm_description)/urdf/arm/arm.urdf.xacro"/>
   <xacro:include filename="$(find pal_sea_arm_description)/urdf/end_effector/end_effector.urdf.xacro"/>
@@ -56,7 +59,5 @@
         <mesh filename="package://pal_sea_arm_description/meshes/arm_tiago_pro/base_link.stl" />
       </geometry>
-      <material name="">
-        <color rgba="0.29804 0.29804 0.29804 1" />
-      </material>
+      <material name="pal/DarkGrey"/>
     </visual>
     <collision>
@@ -67,4 +68,9 @@
     </collision>
   </link>
+  <gazebo reference="arm_root_link">
+    <material>Gazebo/DarkGrey</material>
+    <mu1>0.9</mu1>
+    <mu2>0.9</mu2>
+  </gazebo>
   <!-- ARM -->
   <xacro:pal_sea_arm name="arm" parent="arm_root_link" arm_model="${arm_model}" reflect="1" arm_1_offset="0" arm_2_offset="0" arm_3_offset="0" arm_4_offset="0" arm_5_offset="0" arm_6_offset="0" arm_7_offset="0">

File: pal_sea_arm_description/urdf/arm/arm.urdf.xacro (robot description, xacro)
@@ -39,7 +39,5 @@
             scale="1 1 ${reflect}" />
         </geometry>
-        <material name="">
-          <color rgba="0.29804 0.29804 0.29804 1" />
-        </material>
+        <material name="pal/DarkGrey"/>
       </visual>
       <collision>
@@ -71,7 +69,5 @@
           scale="1 1 ${reflect}" />
         </geometry>
-        <material name="">
-          <color rgba="0.29804 0.29804 0.29804 1" />
-        </material>
+        <material name="pal/DarkGrey"/>
       </visual>
       <collision>
@@ -103,7 +99,5 @@
           scale="1 1 ${reflect}" />
         </geometry>
-        <material name="">
-          <color rgba="0.29804 0.29804 0.29804 1" />
-        </material>
+        <material name="pal/DarkGrey"/>
       </visual>
       <collision>
@@ -137,7 +131,5 @@
           scale="1 1 ${reflect}" />
         </geometry>
-        <material name="">
-          <color rgba="0.29804 0.29804 0.29804 1" />
-        </material>
+        <material name="pal/DarkGrey"/>
       </visual>
       <collision>
@@ -170,7 +162,5 @@
           scale="1 1 ${reflect}" />
         </geometry>
-        <material name="">
-          <color rgba="0.29804 0.29804 0.29804 1" />
-        </material>
+        <material name="pal/DarkGrey"/>
       </visual>
       <collision>
@@ -204,7 +194,5 @@
           scale="1 1 ${reflect}" />
         </geometry>
-        <material name="">
-          <color rgba="0.29804 0.29804 0.29804 1" />
-        </material>
+        <material name="pal/DarkGrey"/>
       </visual>
       <collision>
@@ -238,7 +226,5 @@
           scale="1 1 ${reflect}" />
         </geometry>
-        <material name="">
-          <color rgba="0.29804 0.29804 0.29804 1" />
-        </material>
+        <material name="pal/DarkGrey"/>
       </visual>
       <collision>
@@ -273,7 +259,5 @@
           <cylinder radius="0.005" length="0.005"/>
         </geometry>
-        <material name="">
-          <color rgba="0.29804 0.29804 0.29804 1" />
-        </material>
+        <material name="pal/DarkGrey"/>
       </visual>
       <collision>

File: pal_sea_arm_description/urdf/calibration_constants.urdf.xacro (robot description, xacro)
@@ -5,5 +5,4 @@
 -->
 <robot xmlns:xacro="http://ros.org/wiki/xacro">
- 	<xacro:include filename="$(find pal_sea_arm_description)/urdf/deg_to_rad.xacro" />
 	<!--Constant parameters-->
 	<xacro:property name="arm_1_joint_offset" value="0.0" />

File: pal_sea_arm_description/urdf/end_effector/end_effector.urdf.xacro (robot description, xacro)
@@ -13,6 +13,4 @@
 -->
 <robot xmlns:xacro="http://ros.org/wiki/xacro">
-  <!--File includes-->
-  <xacro:include filename="$(find pal_sea_arm_description)/urdf/deg_to_rad.xacro" />
   <!--
     Utiliy to create a tiago end effector (right or left).

File: pal_sea_arm_description/urdf/sensors/ft_sensor.urdf.xacro (robot description, xacro)
@@ -44,4 +44,9 @@
         </collision>
     </link>
+    <gazebo reference="${name}_ft_link">
+      <material>Gazebo/DarkGrey</material>
+      <mu1>0.9</mu1>
+      <mu2>0.9</mu2>
+    </gazebo>
     <joint name="${name}_ft_joint" type="fixed">
       <parent link="${parent}" />
