Commit message: Change arm_ft_ to wrist_ft to match TIAGo

File: pal_sea_arm_description/robots/pal_sea_arm.urdf.xacro (robot description, xacro)
@@ -34,5 +34,5 @@
   <xacro:property name="has_ft_sensor"           value="${ft_sensor in ['rokubi']}"/>
   <xacro:property name="has_end_effector"        value="${end_effector not in ['false', False, 'no-ee']}"/>
-  <xacro:property name="end_effector_link"       value="${'arm_ft_tool_link' if has_ft_sensor else 'arm_tool_link'}"/>
+  <xacro:property name="end_effector_link"       value="${'wrist_ft_tool_link' if has_ft_sensor else 'arm_tool_link'}"/>
   <link name="world"/>
   <joint name="world_fixed" type="fixed">
@@ -79,5 +79,5 @@
   <xacro:pal_sea_arm_end_effector name="gripper" parent="${end_effector_link}" type="${end_effector}" has_end_effector="${has_end_effector}" reflect="1"/>
   <xacro:if value="${has_ft_sensor}">
-    <xacro:ft_sensor name="arm" parent="arm_tool_link"/>
+    <xacro:ft_sensor name="wrist" parent="arm_tool_link"/>
   </xacro:if>
 </robot>

Commit message: Add namespace to urdf file

File: pal_sea_arm_description/robots/pal_sea_arm.urdf.xacro (robot description, xacro)
@@ -26,7 +26,9 @@
   <xacro:arg name="arm_model" default="pal-sea-arm-standalone"/>
   <xacro:arg name="use_sim" default="false"/>
+  <xacro:arg name="namespace" default=""/>
   <xacro:property name="end_effector" value="$(arg end_effector)" />
   <xacro:property name="ft_sensor" value="$(arg ft_sensor)" />
   <xacro:property name="arm_model" value="$(arg arm_model)" />
+  <xacro:property name="nsp" value="$(arg namespace)" />
   <xacro:if value="${end_effector not in ['no-ee', 'pal-pro-gripper']}">
     <xacro:wrong_end_effector/>

Commit message: Change all occurences of no-ee to no-end-effector

File: pal_sea_arm_description/robots/pal_sea_arm.urdf.xacro (robot description, xacro)
@@ -22,5 +22,5 @@
   <xacro:include filename="$(find pal_sea_arm_description)/ros2_control/ros2_control.urdf.xacro" />
   <xacro:pal_sea_arm_ros2_control use_sim="$(arg use_sim)" />
-  <xacro:arg name="end_effector" default="no-ee"/> <!-- no-ee, pal-pro-gripper -->
+  <xacro:arg name="end_effector" default="pal-pro-gripper"/> <!-- no-end-effector, pal-pro-gripper -->
   <xacro:arg name="ft_sensor" default="rokubi"/> <!-- no-ft-sensor, rokubi-->
   <xacro:arg name="arm_model" default="pal-sea-arm-standalone"/>
@@ -41,5 +41,5 @@
   </xacro:if>
   <xacro:property name="has_ft_sensor"           value="${ft_sensor != 'no-ft-sensor'}"/>
-  <xacro:property name="has_end_effector"        value="${end_effector not in ['no-ee']}"/>
+  <xacro:property name="has_end_effector"        value="${end_effector not in ['no-end-effector'']}"/>
   <xacro:property name="end_effector_link"       value="${'wrist_ft_tool_link' if has_ft_sensor else 'arm_tool_link'}"/>
  <!-- Force Torque sensor -->

File: pal_sea_arm_description/ros2_control/ros2_control.urdf.xacro (robot description, xacro)
@@ -15,5 +15,5 @@
        name="pal_sea_arm" >
     <xacro:macro name="pal_sea_arm_ros2_control" params="use_sim:=^|false">
-    <xacro:arg name="end_effector" default="no-ee"/>
+    <xacro:arg name="end_effector" default="no-end-effector"/>
     <xacro:arg name="ft_sensor" default="no-ft-sensor"/>
     <xacro:property name="end_effector" value="$(arg end_effector)" />

Commit message: Use common sim time arg and set it to True by default for simulation laucnh files

File: pal_sea_arm_description/robots/pal_sea_arm.urdf.xacro (robot description, xacro)
@@ -25,5 +25,5 @@
   <xacro:arg name="ft_sensor" default="rokubi"/> <!-- no-ft-sensor, rokubi-->
   <xacro:arg name="arm_model" default="pal-sea-arm-standalone"/>
-  <xacro:arg name="use_sim" default="false"/>
+  <xacro:arg name="use_sim" default="False"/>
   <xacro:arg name="namespace" default=""/>
   <xacro:property name="end_effector" value="$(arg end_effector)" />
@@ -41,5 +41,5 @@
   </xacro:if>
   <xacro:property name="has_ft_sensor"           value="${ft_sensor != 'no-ft-sensor'}"/>
-  <xacro:property name="has_end_effector"        value="${end_effector not in ['no-end-effector'']}"/>
+  <xacro:property name="has_end_effector"        value="${end_effector not in ['no-end-effector']}"/>
   <xacro:property name="end_effector_link"       value="${'wrist_ft_tool_link' if has_ft_sensor else 'arm_tool_link'}"/>
  <!-- Force Torque sensor -->
