Commit message: Changed arm_model to arm_type in the URDF

File: pal_sea_arm_description/robots/pal_sea_arm.urdf.xacro (robot description, xacro)
@@ -19,15 +19,17 @@
   <xacro:include filename="$(find pal_sea_arm_description)/urdf/end_effector/end_effector.urdf.xacro"/>
   <xacro:include filename="$(find pal_sea_arm_description)/gazebo/gazebo.urdf.xacro" />
-  <xacro:arg name="end_effector" default="pal-pro-gripper"/> <!-- no-end-effector, pal-pro-gripper -->
-  <xacro:arg name="ft_sensor" default="rokubi"/> <!-- no-ft-sensor, rokubi-->
-  <xacro:arg name="arm_model" default="pal-sea-arm-standalone"/>
+  <xacro:arg name="end_effector" default="pal-pro-gripper"/>
+  <!-- no-end-effector, pal-pro-gripper -->
+  <xacro:arg name="ft_sensor" default="rokubi"/>
+  <!-- no-ft-sensor, rokubi-->
+  <xacro:arg name="arm_type" default="pal-sea-arm-standalone"/>
   <xacro:arg name="use_sim" default="False"/>
   <xacro:arg name="namespace" default=""/>
-    <!-- ros2_control -->
+  <!-- ros2_control -->
   <xacro:include filename="$(find pal_sea_arm_description)/ros2_control/ros2_control.urdf.xacro" />
   <xacro:pal_sea_arm_ros2_control use_sim="$(arg use_sim)" />
   <xacro:property name="end_effector" value="$(arg end_effector)" />
   <xacro:property name="ft_sensor" value="$(arg ft_sensor)" />
-  <xacro:property name="arm_model" value="$(arg arm_model)" />
+  <xacro:property name="arm_type" value="$(arg arm_type)" />
   <xacro:property name="nsp" value="$(arg namespace)" />
   <xacro:if value="${end_effector not in ['no-end-effector', 'pal-pro-gripper']}">
@@ -37,11 +39,11 @@
     <xacro:wrong_ft_sensor/>
   </xacro:if>
-  <xacro:if value="${arm_model not in ['pal-sea-arm-standalone', 'tiago-pro', 'tiago-sea', 'tiago-sea-dual']}">
-    <xacro:wrong_arm_model/>
+  <xacro:if value="${arm_type not in ['pal-sea-arm-standalone', 'tiago-pro', 'tiago-sea', 'tiago-sea-dual']}">
+    <xacro:wrong_arm_type/>
   </xacro:if>
-  <xacro:property name="has_ft_sensor"           value="${ft_sensor != 'no-ft-sensor'}"/>
-  <xacro:property name="has_end_effector"        value="${end_effector not in ['no-end-effector']}"/>
-  <xacro:property name="end_effector_link"       value="${'wrist_ft_tool_link' if has_ft_sensor else 'arm_tool_link'}"/>
- <!-- Force Torque sensor -->
+  <xacro:property name="has_ft_sensor" value="${ft_sensor != 'no-ft-sensor'}"/>
+  <xacro:property name="has_end_effector" value="${end_effector not in ['no-end-effector']}"/>
+  <xacro:property name="end_effector_link" value="${'wrist_ft_tool_link' if has_ft_sensor else 'arm_tool_link'}"/>
+  <!-- Force Torque sensor -->
   <xacro:if value="${has_ft_sensor}">
     <xacro:include filename="$(find pal_sea_arm_description)/urdf/sensors/ft_sensor.urdf.xacro" />
@@ -50,7 +52,7 @@
   <link name="world"/>
   <joint name="world_fixed" type="fixed">
-      <origin xyz="0 0 0" rpy="0 0 0"/>
-      <parent link="world"/>
-      <child link="arm_root_link"/>
+    <origin xyz="0 0 0" rpy="0 0 0"/>
+    <parent link="world"/>
+    <child link="arm_root_link"/>
   </joint>
   <!-- BASE LINK -->
@@ -59,11 +61,5 @@
       <origin xyz="0.0 0.0 0.0" rpy="0 0 0" />
       <mass value="0.28971" />
-      <inertia
-        ixx="0.00022379"
-        ixy="1.5836E-20"
-        ixz="5.2063E-21"
-        iyy="0.00022379"
-        iyz="-5.1333E-21"
-        izz="0.00019673" />
+      <inertia ixx="0.00022379" ixy="1.5836E-20" ixz="5.2063E-21" iyy="0.00022379" iyz="-5.1333E-21" izz="0.00019673" />
     </inertial>
     <visual>
@@ -87,5 +83,5 @@
   </gazebo>
   <!-- ARM -->
-  <xacro:pal_sea_arm name="arm" parent="arm_root_link" arm_model="${arm_model}" reflect="1" arm_1_offset="0" arm_2_offset="0" arm_3_offset="0" arm_4_offset="0" arm_5_offset="0" arm_6_offset="0" arm_7_offset="0">
+  <xacro:pal_sea_arm name="arm" parent="arm_root_link" arm_type="${arm_type}" reflect="1" arm_1_offset="0" arm_2_offset="0" arm_3_offset="0" arm_4_offset="0" arm_5_offset="0" arm_6_offset="0" arm_7_offset="0">
     <origin xyz="0 0 0" rpy="0 0 3.1416" />
   </xacro:pal_sea_arm>
@@ -94,5 +90,5 @@
   <xacro:if value="${has_ft_sensor}">
     <xacro:ft_sensor name="wrist" parent="arm_tool_link"/>
-   <!-- <xacro:force_torque_sensor_gazebo name="wrist_ft" update_rate="100"/>-->
+    <!-- <xacro:force_torque_sensor_gazebo name="wrist_ft" update_rate="100"/>-->
   </xacro:if>
 </robot>

File: pal_sea_arm_description/urdf/arm/arm.urdf.xacro (robot description, xacro)
@@ -14,17 +14,15 @@
 <robot xmlns:xacro="http://ros.org/wiki/xacro">
   <!-- Transmissions file -->
-  <xacro:macro name="pal_sea_arm" params="name parent *origin arm_model reflect:=1 arm_1_offset arm_2_offset arm_3_offset arm_4_offset arm_5_offset arm_6_offset arm_7_offset
-                                          no_safety_eps:=False joint_limits_file:='$(find pal_sea_arm_description)/urdf/arm/limits/arm_${arm_model}.limits.xacro'
-                                          arm_properties_file:='$(find pal_sea_arm_description)/urdf/arm/arm_properties/arm_${arm_model}.properties.xacro'">
-    <xacro:property name="arm_eps"       value="${0.00 if no_safety_eps else 0.07}"/>
+  <xacro:macro name="pal_sea_arm" params="name parent *origin arm_type reflect:=1 arm_1_offset arm_2_offset arm_3_offset arm_4_offset arm_5_offset arm_6_offset arm_7_offset no_safety_eps:=False joint_limits_file:='$(find pal_sea_arm_description)/urdf/arm/limits/arm_${arm_type}.limits.xacro' arm_properties_file:='$(find pal_sea_arm_description)/urdf/arm/arm_properties/arm_${arm_type}.properties.xacro'">
+    <xacro:property name="arm_eps" value="${0.00 if no_safety_eps else 0.07}"/>
     <!-- Joint Limits file -->
     <xacro:include filename="${joint_limits_file}"/>
     <xacro:include filename="${arm_properties_file}"/>
     <xacro:property name="mesh_folder"/>
-    <xacro:if value="${arm_model in ['tiago-pro', 'pal-sea-arm-standalone']}">
-      <xacro:property name="mesh_folder"       value="arm_tiago_pro"/>
+    <xacro:if value="${arm_type in ['tiago-pro', 'pal-sea-arm-standalone']}">
+      <xacro:property name="mesh_folder" value="arm_tiago_pro"/>
     </xacro:if>
-    <xacro:if value="${arm_model in ['tiago-sea', 'tiago-sea-dual']}">
-      <xacro:property name="mesh_folder"       value="arm_tiago_sea"/>
+    <xacro:if value="${arm_type in ['tiago-sea', 'tiago-sea-dual']}">
+      <xacro:property name="mesh_folder" value="arm_tiago_sea"/>
     </xacro:if>
     <!-- ARM 1 LINK -->
@@ -34,15 +32,12 @@
         <origin xyz="0 0 0" rpy="0 0 0" />
         <geometry>
-          <mesh
-            filename="package://pal_sea_arm_description/meshes/${mesh_folder}/arm_1_link.stl"
-            scale="1 1 ${reflect}" />
-        </geometry>
-        <material name="pal/DarkGrey"/>
-      </visual>
-      <collision>
-        <origin xyz="0 0 0" rpy="0 0 0" />
-        <geometry>
-          <mesh filename="package://pal_sea_arm_description/meshes/${mesh_folder}/arm_1_link_collision.stl"
-          scale="1 1 ${reflect}" />
+          <mesh filename="package://pal_sea_arm_description/meshes/${mesh_folder}/arm_1_link.stl" scale="1 1 ${reflect}" />
+        </geometry>
+        <material name="pal/DarkGrey"/>
+      </visual>
+      <collision>
+        <origin xyz="0 0 0" rpy="0 0 0" />
+        <geometry>
+          <mesh filename="package://pal_sea_arm_description/meshes/${mesh_folder}/arm_1_link_collision.stl" scale="1 1 ${reflect}" />
         </geometry>
       </collision>
@@ -56,6 +51,5 @@
       <limit lower="${arm_1_joint_lb * deg_to_rad}" upper="${arm_1_joint_ub * deg_to_rad}" effort="${arm_1_max_effort}" velocity="${arm_1_max_velocity}" />
       <dynamics friction="${arm_friction}" damping="${arm_damping}"/>
-      <safety_controller k_position="${arm_k_position}" k_velocity="${arm_k_velocity}" soft_lower_limit="${arm_1_joint_lb  + arm_eps}"
-        soft_upper_limit="${arm_1_joint_ub - arm_eps}" />
+      <safety_controller k_position="${arm_k_position}" k_velocity="${arm_k_velocity}" soft_lower_limit="${arm_1_joint_lb  + arm_eps}" soft_upper_limit="${arm_1_joint_ub - arm_eps}" />
     </joint>
     <!-- ARM 2 LINK -->
@@ -65,14 +59,12 @@
         <origin xyz="0 0 0" rpy="0 0 0" />
         <geometry>
-          <mesh filename="package://pal_sea_arm_description/meshes/${mesh_folder}/arm_2_link.stl"
-          scale="1 1 ${reflect}" />
-        </geometry>
-        <material name="pal/DarkGrey"/>
-      </visual>
-      <collision>
-        <origin xyz="0 0 0" rpy="0 0 0" />
-        <geometry>
-          <mesh filename="package://pal_sea_arm_description/meshes/${mesh_folder}/arm_2_link_collision.stl"
-          scale="1 1 ${reflect}" />
+          <mesh filename="package://pal_sea_arm_description/meshes/${mesh_folder}/arm_2_link.stl" scale="1 1 ${reflect}" />
+        </geometry>
+        <material name="pal/DarkGrey"/>
+      </visual>
+      <collision>
+        <origin xyz="0 0 0" rpy="0 0 0" />
+        <geometry>
+          <mesh filename="package://pal_sea_arm_description/meshes/${mesh_folder}/arm_2_link_collision.stl" scale="1 1 ${reflect}" />
         </geometry>
       </collision>
@@ -86,6 +78,5 @@
       <limit lower="${arm_2_joint_lb * deg_to_rad}" upper="${arm_2_joint_ub * deg_to_rad}" effort="${arm_2_max_effort}" velocity="${arm_2_max_velocity}" />
       <dynamics friction="${arm_friction}" damping="${arm_damping}"/>
-      <safety_controller k_position="${arm_k_position}" k_velocity="${arm_k_velocity}" soft_lower_limit="${arm_2_joint_lb * deg_to_rad  + arm_eps}"
-        soft_upper_limit="${arm_2_joint_ub * deg_to_rad - arm_eps}" />
+      <safety_controller k_position="${arm_k_position}" k_velocity="${arm_k_velocity}" soft_lower_limit="${arm_2_joint_lb * deg_to_rad  + arm_eps}" soft_upper_limit="${arm_2_joint_ub * deg_to_rad - arm_eps}" />
     </joint>
     <!-- ARM 3 LINK -->
@@ -95,14 +86,12 @@
         <origin xyz="0 0 0" rpy="0 0 0" />
         <geometry>
-          <mesh filename="package://pal_sea_arm_description/meshes/${mesh_folder}/arm_3_link.stl"
-          scale="1 1 ${reflect}" />
-        </geometry>
-        <material name="pal/DarkGrey"/>
-      </visual>
-      <collision>
-        <origin xyz="0 0 0" rpy="0 0 0" />
-        <geometry>
-          <mesh filename="package://pal_sea_arm_description/meshes/${mesh_folder}/arm_3_link_collision.stl"
-          scale="1 1 ${reflect}" />
+          <mesh filename="package://pal_sea_arm_description/meshes/${mesh_folder}/arm_3_link.stl" scale="1 1 ${reflect}" />
+        </geometry>
+        <material name="pal/DarkGrey"/>
+      </visual>
+      <collision>
+        <origin xyz="0 0 0" rpy="0 0 0" />
+        <geometry>
+          <mesh filename="package://pal_sea_arm_description/meshes/${mesh_folder}/arm_3_link_collision.stl" scale="1 1 ${reflect}" />
         </geometry>
       </collision>
@@ -114,10 +103,7 @@
       <child link="${name}_3_link" />
       <axis xyz="0 0 1" />
-      <limit lower="${arm_3_joint_lb * deg_to_rad}" upper="${arm_3_joint_ub * deg_to_rad}"
-        effort="${arm_3_max_effort}" velocity="${arm_3_max_velocity}" />
-      <dynamics friction="${arm_friction}" damping="${arm_damping}"/>
-      <safety_controller k_position="${arm_k_position}" k_velocity="${arm_k_velocity}"
-        soft_lower_limit="${arm_3_joint_lb * deg_to_rad  + arm_eps}"
-        soft_upper_limit="${arm_3_joint_ub * deg_to_rad - arm_eps}" />
+      <limit lower="${arm_3_joint_lb * deg_to_rad}" upper="${arm_3_joint_ub * deg_to_rad}" effort="${arm_3_max_effort}" velocity="${arm_3_max_velocity}" />
+      <dynamics friction="${arm_friction}" damping="${arm_damping}"/>
+      <safety_controller k_position="${arm_k_position}" k_velocity="${arm_k_velocity}" soft_lower_limit="${arm_3_joint_lb * deg_to_rad  + arm_eps}" soft_upper_limit="${arm_3_joint_ub * deg_to_rad - arm_eps}" />
     </joint>
     <!-- ARM 4 LINK -->
@@ -127,14 +113,12 @@
         <origin xyz="0 0 0" rpy="0 0 0" />
         <geometry>
-          <mesh filename="package://pal_sea_arm_description/meshes/${mesh_folder}/arm_4_link.stl"
-          scale="1 1 ${reflect}" />
-        </geometry>
-        <material name="pal/DarkGrey"/>
-      </visual>
-      <collision>
-        <origin xyz="0 0 0" rpy="0 0 0" />
-        <geometry>
-          <mesh filename="package://pal_sea_arm_description/meshes/${mesh_folder}/arm_4_link_collision.stl"
-          scale="1 1 ${reflect}" />
+          <mesh filename="package://pal_sea_arm_description/meshes/${mesh_folder}/arm_4_link.stl" scale="1 1 ${reflect}" />
+        </geometry>
+        <material name="pal/DarkGrey"/>
+      </visual>
+      <collision>
+        <origin xyz="0 0 0" rpy="0 0 0" />
+        <geometry>
+          <mesh filename="package://pal_sea_arm_description/meshes/${mesh_folder}/arm_4_link_collision.stl" scale="1 1 ${reflect}" />
         </geometry>
       </collision>
@@ -148,7 +132,5 @@
       <limit lower="${arm_4_joint_lb * deg_to_rad}" upper="${arm_4_joint_ub * deg_to_rad}" effort="${arm_4_max_effort}" velocity="${arm_4_max_velocity}" />
       <dynamics friction="${arm_friction}" damping="${arm_damping}"/>
-      <safety_controller
-        k_position="${arm_k_position}" k_velocity="${arm_k_velocity}" soft_lower_limit="${arm_4_joint_lb * deg_to_rad  + arm_eps}"
-        soft_upper_limit="${arm_4_joint_ub * deg_to_rad - arm_eps}" />
+      <safety_controller k_position="${arm_k_position}" k_velocity="${arm_k_velocity}" soft_lower_limit="${arm_4_joint_lb * deg_to_rad  + arm_eps}" soft_upper_limit="${arm_4_joint_ub * deg_to_rad - arm_eps}" />
     </joint>
     <!-- ARM 5 LINK -->
@@ -158,14 +140,12 @@
         <origin xyz="0 0 0" rpy="0 0 0" />
         <geometry>
-          <mesh filename="package://pal_sea_arm_description/meshes/${mesh_folder}/arm_5_link.stl"
-          scale="1 1 ${reflect}" />
-        </geometry>
-        <material name="pal/DarkGrey"/>
-      </visual>
-      <collision>
-        <origin xyz="0 0 0" rpy="0 0 0" />
-        <geometry>
-          <mesh filename="package://pal_sea_arm_description/meshes/${mesh_folder}/arm_5_link_collision.stl"
-          scale="1 1 ${reflect}" />
+          <mesh filename="package://pal_sea_arm_description/meshes/${mesh_folder}/arm_5_link.stl" scale="1 1 ${reflect}" />
+        </geometry>
+        <material name="pal/DarkGrey"/>
+      </visual>
+      <collision>
+        <origin xyz="0 0 0" rpy="0 0 0" />
+        <geometry>
+          <mesh filename="package://pal_sea_arm_description/meshes/${mesh_folder}/arm_5_link_collision.stl" scale="1 1 ${reflect}" />
         </geometry>
       </collision>
@@ -177,10 +157,7 @@
       <child link="${name}_5_link" />
       <axis xyz="0 0 1" />
-      <limit
-        lower="${arm_5_joint_lb * deg_to_rad}" upper="${arm_5_joint_ub * deg_to_rad}" effort="${arm_5_max_effort}" velocity="${arm_5_max_velocity}" />
-      <dynamics friction="${arm_friction}" damping="${arm_damping}"/>
-      <safety_controller
-        k_position="${arm_k_position}" k_velocity="${arm_k_velocity}" soft_lower_limit="${arm_5_joint_lb * deg_to_rad  + arm_eps}"
-        soft_upper_limit="${arm_5_joint_ub * deg_to_rad - arm_eps}" />
+      <limit lower="${arm_5_joint_lb * deg_to_rad}" upper="${arm_5_joint_ub * deg_to_rad}" effort="${arm_5_max_effort}" velocity="${arm_5_max_velocity}" />
+      <dynamics friction="${arm_friction}" damping="${arm_damping}"/>
+      <safety_controller k_position="${arm_k_position}" k_velocity="${arm_k_velocity}" soft_lower_limit="${arm_5_joint_lb * deg_to_rad  + arm_eps}" soft_upper_limit="${arm_5_joint_ub * deg_to_rad - arm_eps}" />
     </joint>
     <!-- ARM 6 LINK -->
@@ -190,14 +167,12 @@
         <origin xyz="0 0 0" rpy="0 0 0" />
         <geometry>
-          <mesh filename="package://pal_sea_arm_description/meshes/${mesh_folder}/arm_6_link.stl"
-          scale="1 1 ${reflect}" />
-        </geometry>
-        <material name="pal/DarkGrey"/>
-      </visual>
-      <collision>
-        <origin xyz="0 0 0" rpy="0 0 0" />
-        <geometry>
-          <mesh filename="package://pal_sea_arm_description/meshes/${mesh_folder}/arm_6_link_collision.stl"
-          scale="1 1 ${reflect}" />
+          <mesh filename="package://pal_sea_arm_description/meshes/${mesh_folder}/arm_6_link.stl" scale="1 1 ${reflect}" />
+        </geometry>
+        <material name="pal/DarkGrey"/>
+      </visual>
+      <collision>
+        <origin xyz="0 0 0" rpy="0 0 0" />
+        <geometry>
+          <mesh filename="package://pal_sea_arm_description/meshes/${mesh_folder}/arm_6_link_collision.stl" scale="1 1 ${reflect}" />
         </geometry>
       </collision>
@@ -209,10 +184,7 @@
       <child link="${name}_6_link" />
       <axis xyz="0 0 1" />
-      <limit
-        lower="${arm_6_joint_lb * deg_to_rad}" upper="${arm_6_joint_ub * deg_to_rad}" effort="${arm_6_max_effort}" velocity="${arm_6_max_velocity}" />
-      <dynamics friction="${arm_friction}" damping="${arm_damping}"/>
-      <safety_controller
-        k_position="${arm_k_position}" k_velocity="${arm_k_velocity}" soft_lower_limit="${arm_6_joint_lb * deg_to_rad  + arm_eps}"
-        soft_upper_limit="${arm_6_joint_ub * deg_to_rad - arm_eps}" />
+      <limit lower="${arm_6_joint_lb * deg_to_rad}" upper="${arm_6_joint_ub * deg_to_rad}" effort="${arm_6_max_effort}" velocity="${arm_6_max_velocity}" />
+      <dynamics friction="${arm_friction}" damping="${arm_damping}"/>
+      <safety_controller k_position="${arm_k_position}" k_velocity="${arm_k_velocity}" soft_lower_limit="${arm_6_joint_lb * deg_to_rad  + arm_eps}" soft_upper_limit="${arm_6_joint_ub * deg_to_rad - arm_eps}" />
     </joint>
     <!-- ARM 7 LINK -->
@@ -222,14 +194,12 @@
         <origin xyz="0 0 0" rpy="0 0 0" />
         <geometry>
-          <mesh filename="package://pal_sea_arm_description/meshes/${mesh_folder}/arm_7_link.stl"
-          scale="1 1 ${reflect}" />
-        </geometry>
-        <material name="pal/DarkGrey"/>
-      </visual>
-      <collision>
-        <origin xyz="0 0 0" rpy="0 0 0" />
-        <geometry>
-          <mesh filename="package://pal_sea_arm_description/meshes/${mesh_folder}/arm_7_link_collision.stl"
-          scale="1 1 ${reflect}" />
+          <mesh filename="package://pal_sea_arm_description/meshes/${mesh_folder}/arm_7_link.stl" scale="1 1 ${reflect}" />
+        </geometry>
+        <material name="pal/DarkGrey"/>
+      </visual>
+      <collision>
+        <origin xyz="0 0 0" rpy="0 0 0" />
+        <geometry>
+          <mesh filename="package://pal_sea_arm_description/meshes/${mesh_folder}/arm_7_link_collision.stl" scale="1 1 ${reflect}" />
         </geometry>
       </collision>
@@ -241,10 +211,7 @@
       <child link="${name}_7_link" />
       <axis xyz="0 0 1" />
-      <limit
-        lower="${arm_7_joint_lb * deg_to_rad}" upper="${arm_7_joint_ub * deg_to_rad}" effort="${arm_7_max_effort}" velocity="${arm_7_max_velocity}" />
-      <dynamics friction="${arm_friction}" damping="${arm_damping}"/>
-      <safety_controller
-        k_position="${arm_k_position}" k_velocity="${arm_k_velocity}" soft_lower_limit="${arm_7_joint_lb * deg_to_rad  + arm_eps}"
-        soft_upper_limit="${arm_7_joint_ub * deg_to_rad - arm_eps}" />
+      <limit lower="${arm_7_joint_lb * deg_to_rad}" upper="${arm_7_joint_ub * deg_to_rad}" effort="${arm_7_max_effort}" velocity="${arm_7_max_velocity}" />
+      <dynamics friction="${arm_friction}" damping="${arm_damping}"/>
+      <safety_controller k_position="${arm_k_position}" k_velocity="${arm_k_velocity}" soft_lower_limit="${arm_7_joint_lb * deg_to_rad  + arm_eps}" soft_upper_limit="${arm_7_joint_ub * deg_to_rad - arm_eps}" />
     </joint>
     <!--***********************-->
