Commit message: Arm std with new wrist type arg

File: pal_sea_arm_description/robots/pal_sea_arm.urdf.xacro (robot description, xacro)
@@ -13,26 +13,30 @@
  -->
 <robot xmlns:xacro="http://ros.org/wiki/xacro" name="pal_sea_arm">
-  <!--File includes-->
-  <xacro:include filename="$(find pal_urdf_utils)/urdf/deg_to_rad.urdf.xacro" />
-  <xacro:include filename="$(find pal_urdf_utils)/urdf/materials.urdf.xacro" />
-  <xacro:include filename="$(find pal_sea_arm_description)/urdf/arm/arm.urdf.xacro"/>
-  <xacro:include filename="$(find pal_sea_arm_description)/urdf/end_effector/end_effector.urdf.xacro"/>
-  <xacro:include filename="$(find pal_sea_arm_description)/gazebo/gazebo.urdf.xacro" />
+  <!-- ARGUMENTS -->
+  <!-- no-end-effector, pal-pro-gripper -->
   <xacro:arg name="end_effector" default="pal-pro-gripper"/>
-  <!-- no-end-effector, pal-pro-gripper -->
+  <!-- spherical-wrist, straight-wrist -->
+  <xacro:arg name="wrist_model" default="spherical-wrist"/>
+  <!-- no-ft-sensor, rokubi-->
   <xacro:arg name="ft_sensor" default="rokubi"/>
-  <!-- no-ft-sensor, rokubi-->
+  <!-- pal-sea-arm-standalone, tiago-pro, tiago-sea, tiago-sea-dual -->
   <xacro:arg name="arm_type" default="pal-sea-arm-standalone"/>
+  <!-- False, True -->
+  <xacro:arg name="tool_changer" default="True"/>
+  <!-- Common args -->
   <xacro:arg name="use_sim" default="False"/>
   <xacro:arg name="namespace" default=""/>
-  <!-- ros2_control -->
-  <xacro:include filename="$(find pal_sea_arm_description)/ros2_control/ros2_control.urdf.xacro" />
-  <xacro:pal_sea_arm_ros2_control use_sim="$(arg use_sim)" />
+  <!-- PROPERTIES -->
   <xacro:property name="end_effector" value="$(arg end_effector)" />
+  <xacro:property name="wrist_model" value="$(arg wrist_model)" />
   <xacro:property name="ft_sensor" value="$(arg ft_sensor)" />
   <xacro:property name="arm_type" value="$(arg arm_type)" />
+  <xacro:property name="tool_changer" value="$(arg tool_changer)" />
   <xacro:property name="nsp" value="$(arg namespace)" />
   <xacro:if value="${end_effector not in ['no-end-effector', 'pal-pro-gripper']}">
     <xacro:wrong_end_effector/>
+  </xacro:if>
+  <xacro:if value="${wrist_model not in ['straight-wrist', 'spherical-wrist']}">
+    <xacro:wrong_wrist_model/>
   </xacro:if>
   <xacro:if value="${ft_sensor not in ['no-ft-sensor', 'rokubi']}">
@@ -45,4 +49,12 @@
   <xacro:property name="has_end_effector" value="${end_effector not in ['no-end-effector']}"/>
   <xacro:property name="end_effector_link" value="${'wrist_ft_tool_link' if has_ft_sensor else 'arm_tool_link'}"/>
+  <!--INCLUDES -->
+  <xacro:include filename="$(find pal_urdf_utils)/urdf/deg_to_rad.urdf.xacro" />
+  <xacro:include filename="$(find pal_urdf_utils)/urdf/materials.urdf.xacro" />
+  <xacro:include filename="$(find pal_sea_arm_description)/urdf/arm/arm.urdf.xacro"/>
+  <xacro:include filename="$(find pal_sea_arm_description)/urdf/end_effector/end_effector.urdf.xacro"/>
+  <xacro:include filename="$(find pal_sea_arm_description)/gazebo/gazebo.urdf.xacro" />
+  <!-- ROS2 control -->
+  <xacro:include filename="$(find pal_sea_arm_description)/ros2_control/ros2_control.urdf.xacro" />
   <!-- Force Torque sensor -->
   <xacro:if value="${has_ft_sensor}">
@@ -50,4 +62,5 @@
     <xacro:include filename="$(find pal_sea_arm_description)/urdf/sensors/ft_sensor.gazebo.xacro" />
   </xacro:if>
+  <!-- ROBOT DEFINITION -->
   <link name="world"/>
   <joint name="world_fixed" type="fixed">
@@ -83,8 +96,9 @@
   </gazebo>
   <!-- ARM -->
-  <xacro:pal_sea_arm name="arm" parent="arm_root_link" arm_type="${arm_type}" reflect="1" arm_1_offset="0" arm_2_offset="0" arm_3_offset="0" arm_4_offset="0" arm_5_offset="0" arm_6_offset="0" arm_7_offset="0">
+  <xacro:pal_sea_arm name="arm" parent="arm_root_link" arm_type="${arm_type}" wrist_model="${wrist_model}" reflect="1" arm_1_offset="0" arm_2_offset="0" arm_3_offset="0" arm_4_offset="0" arm_5_offset="0" arm_6_offset="0" arm_7_offset="0">
     <origin xyz="0 0 0" rpy="0 0 3.1416" />
   </xacro:pal_sea_arm>
-  <xacro:pal_sea_arm_end_effector name="gripper" parent="${end_effector_link}" type="${end_effector}" has_end_effector="${has_end_effector}" reflect="1"/>
+  <!-- End effector -->
+  <xacro:pal_sea_arm_end_effector name="gripper" parent="${end_effector_link}" type="${end_effector}" tool_changer="${tool_changer}" reflect="1"/>
   <!-- Force Torque sensor-->
   <xacro:if value="${has_ft_sensor}">
@@ -92,3 +106,5 @@
     <!-- <xacro:force_torque_sensor_gazebo name="wrist_ft" update_rate="100"/>-->
   </xacro:if>
+  <!-- ROS2 control -->
+  <xacro:pal_sea_arm_ros2_control use_sim="$(arg use_sim)" />
 </robot>

File: pal_sea_arm_description/ros2_control/ros2_control.urdf.xacro (robot description, xacro)
@@ -12,7 +12,6 @@
   limitations under the License.
  -->
-<robot xmlns:xacro="http://ros.org/wiki/xacro"
-       name="pal_sea_arm" >
-    <xacro:macro name="pal_sea_arm_ros2_control" params="use_sim:=^|false">
+<robot xmlns:xacro="http://ros.org/wiki/xacro" name="pal_sea_arm">
+  <xacro:macro name="pal_sea_arm_ros2_control" params="use_sim:=^|false">
     <xacro:arg name="end_effector" default="no-end-effector"/>
     <xacro:arg name="ft_sensor" default="no-ft-sensor"/>
@@ -22,5 +21,5 @@
     <xacro:include filename="$(find pal_sea_arm_description)/urdf/arm/arm.ros2_control.xacro" />
     <xacro:if value="${end_effector == 'pal-pro-gripper'}">
-        <xacro:include filename="$(find pal_pro_gripper_description)/urdf/pal_pro_gripper.ros2_control.xacro" />
+      <xacro:include filename="$(find pal_pro_gripper_description)/urdf/gripper.ros2_control.xacro" />
     </xacro:if>
     <!-- calibration offsets -->

File: pal_sea_arm_description/urdf/arm/arm.urdf.xacro (robot description, xacro)
@@ -14,16 +14,22 @@
 <robot xmlns:xacro="http://ros.org/wiki/xacro">
   <!-- Transmissions file -->
-  <xacro:macro name="pal_sea_arm" params="name parent *origin arm_type reflect:=1 arm_1_offset arm_2_offset arm_3_offset arm_4_offset arm_5_offset arm_6_offset arm_7_offset no_safety_eps:=False joint_limits_file:='$(find pal_sea_arm_description)/urdf/arm/limits/arm_${arm_type}.limits.xacro' arm_properties_file:='$(find pal_sea_arm_description)/urdf/arm/arm_properties/arm_${arm_type}.properties.xacro'">
+  <xacro:macro name="pal_sea_arm" params="name parent *origin arm_type wrist_model reflect:=1 arm_1_offset arm_2_offset arm_3_offset arm_4_offset arm_5_offset arm_6_offset arm_7_offset no_safety_eps:=False">
+    <!-- PROPERTIES -->
     <xacro:property name="arm_eps" value="${0.00 if no_safety_eps else 0.07}"/>
-    <!-- Joint Limits file -->
-    <xacro:include filename="${joint_limits_file}"/>
-    <xacro:include filename="${arm_properties_file}"/>
     <xacro:property name="mesh_folder"/>
-    <xacro:if value="${arm_type in ['tiago-pro', 'pal-sea-arm-standalone']}">
+    <!-- Tiago Pro -->
+    <xacro:if value="${arm_type in ['tiago-pro']}">
       <xacro:property name="mesh_folder" value="arm_tiago_pro"/>
     </xacro:if>
+    <!-- Tiago SEA -->
     <xacro:if value="${arm_type in ['tiago-sea', 'tiago-sea-dual']}">
       <xacro:property name="mesh_folder" value="arm_tiago_sea"/>
     </xacro:if>
+    <!-- INCLUDES -->
+    <xacro:include filename="$(find pal_sea_arm_description)/urdf/arm/limits/arm_${arm_type}.limits.xacro"/>
+    <xacro:include filename="$(find pal_sea_arm_description)/urdf/arm/arm_properties/${arm_type}/arm.properties.xacro"/>
+    <xacro:include filename="$(find pal_sea_arm_description)/urdf/arm/arm_properties/${arm_type}/arm.properties.xacro"/>
+    <xacro:include filename="$(find pal_sea_arm_description)/urdf/arm/arm_properties/${arm_type}/${wrist_model}.properties.xacro"/>
+    <!-- ARM DEFINITION -->
     <!-- ARM 1 LINK -->
     <link name="${name}_1_link">
@@ -140,12 +146,12 @@
         <origin xyz="0 0 0" rpy="0 0 0" />
         <geometry>
-          <mesh filename="package://pal_sea_arm_description/meshes/${mesh_folder}/arm_5_link.stl" scale="1 1 ${reflect}" />
-        </geometry>
-        <material name="pal/DarkGrey"/>
-      </visual>
-      <collision>
-        <origin xyz="0 0 0" rpy="0 0 0" />
-        <geometry>
-          <mesh filename="package://pal_sea_arm_description/meshes/${mesh_folder}/arm_5_link_collision.stl" scale="1 1 ${reflect}" />
+          <mesh filename="package://pal_sea_arm_description/meshes/${mesh_folder}/${wrist_model}/arm_5_link.stl" scale="1 1 ${reflect}" />
+        </geometry>
+        <material name="pal/DarkGrey"/>
+      </visual>
+      <collision>
+        <origin xyz="0 0 0" rpy="0 0 0" />
+        <geometry>
+          <mesh filename="package://pal_sea_arm_description/meshes/${mesh_folder}/${wrist_model}/arm_5_link_collision.stl" scale="1 1 ${reflect}" />
         </geometry>
       </collision>
@@ -167,12 +173,12 @@
         <origin xyz="0 0 0" rpy="0 0 0" />
         <geometry>
-          <mesh filename="package://pal_sea_arm_description/meshes/${mesh_folder}/arm_6_link.stl" scale="1 1 ${reflect}" />
-        </geometry>
-        <material name="pal/DarkGrey"/>
-      </visual>
-      <collision>
-        <origin xyz="0 0 0" rpy="0 0 0" />
-        <geometry>
-          <mesh filename="package://pal_sea_arm_description/meshes/${mesh_folder}/arm_6_link_collision.stl" scale="1 1 ${reflect}" />
+          <mesh filename="package://pal_sea_arm_description/meshes/${mesh_folder}/${wrist_model}/arm_6_link.stl" scale="1 1 ${reflect}" />
+        </geometry>
+        <material name="pal/DarkGrey"/>
+      </visual>
+      <collision>
+        <origin xyz="0 0 0" rpy="0 0 0" />
+        <geometry>
+          <mesh filename="package://pal_sea_arm_description/meshes/${mesh_folder}/${wrist_model}/arm_6_link_collision.stl" scale="1 1 ${reflect}" />
         </geometry>
       </collision>
@@ -194,12 +200,12 @@
         <origin xyz="0 0 0" rpy="0 0 0" />
         <geometry>
-          <mesh filename="package://pal_sea_arm_description/meshes/${mesh_folder}/arm_7_link.stl" scale="1 1 ${reflect}" />
-        </geometry>
-        <material name="pal/DarkGrey"/>
-      </visual>
-      <collision>
-        <origin xyz="0 0 0" rpy="0 0 0" />
-        <geometry>
-          <mesh filename="package://pal_sea_arm_description/meshes/${mesh_folder}/arm_7_link_collision.stl" scale="1 1 ${reflect}" />
+          <mesh filename="package://pal_sea_arm_description/meshes/${mesh_folder}/${wrist_model}/arm_7_link.stl" scale="1 1 ${reflect}" />
+        </geometry>
+        <material name="pal/DarkGrey"/>
+      </visual>
+      <collision>
+        <origin xyz="0 0 0" rpy="0 0 0" />
+        <geometry>
+          <mesh filename="package://pal_sea_arm_description/meshes/${mesh_folder}/${wrist_model}/arm_7_link_collision.stl" scale="1 1 ${reflect}" />
         </geometry>
       </collision>
@@ -274,4 +280,9 @@
       <mu2>0.9</mu2>
     </gazebo>
+    <gazebo reference="${name}_tool_link">
+      <material>Gazebo/DarkGrey</material>
+      <mu1>0.9</mu1>
+      <mu2>0.9</mu2>
+    </gazebo>
     <gazebo reference="${name}_1_joint">
       <implicitSpringDamper>1</implicitSpringDamper>

File: pal_sea_arm_description/urdf/arm/limits/arm_tiago-pro.limits.xacro (robot description, xacro)
@@ -1,6 +1,6 @@
 <robot xmlns:xacro="http://ros.org/wiki/xacro">
   <!-- Constant parameters -->
-  <xacro:property name="arm_friction"       value="1.0" />
-  <xacro:property name="arm_damping"        value="1.0" />
+  <xacro:property name="arm_friction" value="1.0" />
+  <xacro:property name="arm_damping" value="1.0" />
   <xacro:property name="arm_k_position" value="20"/>
   <xacro:property name="arm_k_velocity" value="20"/>
@@ -19,17 +19,17 @@
   <xacro:property name="arm_7_joint_ub" value="148.97" />
   <xacro:property name="arm_7_joint_lb" value="-148.97" />
-  <xacro:property name="arm_1_max_velocity"      value="1.95" />
-  <xacro:property name="arm_2_max_velocity"      value="1.95" />
-  <xacro:property name="arm_3_max_velocity"      value="2.35" />
-  <xacro:property name="arm_4_max_velocity"      value="2.35" />
-  <xacro:property name="arm_5_max_velocity"      value="2.35" />
-  <xacro:property name="arm_6_max_velocity"      value="2.35" />
-  <xacro:property name="arm_7_max_velocity"      value="2.35" />
-  <xacro:property name="arm_1_max_effort"   value="43.0" />
-  <xacro:property name="arm_2_max_effort"   value="43.0" />
-  <xacro:property name="arm_3_max_effort"   value="26" />
-  <xacro:property name="arm_4_max_effort"   value="26" />
-  <xacro:property name="arm_5_max_effort"   value="26" />
-  <xacro:property name="arm_6_max_effort"   value="26" />
-  <xacro:property name="arm_7_max_effort"   value="26" />
+  <xacro:property name="arm_1_max_velocity" value="1.95" />
+  <xacro:property name="arm_2_max_velocity" value="1.95" />
+  <xacro:property name="arm_3_max_velocity" value="2.35" />
+  <xacro:property name="arm_4_max_velocity" value="2.35" />
+  <xacro:property name="arm_5_max_velocity" value="2.35" />
+  <xacro:property name="arm_6_max_velocity" value="2.35" />
+  <xacro:property name="arm_7_max_velocity" value="2.35" />
+  <xacro:property name="arm_1_max_effort" value="43.0" />
+  <xacro:property name="arm_2_max_effort" value="43.0" />
+  <xacro:property name="arm_3_max_effort" value="26" />
+  <xacro:property name="arm_4_max_effort" value="26" />
+  <xacro:property name="arm_5_max_effort" value="26" />
+  <xacro:property name="arm_6_max_effort" value="26" />
+  <xacro:property name="arm_7_max_effort" value="26" />
 </robot>

File: pal_sea_arm_description/urdf/end_effector/end_effector.urdf.xacro (robot description, xacro)
@@ -20,18 +20,21 @@
     - reflect: Set to 1 for a right end effector, or to -1 for a left end effector
   -->
-  <xacro:macro name="pal_sea_arm_end_effector" params="name parent type has_end_effector reflect is_dual:=false">
-  <!-- No end-effector -->
-  <xacro:if value="${not has_end_effector}">
-    <!-- Add nothing -->
-  </xacro:if>
-  <!-- PAL Pro Gripper -->
-  <xacro:if value="${type == 'pal-pro-gripper'}">
-    <xacro:include filename="$(find pal_pro_gripper_description)/urdf/pro_gripper.urdf.xacro" />
-    <xacro:pal_pro_gripper name="${name}" parent="${parent}" >
-      <origin xyz="0.052 0.0 0.0" rpy="0 ${90 * deg_to_rad} 0"/>
-    </xacro:pal_pro_gripper>
-  </xacro:if>
-  <!-- Custom -->
-  <!-- <xacro:if value="${type == 'custom' and not is_dual}">
+  <xacro:macro name="pal_sea_arm_end_effector" params="name parent type tool_changer reflect">
+    <!-- PAL Pro Gripper -->
+    <xacro:if value="${type == 'pal-pro-gripper'}">
+      <xacro:include filename="$(find pal_pro_gripper_description)/urdf/gripper.urdf.xacro" />
+      <xacro:pal_pro_gripper name="${name}" parent="${parent}" tool_changer="${tool_changer}">
+        <origin xyz="0.0 0.0 0.0" rpy="0 ${90 * deg_to_rad} 0"/>
+      </xacro:pal_pro_gripper>
+    </xacro:if>
+    <!-- PAL Pro Prototype -->
+    <!-- <xacro:if value="${type == 'pal-pro-gripper-prototype'}">
+      <xacro:include filename="$(find pal_pro_gripper_description)/urdf/pro_gripper_prototype.urdf.xacro" />
+      <xacro:pal_pro_gripper_prototype name="${name}" parent="${parent}">
+        <origin xyz="0.052 0.0 0.0" rpy="0 ${90 * deg_to_rad} 0"/>
+      </xacro:pal_pro_gripper_prototype>
+    </xacro:if> -->
+    <!-- Custom -->
+    <!-- <xacro:if value="${type == 'custom' and not is_dual}">
     <xacro:include filename="$(find custom_ee_description)/urdf/end-effector.urdf.xacro" />
     <xacro:end_effector parent="${parent}">
@@ -39,7 +42,7 @@
     </xacro:end_effector>
   </xacro:if> -->
-  <!-- Custom dual-->
-  <!-- <xacro:if value="${type == 'custom' and is_dual}"> -->
-   <!-- If right -->
+    <!-- Custom dual-->
+    <!-- <xacro:if value="${type == 'custom' and is_dual}"> -->
+    <!-- If right -->
     <!-- <xacro:if value="${reflect == 1}">
     <xacro:include filename="$(find custom_dual_ee_description)/urdf/end-effector-right.urdf.xacro" />
@@ -48,5 +51,5 @@
     </xacro:end_effector_right>
     </xacro:if> -->
-     <!-- If left -->
+    <!-- If left -->
     <!-- <xacro:if value="${reflect == -1}">
     <xacro:include filename="$(find custom_dual_ee_description)/urdf/end-effector-left.urdf.xacro" />

Commit message: FT sensor std

File: pal_sea_arm_description/robots/pal_sea_arm.urdf.xacro (robot description, xacro)
@@ -18,5 +18,5 @@
   <!-- spherical-wrist, straight-wrist -->
   <xacro:arg name="wrist_model" default="spherical-wrist"/>
-  <!-- no-ft-sensor, rokubi-->
+  <!-- no-ft-sensor, rokubi, ati-tc -->
   <xacro:arg name="ft_sensor" default="rokubi"/>
   <!-- pal-sea-arm-standalone, tiago-pro, tiago-sea, tiago-sea-dual -->
@@ -40,5 +40,5 @@
     <xacro:wrong_wrist_model/>
   </xacro:if>
-  <xacro:if value="${ft_sensor not in ['no-ft-sensor', 'rokubi']}">
+  <xacro:if value="${ft_sensor not in ['no-ft-sensor', 'rokubi', 'ati-tc']}">
     <xacro:wrong_ft_sensor/>
   </xacro:if>
@@ -59,6 +59,6 @@
   <!-- Force Torque sensor -->
   <xacro:if value="${has_ft_sensor}">
-    <xacro:include filename="$(find pal_sea_arm_description)/urdf/sensors/ft_sensor.urdf.xacro" />
-    <xacro:include filename="$(find pal_sea_arm_description)/urdf/sensors/ft_sensor.gazebo.xacro" />
+    <xacro:include filename="$(find pal_sea_arm_description)/urdf/sensors/ft_sensor/${ft_sensor}.urdf.xacro" />
+    <xacro:include filename="$(find pal_sea_arm_description)/urdf/sensors/ft_sensor/ft_sensor.gazebo.xacro" />
   </xacro:if>
   <!-- ROBOT DEFINITION -->
@@ -100,5 +100,5 @@
   </xacro:pal_sea_arm>
   <!-- End effector -->
-  <xacro:pal_sea_arm_end_effector name="gripper" parent="${end_effector_link}" type="${end_effector}" tool_changer="${tool_changer}" reflect="1"/>
+  <!-- <xacro:pal_sea_arm_end_effector name="gripper" parent="${end_effector_link}" type="${end_effector}" tool_changer="${tool_changer}" reflect="1"/> -->
   <!-- Force Torque sensor-->
   <xacro:if value="${has_ft_sensor}">

File: pal_sea_arm_description/ros2_control/ros2_control.urdf.xacro (robot description, xacro)
@@ -48,5 +48,5 @@
       <!-- Force Torque sensor -->
       <xacro:if value="${has_ft_sensor}">
-        <xacro:include filename="$(find pal_sea_arm_description)/urdf/sensors/sensors.ros2_control.xacro"/>
+        <xacro:include filename="$(find pal_sea_arm_description)/urdf/sensors/ft_sensor/sensor.ros2_control.xacro"/>
         <xacro:ros2_control_force_torque_sensor name="wrist_ft_sensor"/>
       </xacro:if>

File: pal_sea_arm_description/urdf/arm/arm.urdf.xacro (robot description, xacro)
@@ -231,20 +231,26 @@
     <!--        TOOL           -->
     <!--***********************-->
-    <link name="${name}_tool_link">
-      <xacro:inertial_tool_link reflect="${reflect}"/>
-      <visual>
-        <origin xyz="0.001 0 0" rpy="0 ${90.0 * deg_to_rad} 0" />
-        <geometry>
-          <cylinder radius="0.032" length="0.01"/>
-        </geometry>
-        <material name="pal/DarkGrey"/>
-      </visual>
-      <collision>
-        <origin xyz="0.001 0 0" rpy="0 ${90.0 * deg_to_rad} 0" />
-        <geometry>
-          <cylinder radius="0.032" length="0.01"/>
-        </geometry>
-      </collision>
-    </link>
+    <xacro:if value="${tool_changer}">
+      <link name="${name}_tool_link">
+      </link>
+    </xacro:if>
+    <xacro:unless value="${tool_changer}">
+      <link name="${name}_tool_link">
+        <xacro:inertial_tool_link reflect="${reflect}"/>
+        <visual>
+          <origin xyz="0.001 0 0" rpy="0 ${90.0 * deg_to_rad} 0" />
+          <geometry>
+            <cylinder radius="0.032" length="0.01"/>
+          </geometry>
+          <material name="pal/DarkGrey"/>
+        </visual>
+        <collision>
+          <origin xyz="0.001 0 0" rpy="0 ${90.0 * deg_to_rad} 0" />
+          <geometry>
+            <cylinder radius="0.032" length="0.01"/>
+          </geometry>
+        </collision>
+      </link>
+    </xacro:unless>
     <joint name="${name}_tool_joint" type="fixed">
       <parent link="${name}_7_link" />

File: pal_sea_arm_description/urdf/arm/arm_properties/tiago-pro/spherical-wrist.properties.xacro (robot description, xacro)
@@ -35,5 +35,5 @@
     </xacro:macro>
     <xacro:macro name="origin_joint_tool" params="reflect">
-        <origin xyz="0 0 0.0184" rpy="0 ${-90.0 * deg_to_rad} ${90.0 * deg_to_rad}" />
+        <origin xyz="0 0 0.0184" rpy="0 0 ${-90.0 * deg_to_rad}" />
     </xacro:macro>
 </robot>

File: pal_sea_arm_description/urdf/sensors/ft_sensor/rokubi.urdf.xacro (robot description, xacro)
@@ -14,33 +14,32 @@
 <robot xmlns:xacro="http://ros.org/wiki/xacro">
   <xacro:macro name="ft_sensor" params="name parent">
-    <!--************************-->
-    <!--        ft sensor       -->
-    <!--************************-->
+    <!-- FT DEFINITION -->
+    <!-- Body links -->
     <link name="${name}_ft_link">
-        <inertial>
-          <mass value="0.2657" />
-          <inertia ixx="2.9766E-04" ixy="1.87E-06" ixz="8.95E-06" iyy="3.095E-04" iyz="2.07E-06" izz="1.6632E-04" />
-        </inertial>
-        <visual>
-          <origin xyz="0.0 0.0 0.0" rpy="0.0 0.0 0.0"/>
-          <geometry>
-            <mesh filename="package://pal_sea_arm_description/meshes/sensors/rokubi_ft_sensor.STL"/>
-          </geometry>
-          <material name="">
-            <color rgba="0.29804 0.29804 0.29804 1" />
-          </material>
-        </visual>
-        <collision>
-          <origin xyz="0 0 -0.030" rpy="0 0 0" />
-          <geometry>
-            <cylinder radius="0.035" length="0.05"/>
-          </geometry>
-        </collision>
-        <collision>
-          <origin xyz="0.035 0.011 -0.035" rpy="0 0 ${25.0 * deg_to_rad}" />
-          <geometry>
-            <box size="0.0395 0.0496 0.053"/>
-          </geometry>
-        </collision>
+      <inertial>
+        <mass value="0.2657" />
+        <inertia ixx="2.9766E-04" ixy="1.87E-06" ixz="8.95E-06" iyy="3.095E-04" iyz="2.07E-06" izz="1.6632E-04" />
+      </inertial>
+      <visual>
+        <origin xyz="0.0 0.0 0.0" rpy="0.0 0.0 0.0"/>
+        <geometry>
+          <mesh filename="package://pal_sea_arm_description/meshes/sensors/rokubi/rokubi_ft_sensor.stl"/>
+        </geometry>
+        <material name="">
+          <color rgba="0.29804 0.29804 0.29804 1" />
+        </material>
+      </visual>
+      <collision>
+        <origin xyz="0 0 -0.030" rpy="0 0 0" />
+        <geometry>
+          <cylinder radius="0.035" length="0.05"/>
+        </geometry>
+      </collision>
+      <collision>
+        <origin xyz="0.035 0.011 -0.035" rpy="0 0 ${25.0 * deg_to_rad}" />
+        <geometry>
+          <box size="0.0395 0.0496 0.053"/>
+        </geometry>
+      </collision>
     </link>
     <gazebo reference="${name}_ft_link">
@@ -54,7 +53,5 @@
       <origin xyz="0.045 0 0" rpy="${-90.0 * deg_to_rad} ${45.0 * deg_to_rad} ${-90.0 * deg_to_rad}" />
     </joint>
-    <!--***********************-->
-    <!--       FT TOOL         -->
-    <!--***********************-->
+    <!-- FT tool link -->
     <link name="${name}_ft_tool_link">
       <inertial>
@@ -81,4 +78,4 @@
       <origin xyz="0 0 0.005" rpy="${45.0 * deg_to_rad} ${-90.0 * deg_to_rad} ${0.0 * deg_to_rad}" />
     </joint>
-</xacro:macro>
+  </xacro:macro>
 </robot>
