Commit message: Arms versions std

File: pal_sea_arm_description/robots/pal_sea_arm.urdf.xacro (robot description, xacro)
@@ -40,9 +40,22 @@
     <xacro:wrong_wrist_model/>
   </xacro:if>
-  <xacro:if value="${ft_sensor not in ['no-ft-sensor', 'rokubi', 'ati-tc']}">
+  <xacro:if value="${ft_sensor not in ['no-ft-sensor', 'rokubi', 'ati']}">
     <xacro:wrong_ft_sensor/>
   </xacro:if>
   <xacro:if value="${arm_type not in ['pal-sea-arm-standalone', 'tiago-pro', 'tiago-sea', 'tiago-sea-dual']}">
     <xacro:wrong_arm_type/>
+  </xacro:if>
+  <!-- Compatibility check within TC and ft sensors-->
+  <xacro:if value="${ft_sensor == 'rokubi' and wrist_model=='spherical-wrist'}">
+    <xacro:error_rokubi_not_compatible_with_spherical_wrist />
+  </xacro:if>
+  <xacro:if value="${ft_sensor == 'rokubi' and tool_changer}">
+    <xacro:error_rokubi_not_compatible_with_tc />
+  </xacro:if>
+  <xacro:if value="${ft_sensor == 'ati' and not tool_changer}">
+    <xacro:error_ati_not_compatible_without_tc />
+  </xacro:if>
+  <xacro:if value="${not tool_changer and wrist_model=='spherical-wrist'}">
+    <xacro:error_spherical_wrist_always_comes_with_tc />
   </xacro:if>
   <xacro:property name="has_ft_sensor" value="${ft_sensor != 'no-ft-sensor'}"/>
@@ -99,6 +112,4 @@
     <origin xyz="0 0 0" rpy="0 0 3.1416" />
   </xacro:pal_sea_arm>
-  <!-- End effector -->
-  <!-- <xacro:pal_sea_arm_end_effector name="gripper" parent="${end_effector_link}" type="${end_effector}" tool_changer="${tool_changer}" reflect="1"/> -->
   <!-- Force Torque sensor-->
   <xacro:if value="${has_ft_sensor}">
@@ -106,4 +117,6 @@
     <!-- <xacro:force_torque_sensor_gazebo name="wrist_ft" update_rate="100"/>-->
   </xacro:if>
+  <!-- End effector -->
+  <!-- <xacro:pal_sea_arm_end_effector name="gripper" parent="${end_effector_link}" type="${end_effector}" tool_changer="${tool_changer}" reflect="1"/> -->
   <!-- ROS2 control -->
   <xacro:pal_sea_arm_ros2_control use_sim="$(arg use_sim)" />

File: pal_sea_arm_description/urdf/arm/arm.urdf.xacro (robot description, xacro)
@@ -26,5 +26,5 @@
       <xacro:property name="mesh_folder" value="arm_tiago_sea"/>
     </xacro:if>
-    <!-- Compatibility check -->
+    <!-- Compatibility check with wrist model -->
     <xacro:if value="${arm_type == 'tiago-sea' and wrist_model=='spherical-wrist'}">
       <xacro:error_wrist_not_supported />
@@ -233,22 +233,24 @@
     <xacro:if value="${tool_changer}">
       <link name="${name}_tool_link">
+        <xacro:inertial_tool_link reflect="${reflect}"/>
+        <visual>
+          <origin xyz="0 0 0" rpy="0 0 0" />
+          <geometry>
+            <mesh filename="package://pal_sea_arm_description/meshes/${mesh_folder}/tool_changer_link.stl" scale="1 1 ${reflect}" />
+          </geometry>
+          <material name="">
+            <color rgba="0.29804 0.29804 0.29804 1" />
+          </material>
+        </visual>
+        <collision>
+          <origin xyz="0 0 0" rpy="0 0 0" />
+          <geometry>
+            <mesh filename="package://pal_sea_arm_description/meshes/${mesh_folder}/tool_changer_link_collision.stl" scale="1 1 ${reflect}" />
+          </geometry>
+        </collision>
       </link>
     </xacro:if>
     <xacro:unless value="${tool_changer}">
       <link name="${name}_tool_link">
-        <xacro:inertial_tool_link reflect="${reflect}"/>
-        <visual>
-          <origin xyz="0.001 0 0" rpy="0 ${90.0 * deg_to_rad} 0" />
-          <geometry>
-            <cylinder radius="0.032" length="0.01"/>
-          </geometry>
-          <material name="pal/DarkGrey"/>
-        </visual>
-        <collision>
-          <origin xyz="0.001 0 0" rpy="0 ${90.0 * deg_to_rad} 0" />
-          <geometry>
-            <cylinder radius="0.032" length="0.01"/>
-          </geometry>
-        </collision>
       </link>
     </xacro:unless>

File: pal_sea_arm_description/urdf/arm/arm_properties/tiago-pro/arm.properties.xacro (robot description, xacro)
@@ -2,14 +2,14 @@
     <xacro:macro name="inertial_base_link" params="reflect">
         <inertial>
-            <origin xyz="-0.000527606405055313 -0.000692372885949076 -0.0125753324897326" rpy="0 0 0" />
-            <mass value="0.76083968294432" />
-            <inertia ixx="0.000525234695448594" ixy="-8.98818311578796E-06" ixz="-8.92750549423532E-06" iyy="0.000521918163120007" iyz="-6.40745645487785E-06" izz="0.000548487715399327" />
+            <origin xyz="-0.00069237 0.00052761 -0.012575" rpy="0 0 0" />
+            <mass value="0.76084" />
+            <inertia ixx="0.00052192" ixy="8.9882E-06" ixz="-6.4075E-06" iyy="0.00052523" iyz="8.9275E-06" izz="0.00054849" />
         </inertial>
     </xacro:macro>
     <xacro:macro name="inertial_link_1" params="reflect">
         <inertial>
-            <origin xyz="-0.016184 0.0043916 0.15576" rpy="0 0 0" />
+            <origin xyz="0.0043916 0.016184 0.15576" rpy="0 0 0" />
             <mass value="1.1325" />
-            <inertia ixx="0.0023517" ixy="-2.6206E-05" ixz="0.00020617" iyy="0.0025497" iyz="6.2082E-05" izz="0.00097131" />
+            <inertia ixx="0.0025497" ixy="2.6206E-05" ixz="6.2082E-05" iyy="0.0023517" iyz="-0.00020617" izz="0.00097131" />
         </inertial>
     </xacro:macro>

File: pal_sea_arm_description/urdf/arm/arm_properties/tiago-pro/spherical-wrist.properties.xacro (robot description, xacro)
@@ -9,7 +9,7 @@
     <xacro:macro name="inertial_link_6" params="reflect">
         <inertial>
-            <origin xyz="0.031759 -0.0065118 -0.0408" rpy="0 0 0" />
-            <mass value="1.3455" />
-            <inertia ixx="0.0010983" ixy="-0.00012999" ixz="-5.9554E-06" iyy="0.0011642" iyz="-4.7964E-07" izz="0.0011896" />
+            <origin xyz="-0.0083923 -0.00081501 0.039899" rpy="0 0 0" />
+            <mass value="0.83518" />
+            <inertia ixx="0.00077706" ixy="-0.00012999" ixz="-5.9554E-06" iyy="0.00094237" iyz="-1.5002E-06" izz="0.00086922" />
         </inertial>
     </xacro:macro>
@@ -19,7 +19,7 @@
     <xacro:macro name="inertial_link_7" params="reflect">
         <inertial>
-            <origin xyz="0.0019481 0.0017558 0.0085066" rpy="0 0 0" />
-            <mass value="0.12272" />
-            <inertia ixx="5.1385E-05" ixy="8.5364E-07" ixz="-9.0329E-08" iyy="4.7962E-05" iyz="-1.8035E-07" izz="9.2935E-05" />
+            <origin xyz="2.1788E-15 7.5568E-05 -0.037565" rpy="0 0 0" />
+            <mass value="0.51032" />
+            <inertia ixx="0.00032121" ixy="-1.7628E-21" ixz="-7.178E-21" iyy="0.00032034" iyz="-1.0206E-06" izz="0.00022179" />
         </inertial>
     </xacro:macro>
@@ -27,13 +27,14 @@
         <origin xyz="0.07 -0.0534 -0.0422" rpy="1.5708 0 0" />
     </xacro:macro>
+    <!-- Tool changer -->
     <xacro:macro name="inertial_tool_link" params="reflect">
         <inertial>
-            <origin xyz="5.0493E-18 -4.4892E-17 -0.0068514" rpy="0 0 0" />
-            <mass value="0.10189" />
-            <inertia ixx="5.1076E-05" ixy="-1.0374E-21" ixz="-5.9164E-21" iyy="5.0882E-05" iyz="-8.5211E-21" izz="9.705E-05" />
+            <origin xyz="0.0019481 0.0017558 -0.0084934" rpy="0 0 0" />
+            <mass value="0.12272" />
+            <inertia ixx="5.1385E-05" ixy="8.5364E-07" ixz="-9.0329E-08" iyy="4.7962E-05" iyz="-1.8035E-07" izz="9.2935E-05" />
         </inertial>
     </xacro:macro>
     <xacro:macro name="origin_joint_tool" params="reflect">
-        <origin xyz="0 0 0.0184" rpy="0 0 ${-90.0 * deg_to_rad}" />
+        <origin xyz="0 0 0.017" rpy="0 0 0" />
     </xacro:macro>
 </robot>

File: pal_sea_arm_description/urdf/arm/arm_properties/tiago-pro/straight-wrist.properties.xacro (robot description, xacro)
@@ -2,38 +2,39 @@
     <xacro:macro name="inertial_link_5" params="reflect">
         <inertial>
-            <origin xyz="0.0004859 0.00014289 0.129" rpy="0 0 0" />
-            <mass value="0.52538" />
-            <inertia ixx="0.0019111" ixy="-1.4245E-08" ixz="3.8663E-05" iyy="0.0018565" iyz="1.1356E-06" izz="0.00046496" />
+            <origin xyz="8.9806E-06 -0.00053878 0.13058" rpy="0 0 0" />
+            <mass value="0.84847" />
+            <inertia ixx="0.0020531" ixy="-8.9232E-07" ixz="1.6668E-06" iyy="0.0020434" iyz="3.7824E-05" izz="0.00067121" />
         </inertial>
     </xacro:macro>
     <xacro:macro name="inertial_link_6" params="reflect">
         <inertial>
-            <origin xyz="-0.086822 -7.7905E-06 0.0045258" rpy="0 0 0" />
-            <mass value="0.66725" />
-            <inertia ixx="0.00035696" ixy="1.6019E-07" ixz="-9.5191E-05" iyy="0.00073846" iyz="2.118E-08" izz="0.00075321" />
+            <origin xyz="-0.016007 0.052767 3.7676E-05" rpy="0 0 0" />
+            <mass value="0.15792" />
+            <inertia ixx="0.00043323" ixy="9.3978E-05" ixz="-2.1216E-08" iyy="0.00013569" iyz="1.5995E-07" izz="0.00041746" />
         </inertial>
     </xacro:macro>
     <xacro:macro name="origin_joint_6" params="reflect">
-        <origin xyz="0 0 0.165" rpy="0 1.5708 -1.57" />
+        <origin xyz="0 0.0354 0.16489" rpy="1.5708 0 1.5708" />
     </xacro:macro>
     <xacro:macro name="inertial_link_7" params="reflect">
         <inertial>
-            <origin xyz="-6.764E-18 -1.4549E-16 0.018549" rpy="0 0 0" />
-            <mass value="0.10189" />
-            <inertia ixx="5.1076E-05" ixy="-1.0899E-21" ixz="-5.93E-21" iyy="5.0882E-05" iyz="-8.5344E-21" izz="9.705E-05" />
+            <origin xyz="-7.5568E-05 1.3009E-17 -0.037565" rpy="0 0 0" />
+            <mass value="0.51032" />
+            <inertia ixx="0.00032034" ixy="-7.8169E-21" ixz="1.0206E-06" iyy="0.00032121" iyz="7.188E-20" izz="0.00022179" />
         </inertial>
     </xacro:macro>
     <xacro:macro name="origin_joint_7" params="reflect">
-        <origin xyz="-0.1166 0 0" rpy="0 -1.5708 0" />
+        <origin xyz="-0.0354 0.135 0" rpy="-1.5708 0 0" />
     </xacro:macro>
+    <!-- Tool changer -->
     <xacro:macro name="inertial_tool_link" params="reflect">
         <inertial>
-            <origin xyz="5.0493E-18 -4.4892E-17 -0.0068514" rpy="0 0 0" />
-            <mass value="0.10189" />
-            <inertia ixx="5.1076E-05" ixy="-1.0374E-21" ixz="-5.9164E-21" iyy="5.0882E-05" iyz="-8.5211E-21" izz="9.705E-05" />
+            <origin xyz="0.0019481 0.0017558 -0.0084934" rpy="0 0 0" />
+            <mass value="0.12272" />
+            <inertia ixx="5.1385E-05" ixy="8.5364E-07" ixz="-9.0329E-08" iyy="4.7962E-05" iyz="-1.8035E-07" izz="9.2935E-05" />
         </inertial>
     </xacro:macro>
     <xacro:macro name="origin_joint_tool" params="reflect">
-        <origin xyz="0 0 0.0184" rpy="0 ${-90.0 * deg_to_rad} ${90.0 * deg_to_rad}" />
+        <origin xyz="0 0 0.017" rpy="0 0 0" />
     </xacro:macro>
 </robot>

Commit message: No TC working for all combinations

File: pal_sea_arm_description/robots/pal_sea_arm.urdf.xacro (robot description, xacro)
@@ -118,5 +118,5 @@
   </xacro:if>
   <!-- End effector -->
-  <!-- <xacro:pal_sea_arm_end_effector name="gripper" parent="${end_effector_link}" type="${end_effector}" tool_changer="${tool_changer}" reflect="1"/> -->
+  <xacro:pal_sea_arm_end_effector name="gripper" parent="${end_effector_link}" type="${end_effector}" tool_changer="${tool_changer}" reflect="1"/>
   <!-- ROS2 control -->
   <xacro:pal_sea_arm_ros2_control use_sim="$(arg use_sim)" />

File: pal_sea_arm_description/urdf/arm/arm.urdf.xacro (robot description, xacro)
@@ -231,7 +231,8 @@
     <!--        TOOL           -->
     <!--***********************-->
+    <!-- With tool changer (the tool link is the tool changer)-->
     <xacro:if value="${tool_changer}">
       <link name="${name}_tool_link">
-        <xacro:inertial_tool_link reflect="${reflect}"/>
+        <xacro:inertial_tool_changer_link reflect="${reflect}"/>
         <visual>
           <origin xyz="0 0 0" rpy="0 0 0" />
@@ -250,14 +251,19 @@
         </collision>
       </link>
-    </xacro:if>
+      <joint name="${name}_tool_joint" type="fixed">
+        <parent link="${name}_7_link" />
+        <child link="${name}_tool_link" />
+        <xacro:origin_joint_tool_changer reflect="${reflect}"/>
+      </joint>
+    </xacro:if>
+    <!-- Without tool changer (tool link just on top of link 7)-->
     <xacro:unless value="${tool_changer}">
       <link name="${name}_tool_link">
       </link>
+      <joint name="${name}_tool_joint" type="fixed">
+        <parent link="${name}_7_link" />
+        <child link="${name}_tool_link" />
+      </joint>
     </xacro:unless>
-    <joint name="${name}_tool_joint" type="fixed">
-      <parent link="${name}_7_link" />
-      <child link="${name}_tool_link" />
-      <xacro:origin_joint_tool reflect="${reflect}"/>
-    </joint>
     <gazebo reference="${name}_1_link">
       <material>Gazebo/DarkGrey</material>

File: pal_sea_arm_description/urdf/arm/arm_properties/tiago-pro/arm.properties.xacro (robot description, xacro)
@@ -50,3 +50,15 @@
         <origin xyz="-0.0199999999999971 0.17011 -0.037110000000002" rpy="-1.5707963267949 0 0" />
     </xacro:macro>
+    <!-- Tool changer (can be present in both wrists)-->
+    <xacro:macro name="inertial_tool_changer_link" params="reflect">
+        <inertial>
+            <origin xyz="0.0019481 0.0017558 -0.0084934" rpy="0 0 0" />
+            <mass value="0.12272" />
+            <inertia ixx="5.1385E-05" ixy="8.5364E-07" ixz="-9.0329E-08" iyy="4.7962E-05" iyz="-1.8035E-07" izz="9.2935E-05" />
+        </inertial>
+    </xacro:macro>
+    <xacro:macro name="origin_joint_tool_changer" params="reflect">
+        <!-- @Lucien needs to fix -->
+        <origin xyz="0 0 0.017" rpy="0 0 0" />
+    </xacro:macro>
 </robot>

File: pal_sea_arm_description/urdf/arm/arm_properties/tiago-pro/spherical-wrist.properties.xacro (robot description, xacro)
@@ -27,14 +27,3 @@
         <origin xyz="0.07 -0.0534 -0.0422" rpy="1.5708 0 0" />
     </xacro:macro>
-    <!-- Tool changer -->
-    <xacro:macro name="inertial_tool_link" params="reflect">
-        <inertial>
-            <origin xyz="0.0019481 0.0017558 -0.0084934" rpy="0 0 0" />
-            <mass value="0.12272" />
-            <inertia ixx="5.1385E-05" ixy="8.5364E-07" ixz="-9.0329E-08" iyy="4.7962E-05" iyz="-1.8035E-07" izz="9.2935E-05" />
-        </inertial>
-    </xacro:macro>
-    <xacro:macro name="origin_joint_tool" params="reflect">
-        <origin xyz="0 0 0.017" rpy="0 0 0" />
-    </xacro:macro>
 </robot>

File: pal_sea_arm_description/urdf/arm/arm_properties/tiago-pro/straight-wrist.properties.xacro (robot description, xacro)
@@ -27,14 +27,3 @@
         <origin xyz="-0.0354 0.135 0" rpy="-1.5708 0 0" />
     </xacro:macro>
-    <!-- Tool changer -->
-    <xacro:macro name="inertial_tool_link" params="reflect">
-        <inertial>
-            <origin xyz="0.0019481 0.0017558 -0.0084934" rpy="0 0 0" />
-            <mass value="0.12272" />
-            <inertia ixx="5.1385E-05" ixy="8.5364E-07" ixz="-9.0329E-08" iyy="4.7962E-05" iyz="-1.8035E-07" izz="9.2935E-05" />
-        </inertial>
-    </xacro:macro>
-    <xacro:macro name="origin_joint_tool" params="reflect">
-        <origin xyz="0 0 0.017" rpy="0 0 0" />
-    </xacro:macro>
 </robot>

File: pal_sea_arm_description/urdf/end_effector/end_effector.urdf.xacro (robot description, xacro)
@@ -25,5 +25,5 @@
       <xacro:include filename="$(find pal_pro_gripper_description)/urdf/gripper.urdf.xacro" />
       <xacro:pal_pro_gripper name="${name}" parent="${parent}" tool_changer="${tool_changer}">
-        <origin xyz="0.0 0.0 0.0" rpy="0 ${90 * deg_to_rad} 0"/>
+        <origin xyz="0.0 0.0 -0.01" rpy="0 0 0"/>
       </xacro:pal_pro_gripper>
     </xacro:if>

File: pal_sea_arm_description/urdf/sensors/ft_sensor/ati.urdf.xacro (robot description, xacro)
@@ -25,5 +25,5 @@
         <origin xyz="0 0 0" rpy="0 0 0" />
         <geometry>
-          <mesh filename="package://pal_sea_arm_description/meshes/sensors/ati_tc/base_link.stl"/>
+          <mesh filename="package://pal_sea_arm_description/meshes/sensors/ati/base_link.stl"/>
         </geometry>
         <material name="">
@@ -34,5 +34,5 @@
         <origin xyz="0 0 0" rpy="0 0 0" />
         <geometry>
-          <mesh filename="package://pal_sea_arm_description/meshes/sensors/ati_tc/base_link.stl"/>
+          <mesh filename="package://pal_sea_arm_description/meshes/sensors/ati/base_link.stl"/>
         </geometry>
       </collision>
@@ -53,5 +53,5 @@
         <origin xyz="0 0 0" rpy="0 0 0" />
         <geometry>
-          <mesh filename="package://pal_sea_arm_description/meshes/sensors/ati_tc/ft_sensor_link.stl"/>
+          <mesh filename="package://pal_sea_arm_description/meshes/sensors/ati/ft_sensor_link.stl"/>
         </geometry>
         <material name="">
@@ -62,10 +62,10 @@
         <origin xyz="0 0 0" rpy="0 0 0" />
         <geometry>
-          <mesh filename="package://pal_sea_arm_description/meshes/sensors/ati_tc/ft_sensor_link.stl"/>
+          <mesh filename="package://pal_sea_arm_description/meshes/sensors/ati/ft_sensor_link.stl"/>
         </geometry>
       </collision>
     </link>
     <joint name="ft_sensor_joint" type="fixed">
-      <origin xyz="0 0 0.033998" rpy="0 0 0" />
+      <!-- <origin xyz="0 0 0.033998" rpy="0 0 0" /> -->
       <parent link="${name}_ft_sensor_base_link" />
       <child link="${name}_ft_sensor_link" />
@@ -82,5 +82,5 @@
         <origin xyz="0 0 0" rpy="0 0 0" />
         <geometry>
-          <mesh filename="package://pal_sea_arm_description/meshes/sensors/ati_tc/ft_out_link.stl"/>
+          <mesh filename="package://pal_sea_arm_description/meshes/sensors/ati/ft_out_link.stl"/>
         </geometry>
         <material name="">
@@ -91,5 +91,5 @@
         <origin xyz="0 0 0" rpy="0 0 0" />
         <geometry>
-          <mesh filename="package://pal_sea_arm_description/meshes/sensors/ati_tc/ft_out_link.stl"/>
+          <mesh filename="package://pal_sea_arm_description/meshes/sensors/ati/ft_out_link.stl"/>
         </geometry>
       </collision>

File: pal_sea_arm_description/urdf/sensors/ft_sensor/rokubi.urdf.xacro (robot description, xacro)
@@ -51,5 +51,5 @@
       <parent link="${parent}" />
       <child link="${name}_ft_link" />
-      <origin xyz="0.045 0 0" rpy="${-90.0 * deg_to_rad} ${45.0 * deg_to_rad} ${-90.0 * deg_to_rad}" />
+      <origin xyz="0 0 0.04" rpy="0 0 0" />
     </joint>
     <!-- FT tool link -->
@@ -60,5 +60,5 @@
       </inertial>
       <visual>
-        <origin xyz="0.001 0 0" rpy="0 ${90.0 * deg_to_rad} 0" />
+        <origin xyz="0.001 0 0" rpy="0 0 0" />
         <geometry>
           <cylinder radius="0.032" length="0.01"/>
@@ -67,5 +67,5 @@
       </visual>
       <collision>
-        <origin xyz="0.001 0 0" rpy="0 ${90.0 * deg_to_rad} 0" />
+        <origin xyz="0.001 0 0" rpy="0 0 0" />
         <geometry>
           <cylinder radius="0.032" length="0.01"/>
@@ -76,5 +76,4 @@
       <parent link="${name}_ft_link" />
       <child link="${name}_ft_tool_link" />
-      <origin xyz="0 0 0.005" rpy="${45.0 * deg_to_rad} ${-90.0 * deg_to_rad} ${0.0 * deg_to_rad}" />
     </joint>
   </xacro:macro>

Commit message: Final checks

File: pal_sea_arm_description/robots/pal_sea_arm.urdf.xacro (robot description, xacro)
@@ -109,5 +109,5 @@
   </gazebo>
   <!-- ARM -->
-  <xacro:pal_sea_arm name="arm" parent="arm_root_link" arm_type="${arm_type}" wrist_model="${wrist_model}" reflect="1" arm_1_offset="0" arm_2_offset="0" arm_3_offset="0" arm_4_offset="0" arm_5_offset="0" arm_6_offset="0" arm_7_offset="0">
+  <xacro:pal_sea_arm name="arm" parent="arm_root_link" arm_type="${arm_type}" tool_changer="${tool_changer}" wrist_model="${wrist_model}" reflect="1" arm_1_offset="0" arm_2_offset="0" arm_3_offset="0" arm_4_offset="0" arm_5_offset="0" arm_6_offset="0" arm_7_offset="0">
     <origin xyz="0 0 0" rpy="0 0 3.1416" />
   </xacro:pal_sea_arm>

File: pal_sea_arm_description/urdf/arm/arm.urdf.xacro (robot description, xacro)
@@ -14,5 +14,5 @@
 <robot xmlns:xacro="http://ros.org/wiki/xacro">
   <!-- Transmissions file -->
-  <xacro:macro name="pal_sea_arm" params="name parent *origin arm_type wrist_model reflect:=1 arm_1_offset arm_2_offset arm_3_offset arm_4_offset arm_5_offset arm_6_offset arm_7_offset no_safety_eps:=False">
+  <xacro:macro name="pal_sea_arm" params="name parent *origin arm_type tool_changer wrist_model reflect:=1 arm_1_offset arm_2_offset arm_3_offset arm_4_offset arm_5_offset arm_6_offset arm_7_offset no_safety_eps:=False">
     <!-- PROPERTIES -->
     <xacro:property name="arm_eps" value="${0.00 if no_safety_eps else 0.07}"/>

File: pal_sea_arm_description/urdf/sensors/ft_sensor/ati.urdf.xacro (robot description, xacro)
@@ -66,5 +66,5 @@
       </collision>
     </link>
-    <joint name="ft_sensor_joint" type="fixed">
+    <joint name="${name}_ft_sensor_joint" type="fixed">
       <!-- <origin xyz="0 0 0.033998" rpy="0 0 0" /> -->
       <parent link="${name}_ft_sensor_base_link" />

Commit message: Support for different FT models at the same time

File: pal_sea_arm_description/robots/pal_sea_arm.urdf.xacro (robot description, xacro)
@@ -72,5 +72,5 @@
   <!-- Force Torque sensor -->
   <xacro:if value="${has_ft_sensor}">
-    <xacro:include filename="$(find pal_sea_arm_description)/urdf/sensors/ft_sensor/${ft_sensor}.urdf.xacro" />
+    <xacro:include filename="$(find pal_sea_arm_description)/urdf/sensors/ft_sensor/ft_sensor.urdf.xacro" />
     <xacro:include filename="$(find pal_sea_arm_description)/urdf/sensors/ft_sensor/ft_sensor.gazebo.xacro" />
   </xacro:if>
@@ -114,5 +114,5 @@
   <!-- Force Torque sensor-->
   <xacro:if value="${has_ft_sensor}">
-    <xacro:ft_sensor name="wrist" parent="arm_tool_link"/>
+    <xacro:ft_sensor type="${ft_sensor}" name="wrist" parent="arm_tool_link"/>
     <!-- <xacro:force_torque_sensor_gazebo name="wrist_ft" update_rate="100"/>-->
   </xacro:if>

File: pal_sea_arm_description/urdf/sensors/ft_sensor/ati.urdf.xacro (robot description, xacro)
@@ -13,5 +13,5 @@
 -->
 <robot xmlns:xacro="http://ros.org/wiki/xacro">
-  <xacro:macro name="ft_sensor" params="tool_changer:=False name parent">
+  <xacro:macro name="ft_sensor" params="name parent">
     <!-- FT DEFINITION -->
     <!-- Base link -->
