Commit message: Removing checks

File: pal_sea_arm_description/robots/pal_sea_arm.urdf.xacro (robot description, xacro)
@@ -47,5 +47,5 @@
   </xacro:if>
   <!-- Compatibility check within TC and ft sensors-->
-  <xacro:if value="${ft_sensor == 'rokubi' and wrist_model=='spherical-wrist'}">
+  <!-- <xacro:if value="${ft_sensor == 'rokubi' and wrist_model=='spherical-wrist'}">
     <xacro:error_rokubi_not_compatible_with_spherical_wrist />
   </xacro:if>
@@ -58,5 +58,5 @@
   <xacro:if value="${not tool_changer and wrist_model=='spherical-wrist'}">
     <xacro:error_spherical_wrist_always_comes_with_tc />
-  </xacro:if>
+  </xacro:if> -->
   <xacro:property name="has_ft_sensor" value="${ft_sensor != 'no-ft-sensor'}"/>
   <xacro:property name="has_end_effector" value="${end_effector not in ['no-end-effector']}"/>

File: pal_sea_arm_description/urdf/arm/arm.urdf.xacro (robot description, xacro)
@@ -31,10 +31,10 @@
     </xacro:if>
     <!-- Compatibility check with wrist model -->
-    <xacro:if value="${arm_type == 'tiago-sea' and wrist_model=='spherical-wrist'}">
+    <!-- <xacro:if value="${arm_type == 'tiago-sea' and wrist_model=='spherical-wrist'}">
       <xacro:error_wrist_not_supported />
     </xacro:if>
     <xacro:if value="${arm_type == 'tiago-sea-dual' and wrist_model=='spherical-wrist'}">
       <xacro:error_wrist_not_supported />
-    </xacro:if>
+    </xacro:if> -->
     <!-- INCLUDES -->
     <xacro:include filename="$(find pal_sea_arm_description)/urdf/arm/limits/arm_${arm_type}.limits.xacro"/>
@@ -269,5 +269,5 @@
         <child link="${name}_tool_link" />
         <!-- This is added so both grippers are oriented the same -->
-        <origin xyz="0 0 0" rpy="0 0 1.570796" />
+        <!-- <origin xyz="0 0 0.0" rpy="0 0 1.570796" /> -->
       </joint>
     </xacro:unless>

File: pal_sea_arm_description/urdf/arm/arm_properties/tiago-pro/arm.properties.xacro (robot description, xacro)
@@ -60,5 +60,5 @@
     <xacro:macro name="origin_joint_tool_changer" params="reflect">
         <!-- @Lucien needs to fix -->
-        <origin xyz="0 0 0.017" rpy="0 0 1.570796" />
+        <origin xyz="0 0 0.017" rpy="0 0 0" />
     </xacro:macro>
 </robot>

Commit message: Add Inertia version for the new arm

File: pal_sea_arm_description/robots/pal_sea_arm.urdf.xacro (robot description, xacro)
@@ -43,5 +43,5 @@
     <xacro:wrong_ft_sensor/>
   </xacro:if>
-  <xacro:if value="${arm_type not in ['pal-sea-arm-standalone', 'tiago-pro', 'tiago-sea', 'tiago-sea-dual']}">
+  <xacro:if value="${arm_type not in ['pal-sea-arm-standalone', 'tiago-pro', 'tiago-pro-s',  'tiago-sea', 'tiago-sea-dual']}">
     <xacro:wrong_arm_type/>
   </xacro:if>

File: pal_sea_arm_description/urdf/arm/arm.urdf.xacro (robot description, xacro)
@@ -19,6 +19,8 @@
     <xacro:property name="mesh_folder"/>
     <!-- Tiago Pro -->
-    <xacro:if value="${arm_type in ['tiago-pro', 'pal-sea-arm-standalone']}">
+    <xacro:if value="${arm_type in ['tiago-pro', 'tiago-pro-s']}">
       <xacro:property name="mesh_folder" value="arm_tiago_pro"/>
+      <xacro:property name="inertia_version" value="${arm_type}"/>
+      <xacro:property name="arm_type" value="tiago-pro"/>
     </xacro:if>
     <!-- Standalone arm -->

File: pal_sea_arm_description/urdf/arm/arm_properties/tiago-pro/arm.properties.xacro (robot description, xacro)
@@ -1,16 +1,34 @@
 <robot xmlns:xacro="http://ros.org/wiki/xacro">
     <xacro:macro name="inertial_base_link" params="reflect">
-        <inertial>
-            <origin xyz="-0.00069237 0.00052761 -0.012575" rpy="0 0 0" />
-            <mass value="0.76084" />
-            <inertia ixx="0.00052192" ixy="8.9882E-06" ixz="-6.4075E-06" iyy="0.00052523" iyz="8.9275E-06" izz="0.00054849" />
-        </inertial>
+        <xacro:if value="${inertia_version in ['tiago-pro-s']}">
+            <inertial>
+                <origin xyz="-0.00069 0.00053 -0.01258" rpy="0 0 0" />
+                <mass value="0.76084" />
+                <inertia ixx="0.00054" ixy="0.00001" ixz="-0.00001" iyy="0.00055" iyz="0.00001" izz="0.00055" />
+            </inertial>
+        </xacro:if>
+        <xacro:if value="${inertia_version in ['tiago-pro']}">
+            <inertial>
+                <origin xyz="-0.00069237 0.00052761 -0.012575" rpy="0 0 0" />
+                <mass value="0.76084" />
+                <inertia ixx="0.00052192" ixy="8.9882E-06" ixz="-6.4075E-06" iyy="0.00052523" iyz="8.9275E-06" izz="0.00054849" />
+            </inertial>
+        </xacro:if>
     </xacro:macro>
     <xacro:macro name="inertial_link_1" params="reflect">
-        <inertial>
-            <origin xyz="0.0043916 0.016184 0.15576" rpy="0 0 0" />
-            <mass value="1.1325" />
-            <inertia ixx="0.0025497" ixy="2.6206E-05" ixz="6.2082E-05" iyy="0.0023517" iyz="-0.00020617" izz="0.00097131" />
-        </inertial>
+        <xacro:if value="${inertia_version in ['tiago-pro-s']}">
+            <inertial>
+                <origin xyz="0.00476 0.01532 0.15274" rpy="0 0 0" />
+                <mass value="1.21459" />
+                <inertia ixx="0.00434" ixy="0.00004" ixz="0.00016" iyy="0.00421" iyz="-0.00051" izz="0.00121" />
+            </inertial>
+        </xacro:if>
+        <xacro:if value="${inertia_version in ['tiago-pro']}">
+            <inertial>
+                <origin xyz="0.0043916 0.016184 0.15576" rpy="0 0 0" />
+                <mass value="1.1325" />
+                <inertia ixx="0.0025497" ixy="2.6206E-05" ixz="6.2082E-05" iyy="0.0023517" iyz="-0.00020617" izz="0.00097131" />
+            </inertial>
+        </xacro:if>
     </xacro:macro>
     <xacro:macro name="origin_joint_1" params="reflect">
@@ -18,9 +36,18 @@
     </xacro:macro>
     <xacro:macro name="inertial_link_2" params="reflect">
-        <inertial>
-            <origin xyz="0.01786 -0.11956 -0.032097" rpy="0 0 0" />
-            <mass value="1.0436" />
-            <inertia ixx="0.0015021" ixy="0.00011264" ixz="1.0692E-05" iyy="0.00088017" iyz="-0.00015843" izz="0.0016021" />
-        </inertial>
+        <xacro:if value="${inertia_version in ['tiago-pro-s']}">
+            <inertial>
+                <origin xyz="0.01715 -0.11231 -0.03000" rpy="0 0 0" />
+                <mass value="1.13101" />
+                <inertia ixx="0.00357" ixy="0.00029" ixz="0.00007" iyy="0.00117" iyz="-0.00068" izz="0.00352" />
+            </inertial>
+        </xacro:if>
+        <xacro:if value="${inertia_version in ['tiago-pro']}">
+            <inertial>
+                <origin xyz="0.01786 -0.11956 -0.032097" rpy="0 0 0" />
+                <mass value="1.0436" />
+                <inertia ixx="0.0015021" ixy="0.00011264" ixz="1.0692E-05" iyy="0.00088017" iyz="-0.00015843" izz="0.0016021" />
+            </inertial>
+        </xacro:if>
     </xacro:macro>
     <xacro:macro name="origin_joint_2" params="reflect">
@@ -28,9 +55,18 @@
     </xacro:macro>
     <xacro:macro name="inertial_link_3" params="reflect">
-        <inertial>
-            <origin xyz="0.016184 -0.0043916 0.13565" rpy="0 0 0" />
-            <mass value="1.1325" />
-            <inertia ixx="0.0023517" ixy="-2.6206E-05" ixz="-0.00020617" iyy="0.0025497" iyz="-6.2082E-05" izz="0.00097131" />
-        </inertial>
+        <xacro:if value="${inertia_version in ['tiago-pro-s']}">
+            <inertial>
+                <origin xyz="0.01530 -0.00471 0.13242" rpy="0 0 0" />
+                <mass value="1.21628" />
+                <inertia ixx="0.00425" ixy="-0.00004" ixz="-0.00051" iyy="0.00437" iyz="-0.00015" izz="0.00121" />
+            </inertial>
+        </xacro:if>
+        <xacro:if value="${inertia_version in ['tiago-pro']}">
+            <inertial>
+                <origin xyz="0.016184 -0.0043916 0.13565" rpy="0 0 0" />
+                <mass value="1.1325" />
+                <inertia ixx="0.0023517" ixy="-2.6206E-05" ixz="-0.00020617" iyy="0.0025497" iyz="-6.2082E-05" izz="0.00097131" />
+            </inertial>
+        </xacro:if>
     </xacro:macro>
     <xacro:macro name="origin_joint_3" params="reflect">
@@ -38,9 +74,18 @@
     </xacro:macro>
     <xacro:macro name="inertial_link_4" params="reflect">
-        <inertial>
-            <origin xyz="-0.01786 0.11956 -0.032097" rpy="0 0 0" />
-            <mass value="1.0436" />
-            <inertia ixx="0.0015021" ixy="0.00011264" ixz="-1.0692E-05" iyy="0.00088017" iyz="0.00015843" izz="0.0016021" />
-        </inertial>
+        <xacro:if value="${inertia_version in ['tiago-pro-s']}">
+            <inertial>
+                <origin xyz="-0.01715 0.11231 -0.03000" rpy="0 0 0" />
+                <mass value="1.13101" />
+                <inertia ixx="0.00357" ixy="0.00029" ixz="-0.00007" iyy="0.00117" iyz="0.00068" izz="0.00352" />
+            </inertial>
+        </xacro:if>
+        <xacro:if value="${inertia_version in ['tiago-pro']}">
+            <inertial>
+                <origin xyz="-0.01786 0.11956 -0.032097" rpy="0 0 0" />
+                <mass value="1.0436" />
+                <inertia ixx="0.0015021" ixy="0.00011264" ixz="-1.0692E-05" iyy="0.00088017" iyz="0.00015843" izz="0.0016021" />
+            </inertial>
+        </xacro:if>
     </xacro:macro>
     <xacro:macro name="origin_joint_4" params="reflect">

File: pal_sea_arm_description/urdf/arm/arm_properties/tiago-pro/spherical-wrist.properties.xacro (robot description, xacro)
@@ -1,9 +1,18 @@
 <robot xmlns:xacro="http://ros.org/wiki/xacro">
     <xacro:macro name="inertial_link_5" params="reflect">
-        <inertial>
-            <origin xyz="1.1053306160504E-05 -0.027586177392457 0.067845360860401" rpy="0 0 0" />
-            <mass value="0.310763344920608" />
-            <inertia ixx="0.001401450896582" ixy="9.16506225733395E-08" ixz="-9.26253840796548E-08" iyy="0.001399994200261" iyz="0.000327712970358816" izz="0.000402007894416599" />
-        </inertial>
+        <xacro:if value="${inertia_version in ['tiago-pro-s']}">
+            <inertial>
+                <origin xyz="0.00017 -0.02738 0.06749" rpy="0 0 0" />
+                <mass value="0.31298" />
+                <inertia ixx="0.00157" ixy="0.00000" ixz="0.00000" iyy="0.00154" iyz="-0.00038" izz="0.00043" />
+            </inertial>
+        </xacro:if>
+        <xacro:if value="${inertia_version in ['tiago-pro']}">
+            <inertial>
+                <origin xyz="1.1053306160504E-05 -0.027586177392457 0.067845360860401" rpy="0 0 0" />
+                <mass value="0.310763344920608" />
+                <inertia ixx="0.001401450896582" ixy="9.16506225733395E-08" ixz="-9.26253840796548E-08" iyy="0.001399994200261" iyz="0.000327712970358816" izz="0.000402007894416599" />
+            </inertial>
+        </xacro:if>
     </xacro:macro>
     <xacro:macro name="origin_joint_5" params="reflect">
@@ -12,9 +21,18 @@
     </xacro:macro>
     <xacro:macro name="inertial_link_6" params="reflect">
-        <inertial>
-            <origin xyz="0.031765231605914 -0.006515108863227 -0.040804517366422" rpy="0 0 0" />
-            <mass value="1.34587360139295" />
-            <inertia ixx="0.001098855044306" ixy="0.000130003468892" ixz="-5.88209416784623E-06" iyy="0.001164948561169" iyz="4.20092116284985E-07" izz="0.001189837857495" />
-        </inertial>
+        <xacro:if value="${inertia_version in ['tiago-pro-s']}">
+            <inertial>
+                <origin xyz="0.03179 -0.00642 -0.04078" rpy="0 0 0" />
+                <mass value="1.34957" />
+                <inertia ixx="0.00127" ixy="0.00036" ixz="0.00006" iyy="0.00261" iyz="-0.00001" izz="0.00273" />
+            </inertial>
+        </xacro:if>
+        <xacro:if value="${inertia_version in ['tiago-pro']}">
+            <inertial>
+                <origin xyz="0.031765231605914 -0.006515108863227 -0.040804517366422" rpy="0 0 0" />
+                <mass value="1.34587360139295" />
+                <inertia ixx="0.001098855044306" ixy="0.000130003468892" ixz="-5.88209416784623E-06" iyy="0.001164948561169" iyz="4.20092116284985E-07" izz="0.001189837857495" />
+            </inertial>
+        </xacro:if>
     </xacro:macro>
     <xacro:macro name="origin_joint_6" params="reflect">

Commit message: Add allegro hand as end effector

File: pal_sea_arm_description/robots/pal_sea_arm.urdf.xacro (robot description, xacro)
@@ -37,5 +37,5 @@
   <xacro:property name="tool_changer" value="$(arg tool_changer)" />
   <xacro:property name="nsp" value="$(arg namespace)" />
-  <xacro:if value="${end_effector not in ['no-end-effector', 'pal-pro-gripper', 'custom']}">
+  <xacro:if value="${end_effector not in ['no-end-effector', 'pal-pro-gripper', 'allegro-hand', 'custom']}">
     <xacro:wrong_end_effector/>
   </xacro:if>

File: pal_sea_arm_description/urdf/end_effector/end_effector.urdf.xacro (robot description, xacro)
@@ -28,4 +28,79 @@
       </xacro:pal_pro_gripper>
     </xacro:if>
+  <!--Allegro Hand-->
+  <xacro:if value="${type == 'allegro-hand'}">
+    <xacro:include filename="$(find allegro_hand_description)/urdf/allegro_hand.urdf.xacro" />
+    <link name="${name}_coupler_link">
+        <inertial>
+            <origin xyz="-7.7517E-05 -0.00017089 0.003965" rpy="0 0 0"/>
+            <mass value="0.033254"/>
+            <inertia
+                ixx="1.2371E-05" ixy="1.4319E-07" ixz="2.7745E-07"
+                iyy="1.5119E-05" iyz="-2.1946E-08"
+                izz="2.722E-05"/>
+        </inertial>
+        <visual>
+            <geometry>
+                <mesh filename="package://pal_sea_arm_description/meshes/arm_tiago_pro/allegro_coupler_link.STL" scale="${reflect} 1 1" />
+            </geometry>
+            <origin rpy="0 0 0" xyz="0 0 0 "/>
+            <material name="pal/DarkGrey"/>
+        </visual>
+        <collision>
+            <origin xyz="0 0 0.004" rpy="0 0 0"/>
+            <geometry>
+              <cylinder radius="0.0375" length="0.008"/>
+            </geometry>
+        </collision>
+    </link>
+    <gazebo reference="${name}_coupler_link">
+        <material>Gazebo/DarkGrey</material>
+        <mu1>0.9</mu1>
+        <mu2>0.9</mu2>
+    </gazebo>
+    <joint name="${name}_coupler_joint" type="fixed">
+        <parent link="${parent}" />
+        <child link="${name}_coupler_link" />
+        <origin xyz="0.0 0.0 0.0" rpy="0 0 0"/>
+        <axis xyz="0 0 0" />
+    </joint>
+    <link name="${name}_allegro_tc_out_link">
+        <inertial>
+            <origin xyz="-0.00052526 0.0003415 -0.0041487" rpy="0 0 0"/>
+            <mass value="0.03447"/>
+            <inertia
+                ixx="1.6829E-05" ixy="2.9746E-07" ixz="-4.1936E-08"
+                iyy="1.4935E-05" iyz="2.7742E-08"
+                izz="3.0915E-05"/>
+        </inertial>
+        <visual>
+            <geometry>
+                <mesh filename="package://pal_sea_arm_description/meshes/arm_tiago_pro/allegro_tc_out_link.STL" scale="${reflect} 1 1" />
+            </geometry>
+            <origin rpy="0 0 0" xyz="0 0 0 "/>
+            <material name="pal/DarkGrey"/>
+        </visual>
+        <collision>
+            <origin xyz="0 0 -0.006" rpy="0 0 0"/>
+            <geometry>
+              <cylinder radius="0.0375" length="0.012"/>
+            </geometry>
+        </collision>
+    </link>
+    <gazebo reference="${name}_allegro_tc_out_link">
+        <material>Gazebo/DarkGrey</material>
+        <mu1>0.9</mu1>
+        <mu2>0.9</mu2>
+    </gazebo>
+    <joint name="${name}_tc_joint" type="fixed">
+        <parent link="${name}_coupler_link" />
+        <child link="${name}_allegro_tc_out_link" />
+        <origin xyz="0 0 0.018" rpy="0 0 0" />
+        <axis xyz="0 0 0" />
+    </joint>
+    <xacro:allegro_hand name="${name}" parent="${name}_allegro_tc_out_link" reflect="${reflect}">
+      <origin xyz="0.00956 0.001 0.094" rpy="0.0 0.0 0"/>
+    </xacro:allegro_hand>
+  </xacro:if>
     <!-- PAL Pro Prototype -->
     <!-- <xacro:if value="${type == 'pal-pro-gripper-prototype'}">

Commit message: Support in the pal_sea_arm_description

File: pal_sea_arm_description/robots/pal_sea_arm.urdf.xacro (robot description, xacro)
@@ -23,4 +23,6 @@
   <xacro:arg name="arm_type" default="pal-sea-arm-standalone"/>
   <!-- False, True -->
+  <xacro:arg name="torque_estimation" default="False"/>
+  <!-- False, True -->
   <xacro:arg name="tool_changer" default="True"/>
   <!-- Common args -->
@@ -32,4 +34,5 @@
   <xacro:property name="ft_sensor" value="$(arg ft_sensor)" />
   <xacro:property name="arm_type" value="$(arg arm_type)" />
+  <xacro:property name="torque_estimation" value="$(arg torque_estimation)" />
   <xacro:property name="tool_changer" value="$(arg tool_changer)" />
   <xacro:property name="nsp" value="$(arg namespace)" />
@@ -120,4 +123,4 @@
   <xacro:pal_sea_arm_end_effector name="gripper" parent="${end_effector_link}" type="${end_effector}" tool_changer="${tool_changer}" reflect="1"/>
   <!-- ROS2 control -->
-  <xacro:pal_sea_arm_ros2_control use_sim="$(arg use_sim)" />
+  <xacro:pal_sea_arm_ros2_control use_sim="$(arg use_sim)" torque_estimation="${torque_estimation}"/>
 </robot>

File: pal_sea_arm_description/ros2_control/ros2_control.urdf.xacro (robot description, xacro)
@@ -13,5 +13,5 @@
  -->
 <robot xmlns:xacro="http://ros.org/wiki/xacro" name="pal_sea_arm">
-  <xacro:macro name="pal_sea_arm_ros2_control" params="use_sim:=^|false">
+  <xacro:macro name="pal_sea_arm_ros2_control" params="use_sim:=^|false torque_estimation:=false">
     <xacro:arg name="end_effector" default="no-end-effector"/>
     <xacro:arg name="ft_sensor" default="no-ft-sensor"/>
@@ -19,4 +19,5 @@
     <xacro:property name="has_ft_sensor" value="${ft_sensor != 'no-ft-sensor'}" />
     <xacro:property name="ft_sensor" value="$(arg ft_sensor)" />
+    <xacro:property name="torque_estimation" value="$(arg torque_estimation)" />
     <xacro:include filename="$(find pal_sea_arm_description)/urdf/arm/arm.ros2_control.xacro" />
     <xacro:if value="${end_effector == 'pal-pro-gripper'}">
@@ -35,11 +36,11 @@
       </hardware>
       <!-- arm -->
-      <xacro:ros2_control_arm name="arm_1" reduction="121.0" offset_value="${arm_1_joint_offset}"/>
-      <xacro:ros2_control_arm name="arm_2" reduction="121.0" offset_value="${arm_2_joint_offset}"/>
-      <xacro:ros2_control_arm name="arm_3" reduction="101.0" offset_value="${arm_3_joint_offset}"/>
-      <xacro:ros2_control_arm name="arm_4" reduction="101.0" offset_value="${arm_4_joint_offset}"/>
-      <xacro:ros2_control_arm name="arm_5" reduction="101.0" offset_value="${arm_5_joint_offset}"/>
-      <xacro:ros2_control_arm name="arm_6" reduction="101.0" offset_value="${arm_6_joint_offset}"/>
-      <xacro:ros2_control_arm name="arm_7" reduction="101.0" offset_value="${arm_7_joint_offset}"/>
+      <xacro:ros2_control_arm name="arm_1" reduction="121.0" offset_value="${arm_1_joint_offset}" use_sea_transmission="${torque_estimation}"/>
+      <xacro:ros2_control_arm name="arm_2" reduction="121.0" offset_value="${arm_2_joint_offset}" use_sea_transmission="${torque_estimation}"/>
+      <xacro:ros2_control_arm name="arm_3" reduction="101.0" offset_value="${arm_3_joint_offset}" use_sea_transmission="${torque_estimation}"/>
+      <xacro:ros2_control_arm name="arm_4" reduction="101.0" offset_value="${arm_4_joint_offset}" use_sea_transmission="${torque_estimation}"/>
+      <xacro:ros2_control_arm name="arm_5" reduction="101.0" offset_value="${arm_5_joint_offset}" use_sea_transmission="${torque_estimation}"/>
+      <xacro:ros2_control_arm name="arm_6" reduction="101.0" offset_value="${arm_6_joint_offset}" use_sea_transmission="${torque_estimation}"/>
+      <xacro:ros2_control_arm name="arm_7" reduction="101.0" offset_value="${arm_7_joint_offset}" use_sea_transmission="${torque_estimation}"/>
       <xacro:if value="${end_effector == 'pal-pro-gripper'}">
         <!-- pal-pro-gripper -->

Commit message: Fix param use_sim_time name

File: pal_sea_arm_description/robots/pal_sea_arm.urdf.xacro (robot description, xacro)
@@ -27,5 +27,5 @@
   <xacro:arg name="tool_changer" default="True"/>
   <!-- Common args -->
-  <xacro:arg name="use_sim" default="False"/>
+  <xacro:arg name="use_sim_time" default="False"/>
   <xacro:arg name="namespace" default=""/>
   <!-- PROPERTIES -->

File: pal_sea_arm_description/ros2_control/ros2_control.urdf.xacro (robot description, xacro)
@@ -13,5 +13,5 @@
  -->
 <robot xmlns:xacro="http://ros.org/wiki/xacro" name="pal_sea_arm">
-  <xacro:macro name="pal_sea_arm_ros2_control" params="use_sim:=^|false torque_estimation:=false">
+  <xacro:macro name="pal_sea_arm_ros2_control" params="use_sim_time:=^|false torque_estimation:=false">
     <xacro:arg name="end_effector" default="no-end-effector"/>
     <xacro:arg name="ft_sensor" default="no-ft-sensor"/>
@@ -28,8 +28,8 @@
     <ros2_control name="ros2_control_pal_sea_arm_system" type="system">
       <hardware>
-        <xacro:if value="$(arg use_sim)">
+        <xacro:if value="$(arg use_sim_time)">
           <plugin>gazebo_ros2_control/GazeboSystem</plugin>
         </xacro:if>
-        <xacro:unless value="$(arg use_sim)">
+        <xacro:unless value="$(arg use_sim_time)">
           <plugin>robot_control/RobotControl</plugin>
         </xacro:unless>
