Commit message: Added mujoco tags

File: pal_sea_arm_description/robots/pal_sea_arm.urdf.xacro (robot description, xacro)
@@ -29,4 +29,10 @@
   <xacro:arg name="use_sim_time" default="False"/>
   <xacro:arg name="namespace" default=""/>
+  <!-- Mujoco args -->
+  <xacro:arg name="mujoco" default="false" />
+  <xacro:arg name="mj_motor" default="false" />
+  <xacro:arg name="mj_position" default="false" />
+  <xacro:arg name="mj_simulate" default="false" />
+  <xacro:arg name="mj_control" default="false" />
   <!-- PROPERTIES -->
   <xacro:property name="end_effector" value="$(arg end_effector)" />
@@ -37,4 +43,7 @@
   <xacro:property name="tool_changer" value="$(arg tool_changer)" />
   <xacro:property name="nsp" value="$(arg namespace)" />
+  <!-- Mujoco properties -->
+  <xacro:property name="mujoco" value="$(arg mujoco)" />
+  <xacro:property name="mj_control" value="$(arg mj_control)" />
   <xacro:if value="${end_effector not in ['no-end-effector', 'pal-pro-gripper', 'allegro-hand', 'custom']}">
     <xacro:wrong_end_effector/>
@@ -122,4 +131,21 @@
   <!-- End effector -->
   <xacro:pal_sea_arm_end_effector name="gripper" parent="${end_effector_link}" type="${end_effector}" tool_changer="${tool_changer}" reflect="1"/>
+   <!-- Mujoco Tags -->
+  <xacro:include filename="$(find pal_sea_arm_description)/mujoco/mj_tags.xacro" />
+  <xacro:if value="$(arg mujoco)">
+    <mujoco>
+      <xacro:mj_common/>
+      <xacro:if value="$(arg mj_simulate)">
+        <actuator>
+          <xacro:if value="$(arg mj_motor)">
+            <xacro:arm_mj_motor_actuators/>
+          </xacro:if>
+          <xacro:if value="$(arg mj_position)">
+            <xacro:arm_mj_position_actuators/>
+          </xacro:if>
+        </actuator>
+      </xacro:if>
+    </mujoco>
+  </xacro:if>
   <!-- ROS2 control -->
   <xacro:pal_sea_arm_ros2_control use_sim_time="$(arg use_sim_time)" torque_estimation="${torque_estimation}"/>

File: pal_sea_arm_description/ros2_control/ros2_control.urdf.xacro (robot description, xacro)
@@ -29,5 +29,10 @@
       <hardware>
         <xacro:if value="$(arg use_sim_time)">
-          <plugin>gazebo_ros2_control/GazeboSystem</plugin>
+          <xacro:if value="${mj_control}">
+            <plugin>mujoco_ros2_control/MujocoSystem</plugin>
+          </xacro:if>
+          <xacro:unless value="${mj_control}">
+            <plugin>gazebo_ros2_control/GazeboSystem</plugin>
+          </xacro:unless>
         </xacro:if>
         <xacro:unless value="$(arg use_sim_time)">

File: pal_sea_arm_description/urdf/arm/arm.ros2_control.xacro (robot description, xacro)
@@ -14,25 +14,50 @@
 <robot xmlns:xacro="http://ros.org/wiki/xacro">
   <xacro:macro name="ros2_control_arm" params="name reduction offset_value use_sea_transmission:=false">
-    <joint name="${name}_joint">
-      <command_interface name="position" />
-      <command_interface name="velocity" />
-      <command_interface name="effort" />
-      <state_interface name="position" />
-      <state_interface name="velocity" />
-      <state_interface name="effort" />
-      <!-- SEA specific joint interfaces -->
+    <xacro:if value="$(arg mujoco)">
+       <joint name="${name}_joint">
+        <xacro:if value="$(arg mj_position)">
+          <xacro:if value="$(arg mj_simulate)">
+            <command_interface name="position" />
+          </xacro:if>
+          <xacro:unless value="$(arg mj_simulate)">
+            <param name="position_kp">700</param>
+            <param name="position_ki">0</param>
+            <param name="position_kd">1</param>
+            <param name="position_i_max">0</param>
+            <command_interface name="position_pid" />
+          </xacro:unless>
+        </xacro:if>
+        <xacro:unless value="$(arg mj_position)">
+          <command_interface name="effort" />
+          <command_interface name="velocity" />
+        </xacro:unless>
+        <state_interface name="position" />
+        <state_interface name="velocity" />
+        <state_interface name="effort" />
+       </joint>
+    </xacro:if>
+    <xacro:unless value="$(arg mujoco)">
+      <joint name="${name}_joint">
+        <command_interface name="position" />
+        <command_interface name="velocity" />
+        <command_interface name="effort" />
+        <state_interface name="position" />
+        <state_interface name="velocity" />
+        <state_interface name="effort" />
+        <!-- SEA specific joint interfaces -->
+        <xacro:if value="${use_sea_transmission}">
+          <state_interface name="torque"/>
+          <state_interface name="absolute_position"/>
+        </xacro:if>
+      </joint>
+      <xacro:include filename="$(find pal_sea_arm_description)/ros2_control/transmissions.urdf.xacro" />
       <xacro:if value="${use_sea_transmission}">
-        <state_interface name="torque"/>
-        <state_interface name="absolute_position"/>
+        <!-- Reduction needed for the torque estimation -->
+        <xacro:sea_transmission name="${name}" reduction="${reduction}" offset_value="${offset_value}" />
       </xacro:if>
-    </joint>
-    <xacro:include filename="$(find pal_sea_arm_description)/ros2_control/transmissions.urdf.xacro" />
-    <xacro:if value="${use_sea_transmission}">
-      <!-- Reduction needed for the torque estimation -->
-      <xacro:sea_transmission name="${name}" reduction="${reduction}" offset_value="${offset_value}" />
-    </xacro:if>
-    <xacro:unless value="${use_sea_transmission}">
-      <!-- Reduction already applied in the RT layer, harcoded here to 1.0 -->
-      <xacro:simple_transmission name="${name}" reduction="1.0" offset_value="${offset_value}" />
+      <xacro:unless value="${use_sea_transmission}">
+        <!-- Reduction already applied in the RT layer, harcoded here to 1.0 -->
+        <xacro:simple_transmission name="${name}" reduction="1.0" offset_value="${offset_value}" />
+      </xacro:unless>
     </xacro:unless>
   </xacro:macro>

Commit message: changed link definition

File: pal_sea_arm_description/robots/pal_sea_arm.urdf.xacro (robot description, xacro)
@@ -89,37 +89,6 @@
   <!-- ROBOT DEFINITION -->
   <link name="world"/>
-  <joint name="world_fixed" type="fixed">
-    <origin xyz="0 0 0" rpy="0 0 0"/>
-    <parent link="world"/>
-    <child link="arm_root_link"/>
-  </joint>
-  <!-- BASE LINK -->
-  <link name="arm_root_link">
-    <inertial>
-      <origin xyz="0.0 0.0 0.0" rpy="0 0 0" />
-      <mass value="0.28971" />
-      <inertia ixx="0.00022379" ixy="1.5836E-20" ixz="5.2063E-21" iyy="0.00022379" iyz="-5.1333E-21" izz="0.00019673" />
-    </inertial>
-    <visual>
-      <origin xyz="0 0 0" rpy="0 0 0" />
-      <geometry>
-        <mesh filename="package://pal_sea_arm_description/meshes/arm_tiago_pro/base_link.stl" />
-      </geometry>
-      <material name="pal/DarkGrey"/>
-    </visual>
-    <collision>
-      <origin xyz="0 0 0" rpy="0 0 0" />
-      <geometry>
-        <mesh filename="package://pal_sea_arm_description/meshes/arm_tiago_pro/base_link.stl" />
-      </geometry>
-    </collision>
-  </link>
-  <gazebo reference="arm_root_link">
-    <material>Gazebo/DarkGrey</material>
-    <mu1>0.9</mu1>
-    <mu2>0.9</mu2>
-  </gazebo>
   <!-- ARM -->
-  <xacro:pal_sea_arm name="arm" parent="arm_root_link" arm_type="${arm_type}" tool_changer="${tool_changer}" wrist_model="${wrist_model}" reflect="1" arm_1_offset="0" arm_2_offset="0" arm_3_offset="0" arm_4_offset="0" arm_5_offset="0" arm_6_offset="0" arm_7_offset="0">
+  <xacro:pal_sea_arm name="arm" parent="world" arm_type="${arm_type}" tool_changer="${tool_changer}" wrist_model="${wrist_model}" reflect="1" arm_1_offset="0" arm_2_offset="0" arm_3_offset="0" arm_4_offset="0" arm_5_offset="0" arm_6_offset="0" arm_7_offset="0">
     <origin xyz="0 0 0" rpy="0 0 3.1416" />
   </xacro:pal_sea_arm>
@@ -139,8 +108,8 @@
         <actuator>
           <xacro:if value="$(arg mj_motor)">
-            <xacro:arm_mj_motor_actuators/>
+            <xacro:single_arm_mj_motor_actuators/>
           </xacro:if>
           <xacro:if value="$(arg mj_position)">
-            <xacro:arm_mj_position_actuators/>
+            <xacro:single_arm_mj_position_actuators/>
           </xacro:if>
         </actuator>

File: pal_sea_arm_description/urdf/arm/arm.urdf.xacro (robot description, xacro)
@@ -51,4 +51,39 @@
     <xacro:include filename="$(find pal_sea_arm_description)/urdf/arm/arm_properties/${arm_type}/${wrist_model}.properties.xacro"/>
     <!-- ARM DEFINITION -->
+    <!-- BASE LINK -->
+    <link name="${name}_root_link">
+      <inertial>
+        <origin xyz="0.0 0.0 0.0" rpy="0 0 0" />
+        <mass value="0.28971" />
+        <inertia ixx="0.00022379" ixy="1.5836E-20" ixz="5.2063E-21" iyy="0.00022379" iyz="-5.1333E-21" izz="0.00019673" />
+      </inertial>
+      <visual>
+        <origin xyz="0 0 0" rpy="0 0 0" />
+        <geometry>
+          <mesh filename="package://pal_sea_arm_description/meshes/arm_tiago_pro/arm_base_link.stl" />
+        </geometry>
+        <material name="pal/DarkGrey"/>
+      </visual>
+      <collision>
+        <origin xyz="0 0 0" rpy="0 0 0" />
+        <geometry>
+          <mesh filename="package://pal_sea_arm_description/meshes/arm_tiago_pro/arm_base_link.stl" />
+        </geometry>
+      </collision>
+    </link>
+    <joint name="${name}_root_joint" type="fixed">
+        <xacro:insert_block name="origin"/>
+        <parent link="${parent}" />
+        <child link="${name}_root_link" />
+        <axis xyz="0 0 1" />
+        <limit lower="${arm_1_joint_lb * deg_to_rad}" upper="${arm_1_joint_ub * deg_to_rad}" effort="${arm_1_max_effort}" velocity="${arm_1_max_velocity}" />
+        <dynamics friction="${arm_friction}" damping="${arm_damping}"/>
+        <safety_controller k_position="${arm_k_position}" k_velocity="${arm_k_velocity}" soft_lower_limit="${arm_1_joint_lb * deg_to_rad  + arm_eps}" soft_upper_limit="${arm_1_joint_ub * deg_to_rad  - arm_eps}" />
+      </joint>
+    <gazebo reference="arm_root_link">
+      <material>Gazebo/DarkGrey</material>
+      <mu1>0.9</mu1>
+      <mu2>0.9</mu2>
+    </gazebo>
     <!-- ARM 1 LINK -->
     <link name="${name}_1_link">
@@ -70,6 +105,6 @@
     <!-- ARM 1 JOINT -->
     <joint name="${name}_1_joint" type="revolute">
-      <xacro:insert_block name="origin"/>
-      <parent link="${parent}" />
+      <origin xyz="0 0 0" rpy="0 0 0" />
+      <parent link="${name}_root_link" />
       <child link="${name}_1_link" />
       <axis xyz="0 0 1" />

Commit message: Fixed frame orientation

File: pal_sea_arm_description/robots/pal_sea_arm.urdf.xacro (robot description, xacro)
@@ -91,5 +91,5 @@
   <!-- ARM -->
   <xacro:pal_sea_arm name="arm" parent="world" arm_type="${arm_type}" tool_changer="${tool_changer}" wrist_model="${wrist_model}" reflect="1" arm_1_offset="0" arm_2_offset="0" arm_3_offset="0" arm_4_offset="0" arm_5_offset="0" arm_6_offset="0" arm_7_offset="0">
-    <origin xyz="0 0 0" rpy="0 0 3.1416" />
+    <origin xyz="0 0 0" rpy="0 0 0" />
   </xacro:pal_sea_arm>
   <!-- Force Torque sensor-->

Commit message: change xacro parameter and launch argument name

File: pal_sea_arm_description/robots/pal_sea_arm.urdf.xacro (robot description, xacro)
@@ -32,5 +32,5 @@
   <xacro:arg name="sim_type" default="gazebo" />
   <xacro:arg name="mj_control" default="false" />
-  <xacro:arg name="mj_world_name" default="floor" />
+  <xacro:arg name="world_name" default="floor" />
   <!-- PROPERTIES -->
   <xacro:property name="end_effector" value="$(arg end_effector)" />
@@ -43,5 +43,5 @@
   <xacro:property name="sim_type" value="$(arg sim_type)" />
   <xacro:property name="mj_control" value="$(arg mj_control)"/>
-  <xacro:property name="mj_world_name" value="$(arg mj_world_name)"/>
+  <xacro:property name="world_name" value="$(arg world_name)"/>
   <xacro:if value="${end_effector not in ['no-end-effector', 'pal-pro-gripper', 'allegro-hand', 'custom']}">
     <xacro:wrong_end_effector/>
@@ -103,5 +103,5 @@
       <xacro:include filename="$(find pal_sea_arm_description)/mujoco/mj_tags.xacro" />
       <xacro:include filename="$(find pal_pro_gripper_description)/mujoco/mj_tags.xacro" />
-      <xacro:include filename="$(find pal_mujoco_scenes)/scenes/${mj_world_name}.xacro" />
+      <xacro:include filename="$(find pal_mujoco_scenes)/scenes/${world_name}.xacro" />
        <!-- Mujoco environment -->
       <xacro:mj_common light_target="arm_1_link"/>
@@ -110,5 +110,5 @@
         <actuator>
           <!-- Arm -->
-          <xacro:mj_arm_actuators side="arm" arm_type="${arm_type}" wrist_model="${wrist_model}" joint_reflect="1"/>
+          <xacro:mj_arm_actuators name="arm" arm_type="${arm_type}" wrist_model="${wrist_model}" joint_reflect="1"/>
           <xacro:if value="${has_end_effector}">
             <!-- End-effector -->
@@ -120,9 +120,9 @@
           <!-- Equality-->
         <equality>
-          <xacro:mj_gripper_equality side="gripper" anchor_r="0.014 -0.0015 0" anchor_l="0.014 -0.001 0"/>
+          <xacro:mj_gripper_equality name="gripper" anchor_r="0.014 -0.0015 0" anchor_l="0.014 -0.001 0"/>
         </equality>
         <!-- Contact-->
         <contact>
-          <xacro:mj_gripper_contact side="gripper"/>
+          <xacro:mj_gripper_contact name="gripper"/>
         </contact>
       </xacro:if>

Commit message: restored to original version

File: pal_sea_arm_description/robots/pal_sea_arm.urdf.xacro (robot description, xacro)
@@ -87,7 +87,38 @@
   <!-- ROBOT DEFINITION -->
   <link name="world"/>
+  <joint name="world_fixed" type="fixed">
+    <origin xyz="0 0 0" rpy="0 0 0"/>
+    <parent link="world"/>
+    <child link="arm_root_link"/>
+  </joint>
+  <!-- BASE LINK -->
+  <link name="arm_root_link">
+    <inertial>
+      <origin xyz="0.0 0.0 0.0" rpy="0 0 0" />
+      <mass value="0.28971" />
+      <inertia ixx="0.00022379" ixy="1.5836E-20" ixz="5.2063E-21" iyy="0.00022379" iyz="-5.1333E-21" izz="0.00019673" />
+    </inertial>
+    <visual>
+      <origin xyz="0 0 0" rpy="0 0 0" />
+      <geometry>
+        <mesh filename="package://pal_sea_arm_description/meshes/arm_tiago_pro/arm_base_link.stl" />
+      </geometry>
+      <material name="pal/DarkGrey"/>
+    </visual>
+    <collision>
+      <origin xyz="0 0 0" rpy="0 0 0" />
+      <geometry>
+        <mesh filename="package://pal_sea_arm_description/meshes/arm_tiago_pro/arm_base_link.stl" />
+      </geometry>
+    </collision>
+  </link>
+  <gazebo reference="arm_root_link">
+    <material>Gazebo/DarkGrey</material>
+    <mu1>0.9</mu1>
+    <mu2>0.9</mu2>
+  </gazebo>
   <!-- ARM -->
-  <xacro:pal_sea_arm name="arm" parent="world" arm_type="${arm_type}" tool_changer="${tool_changer}" wrist_model="${wrist_model}" reflect="1" arm_1_offset="0" arm_2_offset="0" arm_3_offset="0" arm_4_offset="0" arm_5_offset="0" arm_6_offset="0" arm_7_offset="0">
-    <origin xyz="0 0 0" rpy="0 0 0" />
+  <xacro:pal_sea_arm name="arm" parent="arm_root_link" arm_type="${arm_type}" tool_changer="${tool_changer}" wrist_model="${wrist_model}" reflect="1" arm_1_offset="0" arm_2_offset="0" arm_3_offset="0" arm_4_offset="0" arm_5_offset="0" arm_6_offset="0" arm_7_offset="0">
+    <origin xyz="0 0 0" rpy="0 0 3.1416" />
   </xacro:pal_sea_arm>
   <!-- Force Torque sensor-->

File: pal_sea_arm_description/urdf/arm/arm.urdf.xacro (robot description, xacro)
@@ -51,39 +51,4 @@
     <xacro:include filename="$(find pal_sea_arm_description)/urdf/arm/arm_properties/${arm_type}/${wrist_model}.properties.xacro"/>
     <!-- ARM DEFINITION -->
-    <!-- BASE LINK -->
-    <link name="${name}_root_link">
-      <inertial>
-        <origin xyz="0.0 0.0 0.0" rpy="0 0 0" />
-        <mass value="0.28971" />
-        <inertia ixx="0.00022379" ixy="1.5836E-20" ixz="5.2063E-21" iyy="0.00022379" iyz="-5.1333E-21" izz="0.00019673" />
-      </inertial>
-      <visual>
-        <origin xyz="0 0 0" rpy="0 0 0" />
-        <geometry>
-          <mesh filename="package://pal_sea_arm_description/meshes/arm_tiago_pro/arm_base_link.stl" />
-        </geometry>
-        <material name="pal/DarkGrey"/>
-      </visual>
-      <collision>
-        <origin xyz="0 0 0" rpy="0 0 0" />
-        <geometry>
-          <mesh filename="package://pal_sea_arm_description/meshes/arm_tiago_pro/arm_base_link.stl" />
-        </geometry>
-      </collision>
-    </link>
-    <joint name="${name}_root_joint" type="fixed">
-        <xacro:insert_block name="origin"/>
-        <parent link="${parent}" />
-        <child link="${name}_root_link" />
-        <axis xyz="0 0 1" />
-        <limit lower="${arm_1_joint_lb * deg_to_rad}" upper="${arm_1_joint_ub * deg_to_rad}" effort="${arm_1_max_effort}" velocity="${arm_1_max_velocity}" />
-        <dynamics friction="${arm_friction}" damping="${arm_damping}"/>
-        <safety_controller k_position="${arm_k_position}" k_velocity="${arm_k_velocity}" soft_lower_limit="${arm_1_joint_lb * deg_to_rad  + arm_eps}" soft_upper_limit="${arm_1_joint_ub * deg_to_rad  - arm_eps}" />
-      </joint>
-    <gazebo reference="arm_root_link">
-      <material>Gazebo/DarkGrey</material>
-      <mu1>0.9</mu1>
-      <mu2>0.9</mu2>
-    </gazebo>
     <!-- ARM 1 LINK -->
     <link name="${name}_1_link">
@@ -105,6 +70,6 @@
     <!-- ARM 1 JOINT -->
     <joint name="${name}_1_joint" type="revolute">
-      <origin xyz="0 0 0" rpy="0 0 0" />
-      <parent link="${name}_root_link" />
+      <xacro:insert_block name="origin"/>
+      <parent link="${parent}" />
       <child link="${name}_1_link" />
       <axis xyz="0 0 1" />

File: pal_sea_arm_description/urdf/end_effector/grasping_frames.xacro (robot description, xacro)
@@ -23,5 +23,5 @@
     <!-- Grasping frame X -->
     <joint name="${prefix}grasping_frame_joint" type="fixed">
-      <parent link="${prefix}arm_base_link" />
+      <parent link="${prefix}base_link" />
       <child link="${prefix}grasping_frame" />
       <origin xyz="${xyz}" rpy="0 -1.5708 0" />
@@ -30,5 +30,5 @@
     <!-- Grasping frame Y -->
     <joint name="${prefix}grasping_frame_Y_joint" type="fixed">
-      <parent link="${prefix}arm_base_link" />
+      <parent link="${prefix}base_link" />
       <child link="${prefix}grasping_frame_Y" />
       <origin xyz="${xyz}" rpy="1.5708 0 0" />
@@ -37,5 +37,5 @@
     <!-- Grasping frame Z -->
     <joint name="${prefix}grasping_frame_Z_joint" type="fixed">
-      <parent link="${prefix}arm_base_link" />
+      <parent link="${prefix}base_link" />
       <child link="${prefix}grasping_frame_Z" />
       <origin xyz="${xyz}" rpy="0 0 0" />
