Commit message: Add support for short-wrist

File: pal_sea_arm_description/robots/pal_sea_arm.urdf.xacro (robot description, xacro)
@@ -52,5 +52,5 @@
     <xacro:wrong_end_effector/>
   </xacro:if>
-  <xacro:if value="${wrist_model not in ['straight-wrist', 'spherical-wrist']}">
+  <xacro:if value="${wrist_model not in ['straight-wrist', 'spherical-wrist', 'short-wrist']}">
     <xacro:wrong_wrist_model/>
   </xacro:if>

File: pal_sea_arm_description/urdf/arm/arm.urdf.xacro (robot description, xacro)
@@ -204,58 +204,60 @@
       <dynamics friction="${arm_friction}" damping="${arm_damping}"/>
     </joint>
-    <!-- ARM 6 LINK -->
-    <link name="${name}_6_link">
-      <xacro:inertial_link_6 reflect="${reflect}"/>
-      <visual>
-        <origin xyz="0 0 0" rpy="0 0 0" />
-        <geometry>
-          <mesh filename="package://pal_sea_arm_description/meshes/${mesh_folder}/${wrist_model}/arm_6_link.stl" scale="1 1 ${reflect}" />
-        </geometry>
-        <material name="pal/DarkGrey"/>
-      </visual>
-      <collision>
-        <origin xyz="0 0 0" rpy="0 0 0" />
-        <geometry>
-          <mesh filename="package://pal_sea_arm_description/meshes/${mesh_folder}/${wrist_model}/arm_6_link_collision.stl" scale="1 1 ${reflect}" />
-        </geometry>
-      </collision>
-    </link>
-    <!-- ARM 6 JOINT -->
-    <joint name="${name}_6_joint" type="revolute">
-      <xacro:origin_joint_6 reflect="${reflect}"/>
-      <parent link="${name}_5_link" />
-      <child link="${name}_6_link" />
-      <axis xyz="0 0 ${-1 if wrist_model=='spherical-wrist' else 1}" />
-      <limit lower="${arm_6_joint_lb * deg_to_rad}" upper="${arm_6_joint_ub * deg_to_rad}" effort="${arm_6_max_effort}" velocity="${arm_6_max_velocity}" />
-      <dynamics friction="${arm_friction}" damping="${arm_damping}"/>
-      <safety_controller k_position="${arm_k_position}" k_velocity="${arm_k_velocity}" soft_lower_limit="${arm_6_joint_lb * deg_to_rad  + arm_eps}" soft_upper_limit="${arm_6_joint_ub * deg_to_rad - arm_eps}" />
-    </joint>
+    <xacro:unless value="${wrist_model == 'short-wrist'}">
+      <!-- ARM 6 LINK -->
+      <link name="${name}_6_link">
+        <xacro:inertial_link_6 reflect="${reflect}"/>
+        <visual>
+          <origin xyz="0 0 0" rpy="0 0 0" />
+          <geometry>
+            <mesh filename="package://pal_sea_arm_description/meshes/${mesh_folder}/${wrist_model}/arm_6_link.stl" scale="1 1 ${reflect}" />
+          </geometry>
+          <material name="pal/DarkGrey"/>
+        </visual>
+        <collision>
+          <origin xyz="0 0 0" rpy="0 0 0" />
+          <geometry>
+            <mesh filename="package://pal_sea_arm_description/meshes/${mesh_folder}/${wrist_model}/arm_6_link_collision.stl" scale="1 1 ${reflect}" />
+          </geometry>
+        </collision>
+      </link>
+      <!-- ARM 6 JOINT -->
+      <joint name="${name}_6_joint" type="revolute">
+        <xacro:origin_joint_6 reflect="${reflect}"/>
+        <parent link="${name}_5_link" />
+        <child link="${name}_6_link" />
+        <axis xyz="0 0 ${-1 if wrist_model=='spherical-wrist' else 1}" />
+        <limit lower="${arm_6_joint_lb * deg_to_rad}" upper="${arm_6_joint_ub * deg_to_rad}" effort="${arm_6_max_effort}" velocity="${arm_6_max_velocity}" />
+        <dynamics friction="${arm_friction}" damping="${arm_damping}"/>
+        <safety_controller k_position="${arm_k_position}" k_velocity="${arm_k_velocity}" soft_lower_limit="${arm_6_joint_lb * deg_to_rad  + arm_eps}" soft_upper_limit="${arm_6_joint_ub * deg_to_rad - arm_eps}" />
+      </joint>
     <!-- ARM 7 LINK -->
-    <link name="${name}_7_link">
-      <xacro:inertial_link_7 reflect="${reflect}"/>
-      <visual>
-        <origin xyz="0 0 0" rpy="0 0 0" />
-        <geometry>
-          <mesh filename="package://pal_sea_arm_description/meshes/${mesh_folder}/${wrist_model}/arm_7_link.stl" scale="1 1 ${reflect}" />
-        </geometry>
-        <material name="pal/DarkGrey"/>
-      </visual>
-      <collision>
-        <origin xyz="0 0 0" rpy="0 0 0" />
-        <geometry>
-          <cylinder radius="0.0375" length="0.0366"/>
-        </geometry>
-      </collision>
-    </link>
+      <link name="${name}_7_link">
+        <xacro:inertial_link_7 reflect="${reflect}"/>
+        <visual>
+          <origin xyz="0 0 0" rpy="0 0 0" />
+          <geometry>
+            <mesh filename="package://pal_sea_arm_description/meshes/${mesh_folder}/${wrist_model}/arm_7_link.stl" scale="1 1 ${reflect}" />
+          </geometry>
+          <material name="pal/DarkGrey"/>
+        </visual>
+        <collision>
+          <origin xyz="0 0 0" rpy="0 0 0" />
+          <geometry>
+            <cylinder radius="0.0375" length="0.0366"/>
+          </geometry>
+        </collision>
+      </link>
     <!-- ARM 7 JOINT -->
-    <joint name="${name}_7_joint" type="revolute">
-      <xacro:origin_joint_7 reflect="${reflect}"/>
-      <parent link="${name}_6_link" />
-      <child link="${name}_7_link" />
-      <axis xyz="0 0 1" />
-      <limit lower="${arm_7_joint_lb * deg_to_rad}" upper="${arm_7_joint_ub * deg_to_rad}" effort="${arm_7_max_effort}" velocity="${arm_7_max_velocity}" />
-      <dynamics friction="${arm_friction}" damping="${arm_damping}"/>
-      <safety_controller k_position="${arm_k_position}" k_velocity="${arm_k_velocity}" soft_lower_limit="${arm_7_joint_lb * deg_to_rad  + arm_eps}" soft_upper_limit="${arm_7_joint_ub * deg_to_rad - arm_eps}" />
-    </joint>
+      <joint name="${name}_7_joint" type="revolute">
+        <xacro:origin_joint_7 reflect="${reflect}"/>
+        <parent link="${name}_6_link" />
+        <child link="${name}_7_link" />
+        <axis xyz="0 0 1" />
+        <limit lower="${arm_7_joint_lb * deg_to_rad}" upper="${arm_7_joint_ub * deg_to_rad}" effort="${arm_7_max_effort}" velocity="${arm_7_max_velocity}" />
+        <dynamics friction="${arm_friction}" damping="${arm_damping}"/>
+        <safety_controller k_position="${arm_k_position}" k_velocity="${arm_k_velocity}" soft_lower_limit="${arm_7_joint_lb * deg_to_rad  + arm_eps}" soft_upper_limit="${arm_7_joint_ub * deg_to_rad - arm_eps}" />
+      </joint>
+    </xacro:unless>
     <!--***********************-->
     <!--        TOOL           -->
@@ -265,5 +267,10 @@
       <link name="${name}_tool_link"/>
       <joint name="${name}_tool_joint" type="fixed">
-        <parent link="${name}_7_link" />
+        <xacro:if value="${wrist_model == 'short-wrist'}">
+          <parent link="${name}_5_link" />
+        </xacro:if>
+        <xacro:unless value="${wrist_model == 'short-wrist'}">
+          <parent link="${name}_7_link" />
+        </xacro:unless>
         <child link="${name}_tool_link" />
         <xacro:origin_joint_tool_changer reflect="${reflect}"/>
@@ -272,12 +279,17 @@
     <!-- Without tool changer (tool link just on top of link 7)-->
     <xacro:unless value="${tool_changer}">
-      <link name="${name}_tool_link">
-      </link>
+      <link name="${name}_tool_link"/>
       <joint name="${name}_tool_joint" type="fixed">
-        <parent link="${name}_7_link" />
+        <xacro:if value="${wrist_model == 'short-wrist'}">
+          <parent link="${name}_5_link" />
+        </xacro:if>
+        <xacro:unless value="${wrist_model == 'short-wrist'}">
+          <parent link="${name}_7_link" />
+        </xacro:unless>
         <child link="${name}_tool_link" />
         <origin xyz="0 0 0" rpy="0 ${0 if reflect is 1 else 180 * deg_to_rad} 0.0" />
       </joint>
     </xacro:unless>
+    <!-- GAZEBO PROPERTIES -->
     <gazebo reference="${name}_1_link">
       <material>Gazebo/DarkGrey</material>
@@ -285,4 +297,7 @@
       <mu2>0.9</mu2>
     </gazebo>
+    <gazebo reference="${name}_1_joint">
+      <implicitSpringDamper>1</implicitSpringDamper>
+    </gazebo>
     <gazebo reference="${name}_2_link">
       <material>Gazebo/DarkGrey</material>
@@ -290,4 +305,7 @@
       <mu2>0.9</mu2>
     </gazebo>
+    <gazebo reference="${name}_2_joint">
+      <implicitSpringDamper>1</implicitSpringDamper>
+    </gazebo>
     <gazebo reference="${name}_3_link">
       <material>Gazebo/DarkGrey</material>
@@ -295,4 +313,7 @@
       <mu2>0.9</mu2>
     </gazebo>
+    <gazebo reference="${name}_3_joint">
+      <implicitSpringDamper>1</implicitSpringDamper>
+    </gazebo>
     <gazebo reference="${name}_4_link">
       <material>Gazebo/DarkGrey</material>
@@ -300,4 +321,7 @@
       <mu2>0.9</mu2>
     </gazebo>
+    <gazebo reference="${name}_4_joint">
+      <implicitSpringDamper>1</implicitSpringDamper>
+    </gazebo>
     <gazebo reference="${name}_5_link">
       <material>Gazebo/DarkGrey</material>
@@ -305,4 +329,8 @@
       <mu2>0.9</mu2>
     </gazebo>
+    <gazebo reference="${name}_5_joint">
+      <implicitSpringDamper>1</implicitSpringDamper>
+    </gazebo>
+  <xacro:unless value="${wrist_model == 'short-wrist'}">
     <gazebo reference="${name}_6_link">
       <material>Gazebo/DarkGrey</material>
@@ -310,4 +338,7 @@
       <mu2>0.9</mu2>
     </gazebo>
+    <gazebo reference="${name}_6_joint">
+      <implicitSpringDamper>1</implicitSpringDamper>
+    </gazebo>
     <gazebo reference="${name}_7_link">
       <material>Gazebo/DarkGrey</material>
@@ -315,30 +346,13 @@
       <mu2>0.9</mu2>
     </gazebo>
+    <gazebo reference="${name}_7_joint">
+      <implicitSpringDamper>1</implicitSpringDamper>
+      <provideFeedback>1</provideFeedback>
+    </gazebo>
+  </xacro:unless>
     <gazebo reference="${name}_tool_link">
       <material>Gazebo/DarkGrey</material>
       <mu1>0.9</mu1>
       <mu2>0.9</mu2>
-    </gazebo>
-    <gazebo reference="${name}_1_joint">
-      <implicitSpringDamper>1</implicitSpringDamper>
-    </gazebo>
-    <gazebo reference="${name}_2_joint">
-      <implicitSpringDamper>1</implicitSpringDamper>
-    </gazebo>
-    <gazebo reference="${name}_3_joint">
-      <implicitSpringDamper>1</implicitSpringDamper>
-    </gazebo>
-    <gazebo reference="${name}_4_joint">
-      <implicitSpringDamper>1</implicitSpringDamper>
-    </gazebo>
-    <gazebo reference="${name}_5_joint">
-      <implicitSpringDamper>1</implicitSpringDamper>
-    </gazebo>
-    <gazebo reference="${name}_6_joint">
-      <implicitSpringDamper>1</implicitSpringDamper>
-    </gazebo>
-    <gazebo reference="${name}_7_joint">
-      <implicitSpringDamper>1</implicitSpringDamper>
-      <provideFeedback>1</provideFeedback>
     </gazebo>
   </xacro:macro>

File: pal_sea_arm_description/urdf/arm/arm_properties/tiago-pro/arm.properties.xacro (robot description, xacro)
@@ -112,6 +112,3 @@
         <origin xyz="0.0199999999999993 -0.0371100000000008 0.15989" rpy="1.57079632679489 0 0" />
     </xacro:macro>
-    <xacro:macro name="origin_joint_tool_changer" params="reflect">
-        <origin xyz="0 0 0.017" rpy="0 0 0" />
-    </xacro:macro>
 </robot>

File: pal_sea_arm_description/urdf/arm/arm_properties/tiago-pro/spherical-wrist.properties.xacro (robot description, xacro)
@@ -58,3 +58,6 @@
         <origin xyz="0.07 -0.0534 -0.0422" rpy="1.5708 0 0" />
     </xacro:macro>
+    <xacro:macro name="origin_joint_tool_changer" params="reflect">
+        <origin xyz="0 0 0.017" rpy="0 0 0" />
+    </xacro:macro>
 </robot>

File: pal_sea_arm_description/urdf/arm/arm_properties/tiago-pro/straight-wrist.properties.xacro (robot description, xacro)
@@ -31,3 +31,6 @@
         <origin xyz="0 0.135 0.0354" rpy="-1.5708 0 0" />
     </xacro:macro>
+    <xacro:macro name="origin_joint_tool_changer" params="reflect">
+        <origin xyz="0 0 0.017" rpy="0 0 0" />
+    </xacro:macro>
 </robot>

Commit message: Add new limits values

File: pal_sea_arm_description/robots/pal_sea_arm.urdf.xacro (robot description, xacro)
@@ -34,4 +34,6 @@
   <xacro:arg name="mj_control" default="false" />
   <xacro:arg name="world_name" default="floor" />
+  <!-- Limits v2-->
+  <xacro:arg name="limits_v2" default="False"/>
   <!-- PROPERTIES -->
   <xacro:property name="end_effector" value="$(arg end_effector)" />
@@ -43,4 +45,5 @@
   <xacro:property name="nsp" value="$(arg namespace)" />
   <xacro:property name="gazebo_version" value="$(arg gazebo_version)"/>
+  <xacro:property name="limits_v2" value="$(arg limits_v2)"/>
   <xacro:property name="sim_type" value="$(arg sim_type)" />
   <xacro:property name="mj_control" value="$(arg mj_control)"/>
@@ -121,5 +124,5 @@
   </gazebo>
   <!-- ARM -->
-  <xacro:pal_sea_arm name="arm" parent="arm_root_link" arm_type="${arm_type}" tool_changer="${tool_changer}" wrist_model="${wrist_model}" reflect="1" arm_1_offset="0" arm_2_offset="0" arm_3_offset="0" arm_4_offset="0" arm_5_offset="0" arm_6_offset="0" arm_7_offset="0">
+  <xacro:pal_sea_arm name="arm" parent="arm_root_link" arm_type="${arm_type}" tool_changer="${tool_changer}" wrist_model="${wrist_model}" reflect="1" arm_1_offset="0" arm_2_offset="0" arm_3_offset="0" arm_4_offset="0" arm_5_offset="0" arm_6_offset="0" arm_7_offset="0" limits_v2="${limits_v2}">
     <origin xyz="0 0 0" rpy="0 0 3.1416" />
   </xacro:pal_sea_arm>

File: pal_sea_arm_description/urdf/arm/arm.urdf.xacro (robot description, xacro)
@@ -14,5 +14,5 @@
 <robot xmlns:xacro="http://ros.org/wiki/xacro">
   <!-- Transmissions file -->
-  <xacro:macro name="pal_sea_arm" params="name parent *origin arm_type tool_changer wrist_model reflect:=1 joint_reflect:=1 arm_1_offset arm_2_offset arm_3_offset arm_4_offset arm_5_offset arm_6_offset arm_7_offset no_safety_eps:=False">
+  <xacro:macro name="pal_sea_arm" params="name parent *origin arm_type tool_changer wrist_model reflect:=1 joint_reflect:=1 arm_1_offset arm_2_offset arm_3_offset arm_4_offset arm_5_offset arm_6_offset arm_7_offset no_safety_eps:=False limits_v2:=False">
     <!-- PROPERTIES -->
     <xacro:property name="arm_eps" value="${0.00 if no_safety_eps else 0.07}"/>
@@ -74,7 +74,13 @@
       <child link="${name}_1_link" />
       <axis xyz="0 0 1" />
-      <limit lower="${arm_1_joint_lb * deg_to_rad}" upper="${arm_1_joint_ub * deg_to_rad}" effort="${arm_1_max_effort}" velocity="${arm_1_max_velocity}" />
-      <dynamics friction="${arm_friction}" damping="${arm_damping}"/>
-      <safety_controller k_position="${arm_k_position}" k_velocity="${arm_k_velocity}" soft_lower_limit="${arm_1_joint_lb * deg_to_rad  + arm_eps}" soft_upper_limit="${arm_1_joint_ub * deg_to_rad  - arm_eps}" />
+      <xacro:if value="${limits_v2}">
+        <limit lower="${arm_1_joint_lb_v2 * deg_to_rad}" upper="${arm_1_joint_ub_v2 * deg_to_rad}" effort="${arm_1_max_effort}" velocity="${arm_1_max_velocity}" />
+        <safety_controller k_position="${arm_k_position}" k_velocity="${arm_k_velocity}" soft_lower_limit="${arm_1_joint_lb_v2 * deg_to_rad  + arm_eps}" soft_upper_limit="${arm_1_joint_ub_v2 * deg_to_rad  - arm_eps}" />
+      </xacro:if>
+      <xacro:unless value="${limits_v2}">
+        <limit lower="${arm_1_joint_lb * deg_to_rad}" upper="${arm_1_joint_ub * deg_to_rad}" effort="${arm_1_max_effort}" velocity="${arm_1_max_velocity}" />
+        <safety_controller k_position="${arm_k_position}" k_velocity="${arm_k_velocity}" soft_lower_limit="${arm_1_joint_lb * deg_to_rad  + arm_eps}" soft_upper_limit="${arm_1_joint_ub * deg_to_rad  - arm_eps}" />
+      </xacro:unless>
+      <dynamics friction="${arm_friction}" damping="${arm_damping}"/>
     </joint>
     <!-- ARM 2 LINK -->
@@ -128,7 +134,13 @@
       <child link="${name}_3_link" />
       <axis xyz="0 0 1" />
-      <limit lower="${arm_3_joint_lb * deg_to_rad}" upper="${arm_3_joint_ub * deg_to_rad}" effort="${arm_3_max_effort}" velocity="${arm_3_max_velocity}" />
-      <dynamics friction="${arm_friction}" damping="${arm_damping}"/>
-      <safety_controller k_position="${arm_k_position}" k_velocity="${arm_k_velocity}" soft_lower_limit="${arm_3_joint_lb * deg_to_rad  + arm_eps}" soft_upper_limit="${arm_3_joint_ub * deg_to_rad - arm_eps}" />
+      <xacro:if value="${limits_v2}">
+        <limit lower="${arm_3_joint_lb_v2 * deg_to_rad}" upper="${arm_3_joint_ub_v2 * deg_to_rad}" effort="${arm_3_max_effort}" velocity="${arm_3_max_velocity}" />
+      <safety_controller k_position="${arm_k_position}" k_velocity="${arm_k_velocity}" soft_lower_limit="${arm_3_joint_lb_v2 * deg_to_rad  + arm_eps}" soft_upper_limit="${arm_3_joint_ub_v2 * deg_to_rad - arm_eps}" />
+      </xacro:if>
+      <xacro:unless value="${limits_v2}">
+        <limit lower="${arm_3_joint_lb * deg_to_rad}" upper="${arm_3_joint_ub * deg_to_rad}" effort="${arm_3_max_effort}" velocity="${arm_3_max_velocity}" />
+        <safety_controller k_position="${arm_k_position}" k_velocity="${arm_k_velocity}" soft_lower_limit="${arm_3_joint_lb * deg_to_rad  + arm_eps}" soft_upper_limit="${arm_3_joint_ub * deg_to_rad - arm_eps}" />
+      </xacro:unless>
+      <dynamics friction="${arm_friction}" damping="${arm_damping}"/>
     </joint>
     <!-- ARM 4 LINK -->
@@ -182,7 +194,13 @@
       <child link="${name}_5_link" />
       <axis xyz="0 0 1" />
-      <limit lower="${arm_5_joint_lb * deg_to_rad}" upper="${arm_5_joint_ub * deg_to_rad}" effort="${arm_5_max_effort}" velocity="${arm_5_max_velocity}" />
-      <dynamics friction="${arm_friction}" damping="${arm_damping}"/>
-      <safety_controller k_position="${arm_k_position}" k_velocity="${arm_k_velocity}" soft_lower_limit="${arm_5_joint_lb * deg_to_rad  + arm_eps}" soft_upper_limit="${arm_5_joint_ub * deg_to_rad - arm_eps}" />
+      <xacro:if value="${limits_v2}">
+        <limit lower="${arm_5_joint_lb_v2 * deg_to_rad}" upper="${arm_5_joint_ub_v2 * deg_to_rad}" effort="${arm_5_max_effort}" velocity="${arm_5_max_velocity}" />
+        <safety_controller k_position="${arm_k_position}" k_velocity="${arm_k_velocity}" soft_lower_limit="${arm_5_joint_lb_v2 * deg_to_rad  + arm_eps}" soft_upper_limit="${arm_5_joint_ub_v2 * deg_to_rad - arm_eps}" />
+      </xacro:if>
+      <xacro:unless value="${limits_v2}">
+        <limit lower="${arm_5_joint_lb * deg_to_rad}" upper="${arm_5_joint_ub * deg_to_rad}" effort="${arm_5_max_effort}" velocity="${arm_5_max_velocity}" />
+        <safety_controller k_position="${arm_k_position}" k_velocity="${arm_k_velocity}" soft_lower_limit="${arm_5_joint_lb * deg_to_rad  + arm_eps}" soft_upper_limit="${arm_5_joint_ub * deg_to_rad - arm_eps}" />
+      </xacro:unless>
+      <dynamics friction="${arm_friction}" damping="${arm_damping}"/>
     </joint>
     <!-- ARM 6 LINK -->

File: pal_sea_arm_description/urdf/arm/arm_limits/tiago-pro/arm.limits.xacro (robot description, xacro)
@@ -14,4 +14,9 @@
   <xacro:property name="arm_4_joint_ub" value="65" />
   <xacro:property name="arm_4_joint_lb" value="-140" />
+  <!-- Joint limits v2-->
+  <xacro:property name="arm_1_joint_ub_v2" value="${40 if joint_reflect == 1 else 280}" />
+  <xacro:property name="arm_1_joint_lb_v2" value="${-280 if joint_reflect == 1 else -40}" />
+  <xacro:property name="arm_3_joint_ub_v2" value="160" />
+  <xacro:property name="arm_3_joint_lb_v2" value="-160" />
   <!-- Velocity limits -->
   <xacro:property name="arm_1_max_velocity" value="1.95" />

File: pal_sea_arm_description/urdf/arm/arm_limits/tiago-pro/spherical-wrist.limits.xacro (robot description, xacro)
@@ -7,4 +7,7 @@
   <xacro:property name="arm_7_joint_ub" value="150" />
   <xacro:property name="arm_7_joint_lb" value="-150" />
+  <!-- Joint limtis v2 -->
+  <xacro:property name="arm_5_joint_ub_v2" value="${220 if joint_reflect == 1 else 100}" />
+  <xacro:property name="arm_5_joint_lb_v2" value="${-100 if joint_reflect == 1 else -220}" />
   <!-- Velocity limits -->
   <xacro:property name="arm_5_max_velocity" value="3.95" />
