Commit message: update arm-standalone

File: pal_sea_arm_description/robots/pal_sea_arm.urdf.xacro (robot description, xacro)
@@ -91,28 +91,42 @@
   </xacro:if>
   <!-- ROBOT DEFINITION -->
-  <link name="world"/>
-  <joint name="world_fixed" type="fixed">
-    <origin xyz="0 0 0" rpy="0 0 0"/>
+  <link name="world"></link>
+  <joint name="base_joint" type="fixed">
+    <origin xyz="0 0 0.05" rpy="0 0 0"/>
     <parent link="world"/>
+    <child link="base_link"/>
+  </joint>
+  <link name="base_link">
+    <inertial>
+      <origin xyz="0 0 -0.1" rpy="0 0 0"/>
+      <mass value="0.01" />
+      <inertia ixx="0.001" ixy="0" ixz="0" iyy="0.001" iyz="0" izz="0.001"/>
+    </inertial>
+  </link>
+  <!-- ARM ROOT LINK -->
+  <joint name="arm_root_joint" type="fixed">
+    <origin xyz="0 0 1.272" rpy="0 0 0"/>
+    <parent link="base_link"/>
     <child link="arm_root_link"/>
   </joint>
-  <!-- BASE LINK -->
   <link name="arm_root_link">
     <inertial>
-      <origin xyz="0.0 0.0 0.0" rpy="0 0 0" />
-      <mass value="0.28971" />
-      <inertia ixx="0.00022379" ixy="1.5836E-20" ixz="5.2063E-21" iyy="0.00022379" iyz="-5.1333E-21" izz="0.00019673" />
+      <origin xyz="-0.0023663 -0.0013678 -0.86311" rpy="0 0 2.618" />
+      <mass value="89.317"/>
+      <inertia ixx="6.284" ixy="-2.737E-05" ixz="0.0010106" iyy="6.2841" iyz="0.00058347" izz="3.768" />
     </inertial>
     <visual>
-      <origin xyz="0 0 0" rpy="0 0 0" />
+      <origin xyz="0 0 -0.1" rpy="0 0 2.618 " />
       <geometry>
-        <mesh filename="package://pal_sea_arm_description/meshes/arm_tiago_pro/arm_base_link.stl" />
+        <mesh filename="package://pal_sea_arm_description/meshes/pal_sea_arm_standalone/base_link.stl" />
       </geometry>
-      <material name="pal/DarkGrey"/>
+      <material name="">
+        <color rgba="0.89412 0.91373 0.92941 1" />
+      </material>
     </visual>
     <collision>
-      <origin xyz="0 0 0" rpy="0 0 0" />
+      <origin xyz="0 0 0" rpy="0 0 2.618" />
       <geometry>
-        <mesh filename="package://pal_sea_arm_description/meshes/arm_tiago_pro/arm_base_link.stl" />
+        <mesh filename="package://pal_sea_arm_description/meshes/pal_sea_arm_standalone/base_link.stl" />
       </geometry>
     </collision>
@@ -125,5 +139,5 @@
   <!-- ARM -->
   <xacro:pal_sea_arm name="arm" parent="arm_root_link" arm_type="${arm_type}" tool_changer="${tool_changer}" wrist_model="${wrist_model}" reflect="1" arm_1_offset="0" arm_2_offset="0" arm_3_offset="0" arm_4_offset="0" arm_5_offset="0" arm_6_offset="0" arm_7_offset="0" limits_v2="${limits_v2}">
-    <origin xyz="0 0 0" rpy="0 0 3.1416" />
+    <origin xyz="0.140 0 -0.1" rpy="0 0 0" />
   </xacro:pal_sea_arm>
   <!-- Force Torque sensor-->

File: pal_sea_arm_description/ros2_control/ros2_control.urdf.xacro (robot description, xacro)
@@ -13,5 +13,5 @@
  -->
 <robot xmlns:xacro="http://ros.org/wiki/xacro" name="pal_sea_arm">
-  <xacro:macro name="pal_sea_arm_ros2_control" params="use_sim_time:=^|false torque_estimation:=false">
+  <xacro:macro name="pal_sea_arm_ros2_control" params="use_sim_time:=^|false torque_estimation:=false sim_type:=gazebo">
     <xacro:arg name="end_effector" default="no-end-effector"/>
     <xacro:arg name="ft_sensor" default="no-ft-sensor"/>

File: pal_sea_arm_description/urdf/arm/arm.ros2_control.xacro (robot description, xacro)
@@ -13,5 +13,5 @@
  -->
 <robot xmlns:xacro="http://ros.org/wiki/xacro">
-  <xacro:macro name="ros2_control_arm" params="name reduction offset_value use_sea_transmission:=false">
+  <xacro:macro name="ros2_control_arm" params="name reduction offset_value use_sea_transmission:=false sim_type:=gazebo">
     <joint name="${name}_joint">
       <xacro:if value="${sim_type == 'mujoco-ros2-control'}">

File: pal_sea_arm_description/urdf/arm/arm_limits/pal-sea-arm-standalone/arm.limits.xacro (robot description, xacro)
@@ -6,6 +6,6 @@
   <xacro:property name="arm_k_velocity" value="20"/>
   <!-- Joint limits -->
-  <xacro:property name="arm_1_joint_ub" value="148.97" />
-  <xacro:property name="arm_1_joint_lb" value="-148.97" />
+  <xacro:property name="arm_1_joint_ub" value="120" />
+  <xacro:property name="arm_1_joint_lb" value="-180" />
   <xacro:property name="arm_2_joint_ub" value="63.03" />
   <xacro:property name="arm_2_joint_lb" value="-139.8" />

Commit message: add continuous joint and remove camera param

File: pal_sea_arm_description/robots/pal_sea_arm.urdf.xacro (robot description, xacro)
@@ -43,5 +43,5 @@
   <xacro:property name="torque_estimation" value="$(arg torque_estimation)" />
   <xacro:property name="tool_changer" value="$(arg tool_changer)" />
-  <xacro:property name="nsp" value="$(arg namespace)" />
+  <xacro:property name="namespace" value="$(arg namespace)" />
   <xacro:property name="gazebo_version" value="$(arg gazebo_version)"/>
   <xacro:property name="limits_v2" value="$(arg limits_v2)"/>

File: pal_sea_arm_description/urdf/arm/arm.urdf.xacro (robot description, xacro)
@@ -14,5 +14,5 @@
 <robot xmlns:xacro="http://ros.org/wiki/xacro">
   <!-- Transmissions file -->
-  <xacro:macro name="pal_sea_arm" params="name parent *origin arm_type tool_changer wrist_model reflect:=1 joint_reflect:=1 arm_1_offset arm_2_offset arm_3_offset arm_4_offset arm_5_offset arm_6_offset arm_7_offset no_safety_eps:=False limits_v2:=False">
+  <xacro:macro name="pal_sea_arm" params="name parent use_sim_time:=^|false *origin arm_type tool_changer wrist_model reflect:=1 joint_reflect:=1 arm_1_offset arm_2_offset arm_3_offset arm_4_offset arm_5_offset arm_6_offset arm_7_offset no_safety_eps:=False limits_v2:=False">
     <!-- PROPERTIES -->
     <xacro:property name="arm_eps" value="${0.00 if no_safety_eps else 0.07}"/>
@@ -69,17 +69,20 @@
     </link>
     <!-- ARM 1 JOINT -->
-    <joint name="${name}_1_joint" type="revolute">
+    <xacro:property name="joint_type" value="${'continuous' if arm_type == 'pal-sea-arm-standalone' else 'revolute'}" />
+    <joint name="${name}_1_joint" type="${joint_type}">
       <xacro:insert_block name="origin"/>
       <parent link="${parent}" />
       <child link="${name}_1_link" />
       <axis xyz="0 0 1" />
-      <xacro:if value="${limits_v2}">
-        <limit lower="${arm_1_joint_lb_v2 * deg_to_rad}" upper="${arm_1_joint_ub_v2 * deg_to_rad}" effort="${arm_1_max_effort}" velocity="${arm_1_max_velocity}" />
-        <safety_controller k_position="${arm_k_position}" k_velocity="${arm_k_velocity}" soft_lower_limit="${arm_1_joint_lb_v2 * deg_to_rad  + arm_eps}" soft_upper_limit="${arm_1_joint_ub_v2 * deg_to_rad  - arm_eps}" />
-      </xacro:if>
-      <xacro:unless value="${limits_v2}">
-        <limit lower="${arm_1_joint_lb * deg_to_rad}" upper="${arm_1_joint_ub * deg_to_rad}" effort="${arm_1_max_effort}" velocity="${arm_1_max_velocity}" />
-        <safety_controller k_position="${arm_k_position}" k_velocity="${arm_k_velocity}" soft_lower_limit="${arm_1_joint_lb * deg_to_rad  + arm_eps}" soft_upper_limit="${arm_1_joint_ub * deg_to_rad  - arm_eps}" />
-      </xacro:unless>
+      <xacro:if value="${joint_type == 'revolute'}">
+        <xacro:if value="${limits_v2}">
+          <limit lower="${arm_1_joint_lb_v2 * deg_to_rad}" upper="${arm_1_joint_ub_v2 * deg_to_rad}" effort="${arm_1_max_effort}" velocity="${arm_1_max_velocity}" />
+          <safety_controller k_position="${arm_k_position}" k_velocity="${arm_k_velocity}" soft_lower_limit="${arm_1_joint_lb_v2 * deg_to_rad  + arm_eps}" soft_upper_limit="${arm_1_joint_ub_v2 * deg_to_rad  - arm_eps}" />
+        </xacro:if>
+        <xacro:unless value="${limits_v2}">
+          <limit lower="${arm_1_joint_lb * deg_to_rad}" upper="${arm_1_joint_ub * deg_to_rad}" effort="${arm_1_max_effort}" velocity="${arm_1_max_velocity}" />
+          <safety_controller k_position="${arm_k_position}" k_velocity="${arm_k_velocity}" soft_lower_limit="${arm_1_joint_lb * deg_to_rad  + arm_eps}" soft_upper_limit="${arm_1_joint_ub * deg_to_rad  - arm_eps}" />
+        </xacro:unless>
+      </xacro:if>
       <dynamics friction="${arm_friction}" damping="${arm_damping}"/>
     </joint>

Commit message: fix z_ value of base_link

File: pal_sea_arm_description/robots/pal_sea_arm.urdf.xacro (robot description, xacro)
@@ -117,5 +117,5 @@
     </inertial>
     <visual>
-      <origin xyz="0 0 -0.1" rpy="0 0 2.618 " />
+      <origin xyz="0 0 -0.08" rpy="0 0 2.618 " />
       <geometry>
         <mesh filename="package://pal_sea_arm_description/meshes/pal_sea_arm_standalone/base_link.stl" />
@@ -126,5 +126,5 @@
     </visual>
     <collision>
-      <origin xyz="0 0 0" rpy="0 0 2.618" />
+      <origin xyz="0 0 -0.08" rpy="0 0 2.618" />
       <geometry>
         <mesh filename="package://pal_sea_arm_description/meshes/pal_sea_arm_standalone/base_link.stl" />
@@ -139,5 +139,5 @@
   <!-- ARM -->
   <xacro:pal_sea_arm name="arm" parent="arm_root_link" arm_type="${arm_type}" tool_changer="${tool_changer}" wrist_model="${wrist_model}" reflect="1" arm_1_offset="0" arm_2_offset="0" arm_3_offset="0" arm_4_offset="0" arm_5_offset="0" arm_6_offset="0" arm_7_offset="0" limits_v2="${limits_v2}">
-    <origin xyz="0.140 0 -0.1" rpy="0 0 0" />
+    <origin xyz="0.140 0 -0.08" rpy="0 0 0" />
   </xacro:pal_sea_arm>
   <!-- Force Torque sensor-->

Commit message: add pen-gripper as ee

File: pal_sea_arm_description/robots/pal_sea_arm.urdf.xacro (robot description, xacro)
@@ -49,5 +49,5 @@
   <xacro:property name="mj_control" value="$(arg mj_control)"/>
   <xacro:property name="world_name" value="$(arg world_name)"/>
-  <xacro:if value="${end_effector not in ['no-end-effector', 'pal-pro-gripper', 'allegro-hand', 'custom']}">
+  <xacro:if value="${end_effector not in ['no-end-effector', 'pal-pro-gripper', 'allegro-hand', 'custom', 'pen-gripper']}">
     <xacro:wrong_end_effector/>
   </xacro:if>

File: pal_sea_arm_description/urdf/end_effector/end_effector.urdf.xacro (robot description, xacro)
@@ -27,4 +27,46 @@
         <origin xyz="0.0 0.0 0.0" rpy="0 0 0"/>
       </xacro:pal_pro_gripper>
+    </xacro:if>
+    <!--Pen Gripper-->
+    <xacro:if value="${type == 'pen-gripper'}">
+      <joint name="pen_gripper_joint" type="fixed">
+        <origin xyz="0 0 0" rpy="0 0 0"/>
+        <parent link="arm_tool_link"/>
+        <child link="pen_gripper_base_link"/>
+      </joint>
+      <link name="pen_gripper_base_link">
+        <inertial>
+          <origin xyz="0.00031569 -2.3649E-05 0.022532" rpy="0 0 0"/>
+          <mass value="0.33922"/>
+          <inertia ixx="0.00019797" ixy="5.0773E-08" ixz="3.91E-07" iyy="0.00020508" iyz="-2.2918E-08" izz="0.0002014" />
+        </inertial>
+        <visual>
+          <origin xyz="0 0 0" rpy="0 0 0" />
+          <geometry>
+          <mesh filename="package://pal_sea_arm_description/meshes/pal_sea_arm_standalone/pen_gripper_link.stl" />
+          </geometry>
+          <material name="">
+            <color rgba="0.89412 0.91373 0.92941 1" />
+          </material>
+        </visual>
+        <collision>
+          <origin xyz="0 0 0" rpy="0 0 0" />
+          <geometry>
+            <mesh filename="package://pal_sea_arm_description/meshes/pal_sea_arm_standalone/pen_gripper_link.stl" />
+          </geometry>
+        </collision>
+      </link>
+      <joint name="pen_gripper_tip_joint" type="fixed">
+        <origin xyz="0 0 0.157" rpy="0 0 0"/>
+        <parent link="pen_gripper_base_link"/>
+        <child link="pen_gripper_tip_link"/>
+      </joint>
+      <link name="pen_gripper_tip_link">
+        <inertial>
+          <origin xyz="0 0 0.157" rpy="0 0 0"/>
+          <mass value="0.1"/>
+          <inertia ixx="3.91E-07" ixy="0" ixz="0" iyy="2.2918E-08" iyz="0" izz="2.2918E-08" />
+        </inertial>
+      </link>
     </xacro:if>
   <!--Allegro Hand-->
