Commit message: add geometric calibration

File: pal_sea_arm_description/robots/pal_sea_arm.urdf.xacro (robot description, xacro)
@@ -49,4 +49,102 @@
   <xacro:property name="mj_control" value="$(arg mj_control)"/>
   <xacro:property name="world_name" value="$(arg world_name)"/>
+  <!-- Fallback defaults for geometric calibration deltas: standalone entry point, never
+       includes tiago_pro_description geometric_calibration.urdf.xacro. -->
+	<xacro:property name="arm_left_1_dx" value="0.0" />
+	<xacro:property name="arm_left_1_dy" value="0.0" />
+	<xacro:property name="arm_left_1_dz" value="0.0" />
+	<xacro:property name="arm_left_1_droll" value="0.0" />
+	<xacro:property name="arm_left_1_dpitch" value="0.0" />
+	<xacro:property name="arm_left_1_dyaw" value="0.0" />
+	<xacro:property name="arm_left_2_dx" value="0.0" />
+	<xacro:property name="arm_left_2_dy" value="0.0" />
+	<xacro:property name="arm_left_2_dz" value="0.0" />
+	<xacro:property name="arm_left_2_droll" value="0.0" />
+	<xacro:property name="arm_left_2_dpitch" value="0.0" />
+	<xacro:property name="arm_left_2_dyaw" value="0.0" />
+	<xacro:property name="arm_left_3_dx" value="0.0" />
+	<xacro:property name="arm_left_3_dy" value="0.0" />
+	<xacro:property name="arm_left_3_dz" value="0.0" />
+	<xacro:property name="arm_left_3_droll" value="0.0" />
+	<xacro:property name="arm_left_3_dpitch" value="0.0" />
+	<xacro:property name="arm_left_3_dyaw" value="0.0" />
+	<xacro:property name="arm_left_4_dx" value="0.0" />
+	<xacro:property name="arm_left_4_dy" value="0.0" />
+	<xacro:property name="arm_left_4_dz" value="0.0" />
+	<xacro:property name="arm_left_4_droll" value="0.0" />
+	<xacro:property name="arm_left_4_dpitch" value="0.0" />
+	<xacro:property name="arm_left_4_dyaw" value="0.0" />
+	<xacro:property name="arm_left_5_dx" value="0.0" />
+	<xacro:property name="arm_left_5_dy" value="0.0" />
+	<xacro:property name="arm_left_5_dz" value="0.0" />
+	<xacro:property name="arm_left_5_droll" value="0.0" />
+	<xacro:property name="arm_left_5_dpitch" value="0.0" />
+	<xacro:property name="arm_left_5_dyaw" value="0.0" />
+	<xacro:property name="arm_left_6_dx" value="0.0" />
+	<xacro:property name="arm_left_6_dy" value="0.0" />
+	<xacro:property name="arm_left_6_dz" value="0.0" />
+	<xacro:property name="arm_left_6_droll" value="0.0" />
+	<xacro:property name="arm_left_6_dpitch" value="0.0" />
+	<xacro:property name="arm_left_6_dyaw" value="0.0" />
+	<xacro:property name="arm_left_7_dx" value="0.0" />
+	<xacro:property name="arm_left_7_dy" value="0.0" />
+	<xacro:property name="arm_left_7_dz" value="0.0" />
+	<xacro:property name="arm_left_7_droll" value="0.0" />
+	<xacro:property name="arm_left_7_dpitch" value="0.0" />
+	<xacro:property name="arm_left_7_dyaw" value="0.0" />
+	<xacro:property name="arm_right_1_dx" value="0.0" />
+	<xacro:property name="arm_right_1_dy" value="0.0" />
+	<xacro:property name="arm_right_1_dz" value="0.0" />
+	<xacro:property name="arm_right_1_droll" value="0.0" />
+	<xacro:property name="arm_right_1_dpitch" value="0.0" />
+	<xacro:property name="arm_right_1_dyaw" value="0.0" />
+	<xacro:property name="arm_right_2_dx" value="0.0" />
+	<xacro:property name="arm_right_2_dy" value="0.0" />
+	<xacro:property name="arm_right_2_dz" value="0.0" />
+	<xacro:property name="arm_right_2_droll" value="0.0" />
+	<xacro:property name="arm_right_2_dpitch" value="0.0" />
+	<xacro:property name="arm_right_2_dyaw" value="0.0" />
+	<xacro:property name="arm_right_3_dx" value="0.0" />
+	<xacro:property name="arm_right_3_dy" value="0.0" />
+	<xacro:property name="arm_right_3_dz" value="0.0" />
+	<xacro:property name="arm_right_3_droll" value="0.0" />
+	<xacro:property name="arm_right_3_dpitch" value="0.0" />
+	<xacro:property name="arm_right_3_dyaw" value="0.0" />
+	<xacro:property name="arm_right_4_dx" value="0.0" />
+	<xacro:property name="arm_right_4_dy" value="0.0" />
+	<xacro:property name="arm_right_4_dz" value="0.0" />
+	<xacro:property name="arm_right_4_droll" value="0.0" />
+	<xacro:property name="arm_right_4_dpitch" value="0.0" />
+	<xacro:property name="arm_right_4_dyaw" value="0.0" />
+	<xacro:property name="arm_right_5_dx" value="0.0" />
+	<xacro:property name="arm_right_5_dy" value="0.0" />
+	<xacro:property name="arm_right_5_dz" value="0.0" />
+	<xacro:property name="arm_right_5_droll" value="0.0" />
+	<xacro:property name="arm_right_5_dpitch" value="0.0" />
+	<xacro:property name="arm_right_5_dyaw" value="0.0" />
+	<xacro:property name="arm_right_6_dx" value="0.0" />
+	<xacro:property name="arm_right_6_dy" value="0.0" />
+	<xacro:property name="arm_right_6_dz" value="0.0" />
+	<xacro:property name="arm_right_6_droll" value="0.0" />
+	<xacro:property name="arm_right_6_dpitch" value="0.0" />
+	<xacro:property name="arm_right_6_dyaw" value="0.0" />
+	<xacro:property name="arm_right_7_dx" value="0.0" />
+	<xacro:property name="arm_right_7_dy" value="0.0" />
+	<xacro:property name="arm_right_7_dz" value="0.0" />
+	<xacro:property name="arm_right_7_droll" value="0.0" />
+	<xacro:property name="arm_right_7_dpitch" value="0.0" />
+	<xacro:property name="arm_right_7_dyaw" value="0.0" />
+	<xacro:property name="gripper_left_tool_mount_dx" value="0.0" />
+	<xacro:property name="gripper_left_tool_mount_dy" value="0.0" />
+	<xacro:property name="gripper_left_tool_mount_dz" value="0.0" />
+	<xacro:property name="gripper_left_tool_mount_droll" value="0.0" />
+	<xacro:property name="gripper_left_tool_mount_dpitch" value="0.0" />
+	<xacro:property name="gripper_left_tool_mount_dyaw" value="0.0" />
+	<xacro:property name="gripper_right_tool_mount_dx" value="0.0" />
+	<xacro:property name="gripper_right_tool_mount_dy" value="0.0" />
+	<xacro:property name="gripper_right_tool_mount_dz" value="0.0" />
+	<xacro:property name="gripper_right_tool_mount_droll" value="0.0" />
+	<xacro:property name="gripper_right_tool_mount_dpitch" value="0.0" />
+	<xacro:property name="gripper_right_tool_mount_dyaw" value="0.0" />
   <xacro:if value="${end_effector not in ['no-end-effector', 'pal-pro-gripper', 'allegro-hand', 'custom']}">
     <xacro:wrong_end_effector/>
