Commit message: Adding realsense 435

File: pal_sea_arm_description/urdf/end_effector_camera/end_effector_camera.urdf.xacro (robot description, xacro)
@@ -61,4 +61,43 @@
       </joint>
     </xacro:if>
+    <xacro:if value="${type == 'realsense-d435'}">
+      <link name="${name}_camera_link">
+        <inertial>
+          <origin xyz="-7.7517E-05 -0.00017089 0.003965" rpy="0 0 0"/>
+          <mass
+            value="0.05792613" />
+          <inertia
+            ixx="2.7273E-05" ixy="2.443E-07" ixz="-1.725E-09"
+            iyy="8.09E-06" iyz="-2.777E-09"
+            izz="2.73583E-05" />
+        </inertial>
+        <visual>
+        <origin xyz="0 0 0" rpy="0 0 0" />
+          <geometry>
+            <mesh filename="package://pal_sea_arm_description/meshes/arm_tiago_pro/end_effector_camera_realsense_d435.stl" />
+          </geometry>
+          <material name="">
+            <color rgba="0.75294 0.75294 0.75294 1" />
+          </material>
+        </visual>
+        <collision>
+          <origin xyz="0 0 0" rpy="0 0 0" />
+          <geometry>
+            <mesh filename="package://pal_sea_arm_description/meshes/arm_tiago_pro/end_effector_camera_realsense_d435.stl" />
+          </geometry>
+        </collision>
+      </link>
+      <joint name="${name}_camera_joint" type="fixed">
+        <xacro:if value="${camera_position == 'up'}">
+          <origin xyz="0.0406 0 -0.03" rpy="3.1416 -1.5708 0" />
+        </xacro:if>
+        <xacro:if value="${camera_position == 'down'}">
+          <origin xyz="-0.0406 0 -0.003" rpy="0 -1.5708 0" />
+        </xacro:if>
+        <parent link="${parent}" />
+        <child link="${name}_camera_link" />
+        <axis xyz="0 0 0" />
+      </joint>
+    </xacro:if>
   </xacro:macro>
 </robot>

Commit message: Unifying joint in macro of cameras

File: pal_sea_arm_description/urdf/end_effector_camera/end_effector_camera.urdf.xacro (robot description, xacro)
@@ -14,9 +14,10 @@
 <robot xmlns:xacro="http://ros.org/wiki/xacro">
   <!--
-    Utiliy to create a tiago end effector (right or left).
+    Utiliy to create a tiago end effector camera (right or left).
     Parameters:
     - name: End effector name. The created links and joints are prepended with 'name_'
     - parent: Parent link
-    - reflect: Set to 1 for a right end effector, or to -1 for a left end effector
+    - type: Type of camera to be used. Options are 'realsense-d405' or 'realsense-d435'
+    - camera_position: Position of the camera. Options are 'up' or 'down'.
   -->
   <xacro:macro name="pal_sea_arm_end_effector_camera" params="name parent type camera_position">
@@ -49,15 +50,4 @@
         </collision>
       </link>
-      <joint name="${name}_camera_joint" type="fixed">
-        <xacro:if value="${camera_position == 'up'}">
-          <origin xyz="0.0406 0 -0.003" rpy="3.1416 -1.5708 0" />
-        </xacro:if>
-        <xacro:if value="${camera_position == 'down'}">
-          <origin xyz="-0.0406 0 -0.003" rpy="0 -1.5708 0" />
-        </xacro:if>
-        <parent link="${parent}" />
-        <child link="${name}_camera_link" />
-        <axis xyz="0 0 0" />
-      </joint>
     </xacro:if>
     <xacro:if value="${type == 'realsense-d435'}">
@@ -88,7 +78,8 @@
         </collision>
       </link>
-      <joint name="${name}_camera_joint" type="fixed">
+    </xacro:if>
+          <joint name="${name}_camera_joint" type="fixed">
         <xacro:if value="${camera_position == 'up'}">
-          <origin xyz="0.0406 0 -0.03" rpy="3.1416 -1.5708 0" />
+          <origin xyz="0.0406 0 -0.003" rpy="3.1416 -1.5708 0" />
         </xacro:if>
         <xacro:if value="${camera_position == 'down'}">
@@ -99,5 +90,4 @@
         <axis xyz="0 0 0" />
       </joint>
-    </xacro:if>
   </xacro:macro>
 </robot>

Commit message: Fixing description end effector camera

File: pal_sea_arm_description/urdf/end_effector_camera/end_effector_camera.urdf.xacro (robot description, xacro)
@@ -13,6 +13,6 @@
 -->
 <robot xmlns:xacro="http://ros.org/wiki/xacro">
-  <!--
-    Utiliy to create a tiago end effector camera (right or left).
+  <!--<xacro:macro name="pal_sea_arm_end_effector_camera" params="name parent type camera_position">
+    Utility to create a tiago end effector camera (right or left).
     Parameters:
     - name: End effector name. The created links and joints are prepended with 'name_'
@@ -79,15 +79,15 @@
       </link>
     </xacro:if>
-          <joint name="${name}_camera_joint" type="fixed">
-        <xacro:if value="${camera_position == 'up'}">
-          <origin xyz="0.0406 0 -0.003" rpy="3.1416 -1.5708 0" />
-        </xacro:if>
-        <xacro:if value="${camera_position == 'down'}">
-          <origin xyz="-0.0406 0 -0.003" rpy="0 -1.5708 0" />
-        </xacro:if>
-        <parent link="${parent}" />
-        <child link="${name}_camera_link" />
-        <axis xyz="0 0 0" />
-      </joint>
+    <joint name="${name}_camera_joint" type="fixed">
+      <xacro:if value="${camera_position == 'up'}">
+        <origin xyz="0.0406 0 -0.003" rpy="3.1416 -1.5708 0" />
+      </xacro:if>
+      <xacro:if value="${camera_position == 'down'}">
+        <origin xyz="-0.0406 0 -0.003" rpy="0 -1.5708 0" />
+      </xacro:if>
+      <parent link="${parent}" />
+      <child link="${name}_camera_link" />
+      <axis xyz="0 0 0" />
+    </joint>
   </xacro:macro>
 </robot>

Commit message: Update end_effector_camera.urdf.xacro

File: pal_sea_arm_description/urdf/end_effector_camera/end_effector_camera.urdf.xacro (robot description, xacro)
@@ -79,4 +79,32 @@
       </link>
     </xacro:if>
+    <xacro:if value="${type == 'realsense-d435i'}">
+      <link name="${name}_camera_link">
+        <inertial>
+          <origin xyz="-7.7517E-05 -0.00017089 0.003965" rpy="0 0 0"/>
+          <mass
+            value="0.05792613" />
+          <inertia
+            ixx="2.7273E-05" ixy="2.443E-07" ixz="-1.725E-09"
+            iyy="8.09E-06" iyz="-2.777E-09"
+            izz="2.73583E-05" />
+        </inertial>
+        <visual>
+        <origin xyz="0 0 0" rpy="0 0 0" />
+          <geometry>
+            <mesh filename="package://pal_sea_arm_description/meshes/arm_tiago_pro/end_effector_camera_realsense_d435.stl" />
+          </geometry>
+          <material name="">
+            <color rgba="0.75294 0.75294 0.75294 1" />
+          </material>
+        </visual>
+        <collision>
+          <origin xyz="0 0 0" rpy="0 0 0" />
+          <geometry>
+            <mesh filename="package://pal_sea_arm_description/meshes/arm_tiago_pro/end_effector_camera_realsense_d435.stl" />
+          </geometry>
+        </collision>
+      </link>
+    </xacro:if>
     <joint name="${name}_camera_joint" type="fixed">
       <xacro:if value="${camera_position == 'up'}">
